Commit message: using xml description to initialize simulators and dynamics

File: mppi_examples/mppi_panda/resources/panda/panda.urdf.xacro (robot description, xacro)
@@ -1,8 +1,10 @@
 <?xml version="1.0" encoding="utf-8"?>
-<!-- =================================================================================== -->
-<!-- |    This document was autogenerated by xacro from panda_arm_hand.urdf.xacro      | -->
-<!-- |    EDITING THIS FILE BY HAND IS NOT RECOMMENDED                                 | -->
-<!-- =================================================================================== -->
 <robot name="panda" xmlns:xacro="http://www.ros.org/wiki/xacro">
+  <xacro:arg name="resources_prefix"      default="file:" />
+  <xacro:arg name="resources_directory"   default="$(find mppi_panda)" />
+  <xacro:arg name="collision_format"      default="stl"/>
+  <xacro:property name="resources_prefix"     value="$(arg resources_prefix)" />
+  <xacro:property name="resources_directory"  value="$(arg resources_directory)" />
+  <xacro:property name="collision_format"     value="$(arg collision_format)" />
   <link name="world"/>
   <joint name="panda_joint_world" type="fixed">
@@ -97,14 +99,14 @@
       <origin rpy="0 0 0" xyz="0 0 0"/>
       <geometry>
-        <mesh filename="file:///home/giuseppe/exp_ws/src/mppi/mppi_panda/resources/panda/meshes/visual/link0.dae"/>
-      </geometry>
-      <material name="">
-        <color rgba="1 1 1 1"/>
-      </material>
-    </visual>
-    <collision>
-      <origin rpy="0 0 0" xyz="0 0 0"/>
-      <geometry>
-        <mesh filename="file:///home/giuseppe/exp_ws/src/mppi/mppi_panda/resources/panda/meshes/collision/link0.stl"/>
+        <mesh filename="${resources_prefix}${resources_directory}/resources/panda/meshes/visual/link0.dae"/>
+      </geometry>
+      <material name="">
+        <color rgba="1 1 1 1"/>
+      </material>
+    </visual>
+    <collision>
+      <origin rpy="0 0 0" xyz="0 0 0"/>
+      <geometry>
+        <mesh filename="${resources_prefix}${resources_directory}/resources/panda/meshes/collision/link0.${collision_format}"/>
       </geometry>
     </collision>
@@ -119,14 +121,14 @@
       <origin rpy="0 0 0" xyz="0 0 0"/>
       <geometry>
-        <mesh filename="file:///home/giuseppe/exp_ws/src/mppi/mppi_panda/resources/panda/meshes/visual/link1.dae"/>
-      </geometry>
-      <material name="">
-        <color rgba="1 1 1 1"/>
-      </material>
-    </visual>
-    <collision>
-      <origin rpy="0 0 0" xyz="0 0 0"/>
-      <geometry>
-        <mesh filename="file:///home/giuseppe/exp_ws/src/mppi/mppi_panda/resources/panda/meshes/collision/link1.stl"/>
+        <mesh filename="${resources_prefix}${resources_directory}/resources/panda/meshes/visual/link1.dae"/>
+      </geometry>
+      <material name="">
+        <color rgba="1 1 1 1"/>
+      </material>
+    </visual>
+    <collision>
+      <origin rpy="0 0 0" xyz="0 0 0"/>
+      <geometry>
+        <mesh filename="${resources_prefix}${resources_directory}/resources/panda/meshes/collision/link1.${collision_format}"/>
       </geometry>
     </collision>
@@ -149,14 +151,14 @@
       <origin rpy="0 0 0" xyz="0 0 0"/>
       <geometry>
-        <mesh filename="file:///home/giuseppe/exp_ws/src/mppi/mppi_panda/resources/panda/meshes/visual/link2.dae"/>
-      </geometry>
-      <material name="">
-        <color rgba="1 1 1 1"/>
-      </material>
-    </visual>
-    <collision>
-      <origin rpy="0 0 0" xyz="0 0 0"/>
-      <geometry>
-        <mesh filename="file:///home/giuseppe/exp_ws/src/mppi/mppi_panda/resources/panda/meshes/collision/link2.stl"/>
+        <mesh filename="${resources_prefix}${resources_directory}/resources/panda/meshes/visual/link2.dae"/>
+      </geometry>
+      <material name="">
+        <color rgba="1 1 1 1"/>
+      </material>
+    </visual>
+    <collision>
+      <origin rpy="0 0 0" xyz="0 0 0"/>
+      <geometry>
+        <mesh filename="${resources_prefix}${resources_directory}/resources/panda/meshes/collision/link2.${collision_format}"/>
       </geometry>
     </collision>
@@ -179,14 +181,14 @@
       <origin rpy="0 0 0" xyz="0 0 0"/>
       <geometry>
-        <mesh filename="file:///home/giuseppe/exp_ws/src/mppi/mppi_panda/resources/panda/meshes/visual/link3.dae"/>
-      </geometry>
-      <material name="">
-        <color rgba="1 1 1 1"/>
-      </material>
-    </visual>
-    <collision>
-      <origin rpy="0 0 0" xyz="0 0 0"/>
-      <geometry>
-        <mesh filename="file:///home/giuseppe/exp_ws/src/mppi/mppi_panda/resources/panda/meshes/collision/link3.stl"/>
+        <mesh filename="${resources_prefix}${resources_directory}/resources/panda/meshes/visual/link3.dae"/>
+      </geometry>
+      <material name="">
+        <color rgba="1 1 1 1"/>
+      </material>
+    </visual>
+    <collision>
+      <origin rpy="0 0 0" xyz="0 0 0"/>
+      <geometry>
+        <mesh filename="${resources_prefix}${resources_directory}/resources/panda/meshes/collision/link3.${collision_format}"/>
       </geometry>
     </collision>
@@ -209,14 +211,14 @@
       <origin rpy="0 0 0" xyz="0 0 0"/>
       <geometry>
-        <mesh filename="file:///home/giuseppe/exp_ws/src/mppi/mppi_panda/resources/panda/meshes/visual/link4.dae"/>
-      </geometry>
-      <material name="">
-        <color rgba="1 1 1 1"/>
-      </material>
-    </visual>
-    <collision>
-      <origin rpy="0 0 0" xyz="0 0 0"/>
-      <geometry>
-        <mesh filename="file:///home/giuseppe/exp_ws/src/mppi/mppi_panda/resources/panda/meshes/collision/link4.stl"/>
+        <mesh filename="${resources_prefix}${resources_directory}/resources/panda/meshes/visual/link4.dae"/>
+      </geometry>
+      <material name="">
+        <color rgba="1 1 1 1"/>
+      </material>
+    </visual>
+    <collision>
+      <origin rpy="0 0 0" xyz="0 0 0"/>
+      <geometry>
+        <mesh filename="${resources_prefix}${resources_directory}/resources/panda/meshes/collision/link4.${collision_format}"/>
       </geometry>
     </collision>
@@ -241,14 +243,14 @@
       <origin rpy="0 0 0" xyz="0 0 0"/>
       <geometry>
-        <mesh filename="file:///home/giuseppe/exp_ws/src/mppi/mppi_panda/resources/panda/meshes/visual/link5.dae"/>
-      </geometry>
-      <material name="">
-        <color rgba="1 1 1 1"/>
-      </material>
-    </visual>
-    <collision>
-      <origin rpy="0 0 0" xyz="0 0 0"/>
-      <geometry>
-        <mesh filename="file:///home/giuseppe/exp_ws/src/mppi/mppi_panda/resources/panda/meshes/collision/link5.stl"/>
+        <mesh filename="${resources_prefix}${resources_directory}/resources/panda/meshes/visual/link5.dae"/>
+      </geometry>
+      <material name="">
+        <color rgba="1 1 1 1"/>
+      </material>
+    </visual>
+    <collision>
+      <origin rpy="0 0 0" xyz="0 0 0"/>
+      <geometry>
+        <mesh filename="${resources_prefix}${resources_directory}/resources/panda/meshes/collision/link5.${collision_format}"/>
       </geometry>
     </collision>
@@ -271,14 +273,14 @@
       <origin rpy="0 0 0" xyz="0 0 0"/>
       <geometry>
-        <mesh filename="file:///home/giuseppe/exp_ws/src/mppi/mppi_panda/resources/panda/meshes/visual/link6.dae"/>
-      </geometry>
-      <material name="">
-        <color rgba="1 1 1 1"/>
-      </material>
-    </visual>
-    <collision>
-      <origin rpy="0 0 0" xyz="0 0 0"/>
-      <geometry>
-        <mesh filename="file:///home/giuseppe/exp_ws/src/mppi/mppi_panda/resources/panda/meshes/collision/link6.stl"/>
+        <mesh filename="${resources_prefix}${resources_directory}/resources/panda/meshes/visual/link6.dae"/>
+      </geometry>
+      <material name="">
+        <color rgba="1 1 1 1"/>
+      </material>
+    </visual>
+    <collision>
+      <origin rpy="0 0 0" xyz="0 0 0"/>
+      <geometry>
+        <mesh filename="${resources_prefix}${resources_directory}/resources/panda/meshes/collision/link6.${collision_format}"/>
       </geometry>
     </collision>
@@ -301,14 +303,14 @@
       <origin rpy="0 0 0" xyz="0 0 0"/>
       <geometry>
-        <mesh filename="file:///home/giuseppe/exp_ws/src/mppi/mppi_panda/resources/panda/meshes/visual/link7.dae"/>
-      </geometry>
-      <material name="">
-        <color rgba="1 1 1 1"/>
-      </material>
-    </visual>
-    <collision>
-      <origin rpy="0 0 0" xyz="0 0 0"/>
-      <geometry>
-        <mesh filename="file:///home/giuseppe/exp_ws/src/mppi/mppi_panda/resources/panda/meshes/collision/link7.stl"/>
+        <mesh filename="${resources_prefix}${resources_directory}/resources/panda/meshes/visual/link7.dae"/>
+      </geometry>
+      <material name="">
+        <color rgba="1 1 1 1"/>
+      </material>
+    </visual>
+    <collision>
+      <origin rpy="0 0 0" xyz="0 0 0"/>
+      <geometry>
+        <mesh filename="${resources_prefix}${resources_directory}/resources/panda/meshes/collision/link7.${collision_format}"/>
       </geometry>
     </collision>
@@ -370,14 +372,14 @@
       <origin rpy="0 0 0" xyz="0 0 0"/>
       <geometry>
-        <mesh filename="file:///home/giuseppe/exp_ws/src/mppi/mppi_panda/resources/panda/meshes/visual/hand.dae"/>
-      </geometry>
-      <material name="">
-        <color rgba="1 1 1 1"/>
-      </material>
-    </visual>
-    <collision>
-      <origin rpy="0 0 0" xyz="0 0 0"/>
-      <geometry>
-        urdf   <mesh filename="file:///home/giuseppe/exp_ws/src/mppi/mppi_panda/resources/panda/meshes/collision/hand.stl"/>
+        <mesh filename="${resources_prefix}${resources_directory}/resources/panda/meshes/visual/hand.dae"/>
+      </geometry>
+      <material name="">
+        <color rgba="1 1 1 1"/>
+      </material>
+    </visual>
+    <collision>
+      <origin rpy="0 0 0" xyz="0 0 0"/>
+      <geometry>
+        urdf   <mesh filename="${resources_prefix}${resources_directory}/resources/panda/meshes/collision/hand.${collision_format}"/>
       </geometry>
     </collision>
@@ -392,5 +394,5 @@
 <!--      <origin rpy="0 0 0" xyz="0 0 0"/>-->
 <!--      <geometry>-->
-<!--        <mesh filename="file:///home/giuseppe/exp_ws/src/mppi/mppi_panda/resources/panda/meshes/visual/finger.dae"/>-->
+<!--        <mesh filename="${resources_prefix}${resources_directory}/resources/panda/meshes/visual/finger.dae"/>-->
 <!--      </geometry>-->
 <!--      <material name="">-->
@@ -401,5 +403,5 @@
 <!--      <origin rpy="0 0 0" xyz="0 0 0"/>-->
 <!--      <geometry>-->
-<!--        <mesh filename="file:///home/giuseppe/exp_ws/src/mppi/mppi_panda/resources/panda/meshes/collision/finger.stl"/>-->
+<!--        <mesh filename="${resources_prefix}${resources_directory}/resources/panda/meshes/collision/finger.${collision_format}"/>-->
 <!--      </geometry>-->
 <!--    </collision>-->
@@ -414,5 +416,5 @@
 <!--      <origin rpy="0 0 3.14159265359" xyz="0 0 0"/>-->
 <!--      <geometry>-->
-<!--        <mesh filename="file:///home/giuseppe/exp_ws/src/mppi/mppi_panda/resources/panda/meshes/visual/finger.dae"/>-->
+<!--        <mesh filename="${resources_prefix}${resources_directory}/resources/panda/meshes/visual/finger.dae"/>-->
 <!--      </geometry>-->
 <!--      <material name="">-->
@@ -423,5 +425,5 @@
 <!--      <origin rpy="0 0 3.14159265359" xyz="0 0 0"/>-->
 <!--      <geometry>-->
-<!--        <mesh filename="file:///home/giuseppe/exp_ws/src/mppi/mppi_panda/resources/panda/meshes/collision/finger.stl"/>-->
+<!--        <mesh filename="${resources_prefix}${resources_directory}/resources/panda/meshes/collision/finger.${collision_format}"/>-->
 <!--      </geometry>-->
 <!--    </collision>-->

Commit message: tentative implementation

File: mppi_examples/mppi_panda/resources/panda/panda.urdf.xacro (robot description, xacro)
@@ -105,10 +105,10 @@
       </material>
     </visual>
-    <collision>
-      <origin rpy="0 0 0" xyz="0 0 0"/>
-      <geometry>
-        <mesh filename="${resources_prefix}${resources_directory}/resources/panda/meshes/collision/link0.${collision_format}"/>
-      </geometry>
-    </collision>
+<!--    <collision>-->
+<!--      <origin rpy="0 0 0" xyz="0 0 0"/>-->
+<!--      <geometry>-->
+<!--        <mesh filename="${resources_prefix}${resources_directory}/resources/panda/meshes/collision/link0.${collision_format}"/>-->
+<!--      </geometry>-->
+<!--    </collision>-->
   </link>
   <link name="panda_link1">
@@ -127,10 +127,10 @@
       </material>
     </visual>
-    <collision>
-      <origin rpy="0 0 0" xyz="0 0 0"/>
-      <geometry>
-        <mesh filename="${resources_prefix}${resources_directory}/resources/panda/meshes/collision/link1.${collision_format}"/>
-      </geometry>
-    </collision>
+<!--    <collision>-->
+<!--      <origin rpy="0 0 0" xyz="0 0 0"/>-->
+<!--      <geometry>-->
+<!--        <mesh filename="${resources_prefix}${resources_directory}/resources/panda/meshes/collision/link1.${collision_format}"/>-->
+<!--      </geometry>-->
+<!--    </collision>-->
   </link>
   <joint name="panda_joint1" type="revolute">
@@ -157,10 +157,10 @@
       </material>
     </visual>
-    <collision>
-      <origin rpy="0 0 0" xyz="0 0 0"/>
-      <geometry>
-        <mesh filename="${resources_prefix}${resources_directory}/resources/panda/meshes/collision/link2.${collision_format}"/>
-      </geometry>
-    </collision>
+<!--    <collision>-->
+<!--      <origin rpy="0 0 0" xyz="0 0 0"/>-->
+<!--      <geometry>-->
+<!--        <mesh filename="${resources_prefix}${resources_directory}/resources/panda/meshes/collision/link2.${collision_format}"/>-->
+<!--      </geometry>-->
+<!--    </collision>-->
   </link>
   <joint name="panda_joint2" type="revolute">
@@ -187,10 +187,10 @@
       </material>
     </visual>
-    <collision>
-      <origin rpy="0 0 0" xyz="0 0 0"/>
-      <geometry>
-        <mesh filename="${resources_prefix}${resources_directory}/resources/panda/meshes/collision/link3.${collision_format}"/>
-      </geometry>
-    </collision>
+<!--    <collision>-->
+<!--      <origin rpy="0 0 0" xyz="0 0 0"/>-->
+<!--      <geometry>-->
+<!--        <mesh filename="${resources_prefix}${resources_directory}/resources/panda/meshes/collision/link3.${collision_format}"/>-->
+<!--      </geometry>-->
+<!--    </collision>-->
   </link>
   <joint name="panda_joint3" type="revolute">
@@ -217,10 +217,10 @@
       </material>
     </visual>
-    <collision>
-      <origin rpy="0 0 0" xyz="0 0 0"/>
-      <geometry>
-        <mesh filename="${resources_prefix}${resources_directory}/resources/panda/meshes/collision/link4.${collision_format}"/>
-      </geometry>
-    </collision>
+<!--    <collision>-->
+<!--      <origin rpy="0 0 0" xyz="0 0 0"/>-->
+<!--      <geometry>-->
+<!--        <mesh filename="${resources_prefix}${resources_directory}/resources/panda/meshes/collision/link4.${collision_format}"/>-->
+<!--      </geometry>-->
+<!--    </collision>-->
   </link>
   <joint name="panda_joint4" type="revolute">
@@ -249,10 +249,10 @@
       </material>
     </visual>
-    <collision>
-      <origin rpy="0 0 0" xyz="0 0 0"/>
-      <geometry>
-        <mesh filename="${resources_prefix}${resources_directory}/resources/panda/meshes/collision/link5.${collision_format}"/>
-      </geometry>
-    </collision>
+<!--    <collision>-->
+<!--      <origin rpy="0 0 0" xyz="0 0 0"/>-->
+<!--      <geometry>-->
+<!--        <mesh filename="${resources_prefix}${resources_directory}/resources/panda/meshes/collision/link5.${collision_format}"/>-->
+<!--      </geometry>-->
+<!--    </collision>-->
   </link>
   <joint name="panda_joint5" type="revolute">
@@ -279,10 +279,10 @@
       </material>
     </visual>
-    <collision>
-      <origin rpy="0 0 0" xyz="0 0 0"/>
-      <geometry>
-        <mesh filename="${resources_prefix}${resources_directory}/resources/panda/meshes/collision/link6.${collision_format}"/>
-      </geometry>
-    </collision>
+<!--    <collision>-->
+<!--      <origin rpy="0 0 0" xyz="0 0 0"/>-->
+<!--      <geometry>-->
+<!--        <mesh filename="${resources_prefix}${resources_directory}/resources/panda/meshes/collision/link6.${collision_format}"/>-->
+<!--      </geometry>-->
+<!--    </collision>-->
   </link>
   <joint name="panda_joint6" type="revolute">
@@ -309,10 +309,10 @@
       </material>
     </visual>
-    <collision>
-      <origin rpy="0 0 0" xyz="0 0 0"/>
-      <geometry>
-        <mesh filename="${resources_prefix}${resources_directory}/resources/panda/meshes/collision/link7.${collision_format}"/>
-      </geometry>
-    </collision>
+<!--    <collision>-->
+<!--      <origin rpy="0 0 0" xyz="0 0 0"/>-->
+<!--      <geometry>-->
+<!--        <mesh filename="${resources_prefix}${resources_directory}/resources/panda/meshes/collision/link7.${collision_format}"/>-->
+<!--      </geometry>-->
+<!--    </collision>-->
   </link>
   <joint name="panda_joint7" type="revolute">
@@ -378,10 +378,10 @@
       </material>
     </visual>
-    <collision>
-      <origin rpy="0 0 0" xyz="0 0 0"/>
-      <geometry>
-        urdf   <mesh filename="${resources_prefix}${resources_directory}/resources/panda/meshes/collision/hand.${collision_format}"/>
-      </geometry>
-    </collision>
+<!--    <collision>-->
+<!--      <origin rpy="0 0 0" xyz="0 0 0"/>-->
+<!--      <geometry>-->
+<!--        urdf   <mesh filename="${resources_prefix}${resources_directory}/resources/panda/meshes/collision/hand.${collision_format}"/>-->
+<!--      </geometry>-->
+<!--    </collision>-->
   </link>
 <!--  <link name="panda_leftfinger">-->
