Commit message: replacing urdf path with robot description

File: mppi_examples/mppi_panda/resources/panda/panda.urdf.xacro (robot description, xacro)
@@ -1,8 +1,10 @@
 <?xml version="1.0" encoding="utf-8"?>
-<!-- =================================================================================== -->
-<!-- |    This document was autogenerated by xacro from panda_arm_hand.urdf.xacro      | -->
-<!-- |    EDITING THIS FILE BY HAND IS NOT RECOMMENDED                                 | -->
-<!-- =================================================================================== -->
 <robot name="panda" xmlns:xacro="http://www.ros.org/wiki/xacro">
+  <xacro:arg name="resources_prefix"      default="" />
+  <xacro:arg name="resources_directory"   default="$(find mppi_panda)" />
+  <xacro:arg name="collision_format"      default="stl"/>
+  <xacro:property name="resources_prefix"     value="$(arg resources_prefix)" />
+  <xacro:property name="resources_directory"  value="$(arg resources_directory)" />
+  <xacro:property name="collision_format"     value="$(arg collision_format)" />
   <link name="world"/>
   <joint name="panda_joint_world" type="fixed">
@@ -97,16 +99,16 @@
       <origin rpy="0 0 0" xyz="0 0 0"/>
       <geometry>
-        <mesh filename="/home/giuseppe/exp_ws/src/mppi/mppi_panda/resources/panda/meshes/visual/link0.dae"/>
-      </geometry>
-      <material name="">
-        <color rgba="1 1 1 1"/>
-      </material>
-    </visual>
-    <collision>
-      <origin rpy="0 0 0" xyz="0 0 0"/>
-      <geometry>
-        <mesh filename="/home/giuseppe/exp_ws/src/mppi/mppi_panda/resources/panda/meshes/collision/link0.stl"/>
-      </geometry>
-    </collision>
+        <mesh filename="${resources_prefix}${resources_directory}/resources/panda/meshes/visual/link0.dae"/>
+      </geometry>
+      <material name="">
+        <color rgba="1 1 1 1"/>
+      </material>
+    </visual>
+<!--    <collision>-->
+<!--      <origin rpy="0 0 0" xyz="0 0 0"/>-->
+<!--      <geometry>-->
+<!--        <mesh filename="${resources_prefix}${resources_directory}/resources/panda/meshes/collision/link0.${collision_format}"/>-->
+<!--      </geometry>-->
+<!--    </collision>-->
   </link>
   <link name="panda_link1">
@@ -119,16 +121,16 @@
       <origin rpy="0 0 0" xyz="0 0 0"/>
       <geometry>
-        <mesh filename="/home/giuseppe/exp_ws/src/mppi/mppi_panda/resources/panda/meshes/visual/link1.dae"/>
-      </geometry>
-      <material name="">
-        <color rgba="1 1 1 1"/>
-      </material>
-    </visual>
-    <collision>
-      <origin rpy="0 0 0" xyz="0 0 0"/>
-      <geometry>
-        <mesh filename="/home/giuseppe/exp_ws/src/mppi/mppi_panda/resources/panda/meshes/collision/link1.stl"/>
-      </geometry>
-    </collision>
+        <mesh filename="${resources_prefix}${resources_directory}/resources/panda/meshes/visual/link1.dae"/>
+      </geometry>
+      <material name="">
+        <color rgba="1 1 1 1"/>
+      </material>
+    </visual>
+<!--    <collision>-->
+<!--      <origin rpy="0 0 0" xyz="0 0 0"/>-->
+<!--      <geometry>-->
+<!--        <mesh filename="${resources_prefix}${resources_directory}/resources/panda/meshes/collision/link1.${collision_format}"/>-->
+<!--      </geometry>-->
+<!--    </collision>-->
   </link>
   <joint name="panda_joint1" type="revolute">
@@ -149,16 +151,16 @@
       <origin rpy="0 0 0" xyz="0 0 0"/>
       <geometry>
-        <mesh filename="/home/giuseppe/exp_ws/src/mppi/mppi_panda/resources/panda/meshes/visual/link2.dae"/>
-      </geometry>
-      <material name="">
-        <color rgba="1 1 1 1"/>
-      </material>
-    </visual>
-    <collision>
-      <origin rpy="0 0 0" xyz="0 0 0"/>
-      <geometry>
-        <mesh filename="/home/giuseppe/exp_ws/src/mppi/mppi_panda/resources/panda/meshes/collision/link2.stl"/>
-      </geometry>
-    </collision>
+        <mesh filename="${resources_prefix}${resources_directory}/resources/panda/meshes/visual/link2.dae"/>
+      </geometry>
+      <material name="">
+        <color rgba="1 1 1 1"/>
+      </material>
+    </visual>
+<!--    <collision>-->
+<!--      <origin rpy="0 0 0" xyz="0 0 0"/>-->
+<!--      <geometry>-->
+<!--        <mesh filename="${resources_prefix}${resources_directory}/resources/panda/meshes/collision/link2.${collision_format}"/>-->
+<!--      </geometry>-->
+<!--    </collision>-->
   </link>
   <joint name="panda_joint2" type="revolute">
@@ -179,16 +181,16 @@
       <origin rpy="0 0 0" xyz="0 0 0"/>
       <geometry>
-        <mesh filename="/home/giuseppe/exp_ws/src/mppi/mppi_panda/resources/panda/meshes/visual/link3.dae"/>
-      </geometry>
-      <material name="">
-        <color rgba="1 1 1 1"/>
-      </material>
-    </visual>
-    <collision>
-      <origin rpy="0 0 0" xyz="0 0 0"/>
-      <geometry>
-        <mesh filename="/home/giuseppe/exp_ws/src/mppi/mppi_panda/resources/panda/meshes/collision/link3.stl"/>
-      </geometry>
-    </collision>
+        <mesh filename="${resources_prefix}${resources_directory}/resources/panda/meshes/visual/link3.dae"/>
+      </geometry>
+      <material name="">
+        <color rgba="1 1 1 1"/>
+      </material>
+    </visual>
+<!--    <collision>-->
+<!--      <origin rpy="0 0 0" xyz="0 0 0"/>-->
+<!--      <geometry>-->
+<!--        <mesh filename="${resources_prefix}${resources_directory}/resources/panda/meshes/collision/link3.${collision_format}"/>-->
+<!--      </geometry>-->
+<!--    </collision>-->
   </link>
   <joint name="panda_joint3" type="revolute">
@@ -209,16 +211,16 @@
       <origin rpy="0 0 0" xyz="0 0 0"/>
       <geometry>
-        <mesh filename="/home/giuseppe/exp_ws/src/mppi/mppi_panda/resources/panda/meshes/visual/link4.dae"/>
-      </geometry>
-      <material name="">
-        <color rgba="1 1 1 1"/>
-      </material>
-    </visual>
-    <collision>
-      <origin rpy="0 0 0" xyz="0 0 0"/>
-      <geometry>
-        <mesh filename="/home/giuseppe/exp_ws/src/mppi/mppi_panda/resources/panda/meshes/collision/link4.stl"/>
-      </geometry>
-    </collision>
+        <mesh filename="${resources_prefix}${resources_directory}/resources/panda/meshes/visual/link4.dae"/>
+      </geometry>
+      <material name="">
+        <color rgba="1 1 1 1"/>
+      </material>
+    </visual>
+<!--    <collision>-->
+<!--      <origin rpy="0 0 0" xyz="0 0 0"/>-->
+<!--      <geometry>-->
+<!--        <mesh filename="${resources_prefix}${resources_directory}/resources/panda/meshes/collision/link4.${collision_format}"/>-->
+<!--      </geometry>-->
+<!--    </collision>-->
   </link>
   <joint name="panda_joint4" type="revolute">
@@ -241,16 +243,16 @@
       <origin rpy="0 0 0" xyz="0 0 0"/>
       <geometry>
-        <mesh filename="/home/giuseppe/exp_ws/src/mppi/mppi_panda/resources/panda/meshes/visual/link5.dae"/>
-      </geometry>
-      <material name="">
-        <color rgba="1 1 1 1"/>
-      </material>
-    </visual>
-    <collision>
-      <origin rpy="0 0 0" xyz="0 0 0"/>
-      <geometry>
-        <mesh filename="/home/giuseppe/exp_ws/src/mppi/mppi_panda/resources/panda/meshes/collision/link5.stl"/>
-      </geometry>
-    </collision>
+        <mesh filename="${resources_prefix}${resources_directory}/resources/panda/meshes/visual/link5.dae"/>
+      </geometry>
+      <material name="">
+        <color rgba="1 1 1 1"/>
+      </material>
+    </visual>
+<!--    <collision>-->
+<!--      <origin rpy="0 0 0" xyz="0 0 0"/>-->
+<!--      <geometry>-->
+<!--        <mesh filename="${resources_prefix}${resources_directory}/resources/panda/meshes/collision/link5.${collision_format}"/>-->
+<!--      </geometry>-->
+<!--    </collision>-->
   </link>
   <joint name="panda_joint5" type="revolute">
@@ -271,16 +273,16 @@
       <origin rpy="0 0 0" xyz="0 0 0"/>
       <geometry>
-        <mesh filename="/home/giuseppe/exp_ws/src/mppi/mppi_panda/resources/panda/meshes/visual/link6.dae"/>
-      </geometry>
-      <material name="">
-        <color rgba="1 1 1 1"/>
-      </material>
-    </visual>
-    <collision>
-      <origin rpy="0 0 0" xyz="0 0 0"/>
-      <geometry>
-        <mesh filename="/home/giuseppe/exp_ws/src/mppi/mppi_panda/resources/panda/meshes/collision/link6.stl"/>
-      </geometry>
-    </collision>
+        <mesh filename="${resources_prefix}${resources_directory}/resources/panda/meshes/visual/link6.dae"/>
+      </geometry>
+      <material name="">
+        <color rgba="1 1 1 1"/>
+      </material>
+    </visual>
+<!--    <collision>-->
+<!--      <origin rpy="0 0 0" xyz="0 0 0"/>-->
+<!--      <geometry>-->
+<!--        <mesh filename="${resources_prefix}${resources_directory}/resources/panda/meshes/collision/link6.${collision_format}"/>-->
+<!--      </geometry>-->
+<!--    </collision>-->
   </link>
   <joint name="panda_joint6" type="revolute">
@@ -301,16 +303,16 @@
       <origin rpy="0 0 0" xyz="0 0 0"/>
       <geometry>
-        <mesh filename="/home/giuseppe/exp_ws/src/mppi/mppi_panda/resources/panda/meshes/visual/link7.dae"/>
-      </geometry>
-      <material name="">
-        <color rgba="1 1 1 1"/>
-      </material>
-    </visual>
-    <collision>
-      <origin rpy="0 0 0" xyz="0 0 0"/>
-      <geometry>
-        <mesh filename="/home/giuseppe/exp_ws/src/mppi/mppi_panda/resources/panda/meshes/collision/link7.stl"/>
-      </geometry>
-    </collision>
+        <mesh filename="${resources_prefix}${resources_directory}/resources/panda/meshes/visual/link7.dae"/>
+      </geometry>
+      <material name="">
+        <color rgba="1 1 1 1"/>
+      </material>
+    </visual>
+<!--    <collision>-->
+<!--      <origin rpy="0 0 0" xyz="0 0 0"/>-->
+<!--      <geometry>-->
+<!--        <mesh filename="${resources_prefix}${resources_directory}/resources/panda/meshes/collision/link7.${collision_format}"/>-->
+<!--      </geometry>-->
+<!--    </collision>-->
   </link>
   <joint name="panda_joint7" type="revolute">
@@ -370,16 +372,16 @@
       <origin rpy="0 0 0" xyz="0 0 0"/>
       <geometry>
-        <mesh filename="/home/giuseppe/exp_ws/src/mppi/mppi_panda/resources/panda/meshes/visual/hand.dae"/>
-      </geometry>
-      <material name="">
-        <color rgba="1 1 1 1"/>
-      </material>
-    </visual>
-    <collision>
-      <origin rpy="0 0 0" xyz="0 0 0"/>
-      <geometry>
-        urdf   <mesh filename="/home/giuseppe/exp_ws/src/mppi/mppi_panda/resources/panda/meshes/collision/hand.stl"/>
-      </geometry>
-    </collision>
+        <mesh filename="${resources_prefix}${resources_directory}/resources/panda/meshes/visual/hand.dae"/>
+      </geometry>
+      <material name="">
+        <color rgba="1 1 1 1"/>
+      </material>
+    </visual>
+<!--    <collision>-->
+<!--      <origin rpy="0 0 0" xyz="0 0 0"/>-->
+<!--      <geometry>-->
+<!--        urdf   <mesh filename="${resources_prefix}${resources_directory}/resources/panda/meshes/collision/hand.${collision_format}"/>-->
+<!--      </geometry>-->
+<!--    </collision>-->
   </link>
 <!--  <link name="panda_leftfinger">-->
@@ -392,5 +394,5 @@
 <!--      <origin rpy="0 0 0" xyz="0 0 0"/>-->
 <!--      <geometry>-->
-<!--        <mesh filename="/home/giuseppe/exp_ws/src/mppi/mppi_panda/resources/panda/meshes/visual/finger.dae"/>-->
+<!--        <mesh filename="${resources_prefix}${resources_directory}/resources/panda/meshes/visual/finger.dae"/>-->
 <!--      </geometry>-->
 <!--      <material name="">-->
@@ -401,5 +403,5 @@
 <!--      <origin rpy="0 0 0" xyz="0 0 0"/>-->
 <!--      <geometry>-->
-<!--        <mesh filename="/home/giuseppe/exp_ws/src/mppi/mppi_panda/resources/panda/meshes/collision/finger.stl"/>-->
+<!--        <mesh filename="${resources_prefix}${resources_directory}/resources/panda/meshes/collision/finger.${collision_format}"/>-->
 <!--      </geometry>-->
 <!--    </collision>-->
@@ -414,5 +416,5 @@
 <!--      <origin rpy="0 0 3.14159265359" xyz="0 0 0"/>-->
 <!--      <geometry>-->
-<!--        <mesh filename="/home/giuseppe/exp_ws/src/mppi/mppi_panda/resources/panda/meshes/visual/finger.dae"/>-->
+<!--        <mesh filename="${resources_prefix}${resources_directory}/resources/panda/meshes/visual/finger.dae"/>-->
 <!--      </geometry>-->
 <!--      <material name="">-->
@@ -423,5 +425,5 @@
 <!--      <origin rpy="0 0 3.14159265359" xyz="0 0 0"/>-->
 <!--      <geometry>-->
-<!--        <mesh filename="/home/giuseppe/exp_ws/src/mppi/mppi_panda/resources/panda/meshes/collision/finger.stl"/>-->
+<!--        <mesh filename="${resources_prefix}${resources_directory}/resources/panda/meshes/collision/finger.${collision_format}"/>-->
 <!--      </geometry>-->
 <!--    </collision>-->

Commit message: removed all hard coded paths

File: mppi_examples/mppi_panda/resources/panda/panda.urdf.xacro (robot description, xacro)
@@ -7,7 +7,7 @@
   <xacro:property name="resources_directory"  value="$(arg resources_directory)" />
   <xacro:property name="collision_format"     value="$(arg collision_format)" />
-  <link name="world"/>
-  <joint name="panda_joint_world" type="fixed">
-    <parent link="world"/>
+  <xacro:macro name="panda_robot" params="parent_link:='world'">
+  <joint name="panda_joint_${parent_link}" type="fixed">
+    <parent link="${parent_link}"/>
     <child link="panda_link0"/>
     <origin rpy="0 0 0" xyz="0 0 0"/>
@@ -105,10 +105,10 @@
       </material>
     </visual>
-<!--    <collision>-->
-<!--      <origin rpy="0 0 0" xyz="0 0 0"/>-->
-<!--      <geometry>-->
-<!--        <mesh filename="${resources_prefix}${resources_directory}/resources/panda/meshes/collision/link0.${collision_format}"/>-->
-<!--      </geometry>-->
-<!--    </collision>-->
+    <collision>
+      <origin rpy="0 0 0" xyz="0 0 0"/>
+      <geometry>
+        <mesh filename="${resources_prefix}${resources_directory}/resources/panda/meshes/collision/link0.${collision_format}"/>
+      </geometry>
+    </collision>
   </link>
   <link name="panda_link1">
@@ -127,10 +127,10 @@
       </material>
     </visual>
-<!--    <collision>-->
-<!--      <origin rpy="0 0 0" xyz="0 0 0"/>-->
-<!--      <geometry>-->
-<!--        <mesh filename="${resources_prefix}${resources_directory}/resources/panda/meshes/collision/link1.${collision_format}"/>-->
-<!--      </geometry>-->
-<!--    </collision>-->
+    <collision>
+      <origin rpy="0 0 0" xyz="0 0 0"/>
+      <geometry>
+        <mesh filename="${resources_prefix}${resources_directory}/resources/panda/meshes/collision/link1.${collision_format}"/>
+      </geometry>
+    </collision>
   </link>
   <joint name="panda_joint1" type="revolute">
@@ -157,10 +157,10 @@
       </material>
     </visual>
-<!--    <collision>-->
-<!--      <origin rpy="0 0 0" xyz="0 0 0"/>-->
-<!--      <geometry>-->
-<!--        <mesh filename="${resources_prefix}${resources_directory}/resources/panda/meshes/collision/link2.${collision_format}"/>-->
-<!--      </geometry>-->
-<!--    </collision>-->
+    <collision>
+      <origin rpy="0 0 0" xyz="0 0 0"/>
+      <geometry>
+        <mesh filename="${resources_prefix}${resources_directory}/resources/panda/meshes/collision/link2.${collision_format}"/>
+      </geometry>
+    </collision>
   </link>
   <joint name="panda_joint2" type="revolute">
@@ -187,10 +187,10 @@
       </material>
     </visual>
-<!--    <collision>-->
-<!--      <origin rpy="0 0 0" xyz="0 0 0"/>-->
-<!--      <geometry>-->
-<!--        <mesh filename="${resources_prefix}${resources_directory}/resources/panda/meshes/collision/link3.${collision_format}"/>-->
-<!--      </geometry>-->
-<!--    </collision>-->
+    <collision>
+      <origin rpy="0 0 0" xyz="0 0 0"/>
+      <geometry>
+        <mesh filename="${resources_prefix}${resources_directory}/resources/panda/meshes/collision/link3.${collision_format}"/>
+      </geometry>
+    </collision>
   </link>
   <joint name="panda_joint3" type="revolute">
@@ -217,10 +217,10 @@
       </material>
     </visual>
-<!--    <collision>-->
-<!--      <origin rpy="0 0 0" xyz="0 0 0"/>-->
-<!--      <geometry>-->
-<!--        <mesh filename="${resources_prefix}${resources_directory}/resources/panda/meshes/collision/link4.${collision_format}"/>-->
-<!--      </geometry>-->
-<!--    </collision>-->
+    <collision>
+      <origin rpy="0 0 0" xyz="0 0 0"/>
+      <geometry>
+        <mesh filename="${resources_prefix}${resources_directory}/resources/panda/meshes/collision/link4.${collision_format}"/>
+      </geometry>
+    </collision>
   </link>
   <joint name="panda_joint4" type="revolute">
@@ -249,10 +249,10 @@
       </material>
     </visual>
-<!--    <collision>-->
-<!--      <origin rpy="0 0 0" xyz="0 0 0"/>-->
-<!--      <geometry>-->
-<!--        <mesh filename="${resources_prefix}${resources_directory}/resources/panda/meshes/collision/link5.${collision_format}"/>-->
-<!--      </geometry>-->
-<!--    </collision>-->
+    <collision>
+      <origin rpy="0 0 0" xyz="0 0 0"/>
+      <geometry>
+        <mesh filename="${resources_prefix}${resources_directory}/resources/panda/meshes/collision/link5.${collision_format}"/>
+      </geometry>
+    </collision>
   </link>
   <joint name="panda_joint5" type="revolute">
@@ -279,10 +279,10 @@
       </material>
     </visual>
-<!--    <collision>-->
-<!--      <origin rpy="0 0 0" xyz="0 0 0"/>-->
-<!--      <geometry>-->
-<!--        <mesh filename="${resources_prefix}${resources_directory}/resources/panda/meshes/collision/link6.${collision_format}"/>-->
-<!--      </geometry>-->
-<!--    </collision>-->
+    <collision>
+      <origin rpy="0 0 0" xyz="0 0 0"/>
+      <geometry>
+        <mesh filename="${resources_prefix}${resources_directory}/resources/panda/meshes/collision/link6.${collision_format}"/>
+      </geometry>
+    </collision>
   </link>
   <joint name="panda_joint6" type="revolute">
@@ -309,10 +309,10 @@
       </material>
     </visual>
-<!--    <collision>-->
-<!--      <origin rpy="0 0 0" xyz="0 0 0"/>-->
-<!--      <geometry>-->
-<!--        <mesh filename="${resources_prefix}${resources_directory}/resources/panda/meshes/collision/link7.${collision_format}"/>-->
-<!--      </geometry>-->
-<!--    </collision>-->
+    <collision>
+      <origin rpy="0 0 0" xyz="0 0 0"/>
+      <geometry>
+        <mesh filename="${resources_prefix}${resources_directory}/resources/panda/meshes/collision/link7.${collision_format}"/>
+      </geometry>
+    </collision>
   </link>
   <joint name="panda_joint7" type="revolute">
@@ -378,10 +378,10 @@
       </material>
     </visual>
-<!--    <collision>-->
-<!--      <origin rpy="0 0 0" xyz="0 0 0"/>-->
-<!--      <geometry>-->
-<!--        urdf   <mesh filename="${resources_prefix}${resources_directory}/resources/panda/meshes/collision/hand.${collision_format}"/>-->
-<!--      </geometry>-->
-<!--    </collision>-->
+    <collision>
+      <origin rpy="0 0 0" xyz="0 0 0"/>
+      <geometry>
+        <mesh filename="${resources_prefix}${resources_directory}/resources/panda/meshes/collision/hand.${collision_format}"/>
+      </geometry>
+    </collision>
   </link>
 <!--  <link name="panda_leftfinger">-->
@@ -443,3 +443,4 @@
 <!--    <limit effort="20" lower="-0.001" upper="0.04" velocity="0.3"/>-->
 <!--  </joint>-->
+  </xacro:macro>
 </robot>

File: test.urdf (robot description, URDF)
Before this commit: robot panda, 11 links, 10 joints
Links:
- link panda_hand: geometry collision mesh filename=file:///home/giuseppe/student_projects_ws/src/sampling_base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; visual mesh filename=file:///home/giuseppe/student_projects_ws/src/sampling_base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
- link panda_link0: geometry collision mesh filename=file:///home/giuseppe/student_projects_ws/src/sampling_base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; visual mesh filename=file:///home/giuseppe/student_projects_ws/src/sampling_base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
- link panda_link1: geometry collision mesh filename=file:///home/giuseppe/student_projects_ws/src/sampling_base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; visual mesh filename=file:///home/giuseppe/student_projects_ws/src/sampling_base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
- link panda_link2: geometry collision mesh filename=file:///home/giuseppe/student_projects_ws/src/sampling_base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; visual mesh filename=file:///home/giuseppe/student_projects_ws/src/sampling_base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
- link panda_link3: geometry collision mesh filename=file:///home/giuseppe/student_projects_ws/src/sampling_base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; visual mesh filename=file:///home/giuseppe/student_projects_ws/src/sampling_base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
- link panda_link4: geometry collision mesh filename=file:///home/giuseppe/student_projects_ws/src/sampling_base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; visual mesh filename=file:///home/giuseppe/student_projects_ws/src/sampling_base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
- link panda_link5: geometry collision mesh filename=file:///home/giuseppe/student_projects_ws/src/sampling_base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; visual mesh filename=file:///home/giuseppe/student_projects_ws/src/sampling_base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
- link panda_link6: geometry collision mesh filename=file:///home/giuseppe/student_projects_ws/src/sampling_base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; visual mesh filename=file:///home/giuseppe/student_projects_ws/src/sampling_base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
- link panda_link7: geometry collision mesh filename=file:///home/giuseppe/student_projects_ws/src/sampling_base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; visual mesh filename=file:///home/giuseppe/student_projects_ws/src/sampling_base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
