Commit message: optional collision elements

File: mppi_examples/mppi_panda/resources/panda/panda.urdf.xacro (robot description, xacro)
@@ -4,7 +4,9 @@
   <xacro:arg name="resources_directory"   default="$(find mppi_panda)" />
   <xacro:arg name="collision_format"      default="stl"/>
+  <xacro:arg name="collision"             default="true"/>
   <xacro:property name="resources_prefix"     value="$(arg resources_prefix)" />
   <xacro:property name="resources_directory"  value="$(arg resources_directory)" />
   <xacro:property name="collision_format"     value="$(arg collision_format)" />
+  <xacro:property name="collision"            value="$(arg collision)" />
   <link name="world"/>
   <joint name="panda_joint_world" type="fixed">
@@ -105,10 +107,12 @@
       </material>
     </visual>
-    <collision>
-      <origin rpy="0 0 0" xyz="0 0 0"/>
-      <geometry>
-        <mesh filename="${resources_prefix}${resources_directory}/resources/panda/meshes/collision/link0.${collision_format}"/>
-      </geometry>
+    <xacro:if value="${collision}">
+      <collision>
+        <origin rpy="0 0 0" xyz="0 0 0"/>
+        <geometry>
+          <mesh filename="${resources_prefix}${resources_directory}/resources/panda/meshes/collision/link0.${collision_format}"/>
+        </geometry>
     </collision>
+    </xacro:if>
   </link>
   <link name="panda_link1">
@@ -127,10 +131,12 @@
       </material>
     </visual>
-    <collision>
-      <origin rpy="0 0 0" xyz="0 0 0"/>
-      <geometry>
-        <mesh filename="${resources_prefix}${resources_directory}/resources/panda/meshes/collision/link1.${collision_format}"/>
-      </geometry>
-    </collision>
+    <xacro:if value="${collision}">
+      <collision>
+        <origin rpy="0 0 0" xyz="0 0 0"/>
+        <geometry>
+          <mesh filename="${resources_prefix}${resources_directory}/resources/panda/meshes/collision/link1.${collision_format}"/>
+        </geometry>
+      </collision>
+    </xacro:if>
   </link>
   <joint name="panda_joint1" type="revolute">
@@ -157,10 +163,12 @@
       </material>
     </visual>
-    <collision>
-      <origin rpy="0 0 0" xyz="0 0 0"/>
-      <geometry>
-        <mesh filename="${resources_prefix}${resources_directory}/resources/panda/meshes/collision/link2.${collision_format}"/>
-      </geometry>
-    </collision>
+      <xacro:if value="${collision}">
+        <collision>
+          <origin rpy="0 0 0" xyz="0 0 0"/>
+          <geometry>
+            <mesh filename="${resources_prefix}${resources_directory}/resources/panda/meshes/collision/link2.${collision_format}"/>
+          </geometry>
+        </collision>
+      </xacro:if>
   </link>
   <joint name="panda_joint2" type="revolute">
@@ -187,10 +195,12 @@
       </material>
     </visual>
-    <collision>
-      <origin rpy="0 0 0" xyz="0 0 0"/>
-      <geometry>
-        <mesh filename="${resources_prefix}${resources_directory}/resources/panda/meshes/collision/link3.${collision_format}"/>
-      </geometry>
-    </collision>
+    <xacro:if value="${collision}">
+      <collision>
+        <origin rpy="0 0 0" xyz="0 0 0"/>
+        <geometry>
+          <mesh filename="${resources_prefix}${resources_directory}/resources/panda/meshes/collision/link3.${collision_format}"/>
+        </geometry>
+      </collision>
+    </xacro:if>
   </link>
   <joint name="panda_joint3" type="revolute">
@@ -217,10 +227,12 @@
       </material>
     </visual>
-    <collision>
-      <origin rpy="0 0 0" xyz="0 0 0"/>
-      <geometry>
-        <mesh filename="${resources_prefix}${resources_directory}/resources/panda/meshes/collision/link4.${collision_format}"/>
-      </geometry>
-    </collision>
+      <xacro:if value="${collision}">
+        <collision>
+          <origin rpy="0 0 0" xyz="0 0 0"/>
+          <geometry>
+            <mesh filename="${resources_prefix}${resources_directory}/resources/panda/meshes/collision/link4.${collision_format}"/>
+          </geometry>
+        </collision>
+      </xacro:if>
   </link>
   <joint name="panda_joint4" type="revolute">
@@ -249,10 +261,12 @@
       </material>
     </visual>
-    <collision>
-      <origin rpy="0 0 0" xyz="0 0 0"/>
-      <geometry>
-        <mesh filename="${resources_prefix}${resources_directory}/resources/panda/meshes/collision/link5.${collision_format}"/>
-      </geometry>
-    </collision>
+    <xacro:if value="${collision}">
+      <collision>
+        <origin rpy="0 0 0" xyz="0 0 0"/>
+        <geometry>
+          <mesh filename="${resources_prefix}${resources_directory}/resources/panda/meshes/collision/link5.${collision_format}"/>
+        </geometry>
+      </collision>
+    </xacro:if>
   </link>
   <joint name="panda_joint5" type="revolute">
@@ -279,10 +293,12 @@
       </material>
     </visual>
-    <collision>
-      <origin rpy="0 0 0" xyz="0 0 0"/>
-      <geometry>
-        <mesh filename="${resources_prefix}${resources_directory}/resources/panda/meshes/collision/link6.${collision_format}"/>
-      </geometry>
-    </collision>
+    <xacro:if value="${collision}">
+      <collision>
+        <origin rpy="0 0 0" xyz="0 0 0"/>
+        <geometry>
+          <mesh filename="${resources_prefix}${resources_directory}/resources/panda/meshes/collision/link6.${collision_format}"/>
+        </geometry>
+      </collision>
+    </xacro:if>
   </link>
   <joint name="panda_joint6" type="revolute">
@@ -309,10 +325,12 @@
       </material>
     </visual>
-    <collision>
-      <origin rpy="0 0 0" xyz="0 0 0"/>
-      <geometry>
-        <mesh filename="${resources_prefix}${resources_directory}/resources/panda/meshes/collision/link7.${collision_format}"/>
-      </geometry>
-    </collision>
+    <xacro:if value="${collision}">
+      <collision>
+        <origin rpy="0 0 0" xyz="0 0 0"/>
+        <geometry>
+          <mesh filename="${resources_prefix}${resources_directory}/resources/panda/meshes/collision/link7.${collision_format}"/>
+        </geometry>
+      </collision>
+    </xacro:if>
   </link>
   <joint name="panda_joint7" type="revolute">
@@ -378,10 +396,12 @@
       </material>
     </visual>
-    <collision>
-      <origin rpy="0 0 0" xyz="0 0 0"/>
-      <geometry>
-        <mesh filename="${resources_prefix}${resources_directory}/resources/panda/meshes/collision/hand.${collision_format}"/>
-      </geometry>
-    </collision>
+    <xacro:if value="${collision}">
+      <collision>
+        <origin rpy="0 0 0" xyz="0 0 0"/>
+        <geometry>
+          <mesh filename="${resources_prefix}${resources_directory}/resources/panda/meshes/collision/hand.${collision_format}"/>
+        </geometry>
+      </collision>
+    </xacro:if>
   </link>
 <!--  <link name="panda_leftfinger">-->

Commit message: optional fingers

File: mppi_examples/mppi_panda/resources/panda/panda.urdf.xacro (robot description, xacro)
@@ -5,8 +5,10 @@
   <xacro:arg name="collision_format"      default="stl"/>
   <xacro:arg name="collision"             default="true"/>
+  <xacro:arg name="add_finger"            default="false"/>
   <xacro:property name="resources_prefix"     value="$(arg resources_prefix)" />
   <xacro:property name="resources_directory"  value="$(arg resources_directory)" />
   <xacro:property name="collision_format"     value="$(arg collision_format)" />
   <xacro:property name="collision"            value="$(arg collision)" />
+  <xacro:property name="add_finger"           value="$(arg add_finger)" />
   <link name="world"/>
   <joint name="panda_joint_world" type="fixed">
@@ -360,25 +362,4 @@
     <origin rpy="0 0 -0.785398163397" xyz="0 0 0"/>
   </joint>
-<!--  <gazebo reference="panda_hand"/>-->
-<!--  <gazebo reference="panda_leftfinger"/>-->
-<!--  <gazebo reference="panda_rightfinger"/>-->
-<!--  <transmission name="panda_finger_joint1_trans">-->
-<!--    <type>transmission_interface/SimpleTransmission</type>-->
-<!--    <joint name="panda_finger_joint1">-->
-<!--      <hardwareInterface>hardware_interface/PositionJointInterface</hardwareInterface>-->
-<!--    </joint>-->
-<!--    <actuator name="panda_finger_joint1_motor">-->
-<!--      <mechanicalReduction>1</mechanicalReduction>-->
-<!--    </actuator>-->
-<!--  </transmission>-->
-<!--  <transmission name="panda_finger_joint2_trans">-->
-<!--    <type>transmission_interface/SimpleTransmission</type>-->
-<!--    <joint name="panda_finger_joint2">-->
-<!--      <hardwareInterface>hardware_interface/PositionJointInterface</hardwareInterface>-->
-<!--    </joint>-->
-<!--    <actuator name="panda_finger_joint2_motor">-->
-<!--      <mechanicalReduction>1</mechanicalReduction>-->
-<!--    </actuator>-->
-<!--  </transmission>-->
   <link name="panda_hand">
     <inertial>
@@ -405,61 +386,84 @@
     </xacro:if>
   </link>
-<!--  <link name="panda_leftfinger">-->
-<!--    <inertial>-->
-<!--      <mass value="0.1"/>-->
-<!--      <origin rpy="0 0 0" xyz="0 0.0145644 0.0227941"/>-->
-<!--      <inertia ixx="3.01220925051e-05" ixy="0.0" ixz="0.0" iyy="2.95873808038e-05" iyz="0.0" izz="6.95125211657e-06"/>-->
-<!--    </inertial>-->
-<!--    <visual>-->
-<!--      <origin rpy="0 0 0" xyz="0 0 0"/>-->
-<!--      <geometry>-->
-<!--        <mesh filename="${resources_prefix}${resources_directory}/resources/panda/meshes/visual/finger.dae"/>-->
-<!--      </geometry>-->
-<!--      <material name="">-->
-<!--        <color rgba="1 1 1 1"/>-->
-<!--      </material>-->
-<!--    </visual>-->
-<!--    <collision>-->
-<!--      <origin rpy="0 0 0" xyz="0 0 0"/>-->
-<!--      <geometry>-->
-<!--        <mesh filename="${resources_prefix}${resources_directory}/resources/panda/meshes/collision/finger.${collision_format}"/>-->
-<!--      </geometry>-->
-<!--    </collision>-->
-<!--  </link>-->
-<!--  <link name="panda_rightfinger">-->
-<!--    <inertial>-->
-<!--      <mass value="0.1"/>-->
-<!--      <origin rpy="0 0 3.14159265359" xyz="0 0.0145644 0.0227941"/>-->
-<!--      <inertia ixx="3.01220925051e-05" ixy="0.0" ixz="0.0" iyy="2.95873808038e-05" iyz="0.0" izz="6.95125211657e-06"/>-->
-<!--    </inertial>-->
-<!--    <visual>-->
-<!--      <origin rpy="0 0 3.14159265359" xyz="0 0 0"/>-->
-<!--      <geometry>-->
-<!--        <mesh filename="${resources_prefix}${resources_directory}/resources/panda/meshes/visual/finger.dae"/>-->
-<!--      </geometry>-->
-<!--      <material name="">-->
-<!--        <color rgba="1 1 1 1"/>-->
-<!--      </material>-->
-<!--    </visual>-->
-<!--    <collision>-->
-<!--      <origin rpy="0 0 3.14159265359" xyz="0 0 0"/>-->
-<!--      <geometry>-->
-<!--        <mesh filename="${resources_prefix}${resources_directory}/resources/panda/meshes/collision/finger.${collision_format}"/>-->
-<!--      </geometry>-->
-<!--    </collision>-->
-<!--  </link>-->
-<!--  <joint name="panda_finger_joint1" type="prismatic">-->
-<!--    <parent link="panda_hand"/>-->
-<!--    <child link="panda_leftfinger"/>-->
-<!--    <origin rpy="0 0 0" xyz="0 0 0.0584"/>-->
-<!--    <axis xyz="0 1 0"/>-->
-<!--    <limit effort="20" lower="-0.001" upper="0.04" velocity="0.3"/>-->
-<!--  </joint>-->
-<!--  <joint name="panda_finger_joint2" type="prismatic">-->
-<!--    <parent link="panda_hand"/>-->
-<!--    <child link="panda_rightfinger"/>-->
-<!--    <origin rpy="0 0 0" xyz="0 0 0.0584"/>-->
-<!--    <axis xyz="0 -1 0"/>-->
-<!--    <limit effort="20" lower="-0.001" upper="0.04" velocity="0.3"/>-->
-<!--  </joint>-->
+  <xacro:if value="${add_finger}">
+    <gazebo reference="panda_hand"/>
+    <gazebo reference="panda_leftfinger"/>
+    <gazebo reference="panda_rightfinger"/>
+    <transmission name="panda_finger_joint1_trans">
+      <type>transmission_interface/SimpleTransmission</type>
+      <joint name="panda_finger_joint1">
+        <hardwareInterface>hardware_interface/PositionJointInterface</hardwareInterface>
+      </joint>
+      <actuator name="panda_finger_joint1_motor">
+        <mechanicalReduction>1</mechanicalReduction>
+      </actuator>
+    </transmission>
+    <transmission name="panda_finger_joint2_trans">
+      <type>transmission_interface/SimpleTransmission</type>
+      <joint name="panda_finger_joint2">
+        <hardwareInterface>hardware_interface/PositionJointInterface</hardwareInterface>
+      </joint>
+      <actuator name="panda_finger_joint2_motor">
+        <mechanicalReduction>1</mechanicalReduction>
+      </actuator>
+    </transmission>
+    <link name="panda_leftfinger">
+      <inertial>
+        <mass value="0.1"/>
+        <origin rpy="0 0 0" xyz="0 0.0145644 0.0227941"/>
+        <inertia ixx="3.01220925051e-05" ixy="0.0" ixz="0.0" iyy="2.95873808038e-05" iyz="0.0" izz="6.95125211657e-06"/>
+      </inertial>
+      <visual>
+        <origin rpy="0 0 0" xyz="0 0 0"/>
+        <geometry>
+          <mesh filename="${resources_prefix}${resources_directory}/resources/panda/meshes/visual/finger.dae"/>
+        </geometry>
+        <material name="">
+          <color rgba="1 1 1 1"/>
+        </material>
+      </visual>
+      <collision>
+        <origin rpy="0 0 0" xyz="0 0 0"/>
+        <geometry>
+          <mesh filename="${resources_prefix}${resources_directory}/resources/panda/meshes/collision/finger.${collision_format}"/>
+        </geometry>
+      </collision>
+    </link>
+    <link name="panda_rightfinger">
+      <inertial>
+        <mass value="0.1"/>
+        <origin rpy="0 0 3.14159265359" xyz="0 0.0145644 0.0227941"/>
+        <inertia ixx="3.01220925051e-05" ixy="0.0" ixz="0.0" iyy="2.95873808038e-05" iyz="0.0" izz="6.95125211657e-06"/>
+      </inertial>
+      <visual>
+        <origin rpy="0 0 3.14159265359" xyz="0 0 0"/>
+        <geometry>
+          <mesh filename="${resources_prefix}${resources_directory}/resources/panda/meshes/visual/finger.dae"/>
+        </geometry>
+        <material name="">
+          <color rgba="1 1 1 1"/>
+        </material>
+      </visual>
+      <collision>
+        <origin rpy="0 0 3.14159265359" xyz="0 0 0"/>
+        <geometry>
+          <mesh filename="${resources_prefix}${resources_directory}/resources/panda/meshes/collision/finger.${collision_format}"/>
+        </geometry>
+      </collision>
+    </link>
+    <joint name="panda_finger_joint1" type="prismatic">
+      <parent link="panda_hand"/>
+      <child link="panda_leftfinger"/>
+      <origin rpy="0 0 0" xyz="0 0 0.0584"/>
+      <axis xyz="0 1 0"/>
+      <limit effort="20" lower="-0.001" upper="0.04" velocity="0.3"/>
+    </joint>
+    <joint name="panda_finger_joint2" type="prismatic">
+      <parent link="panda_hand"/>
+      <child link="panda_rightfinger"/>
+      <origin rpy="0 0 0" xyz="0 0 0.0584"/>
+      <axis xyz="0 -1 0"/>
+      <limit effort="20" lower="-0.001" upper="0.04" velocity="0.3"/>
+    </joint>
+  </xacro:if>
 </robot>

Commit message: simplified collision shape for finger and hand

File: mppi_examples/mppi_panda/resources/panda/panda.urdf.xacro (robot description, xacro)
@@ -4,10 +4,14 @@
   <xacro:arg name="resources_directory"   default="$(find mppi_panda)" />
   <xacro:arg name="collision_format"      default="stl"/>
-  <xacro:arg name="collision"             default="true"/>
+  <xacro:arg name="collision_links"       default="true"/>
+  <xacro:arg name="collision_hand"        default="true"/>
+  <xacro:arg name="collision_finger"      default="true"/>
   <xacro:arg name="add_finger"            default="false"/>
   <xacro:property name="resources_prefix"     value="$(arg resources_prefix)" />
   <xacro:property name="resources_directory"  value="$(arg resources_directory)" />
   <xacro:property name="collision_format"     value="$(arg collision_format)" />
-  <xacro:property name="collision"            value="$(arg collision)" />
+  <xacro:property name="collision_links"      value="$(arg collision_links)"/>
+  <xacro:property name="collision_hand"       value="$(arg collision_hand)"/>
+  <xacro:property name="collision_finger"     value="$(arg collision_finger)"/>
   <xacro:property name="add_finger"           value="$(arg add_finger)" />
   <xacro:macro name="panda_robot" params="parent_link:='world'">
@@ -109,5 +113,5 @@
       </material>
     </visual>
-    <xacro:if value="${collision}">
+    <xacro:if value="${collision_links}">
       <collision>
         <origin rpy="0 0 0" xyz="0 0 0"/>
@@ -133,5 +137,5 @@
       </material>
     </visual>
-    <xacro:if value="${collision}">
+    <xacro:if value="${collision_links}">
       <collision>
         <origin rpy="0 0 0" xyz="0 0 0"/>
@@ -165,5 +169,5 @@
       </material>
     </visual>
-      <xacro:if value="${collision}">
+      <xacro:if value="${collision_links}">
         <collision>
           <origin rpy="0 0 0" xyz="0 0 0"/>
@@ -197,5 +201,5 @@
       </material>
     </visual>
-    <xacro:if value="${collision}">
+    <xacro:if value="${collision_links}">
       <collision>
         <origin rpy="0 0 0" xyz="0 0 0"/>
@@ -229,5 +233,5 @@
       </material>
     </visual>
-      <xacro:if value="${collision}">
+      <xacro:if value="${collision_links}">
         <collision>
           <origin rpy="0 0 0" xyz="0 0 0"/>
@@ -263,5 +267,5 @@
       </material>
     </visual>
-    <xacro:if value="${collision}">
+    <xacro:if value="${collision_links}">
       <collision>
         <origin rpy="0 0 0" xyz="0 0 0"/>
@@ -295,5 +299,5 @@
       </material>
     </visual>
-    <xacro:if value="${collision}">
+    <xacro:if value="${collision_links}">
       <collision>
         <origin rpy="0 0 0" xyz="0 0 0"/>
@@ -327,5 +331,5 @@
       </material>
     </visual>
-    <xacro:if value="${collision}">
+    <xacro:if value="${collision_links}">
       <collision>
         <origin rpy="0 0 0" xyz="0 0 0"/>
@@ -377,9 +381,11 @@
       </material>
     </visual>
-    <xacro:if value="${collision}">
-      <collision>
-        <origin rpy="0 0 0" xyz="0 0 0"/>
-        <geometry>
-          <mesh filename="${resources_prefix}${resources_directory}/resources/panda/meshes/collision/hand.${collision_format}"/>
+    <xacro:if value="${collision_hand}">
+      <collision>
+        <!--origin rpy="0 0 0" xyz="0 0 0"/-->
+        <origin rpy="0 0 0" xyz="0 0 0.0333"/>
+        <geometry>
+          <!--mesh filename="${resources_prefix}${resources_directory}/resources/panda/meshes/collision/hand.${collision_format}"/!-->
+          <box size="0.035 0.19 0.065"/>
         </geometry>
       </collision>
@@ -423,9 +429,11 @@
         </material>
       </visual>
-      <xacro:if value="${collision}">
+      <xacro:if value="${collision_finger}">
         <collision>
-          <origin rpy="0 0 0" xyz="0 0 0"/>
+          <!--origin rpy="0 0 0" xyz="0 0 0"/-->
+          <origin rpy="0 0 3.14159265359" xyz="0 0.01 0.028"/>
           <geometry>
-            <mesh filename="${resources_prefix}${resources_directory}/resources/panda/meshes/collision/finger.${collision_format}"/>
+            <!--mesh filename="${resources_prefix}${resources_directory}/resources/panda/meshes/collision/finger.${collision_format}"/-->
+            <box size="0.02 0.02 0.05"/>
           </geometry>
         </collision>
@@ -447,9 +455,11 @@
         </material>
       </visual>
-      <xacro:if value="${collision}">
+      <xacro:if value="${collision_finger}">
         <collision>
-          <origin rpy="0 0 3.14159265359" xyz="0 0 0"/>
+          <!-- origin rpy="0 0 3.14159265359" xyz="0 0 0"/ -->
+          <origin rpy="0 0 3.14159265359" xyz="0 -0.01 0.028"/>
           <geometry>
-            <mesh filename="${resources_prefix}${resources_directory}/resources/panda/meshes/collision/finger.${collision_format}"/>
+            <!--mesh filename="${resources_prefix}${resources_directory}/resources/panda/meshes/collision/finger.${collision_format}"/-->
+            <box size="0.02 0.02 0.05"/>
           </geometry>
         </collision>
