Commit message: optional position limits

File: mppi_examples/mppi_panda/resources/panda/panda.urdf.xacro (robot description, xacro)
@@ -7,4 +7,5 @@
   <xacro:arg name="collision_hand"        default="true"/>
   <xacro:arg name="collision_finger"      default="true"/>
+  <xacro:arg name="no_position_limits"      default="true"/>
   <xacro:arg name="add_finger"            default="false"/>
   <xacro:property name="resources_prefix"     value="$(arg resources_prefix)" />
@@ -14,4 +15,5 @@
   <xacro:property name="collision_hand"       value="$(arg collision_hand)"/>
   <xacro:property name="collision_finger"     value="$(arg collision_finger)"/>
+  <xacro:property name="no_position_limits"   value="$(arg no_position_limits)"/>
   <xacro:property name="add_finger"           value="$(arg add_finger)" />
   <xacro:macro name="panda_robot" params="parent_link:='world'">
@@ -152,5 +154,10 @@
     <child link="panda_link1"/>
     <axis xyz="0 0 1"/>
-    <limit effort="87" lower="-2.8973" upper="2.8973" velocity="2.1750"/>
+    <xacro:if value="${no_position_limits}">
+      <limit effort="87" lower="-20" upper="20" velocity="2.1750"/>
+    </xacro:if>
+    <xacro:unless value="${no_position_limits}">
+      <limit effort="87" lower="-2.8973" upper="2.8973" velocity="2.1750"/>
+    </xacro:unless>
   </joint>
   <link name="panda_link2">
@@ -184,5 +191,10 @@
     <child link="panda_link2"/>
     <axis xyz="0 0 1"/>
-    <limit effort="87" lower="-1.7628" upper="1.7628" velocity="2.1750"/>
+    <xacro:if value="${no_position_limits}">
+      <limit effort="87" lower="-20" upper="20" velocity="2.1750"/>
+    </xacro:if>
+    <xacro:unless value="${no_position_limits}">
+      <limit effort="87" lower="-1.7628" upper="1.7628" velocity="2.1750"/>
+    </xacro:unless>
   </joint>
   <link name="panda_link3">
@@ -216,5 +228,10 @@
     <child link="panda_link3"/>
     <axis xyz="0 0 1"/>
-    <limit effort="87" lower="-2.8973" upper="2.8973" velocity="2.1750"/>
+    <xacro:if value="${no_position_limits}">
+      <limit effort="87" lower="-20" upper="20" velocity="2.1750"/>
+    </xacro:if>
+    <xacro:unless value="${no_position_limits}">
+      <limit effort="87" lower="-2.8973" upper="2.8973" velocity="2.1750"/>
+    </xacro:unless>
   </joint>
   <link name="panda_link4">
@@ -249,6 +266,11 @@
     <child link="panda_link4"/>
     <axis xyz="0 0 1"/>
-    <limit effort="87" lower="-3.0718" upper="0.0698" velocity="2.1750"/>
-    <!-- upper should be -0.0698, but that brakes simulation when initial position for this joint is 0.0 -->
+    <xacro:if value="${no_position_limits}">
+      <limit effort="87" lower="-20" upper="20" velocity="2.1750"/>
+    </xacro:if>
+    <xacro:unless value="${no_position_limits}">
+      <limit effort="87" lower="-3.0718" upper="0.0698" velocity="2.1750"/>
+      <!-- upper should be -0.0698, but that brakes simulation when initial position for this joint is 0.0 -->
+    </xacro:unless>
   </joint>
   <link name="panda_link5">
@@ -282,5 +304,10 @@
     <child link="panda_link5"/>
     <axis xyz="0 0 1"/>
-    <limit effort="12" lower="-2.8973" upper="2.8973" velocity="2.6100"/>
+    <xacro:if value="${no_position_limits}">
+      <limit effort="12" lower="-20" upper="20" velocity="2.6100"/>
+    </xacro:if>
+    <xacro:unless value="${no_position_limits}">
+      <limit effort="12" lower="-2.8973" upper="2.8973" velocity="2.6100"/>
+    </xacro:unless>
   </joint>
   <link name="panda_link6">
@@ -314,5 +341,10 @@
     <child link="panda_link6"/>
     <axis xyz="0 0 1"/>
-    <limit effort="12" lower="-0.0175" upper="3.7525" velocity="2.6100"/>
+    <xacro:if value="${no_position_limits}">
+      <limit effort="12" lower="-20" upper="20" velocity="2.6100"/>
+    </xacro:if>
+    <xacro:unless value="${no_position_limits}">
+      <limit effort="12" lower="-0.0175" upper="3.7525" velocity="2.6100"/>
+    </xacro:unless>
   </joint>
   <link name="panda_link7">
@@ -346,5 +378,10 @@
     <child link="panda_link7"/>
     <axis xyz="0 0 1"/>
-    <limit effort="12" lower="-2.8973" upper="2.8973" velocity="2.6100"/>
+    <xacro:if value="${no_position_limits}">
+      <limit effort="12" lower="-20" upper="20" velocity="2.6100"/>
+    </xacro:if>
+    <xacro:unless value="${no_position_limits}">
+      <limit effort="12" lower="-2.8973" upper="2.8973" velocity="2.6100"/>
+    </xacro:unless>
   </joint>
   <link name="panda_link8">
