Commit message: clang format

File: mppi_examples/mppi_panda/resources/panda/panda.urdf.xacro (robot description, xacro)
@@ -1,521 +1,539 @@
 <?xml version="1.0" encoding="utf-8"?>
 <robot name="panda" xmlns:xacro="http://www.ros.org/wiki/xacro">
-  <xacro:arg name="resources_prefix"      default="" />
-  <xacro:arg name="resources_directory"   default="$(find mppi_panda)" />
-  <xacro:arg name="collision_format"      default="stl"/>
-  <xacro:arg name="collision_links"       default="true"/>
-  <xacro:arg name="collision_hand"        default="true"/>
-  <xacro:arg name="collision_finger"      default="true"/>
-  <xacro:arg name="no_position_limits"      default="true"/>
-  <xacro:arg name="add_finger"            default="false"/>
-  <xacro:property name="resources_prefix"     value="$(arg resources_prefix)" />
-  <xacro:property name="resources_directory"  value="$(arg resources_directory)" />
-  <xacro:property name="collision_format"     value="$(arg collision_format)" />
-  <xacro:property name="collision_links"      value="$(arg collision_links)"/>
-  <xacro:property name="collision_hand"       value="$(arg collision_hand)"/>
-  <xacro:property name="collision_finger"     value="$(arg collision_finger)"/>
-  <xacro:property name="no_position_limits"   value="$(arg no_position_limits)"/>
-  <xacro:property name="add_finger"           value="$(arg add_finger)" />
-  <xacro:macro name="panda_robot" params="parent_link:='world'">
-  <joint name="panda_joint_${parent_link}" type="fixed">
-    <parent link="${parent_link}"/>
-    <child link="panda_link0"/>
-    <origin rpy="0 0 0" xyz="0 0 0"/>
-  </joint>
-  <gazebo>
-    <plugin filename="libgazebo_ros_control.so" name="gazebo_ros_control">
-      <robotNamespace>/</robotNamespace>
-    </plugin>
-  </gazebo>
-  <gazebo reference="panda_link0"/>
-  <gazebo reference="panda_link1"/>
-  <gazebo reference="panda_link2"/>
-  <gazebo reference="panda_link3"/>
-  <gazebo reference="panda_link4"/>
-  <gazebo reference="panda_link5"/>
-  <gazebo reference="panda_link6"/>
-  <gazebo reference="panda_link7"/>
-  <gazebo reference="panda_link8"/>
-  <transmission name="panda_joint1_trans">
-    <type>transmission_interface/SimpleTransmission</type>
-    <joint name="panda_joint1">
-      <hardwareInterface>hardware_interface/PositionJointInterface</hardwareInterface>
-    </joint>
-    <actuator name="panda_joint1_motor">
-      <mechanicalReduction>1</mechanicalReduction>
-    </actuator>
-  </transmission>
-  <transmission name="panda_joint2_trans">
-    <type>transmission_interface/SimpleTransmission</type>
-    <joint name="panda_joint2">
-      <hardwareInterface>hardware_interface/PositionJointInterface</hardwareInterface>
-    </joint>
-    <actuator name="panda_joint2_motor">
-      <mechanicalReduction>1</mechanicalReduction>
-    </actuator>
-  </transmission>
-  <transmission name="panda_joint3_trans">
-    <type>transmission_interface/SimpleTransmission</type>
-    <joint name="panda_joint3">
-      <hardwareInterface>hardware_interface/PositionJointInterface</hardwareInterface>
-    </joint>
-    <actuator name="panda_joint3_motor">
-      <mechanicalReduction>1</mechanicalReduction>
-    </actuator>
-  </transmission>
-  <transmission name="panda_joint4_trans">
-    <type>transmission_interface/SimpleTransmission</type>
-    <joint name="panda_joint4">
-      <hardwareInterface>hardware_interface/PositionJointInterface</hardwareInterface>
-    </joint>
-    <actuator name="panda_joint4_motor">
-      <mechanicalReduction>1</mechanicalReduction>
-    </actuator>
-  </transmission>
-  <transmission name="panda_joint5_trans">
-    <type>transmission_interface/SimpleTransmission</type>
-    <joint name="panda_joint5">
-      <hardwareInterface>hardware_interface/PositionJointInterface</hardwareInterface>
-    </joint>
-    <actuator name="panda_joint5_motor">
-      <mechanicalReduction>1</mechanicalReduction>
-    </actuator>
-  </transmission>
-  <transmission name="panda_joint6_trans">
-    <type>transmission_interface/SimpleTransmission</type>
-    <joint name="panda_joint6">
-      <hardwareInterface>hardware_interface/PositionJointInterface</hardwareInterface>
-    </joint>
-    <actuator name="panda_joint6_motor">
-      <mechanicalReduction>1</mechanicalReduction>
-    </actuator>
-  </transmission>
-  <transmission name="panda_joint7_trans">
-    <type>transmission_interface/SimpleTransmission</type>
-    <joint name="panda_joint7">
-      <hardwareInterface>hardware_interface/PositionJointInterface</hardwareInterface>
-    </joint>
-    <actuator name="panda_joint7_motor">
-      <mechanicalReduction>1</mechanicalReduction>
-    </actuator>
-  </transmission>
-  <link name="panda_link0">
-    <inertial>
-      <mass value="2.92"/>
-      <origin rpy="0 0 0" xyz="-0.025566 -2.88e-05 0.057332"/>
-      <inertia ixx="0.00782229414331" ixy="-1.56191622996e-05" ixz="-0.00126005738123" iyy="0.0109027971813" iyz="1.08233858202e-05" izz="0.0102355503949"/>
-    </inertial>
-    <visual>
-      <origin rpy="0 0 0" xyz="0 0 0"/>
-      <geometry>
-        <mesh filename="${resources_prefix}${resources_directory}/resources/panda/meshes/visual/link0.dae"/>
-      </geometry>
-      <material name="">
-        <color rgba="1 1 1 1"/>
-      </material>
-    </visual>
-    <xacro:if value="${collision_links}">
-      <collision>
-        <origin rpy="0 0 0" xyz="0 0 0"/>
-        <geometry>
-          <mesh filename="${resources_prefix}${resources_directory}/resources/panda/meshes/collision/link0.${collision_format}"/>
-        </geometry>
-    </collision>
-    </xacro:if>
-  </link>
-  <link name="panda_link1">
-    <inertial>
-      <mass value="2.74"/>
-      <origin rpy="0 0 0" xyz="0 -0.0324958 -0.0675818"/>
-      <inertia ixx="0.0180416958283" ixy="0.0" ixz="0.0" iyy="0.0159136071891" iyz="0.0046758424612" izz="0.00620690827127"/>
-    </inertial>
-    <visual>
-      <origin rpy="0 0 0" xyz="0 0 0"/>
-      <geometry>
-        <mesh filename="${resources_prefix}${resources_directory}/resources/panda/meshes/visual/link1.dae"/>
-      </geometry>
-      <material name="">
-        <color rgba="1 1 1 1"/>
-      </material>
-    </visual>
-    <xacro:if value="${collision_links}">
-      <collision>
-        <origin rpy="0 0 0" xyz="0 0 0"/>
-        <geometry>
-          <mesh filename="${resources_prefix}${resources_directory}/resources/panda/meshes/collision/link1.${collision_format}"/>
-        </geometry>
-      </collision>
-    </xacro:if>
-  </link>
-  <joint name="panda_joint1" type="revolute">
-    <safety_controller k_position="100.0" k_velocity="40.0" soft_lower_limit="-2.8973" soft_upper_limit="2.8973"/>
-    <origin rpy="0 0 0" xyz="0 0 0.333"/>
-    <parent link="panda_link0"/>
-    <child link="panda_link1"/>
-    <axis xyz="0 0 1"/>
-    <xacro:if value="${no_position_limits}">
-      <limit effort="87" lower="-20" upper="20" velocity="2.1750"/>
-    </xacro:if>
-    <xacro:unless value="${no_position_limits}">
-      <limit effort="87" lower="-2.8973" upper="2.8973" velocity="2.1750"/>
-    </xacro:unless>
-  </joint>
-  <link name="panda_link2">
-    <inertial>
-      <mass value="2.74"/>
-      <origin rpy="0 0 0" xyz="0 -0.06861 0.0322285"/>
-      <inertia ixx="0.0182856182281" ixy="0.0" ixz="0.0" iyy="0.00621358421175" iyz="-0.00472844221905" izz="0.0161514346309"/>
-    </inertial>
-    <visual>
-      <origin rpy="0 0 0" xyz="0 0 0"/>
-      <geometry>
-        <mesh filename="${resources_prefix}${resources_directory}/resources/panda/meshes/visual/link2.dae"/>
-      </geometry>
-      <material name="">
-        <color rgba="1 1 1 1"/>
-      </material>
-    </visual>
-      <xacro:if value="${collision_links}">
-        <collision>
-          <origin rpy="0 0 0" xyz="0 0 0"/>
-          <geometry>
-            <mesh filename="${resources_prefix}${resources_directory}/resources/panda/meshes/collision/link2.${collision_format}"/>
-          </geometry>
-        </collision>
-      </xacro:if>
-  </link>
-  <joint name="panda_joint2" type="revolute">
-    <safety_controller k_position="100.0" k_velocity="40.0" soft_lower_limit="-1.7628" soft_upper_limit="1.7628"/>
-    <origin rpy="-1.57079632679 0 0" xyz="0 0 0"/>
-    <parent link="panda_link1"/>
-    <child link="panda_link2"/>
-    <axis xyz="0 0 1"/>
-    <xacro:if value="${no_position_limits}">
-      <limit effort="87" lower="-20" upper="20" velocity="2.1750"/>
-    </xacro:if>
-    <xacro:unless value="${no_position_limits}">
-      <limit effort="87" lower="-1.7628" upper="1.7628" velocity="2.1750"/>
-    </xacro:unless>
-  </joint>
-  <link name="panda_link3">
-    <inertial>
-      <mass value="2.38"/>
-      <origin rpy="0 0 0" xyz="0.0469893 0.0316374 -0.031704"/>
-      <inertia ixx="0.00771376630908" ixy="-0.00248490625138" ixz="-0.00332147581033" iyy="0.00989108008727" iyz="-0.00217796151484" izz="0.00811723558464"/>
-    </inertial>
-    <visual>
-      <origin rpy="0 0 0" xyz="0 0 0"/>
-      <geometry>
-        <mesh filename="${resources_prefix}${resources_directory}/resources/panda/meshes/visual/link3.dae"/>
-      </geometry>
-      <material name="">
-        <color rgba="1 1 1 1"/>
-      </material>
-    </visual>
-    <xacro:if value="${collision_links}">
-      <collision>
-        <origin rpy="0 0 0" xyz="0 0 0"/>
-        <geometry>
-          <mesh filename="${resources_prefix}${resources_directory}/resources/panda/meshes/collision/link3.${collision_format}"/>
-        </geometry>
-      </collision>
-    </xacro:if>
-  </link>
-  <joint name="panda_joint3" type="revolute">
-    <safety_controller k_position="100.0" k_velocity="40.0" soft_lower_limit="-2.8973" soft_upper_limit="2.8973"/>
-    <origin rpy="1.57079632679 0 0" xyz="0 -0.316 0"/>
-    <parent link="panda_link2"/>
-    <child link="panda_link3"/>
-    <axis xyz="0 0 1"/>
-    <xacro:if value="${no_position_limits}">
-      <limit effort="87" lower="-20" upper="20" velocity="2.1750"/>
-    </xacro:if>
-    <xacro:unless value="${no_position_limits}">
-      <limit effort="87" lower="-2.8973" upper="2.8973" velocity="2.1750"/>
-    </xacro:unless>
-  </joint>
-  <link name="panda_link4">
-    <inertial>
-      <mass value="2.38"/>
-      <origin rpy="0 0 0" xyz="-0.0360446 0.0336853 0.031882"/>
-      <inertia ixx="0.00799663881132" ixy="0.00347095570217" ixz="-0.00241222942995" iyy="0.00825390705278" iyz="0.00235774044121" izz="0.0102515004345"/>
-    </inertial>
-    <visual>
-      <origin rpy="0 0 0" xyz="0 0 0"/>
-      <geometry>
-        <mesh filename="${resources_prefix}${resources_directory}/resources/panda/meshes/visual/link4.dae"/>
-      </geometry>
-      <material name="">
-        <color rgba="1 1 1 1"/>
-      </material>
-    </visual>
-      <xacro:if value="${collision_links}">
-        <collision>
-          <origin rpy="0 0 0" xyz="0 0 0"/>
-          <geometry>
-            <mesh filename="${resources_prefix}${resources_directory}/resources/panda/meshes/collision/link4.${collision_format}"/>
-          </geometry>
-        </collision>
-      </xacro:if>
-  </link>
-  <joint name="panda_joint4" type="revolute">
-    <safety_controller k_position="100.0" k_velocity="40.0" soft_lower_limit="-3.0718" soft_upper_limit="0.0698"/>
-    <!-- soft_upper_limitr should be -0.0698, but that brakes simulation when initial position for this joint is 0.0 -->
-    <origin rpy="1.57079632679 0 0" xyz="0.0825 0 0"/>
-    <parent link="panda_link3"/>
-    <child link="panda_link4"/>
-    <axis xyz="0 0 1"/>
-    <xacro:if value="${no_position_limits}">
-      <limit effort="87" lower="-20" upper="20" velocity="2.1750"/>
-    </xacro:if>
-    <xacro:unless value="${no_position_limits}">
-      <limit effort="87" lower="-3.0718" upper="0.0698" velocity="2.1750"/>
-      <!-- upper should be -0.0698, but that brakes simulation when initial position for this joint is 0.0 -->
-    </xacro:unless>
-  </joint>
-  <link name="panda_link5">
-    <inertial>
-      <mass value="2.74"/>
-      <origin rpy="0 0 0" xyz="0 0.0610427 -0.104176"/>
-      <inertia ixx="0.030371374513" ixy="6.50283587108e-07" ixz="-1.05129179916e-05" iyy="0.0288752887402" iyz="-0.00775653445787" izz="0.00444134056164"/>
-    </inertial>
-    <visual>
-      <origin rpy="0 0 0" xyz="0 0 0"/>
-      <geometry>
-        <mesh filename="${resources_prefix}${resources_directory}/resources/panda/meshes/visual/link5.dae"/>
-      </geometry>
-      <material name="">
-        <color rgba="1 1 1 1"/>
-      </material>
-    </visual>
-    <xacro:if value="${collision_links}">
-      <collision>
-        <origin rpy="0 0 0" xyz="0 0 0"/>
-        <geometry>
-          <mesh filename="${resources_prefix}${resources_directory}/resources/panda/meshes/collision/link5.${collision_format}"/>
-        </geometry>
-      </collision>
-    </xacro:if>
-  </link>
-  <joint name="panda_joint5" type="revolute">
-    <safety_controller k_position="100.0" k_velocity="40.0" soft_lower_limit="-2.8973" soft_upper_limit="2.8973"/>
-    <origin rpy="-1.57079632679 0 0" xyz="-0.0825 0.384 0"/>
-    <parent link="panda_link4"/>
-    <child link="panda_link5"/>
-    <axis xyz="0 0 1"/>
-    <xacro:if value="${no_position_limits}">
-      <limit effort="12" lower="-20" upper="20" velocity="2.6100"/>
-    </xacro:if>
-    <xacro:unless value="${no_position_limits}">
-      <limit effort="12" lower="-2.8973" upper="2.8973" velocity="2.6100"/>
-    </xacro:unless>
-  </joint>
-  <link name="panda_link6">
-    <inertial>
-      <mass value="1.55"/>
-      <origin rpy="0 0 0" xyz="0.0510509 0.009108 0.0106343"/>
-      <inertia ixx="0.00303336450376" ixy="-0.000437276865508" ixz="0.000629257294877" iyy="0.00404479911567" iyz="0.000130472021025" izz="0.00558234286039"/>
-    </inertial>
-    <visual>
-      <origin rpy="0 0 0" xyz="0 0 0"/>
-      <geometry>
-        <mesh filename="${resources_prefix}${resources_directory}/resources/panda/meshes/visual/link6.dae"/>
-      </geometry>
-      <material name="">
-        <color rgba="1 1 1 1"/>
-      </material>
-    </visual>
-    <xacro:if value="${collision_links}">
-      <collision>
-        <origin rpy="0 0 0" xyz="0 0 0"/>
-        <geometry>
-          <mesh filename="${resources_prefix}${resources_directory}/resources/panda/meshes/collision/link6.${collision_format}"/>
-        </geometry>
-      </collision>
-    </xacro:if>
-  </link>
-  <joint name="panda_joint6" type="revolute">
-    <safety_controller k_position="100.0" k_velocity="40.0" soft_lower_limit="-0.0175" soft_upper_limit="3.7525"/>
-    <origin rpy="1.57079632679 0 0" xyz="0 0 0"/>
-    <parent link="panda_link5"/>
-    <child link="panda_link6"/>
-    <axis xyz="0 0 1"/>
-    <xacro:if value="${no_position_limits}">
-      <limit effort="12" lower="-20" upper="20" velocity="2.6100"/>
-    </xacro:if>
-    <xacro:unless value="${no_position_limits}">
-      <limit effort="12" lower="-0.0175" upper="3.7525" velocity="2.6100"/>
-    </xacro:unless>
-  </joint>
-  <link name="panda_link7">
-    <inertial>
-      <mass value="0.54"/>
-      <origin rpy="0 0 0" xyz="0.0109695 0.0107965 0.0650411"/>
-      <inertia ixx="0.000888868887021" ixy="-0.00012239074652" ixz="3.98699829666e-05" iyy="0.000888001373233" iyz="-9.33825115206e-05" izz="0.0007176834609"/>
-    </inertial>
-    <visual>
-      <origin rpy="0 0 0" xyz="0 0 0"/>
-      <geometry>
-        <mesh filename="${resources_prefix}${resources_directory}/resources/panda/meshes/visual/link7.dae"/>
-      </geometry>
-      <material name="">
-        <color rgba="1 1 1 1"/>
-      </material>
-    </visual>
-    <xacro:if value="${collision_links}">
-      <collision>
-        <origin rpy="0 0 0" xyz="0 0 0"/>
-        <geometry>
-          <mesh filename="${resources_prefix}${resources_directory}/resources/panda/meshes/collision/link7.${collision_format}"/>
-        </geometry>
-      </collision>
-    </xacro:if>
-  </link>
-  <joint name="panda_joint7" type="revolute">
-    <safety_controller k_position="100.0" k_velocity="40.0" soft_lower_limit="-2.8973" soft_upper_limit="2.8973"/>
-    <origin rpy="1.57079632679 0 0" xyz="0.088 0 0"/>
-    <parent link="panda_link6"/>
-    <child link="panda_link7"/>
-    <axis xyz="0 0 1"/>
-    <xacro:if value="${no_position_limits}">
-      <limit effort="12" lower="-20" upper="20" velocity="2.6100"/>
-    </xacro:if>
-    <xacro:unless value="${no_position_limits}">
-      <limit effort="12" lower="-2.8973" upper="2.8973" velocity="2.6100"/>
-    </xacro:unless>
-  </joint>
-  <link name="panda_link8">
-    <inertial>
-      <mass value="0.0"/>
-      <origin rpy="0 0 0" xyz="0.0 0.0 0.0"/>
-      <inertia ixx="0.0" ixy="0.0" ixz="0" iyy="0.0" iyz="0.0" izz="0.0"/>
-    </inertial>
-  </link>
-  <joint name="panda_joint8" type="fixed">
-    <origin rpy="0 0 0" xyz="0 0 0.107"/>
-    <parent link="panda_link7"/>
-    <child link="panda_link8"/>
-    <axis xyz="0 0 0"/>
-  </joint>
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
File: mppi_examples/mppi_panda/resources/panda/panda_standalone.urdf.xacro (robot description, xacro)
@@ -1,5 +1,5 @@
 <?xml version="1.0"?>
 <robot xmlns:xacro="http://www.ros.org/wiki/xacro" name="panda">
-    <xacro:include filename="$(find mppi_panda)/resources/panda/panda.urdf.xacro" />
+    <xacro:include filename="$(find mppi_panda)/resources/panda/panda.urdf.xacro"/>
     <link name="world"/>
     <xacro:panda_robot parent_link="world"/>

File: mppi_examples/mppi_panda_mobile/resources/panda/base.urdf.xacro (robot description, xacro)
@@ -1,20 +1,20 @@
 <?xml version="1.0" encoding="utf-8"?>
 <robot name="panda_mobile" xmlns:xacro="http://www.ros.org/wiki/xacro">
-  <xacro:macro name="panda_base" params="base_link:='base'">
-    <link name="${base_link}">
-    <collision>
-      <origin xyz="0 0 0" rpy="0 0 0"/>
-      <geometry>
-        <box size="0.5 0.5 0.25"/>
-      </geometry>
-    </collision>
-    <visual>
-      <origin xyz="0 0 0" rpy="0 0 0"/>
-      <geometry>
-        <box size="0.5 0.5 0.25"/>
-      </geometry>
-      <material name="green"/>
-    </visual>
-    </link>
-  </xacro:macro>
+    <xacro:macro name="panda_base" params="base_link:='base'">
+        <link name="${base_link}">
+            <collision>
+                <origin xyz="0 0 0" rpy="0 0 0"/>
+                <geometry>
+                    <box size="0.5 0.5 0.25"/>
+                </geometry>
+            </collision>
+            <visual>
+                <origin xyz="0 0 0" rpy="0 0 0"/>
+                <geometry>
+                    <box size="0.5 0.5 0.25"/>
+                </geometry>
+                <material name="green"/>
+            </visual>
+        </link>
+    </xacro:macro>
 </robot>

File: mppi_examples/mppi_panda_mobile/resources/panda/panda_mobile.urdf.xacro (robot description, xacro)
@@ -1,8 +1,8 @@
 <?xml version="1.0" encoding="utf-8"?>
 <robot name="panda" xmlns:xacro="http://www.ros.org/wiki/xacro">
-  <xacro:include filename="$(find mppi_panda)/resources/panda/panda.urdf.xacro" />
-  <xacro:include filename="$(find mppi_panda_mobile)/resources/panda/base.urdf.xacro" />
-  <xacro:property name="base_name" value="base"/>
-  <xacro:panda_base base_link="${base_name}"/>
-  <xacro:panda_robot parent_link="${base_name}"/>
+    <xacro:include filename="$(find mppi_panda)/resources/panda/panda.urdf.xacro"/>
+    <xacro:include filename="$(find mppi_panda_mobile)/resources/panda/base.urdf.xacro"/>
+    <xacro:property name="base_name" value="base"/>
+    <xacro:panda_base base_link="${base_name}"/>
+    <xacro:panda_robot parent_link="${base_name}"/>
 </robot>

File: mppi_examples/mppi_panda_raisim/data/panda_grasp.urdf.xacro (robot description, xacro)
@@ -1,5 +1,5 @@
 <?xml version="1.0"?>
 <robot xmlns:xacro="http://www.ros.org/wiki/xacro" name="panda">
-    <xacro:include filename="$(find mppi_panda)/resources/panda/panda.urdf.xacro" />
+    <xacro:include filename="$(find mppi_panda)/resources/panda/panda.urdf.xacro"/>
     <link name="world"/>
     <xacro:panda_robot parent_link="world"/>

Commit message: real simplifed finger contact model

File: mppi_examples/mppi_panda/resources/panda/panda.urdf.xacro (robot description, xacro)
@@ -486,9 +486,19 @@
                 <xacro:if value="${collision_finger}">
                     <collision>
-                        <!--origin rpy="0 0 0" xyz="0 0 0"/-->
-                        <origin rpy="0 0 3.14159265359" xyz="0 0.01 0.028"/>
+                        <origin rpy="0.0 0 0.0" xyz="0 0.018 0.01"/>
                         <geometry>
-                            <!--mesh filename="${resources_prefix}${resources_directory}/resources/panda/meshes/collision/finger.${collision_format}"/-->
-                            <box size="0.02 0.02 0.05"/>
+                            <box size="0.0222 0.015 0.02"/>
+                        </geometry>
+                    </collision>
+                    <collision>
+                        <origin rpy="${3.14 * 30 / 180.0} 0 0.0" xyz="0 0.017 0.027"/>
+                        <geometry>
+                            <box size="0.0222 0.007 0.025"/>
+                        </geometry>
+                    </collision>
+                    <collision>
+                        <origin rpy="0.0 0 0.0" xyz="0 0.007 0.045"/>
+                        <geometry>
+                            <box size="0.0222 0.0145 0.018"/>
                         </geometry>
                     </collision>
@@ -513,9 +523,19 @@
                 <xacro:if value="${collision_finger}">
                     <collision>
-                        <!-- origin rpy="0 0 3.14159265359" xyz="0 0 0"/ -->
-                        <origin rpy="0 0 3.14159265359" xyz="0 -0.01 0.028"/>
+                        <origin rpy="0.0 0 0.0" xyz="0 -0.018 0.01"/>
                         <geometry>
-                            <!--mesh filename="${resources_prefix}${resources_directory}/resources/panda/meshes/collision/finger.${collision_format}"/-->
-                            <box size="0.02 0.02 0.05"/>
+                            <box size="0.0222 0.015 0.02"/>
+                        </geometry>
+                    </collision>
+                    <collision>
+                        <origin rpy="${-3.14 * 30 / 180.0} 0 0.0" xyz="0 -0.017 0.027"/>
+                        <geometry>
+                            <box size="0.0222 0.007 0.025"/>
+                        </geometry>
+                    </collision>
+                    <collision>
+                        <origin rpy="0.0 0 0.0" xyz="0 -0.007 0.045"/>
+                        <geometry>
+                            <box size="0.0222 0.0145 0.018"/>
                         </geometry>
                     </collision>
