Commit message: optional panda damping

File: mppi_examples/mppi_panda/resources/panda/panda.urdf.xacro (robot description, xacro)
@@ -9,4 +9,6 @@
     <xacro:arg name="custom_fingers" default="false"/>
     <xacro:arg name="no_position_limits" default="true"/>
+    <xacro:arg name="friction" default="0.0"/>
+    <xacro:arg name="damping"  default="0.0"/>
     <xacro:arg name="add_finger" default="false"/>
     <xacro:property name="resources_prefix" value="$(arg resources_prefix)"/>
@@ -18,4 +20,6 @@
     <xacro:property name="no_position_limits" value="$(arg no_position_limits)"/>
     <xacro:property name="add_finger" value="$(arg add_finger)"/>
+    <xacro:property name="friction" default="$(arg friction)"/>
+    <xacro:property name="damping"  default="$(arg damping)"/>
     <xacro:include filename="$(find mppi_panda)/resources/panda/custom_fingers.urdf"/>
     <xacro:macro name="panda_robot" params="parent_link:='world' robot_description:=''">
@@ -166,4 +170,5 @@
                 <limit effort="87" lower="-2.8973" upper="2.8973" velocity="2.1750"/>
             </xacro:unless>
+            <dynamics damping="${damping}" friction="${friction}"/>
         </joint>
         <link name="panda_link2">
@@ -205,4 +210,5 @@
                 <limit effort="87" lower="-1.7628" upper="1.7628" velocity="2.1750"/>
             </xacro:unless>
+            <dynamics damping="${damping}" friction="${friction}"/>
         </joint>
         <link name="panda_link3">
@@ -244,4 +250,5 @@
                 <limit effort="87" lower="-2.8973" upper="2.8973" velocity="2.1750"/>
             </xacro:unless>
+            <dynamics damping="${damping}" friction="${friction}"/>
         </joint>
         <link name="panda_link4">
@@ -285,4 +292,5 @@
                 <!-- upper should be -0.0698, but that brakes simulation when initial position for this joint is 0.0 -->
             </xacro:unless>
+            <dynamics damping="${damping}" friction="${friction}"/>
         </joint>
         <link name="panda_link5">
@@ -324,4 +332,5 @@
                 <limit effort="12" lower="-2.8973" upper="2.8973" velocity="2.6100"/>
             </xacro:unless>
+            <dynamics damping="${damping}" friction="${friction}"/>
         </joint>
         <link name="panda_link6">
@@ -363,4 +372,5 @@
                 <limit effort="12" lower="-0.0175" upper="3.7525" velocity="2.6100"/>
             </xacro:unless>
+            <dynamics damping="${damping}" friction="${friction}"/>
         </joint>
         <link name="panda_link7">
@@ -402,4 +412,5 @@
                 <limit effort="12" lower="-2.8973" upper="2.8973" velocity="2.6100"/>
             </xacro:unless>
+            <dynamics damping="${damping}" friction="${friction}"/>
         </joint>
         <link name="panda_link8">

Commit message: finger distance was wrong

File: mppi_examples/mppi_panda/resources/panda/panda.urdf.xacro (robot description, xacro)
@@ -581,5 +581,5 @@
                 <parent link="panda_hand"/>
                 <child link="panda_leftfinger"/>
-                <origin rpy="0 0 0" xyz="0 0 0.0584"/>
+                <origin rpy="0 0 0" xyz="0 0 0.064"/> <!-- 0.0584 -->
                 <axis xyz="0 1 0"/>
                 <limit effort="20" lower="-0.001" upper="0.04" velocity="0.3"/>
@@ -588,5 +588,5 @@
                 <parent link="panda_hand"/>
                 <child link="panda_rightfinger"/>
-                <origin rpy="0 0 0" xyz="0 0 0.0584"/>
+                <origin rpy="0 0 0" xyz="0 0 0.064"/> <!-- 0.0584 -->
                 <axis xyz="0 -1 0"/>
                 <limit effort="20" lower="-0.001" upper="0.04" velocity="0.3"/>

Commit message: apparently the offset was right

File: mppi_examples/mppi_panda/resources/panda/panda.urdf.xacro (robot description, xacro)
@@ -581,5 +581,5 @@
                 <parent link="panda_hand"/>
                 <child link="panda_leftfinger"/>
-                <origin rpy="0 0 0" xyz="0 0 0.064"/> <!-- 0.0584 -->
+                <origin rpy="0 0 0" xyz="0 0 0.0584"/> <!-- 0.0584 -->
                 <axis xyz="0 1 0"/>
                 <limit effort="20" lower="-0.001" upper="0.04" velocity="0.3"/>
@@ -588,5 +588,5 @@
                 <parent link="panda_hand"/>
                 <child link="panda_rightfinger"/>
-                <origin rpy="0 0 0" xyz="0 0 0.064"/> <!-- 0.0584 -->
+                <origin rpy="0 0 0" xyz="0 0 0.0584"/> <!-- 0.064 -->
                 <axis xyz="0 -1 0"/>
                 <limit effort="20" lower="-0.001" upper="0.04" velocity="0.3"/>

Commit message: add bota sensor

File: mppi_examples/mppi_panda/resources/panda/panda.urdf.xacro (robot description, xacro)
@@ -11,4 +11,5 @@
     <xacro:arg name="friction" default="0.0"/>
     <xacro:arg name="damping"  default="0.0"/>
+    <xacro:arg name="add_wrench_sensor" default="false"/>
     <xacro:arg name="add_finger" default="false"/>
     <xacro:property name="resources_prefix" value="$(arg resources_prefix)"/>
@@ -22,5 +23,7 @@
     <xacro:property name="friction" default="$(arg friction)"/>
     <xacro:property name="damping"  default="$(arg damping)"/>
+    <xacro:property name="add_wrench_sensor" default="$(arg add_wrench_sensor)"/>
     <xacro:include filename="$(find mppi_panda)/resources/panda/custom_fingers.urdf"/>
+    <xacro:include filename="$(find mppi_panda)/sensors/bota/urdf/BFT_SENS_SER_M8.urdf.xacro"/>
     <xacro:macro name="panda_robot" params="parent_link:='world' robot_description:=''">
         <joint name="panda_joint_${parent_link}" type="fixed">
@@ -427,8 +430,27 @@
             <axis xyz="0 0 0"/>
         </joint>
+        <!-- Common link to connect the hand (with or without the sensor) -->
+        <link name="hand_flange"/>
+        <xacro:if value="${add_wrench_sensor}">
+            <xacro:BFT_SENS_SER_M8 parent="panda_link8">
+                <origin xyz="0 0 0" rpy="0 0 ${3.14/2}"/>
+            </xacro:BFT_SENS_SER_M8>
+            <joint name="hand_flange_joint" type="fixed">
+                <origin xyz="0 0 0" rpy="0 0 0"/>
+                <parent link="ft_sensor0_wrench"/>
+                <child link="hand_flange"/>
+            </joint>
+        </xacro:if>
+        <xacro:unless>
+            <joint name="hand_flange_joint" type="fixed">
+                <origin xyz="0 0 0" rpy="0 0 -0.785398163397"/>
+                <parent link="panda_link8"/>
+                <child link="hand_flange"/>
+            </joint>
+        </xacro:unless>
         <joint name="panda_hand_joint" type="fixed">
-            <parent link="panda_link8"/>
+            <parent link="hand_flange"/>
             <child link="panda_hand"/>
-            <origin rpy="0 0 -0.785398163397" xyz="0 0 0"/>
+            <origin rpy="0 0 0.0" xyz="0 0 0"/>
         </joint>
         <link name="panda_hand">
