Commit message: door integrated in simulation and control but something fishy when in collision with the door

File: mppi_examples/mppi_panda_raisim/data/door.urdf (robot description, URDF)
Before this commit: robot door, 4 links, 3 joints
Joints:
- joint fixed: origin xyz=0 0 0 -> xyz=0.65 0 0.01 rpy=0 0 3.14

Commit message: working solution with velocity control

File: mppi_examples/mppi_panda_raisim/data/door.urdf (robot description, URDF)
Before this commit: robot door, 4 links, 3 joints
Links:
- removed link door_base_link
- added link door_frame, mass 1.0; collision box size=0.05 0.6 0.5; visual box size=0.05 0.6 0.5
Joints:
- joint door_joint: origin xyz=0 0 0 -> xyz=0.036 0 0; parent door_base_link -> door_frame
- joint fixed: child door_base_link -> door_frame

Commit message: updated urdf

File: mppi_examples/mppi_panda_raisim/data/door.urdf (robot description, URDF)
Before this commit: robot door, 4 links, 3 joints
Links:
- link door_frame: mass 1.0 -> None

Commit message: moving door on the side

File: mppi_examples/mppi_panda_raisim/data/door.urdf (robot description, URDF)
Before this commit: robot door, 4 links, 3 joints
Joints:
- joint fixed: origin xyz=0.65 0 0.01 rpy=0 0 3.14 -> xyz=0.65 0.3 0.01 rpy=0 0 3.14

Commit message: grasping in the cost function

File: mppi_examples/mppi_panda_raisim/data/door.urdf (robot description, URDF)
Before this commit: robot door, 4 links, 3 joints
Joints:
- joint door_joint: limit (none) -> lower=0 upper=1.57 effort=100 velocity=10.0; type continuous -> revolute

Commit message: working door openinggit add -A!

File: mppi_examples/mppi_panda_raisim/data/door.urdf (robot description, URDF)
Before this commit: robot door, 4 links, 3 joints
Joints:
- joint door_joint: origin xyz=0.036 0 0 -> xyz=0.046 0 0

File: mppi_examples/mppi_panda_raisim/data/panda_grasp.urdf.xacro (robot description, xacro)
@@ -10,5 +10,5 @@
             <child link="panda_grasp"/>
             <axis xyz="0 1 0"/>
-            <origin xyz="0 0 0.09" rpy="0 0 0"/>
+            <origin xyz="0 0 0.1" rpy="0 0 0"/>
         </joint>
     </xacro:if>

Commit message: adding door step]

File: mppi_examples/mppi_panda_raisim/data/door.urdf (robot description, URDF)
Before this commit: robot door, 4 links, 3 joints
Links:
- added link door_frame_step; collision box size=0.081 0.6 0.5; visual box size=0.081 0.6 0.10
Joints:
- added joint step_joint: type fixed, parent door_frame, child door_frame_step, origin xyz=0.0155 0 0.31 rpy=0 0 0, axis 0 1 0

Commit message: adding contact state

File: mppi_examples/mppi_panda_raisim/data/door.urdf (robot description, URDF)
Before this commit: robot door, 5 links, 4 joints
Links:
- link door_frame_step: geometry collision box size=0.081 0.6 0.10; visual box size=0.081 0.6 0.10
Joints:
- joint handle_joint: origin xyz=0.035 0 0.47 rpy=1.5708 0 0 -> xyz=0.155 0 0.47 rpy=1.5708 0 0

File: mppi_examples/mppi_panda_raisim/data/panda.urdf (robot description, URDF)
Before this commit: robot panda, 13 links, 12 joints
Links:
- link panda_hand: geometry collision box size=0.035 0.19 0.065; visual mesh filename=/home/giuseppe/student_projects_ws/src/sampling_based_contr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
- link panda_leftfinger: geometry collision box size=0.02 0.02 0.05; visual mesh filename=/home/giuseppe/student_projects_ws/src/sampling_based_contr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
- link panda_rightfinger: geometry collision box size=0.02 0.02 0.05; visual mesh filename=/home/giuseppe/student_projects_ws/src/sampling_based_contr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
Joints:
- joint panda_joint1: limit lower=-2.8973 upper=2.8973 effort=87 velocity=2.1750 -> lower=-20 upper=20 effort=87 velocity=2.1750
- joint panda_joint2: limit lower=-1.7628 upper=1.7628 effort=87 velocity=2.1750 -> lower=-20 upper=20 effort=87 velocity=2.1750
- joint panda_joint3: limit lower=-2.8973 upper=2.8973 effort=87 velocity=2.1750 -> lower=-20 upper=20 effort=87 velocity=2.1750
- joint panda_joint4: limit lower=-3.0718 upper=0.0698 effort=87 velocity=2.1750 -> lower=-20 upper=20 effort=87 velocity=2.1750
- joint panda_joint5: limit lower=-2.8973 upper=2.8973 effort=12 velocity=2.6100 -> lower=-20 upper=20 effort=12 velocity=2.6100
- joint panda_joint6: limit lower=-0.0175 upper=3.7525 effort=12 velocity=2.6100 -> lower=-20 upper=20 effort=12 velocity=2.6100
- joint panda_joint7: limit lower=-2.8973 upper=2.8973 effort=12 velocity=2.6100 -> lower=-20 upper=20 effort=12 velocity=2.6100

Commit message: contact state and cost

File: mppi_examples/mppi_panda_raisim/data/door.urdf (robot description, URDF)
Before this commit: robot door, 5 links, 4 joints
Links:
- removed link door_frame_step
Joints:
- removed joint step_joint
- joint handle_joint: origin xyz=0.155 0 0.47 rpy=1.5708 0 0 -> xyz=0.055 0 0.47 rpy=1.5708 0 0
