Commit message: working with microwave

File: mppi_examples/mppi_manipulation/data/valve.urdf.xacro (robot description, xacro)
@@ -1,11 +1,11 @@
 <?xml version="1.0" ?>
 <robot name="valve">
-    <arg name="resource_prefix" default="file://"/>
-    <arg name="resource_directory" default="$(find mppi_panda_raisim)/data/meshes"/>
+    <arg name="resource_prefix" default=""/>
+    <arg name="resource_directory" default="$(find mppi_manipulation)/data/meshes"/>
     <link name="world"/>
     <joint name="fixed" type="fixed">
         <parent link="world"/>
         <child link="valve_base"/>
-        <origin xyz="0 0 0" rpy="0 0 0"/>
+        <origin xyz="0.7 0.0 0.4" rpy="1.57 0 0"/>
     </joint>
     <link name="valve_base"/>
@@ -19,5 +19,5 @@
             <origin rpy="0 0 0" xyz="0 0 0"/>
             <geometry>
-                <mesh filename="$(arg resource_prefix)$(arg resource_directory)/valve_visual.dae"/>
+                <mesh filename="$(arg resource_prefix)$(arg resource_directory)/valve_visual.obj"/>
             </geometry>
         </visual>
@@ -25,9 +25,9 @@
             <origin rpy="0 0 0" xyz="0 0 0"/>
 	    <geometry>
-                <mesh  filename="$(arg resource_prefix)$(arg resource_directory)/valve_collision.dae"/>
+                <mesh  filename="$(arg resource_prefix)$(arg resource_directory)/valve_simple_collision.obj"/>
             </geometry>
         </collision>
     </link>
-    <joint name="handle_joint" type="revolute">
+    <joint name="articulation_joint" type="revolute">
         <parent link="valve_base"/>
         <child link="handle_link"/>

Commit message: fixing valve stuff

File: mppi_examples/mppi_manipulation/data/valve.urdf.xacro (robot description, xacro)
@@ -25,5 +25,5 @@
             <origin rpy="0 0 0" xyz="0 0 0"/>
 	    <geometry>
-                <mesh  filename="$(arg resource_prefix)$(arg resource_directory)/valve_simple_collision.obj"/>
+                <mesh  filename="$(arg resource_prefix)$(arg resource_directory)/valve_collision.obj"/>
             </geometry>
         </collision>
@@ -34,5 +34,5 @@
         <origin xyz="0 0 0" rpy="0 0 0"/>
         <dynamics damping="1.0" friction="2.0"/>
-        <axis xyz="0 0 1"/>
+        <axis xyz="0 1 0"/>
         <limit upper="3.14" lower="3.14" effort="100" velocity="1.0"/>
     </joint>
