Commit message: replacing threadpool with openmp

File: mppi_examples/mppi_manipulation/data/valve.urdf (robot description, URDF)
Before this commit: robot valve, 3 links, 2 joints
Links:
- link handle_link: geometry collision mesh filename=/home/giuseppe/student_projects_ws/src/sampling_based_contr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; visual mesh filename=/home/giuseppe/student_projects_ws/src/sampling_based_contr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
Joints:
- removed joint handle_joint
- added joint articulation_joint: type revolute, parent valve_base, child handle_link, origin xyz=0 0 0 rpy=0 0 0, axis 0 1 0, limit lower=3.14 upper=3.14 effort=100 velocity=1.0
- joint fixed: origin xyz=0 0 0 rpy=0 0 0 -> xyz=0.7 0.0 0.4 rpy=1.57 0 0
