Commit message: working state assembler in dummy simulation

File: mppi_examples/mppi_manipulation/data/shelf.urdf.xacro (robot description, xacro)
@@ -31,9 +31,16 @@
         </collision>
     </link>
+    <link name="door_hinge"/>
+    <joint name="door_hinge_joint" type="fixed">
+        <parent link="shelf"/>
+        <child link="door_hinge"/>
+        <dynamics damping="2.0" friction="4.0"/>
+        <origin xyz="0 -${door_length} ${door_height/2}"/>
+    </joint>
     <joint name="articulation_joint" type="revolute">
-        <parent link="shelf"/>
+        <parent link="door_hinge"/>
         <child link="door"/>
         <dynamics damping="2.0" friction="4.0"/>
-        <origin xyz="0 -${door_length} ${door_height/2}"/>
+        <origin xyz="0 0 0"/>
         <axis xyz="0 0 -1"/>
         <limit effort="100" lower="0" upper="1.57" velocity="10.0"/>
