Commit message: observer working in sim

File: mppi_examples/mppi_manipulation/data/panda_mobile_gazebo.urdf.xacro (robot description, xacro)
@@ -13,5 +13,5 @@
     </joint>
     <link name="franka_mount_link"/>
-    <xacro:panda_robot parent_link="franka_mount_link"/>
+    <xacro:panda_robot parent_link="franka_mount_link" robot_description="/robot_description_for_gazebo"/>
     <!--    Add utility grasp frame-->
     <xacro:if value="${add_finger}">

File: mppi_examples/mppi_manipulation/data/ridgeback.urdf.xacro (robot description, xacro)
@@ -22,4 +22,18 @@
             <child link="reference_link"/>
         </joint>
+<!--        Just an hack to get the reference pose from gazebo: using a movable joint does not cause collapse of the model-->
+        <link name="reference_link_gazebo">
+            <inertial>
+                <mass value="0.001"/>
+                <origin xyz="0 0 0" rpy="0 0 0"/>
+                <inertia ixx="${dummy_inertia}" ixy="0.0" ixz="0.0" iyy="${dummy_inertia}" iyz="0.0" izz="${dummy_inertia}"/>
+            </inertial>
+        </link>
+        <joint name="reference_link_gazeb_joint" type="revolute">
+            <origin xyz="-0.343 0 0.77" rpy="0 0 0"/>
+            <parent link="mid_mount"/>
+            <child link="reference_link_gazebo"/>
+            <limit upper="0.0" lower="0.0" effort="0.0" velocity="0.0"/>
+        </joint>
     </xacro:macro>
 </robot>

File: mppi_examples/mppi_panda/resources/panda/panda.urdf.xacro (robot description, xacro)
@@ -17,5 +17,5 @@
     <xacro:property name="no_position_limits" value="$(arg no_position_limits)"/>
     <xacro:property name="add_finger" value="$(arg add_finger)"/>
-    <xacro:macro name="panda_robot" params="parent_link:='world'">
+    <xacro:macro name="panda_robot" params="parent_link:='world' robot_description:=''">
         <joint name="panda_joint_${parent_link}" type="fixed">
             <parent link="${parent_link}"/>
@@ -26,4 +26,5 @@
             <plugin filename="libgazebo_ros_control.so" name="gazebo_ros_control">
                 <robotNamespace>/</robotNamespace>
+                <robotParam>/${robot_description}</robotParam>
             </plugin>
         </gazebo>
