Commit message: refactoring for remote visualization

File: mppi_examples/mppi_manipulation/data/ridgeback.urdf.xacro (robot description, xacro)
@@ -5,9 +5,9 @@
         <!-- Sensor mount -->
         <link name="ridgeback_sensor_mount_link">
-            <visual>
+<!--             <visual>
                 <geometry>
-                    <mesh filename="${resources_prefix}$(find mppi_manipulation)/data/meshes/ridgeback_sensor_mount.dae"/>
+                    <mesh filename="package://mppi_manipulation/data/meshes/ridgeback_sensor_mount.dae"/>
                 </geometry>
-            </visual>
+            </visual> -->
         </link>
         <joint name="ridgeback_sensor_mount_joint" type="fixed">

File: mppi_examples/mppi_manipulation/data/ridgeback.xacro (robot description, xacro)
@@ -1,4 +1,6 @@
 <?xml version="1.0"?>
 <robot name="ridgeback" xmlns:xacro="http://ros.org/wiki/xacro">
+    <xacro:arg name='ridgeback_resources_prefix' default='package://ridgeback_description'/>
+    <xacro:property name='ridgeback_resources_prefix' default="$(arg ridgeback_resources_prefix)"/>
     <xacro:property name="PI" value="3.1415926535897931" />
     <xacro:property name="wheel_radius" value="0.0759" />
@@ -48,5 +50,5 @@
             <origin xyz="0 0 0" rpy="0 0 0" />
             <geometry>
-                <mesh filename="${resources_prefix}$(find ridgeback_description)/meshes/body.stl"/>
+                <mesh filename="${ridgeback_resources_prefix}/meshes/body.stl"/>
             </geometry>
             <material name="black" />
@@ -75,5 +77,5 @@
             <origin xyz="0 0 0" rpy="0 0 ${PI}" />
             <geometry>
-                <mesh filename="${resources_prefix}$(find ridgeback_description)/meshes/side-cover.stl"/>
+                <mesh filename="${ridgeback_resources_prefix}/meshes/side-cover.stl"/>
             </geometry>
             <material name="yellow" />
@@ -84,5 +86,5 @@
             <origin xyz="0 0 0" rpy="0 0 0" />
             <geometry>
-                <mesh filename="${resources_prefix}$(find ridgeback_description)/meshes/side-cover.stl"/>
+                <mesh filename="${ridgeback_resources_prefix}/meshes/side-cover.stl"/>
             </geometry>
             <material name="yellow" />
@@ -98,5 +100,5 @@
             <origin xyz="0 0 0" rpy="0 0 0" />
             <geometry>
-                <mesh filename="${resources_prefix}$(find ridgeback_description)/meshes/end-cover.stl" />
+                <mesh filename="${ridgeback_resources_prefix}/meshes/end-cover.stl" />
             </geometry>
             <material name="black" />
@@ -112,5 +114,5 @@
             <origin xyz="0 0 0" rpy="0 0 ${PI}" />
             <geometry>
-                <mesh filename="${resources_prefix}$(find ridgeback_description)/meshes/end-cover.stl" />
+                <mesh filename="${ridgeback_resources_prefix}/meshes/end-cover.stl" />
             </geometry>
             <material name="black" />
@@ -131,5 +133,5 @@
             <origin xyz="0 0 0" rpy="0 0 0" />
             <geometry>
-                <mesh filename="${resources_prefix}$(find ridgeback_description)/meshes/lights.stl" />
+                <mesh filename="${ridgeback_resources_prefix}/meshes/lights.stl" />
             </geometry>
             <material name="white" />
@@ -140,5 +142,5 @@
             <origin xyz="0 0 0" rpy="0 0 ${PI}" />
             <geometry>
-                <mesh filename="${resources_prefix}$(find ridgeback_description)/meshes/lights.stl" />
+                <mesh filename="${ridgeback_resources_prefix}/meshes/lights.stl" />
             </geometry>
             <material name="red" />
@@ -154,5 +156,5 @@
             <origin xyz="0 0 0" rpy="0 0 0" />
             <geometry>
-                <mesh filename="${resources_prefix}$(find ridgeback_description)/meshes/top.stl" />
+                <mesh filename="${ridgeback_resources_prefix}/meshes/top.stl" />
             </geometry>
             <material name="black" />
@@ -168,5 +170,5 @@
             <origin xyz="0 0 0" rpy="0 ${PI/2} 0" />
             <geometry>
-                <mesh filename="${resources_prefix}$(find ridgeback_description)/meshes/axle.stl" />
+                <mesh filename="${ridgeback_resources_prefix}/meshes/axle.stl" />
             </geometry>
             <material name="black" />

File: mppi_examples/mppi_manipulation/data/ridgeback_gazebo.urdf.xacro (robot description, xacro)
@@ -12,5 +12,5 @@
                 <origin xyz="0 0 0" rpy="${PI/2} 0 0"/>
                 <geometry>
-                    <mesh filename="${resources_prefix}$(find ridgeback_description)/meshes/wheel.stl"/>
+                    <mesh filename="package://ridgeback_description/meshes/wheel.stl"/>
                 </geometry>
                 <material name="black"/>
@@ -60,5 +60,5 @@
                 <origin xyz="0 0 0" rpy="${PI/2} 0 ${PI/2}"/>
                 <geometry>
-                    <mesh filename="${resources_prefix}$(find ridgeback_description)/meshes/rocker.stl"/>
+                    <mesh filename="package://ridgeback_description/meshes/rocker.stl"/>
                 </geometry>
                 <material name="black"/>
