Commit message: minor fixes

File: mppi_examples/mppi_manipulation/data/planar_base.urdf.xacro (robot description, xacro)
@@ -41,5 +41,5 @@
             <origin rpy="0 0 0" xyz="0.0 0.0 0.0"/>
             <axis xyz="1 0 0"/>
-            <limit effort="1000.0" lower="-100" upper="100" velocity="1.0"/>
+            <limit effort="1000.0" lower="-10" upper="10" velocity="1.0"/>
             <dynamics damping="10.0" friction="10"/>
         </joint>
@@ -50,5 +50,5 @@
             <origin rpy="0 0 0" xyz="0.0 0.0 0.0"/>
             <axis xyz="0 1 0"/>
-            <limit effort="1000.0" lower="-100" upper="100" velocity="1.0"/>
+            <limit effort="1000.0" lower="-10" upper="10" velocity="1.0"/>
             <dynamics damping="10.0" friction="10"/>
         </joint>

Commit message: chaning dynamic properties of the base

File: mppi_examples/mppi_manipulation/data/planar_base.urdf.xacro (robot description, xacro)
@@ -18,5 +18,5 @@
             <inertial>
                 <origin rpy="0 0 0" xyz="0.0 0.0 0.0"/>
-                <mass value="10.0"/>
+                <mass value="1.0"/>
                 <inertia ixx="1.0" ixy="0.0" ixz="0.0" iyy="1.0" iyz="0.0" izz="1.0"/>
             </inertial>
@@ -25,5 +25,5 @@
             <inertial>
                 <origin rpy="0 0 0" xyz="0.0 0.0 0.0"/>
-                <mass value="10.0"/>
+                <mass value="1.0"/>
                 <inertia ixx="1.0" ixy="0.0" ixz="0.0" iyy="1.0" iyz="0.0" izz="1.0"/>
             </inertial>
@@ -32,5 +32,5 @@
             <inertial>
                 <origin rpy="0 0 0" xyz="0.0 0.0 0.0"/>
-                <mass value="10.0"/>
+                <mass value="1.0"/>
                 <inertia ixx="1.0" ixy="0.0" ixz="0.0" iyy="1.0" iyz="0.0" izz="1.0"/>
             </inertial>
@@ -42,5 +42,5 @@
             <axis xyz="1 0 0"/>
             <limit effort="1000.0" lower="-10" upper="10" velocity="1.0"/>
-            <dynamics damping="10.0" friction="10"/>
+            <dynamics damping="1.0" friction="1"/>
         </joint>
         <xacro:add_transmission joint_name="x_base_joint"/>
@@ -51,5 +51,5 @@
             <axis xyz="0 1 0"/>
             <limit effort="1000.0" lower="-10" upper="10" velocity="1.0"/>
-            <dynamics damping="10.0" friction="10"/>
+            <dynamics damping="1.0" friction="1"/>
         </joint>
         <xacro:add_transmission joint_name="y_base_joint"/>
@@ -60,5 +60,5 @@
             <axis xyz="0 0 1"/>
             <limit effort="1000.0" velocity="1.0" upper="10.0" lower="-10.0"/>
-            <dynamics damping="10.0" friction="10"/>
+            <dynamics damping="1.0" friction="1"/>
         </joint>
         <xacro:add_transmission joint_name="pivot_joint"/>

Commit message: base revolute joint is the first joint

File: mppi_examples/mppi_manipulation/data/planar_base.urdf.xacro (robot description, xacro)
@@ -36,6 +36,15 @@
             </inertial>
         </link>
+        <joint name="pivot_joint" type="revolute">
+            <parent link="omni_base_root_link"/>
+            <child link="pivot"/>
+            <origin rpy="0 0 0" xyz="0.0 0.0 0.0"/>
+            <axis xyz="0 0 1"/>
+            <limit effort="1000.0" velocity="1.0" upper="10.0" lower="-10.0"/>
+            <dynamics damping="1.0" friction="1"/>
+        </joint>
+        <xacro:add_transmission joint_name="pivot_joint"/>
         <joint name="x_base_joint" type="prismatic">
-            <parent link="omni_base_root_link"/>
+            <parent link="pivot"/>
             <child link="x_slider"/>
             <origin rpy="0 0 0" xyz="0.0 0.0 0.0"/>
@@ -54,15 +63,6 @@
         </joint>
         <xacro:add_transmission joint_name="y_base_joint"/>
-        <joint name="pivot_joint" type="revolute">
+        <joint name="omni_base_flange" type="fixed">
             <parent link="y_slider"/>
-            <child link="pivot"/>
-            <origin rpy="0 0 0" xyz="0.0 0.0 0.0"/>
-            <axis xyz="0 0 1"/>
-            <limit effort="1000.0" velocity="1.0" upper="10.0" lower="-10.0"/>
-            <dynamics damping="1.0" friction="1"/>
-        </joint>
-        <xacro:add_transmission joint_name="pivot_joint"/>
-        <joint name="omni_base_flange" type="fixed">
-            <parent link="pivot"/>
             <child link="${connect_to}"/>
         </joint>

Commit message: Revert "base revolute joint is the first joint"
This reverts commit f99cc8a6af46db51a483d45117b6b8d0471a77c1.

File: mppi_examples/mppi_manipulation/data/planar_base.urdf.xacro (robot description, xacro)
@@ -36,15 +36,6 @@
             </inertial>
         </link>
-        <joint name="pivot_joint" type="revolute">
+        <joint name="x_base_joint" type="prismatic">
             <parent link="omni_base_root_link"/>
-            <child link="pivot"/>
-            <origin rpy="0 0 0" xyz="0.0 0.0 0.0"/>
-            <axis xyz="0 0 1"/>
-            <limit effort="1000.0" velocity="1.0" upper="10.0" lower="-10.0"/>
-            <dynamics damping="1.0" friction="1"/>
-        </joint>
-        <xacro:add_transmission joint_name="pivot_joint"/>
-        <joint name="x_base_joint" type="prismatic">
-            <parent link="pivot"/>
             <child link="x_slider"/>
             <origin rpy="0 0 0" xyz="0.0 0.0 0.0"/>
@@ -63,6 +54,15 @@
         </joint>
         <xacro:add_transmission joint_name="y_base_joint"/>
+        <joint name="pivot_joint" type="revolute">
+            <parent link="y_slider"/>
+            <child link="pivot"/>
+            <origin rpy="0 0 0" xyz="0.0 0.0 0.0"/>
+            <axis xyz="0 0 1"/>
+            <limit effort="1000.0" velocity="1.0" upper="10.0" lower="-10.0"/>
+            <dynamics damping="1.0" friction="1"/>
+        </joint>
+        <xacro:add_transmission joint_name="pivot_joint"/>
         <joint name="omni_base_flange" type="fixed">
-            <parent link="y_slider"/>
+            <parent link="pivot"/>
             <child link="${connect_to}"/>
         </joint>

Commit message: adding greater rotational inertia

File: mppi_examples/mppi_manipulation/data/planar_base.urdf.xacro (robot description, xacro)
@@ -33,5 +33,5 @@
                 <origin rpy="0 0 0" xyz="0.0 0.0 0.0"/>
                 <mass value="1.0"/>
-                <inertia ixx="1.0" ixy="0.0" ixz="0.0" iyy="1.0" iyz="0.0" izz="1.0"/>
+                <inertia ixx="1.0" ixy="0.0" ixz="0.0" iyy="1.0" iyz="0.0" izz="4.0"/>
             </inertial>
         </link>
@@ -59,6 +59,6 @@
             <origin rpy="0 0 0" xyz="0.0 0.0 0.0"/>
             <axis xyz="0 0 1"/>
-            <limit effort="1000.0" velocity="1.0" upper="10.0" lower="-10.0"/>
-            <dynamics damping="1.0" friction="1"/>
+            <limit effort="10.0" velocity="1.0" upper="10.0" lower="-10.0"/>
+            <dynamics damping="5.0" friction="1"/>
         </joint>
         <xacro:add_transmission joint_name="pivot_joint"/>

Commit message: saturday tests

File: mppi_examples/mppi_manipulation/data/planar_base.urdf.xacro (robot description, xacro)
@@ -18,6 +18,6 @@
             <inertial>
                 <origin rpy="0 0 0" xyz="0.0 0.0 0.0"/>
-                <mass value="1.0"/>
-                <inertia ixx="1.0" ixy="0.0" ixz="0.0" iyy="1.0" iyz="0.0" izz="1.0"/>
+                <mass value="0.01"/>
+                <inertia ixx="0.01" ixy="0.0" ixz="0.0" iyy="0.01" iyz="0.0" izz="0.01"/>
             </inertial>
         </link>
@@ -25,6 +25,6 @@
             <inertial>
                 <origin rpy="0 0 0" xyz="0.0 0.0 0.0"/>
-                <mass value="1.0"/>
-                <inertia ixx="1.0" ixy="0.0" ixz="0.0" iyy="1.0" iyz="0.0" izz="1.0"/>
+                <mass value="0.01"/>
+                <inertia ixx="0.01" ixy="0.0" ixz="0.0" iyy="0.01" iyz="0.0" izz="0.01"/>
             </inertial>
         </link>
@@ -32,6 +32,6 @@
             <inertial>
                 <origin rpy="0 0 0" xyz="0.0 0.0 0.0"/>
-                <mass value="1.0"/>
-                <inertia ixx="1.0" ixy="0.0" ixz="0.0" iyy="1.0" iyz="0.0" izz="4.0"/>
+                <mass value="0.01"/>
+                <inertia ixx="0.01" ixy="0.0" ixz="0.0" iyy="0.01" iyz="0.0" izz="0.01"/>
             </inertial>
         </link>
@@ -42,5 +42,5 @@
             <axis xyz="1 0 0"/>
             <limit effort="1000.0" lower="-10" upper="10" velocity="1.0"/>
-            <dynamics damping="1.0" friction="1"/>
+            <dynamics damping="0.0" friction="10"/>
         </joint>
         <xacro:add_transmission joint_name="x_base_joint"/>
@@ -51,5 +51,5 @@
             <axis xyz="0 1 0"/>
             <limit effort="1000.0" lower="-10" upper="10" velocity="1.0"/>
-            <dynamics damping="1.0" friction="1"/>
+            <dynamics damping="0.0" friction="10"/>
         </joint>
         <xacro:add_transmission joint_name="y_base_joint"/>
@@ -59,6 +59,6 @@
             <origin rpy="0 0 0" xyz="0.0 0.0 0.0"/>
             <axis xyz="0 0 1"/>
-            <limit effort="10.0" velocity="1.0" upper="10.0" lower="-10.0"/>
-            <dynamics damping="5.0" friction="1"/>
+            <limit effort="1000.0" velocity="1.0" upper="10.0" lower="-10.0"/>
+            <dynamics damping="0.0" friction="10"/>
         </joint>
         <xacro:add_transmission joint_name="pivot_joint"/>
