Commit message: add object_modeling pkg

File: mppi_examples/mppi_manipulation/data/panda.urdf (robot description, URDF)
Before this commit: robot panda, 13 links, 12 joints
Links:
- link panda_hand: geometry collision box size=0.035 0.19 0.065; visual mesh filename=/home/boyang/catkin_ws/src/sampling_based_control/mppi_exam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
- link panda_leftfinger: geometry collision box size=0.02 0.02 0.05; visual mesh filename=/home/boyang/catkin_ws/src/sampling_based_control/mppi_exam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
- link panda_link0: geometry collision mesh filename=/home/boyang/catkin_ws/src/sampling_based_control/mppi_exam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; visual mesh filename=/home/boyang/catkin_ws/src/sampling_based_control/mppi_exam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
- link panda_link1: geometry collision mesh filename=/home/boyang/catkin_ws/src/sampling_based_control/mppi_exam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; visual mesh filename=/home/boyang/catkin_ws/src/sampling_based_control/mppi_exam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
- link panda_link2: geometry collision mesh filename=/home/boyang/catkin_ws/src/sampling_based_control/mppi_exam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; visual mesh filename=/home/boyang/catkin_ws/src/sampling_based_control/mppi_exam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
- link panda_link3: geometry collision mesh filename=/home/boyang/catkin_ws/src/sampling_based_control/mppi_exam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; visual mesh filename=/home/boyang/catkin_ws/src/sampling_based_control/mppi_exam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
- link panda_link4: geometry collision mesh filename=/home/boyang/catkin_ws/src/sampling_based_control/mppi_exam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; visual mesh filename=/home/boyang/catkin_ws/src/sampling_based_control/mppi_exam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
- link panda_link5: geometry collision mesh filename=/home/boyang/catkin_ws/src/sampling_based_control/mppi_exam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; visual mesh filename=/home/boyang/catkin_ws/src/sampling_based_control/mppi_exam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
- link panda_link6: geometry collision mesh filename=/home/boyang/catkin_ws/src/sampling_based_control/mppi_exam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; visual mesh filename=/home/boyang/catkin_ws/src/sampling_based_control/mppi_exam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
- link panda_link7: geometry collision mesh filename=/home/boyang/catkin_ws/src/sampling_based_control/mppi_exam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; visual mesh filename=/home/boyang/catkin_ws/src/sampling_based_control/mppi_exam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
- link panda_rightfinger: geometry collision box size=0.02 0.02 0.05; visual mesh filename=/home/boyang/catkin_ws/src/sampling_based_control/mppi_exam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

File: mppi_examples/mppi_manipulation/data/panda_mobile_fixed.urdf (robot description, URDF)
Before this commit: robot panda, 29 links, 28 joints
Links:
- link axle_link: geometry visual mesh filename=/home/boyang/catkin_ws/src/ridgeback/ridgeback_description/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
- link chassis_link: geometry visual mesh filename=/home/boyang/catkin_ws/src/ridgeback/ridgeback_description/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
- link front_cover_link: geometry visual mesh filename=/home/boyang/catkin_ws/src/ridgeback/ridgeback_description/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
- link front_lights_link: geometry visual mesh filename=/home/boyang/catkin_ws/src/ridgeback/ridgeback_description/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
- link left_side_cover_link: geometry visual mesh filename=/home/boyang/catkin_ws/src/ridgeback/ridgeback_description/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
- link panda_hand: geometry collision box size=0.035 0.19 0.065; visual mesh filename=/home/boyang/catkin_ws/src/sampling_based_control/mppi_exam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
- link panda_leftfinger: geometry collision box size=0.02 0.02 0.05; visual mesh filename=/home/boyang/catkin_ws/src/sampling_based_control/mppi_exam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
- link panda_link0: geometry collision mesh filename=/home/boyang/catkin_ws/src/sampling_based_control/mppi_exam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; visual mesh filename=/home/boyang/catkin_ws/src/sampling_based_control/mppi_exam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
- link panda_link1: geometry collision mesh filename=/home/boyang/catkin_ws/src/sampling_based_control/mppi_exam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; visual mesh filename=/home/boyang/catkin_ws/src/sampling_based_control/mppi_exam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
- link panda_link2: geometry collision mesh filename=/home/boyang/catkin_ws/src/sampling_based_control/mppi_exam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; visual mesh filename=/home/boyang/catkin_ws/src/sampling_based_control/mppi_exam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
- link panda_link3: geometry collision mesh filename=/home/boyang/catkin_ws/src/sampling_based_control/mppi_exam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; visual mesh filename=/home/boyang/catkin_ws/src/sampling_based_control/mppi_exam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
- link panda_link4: geometry collision mesh filename=/home/boyang/catkin_ws/src/sampling_based_control/mppi_exam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; visual mesh filename=/home/boyang/catkin_ws/src/sampling_based_control/mppi_exam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
- link panda_link5: geometry collision mesh filename=/home/boyang/catkin_ws/src/sampling_based_control/mppi_exam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; visual mesh filename=/home/boyang/catkin_ws/src/sampling_based_control/mppi_exam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
- link panda_link6: geometry collision mesh filename=/home/boyang/catkin_ws/src/sampling_based_control/mppi_exam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; visual mesh filename=/home/boyang/catkin_ws/src/sampling_based_control/mppi_exam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
- link panda_link7: geometry collision mesh filename=/home/boyang/catkin_ws/src/sampling_based_control/mppi_exam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; visual mesh filename=/home/boyang/catkin_ws/src/sampling_based_control/mppi_exam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
- link panda_rightfinger: geometry collision box size=0.02 0.02 0.05; visual mesh filename=/home/boyang/catkin_ws/src/sampling_based_control/mppi_exam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
- link rear_cover_link: geometry visual mesh filename=/home/boyang/catkin_ws/src/ridgeback/ridgeback_description/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
- link rear_lights_link: geometry visual mesh filename=/home/boyang/catkin_ws/src/ridgeback/ridgeback_description/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
- link ridgeback_sensor_mount_link: geometry visual mesh filename=/home/boyang/catkin_ws/src/sampling_based_control/mppi_exam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
- link right_side_cover_link: geometry visual mesh filename=/home/boyang/catkin_ws/src/ridgeback/ridgeback_description/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
- link top_link: geometry visual mesh filename=/home/boyang/catkin_ws/src/ridgeback/ridgeback_description/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

File: mppi_examples/mppi_panda/resources/panda/panda.urdf (robot description, URDF)
Before this commit: robot panda, 11 links, 10 joints
Links:
- link panda_hand: geometry collision box size=0.035 0.19 0.065; visual mesh filename=file:///home/boyang/catkin_ws/src/sampling_based_control/mp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
- link panda_link0: geometry collision mesh filename=file:///home/boyang/catkin_ws/src/sampling_based_control/mp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; visual mesh filename=file:///home/boyang/catkin_ws/src/sampling_based_control/mp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
- link panda_link1: geometry collision mesh filename=file:///home/boyang/catkin_ws/src/sampling_based_control/mp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; visual mesh filename=file:///home/boyang/catkin_ws/src/sampling_based_control/mp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
- link panda_link2: geometry collision mesh filename=file:///home/boyang/catkin_ws/src/sampling_based_control/mp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; visual mesh filename=file:///home/boyang/catkin_ws/src/sampling_based_control/mp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
- link panda_link3: geometry collision mesh filename=file:///home/boyang/catkin_ws/src/sampling_based_control/mp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; visual mesh filename=file:///home/boyang/catkin_ws/src/sampling_based_control/mp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
- link panda_link4: geometry collision mesh filename=file:///home/boyang/catkin_ws/src/sampling_based_control/mp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; visual mesh filename=file:///home/boyang/catkin_ws/src/sampling_based_control/mp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
- link panda_link5: geometry collision mesh filename=file:///home/boyang/catkin_ws/src/sampling_based_control/mp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; visual mesh filename=file:///home/boyang/catkin_ws/src/sampling_based_control/mp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
- link panda_link6: geometry collision mesh filename=file:///home/boyang/catkin_ws/src/sampling_based_control/mp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; visual mesh filename=file:///home/boyang/catkin_ws/src/sampling_based_control/mp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
- link panda_link7: geometry collision mesh filename=file:///home/boyang/catkin_ws/src/sampling_based_control/mp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; visual mesh filename=file:///home/boyang/catkin_ws/src/sampling_based_control/mp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

File: mppi_examples/mppi_sliding/data/objects/valve.urdf (robot description, URDF)
Before this commit: robot valve, 3 links, 2 joints
Links:
- link handle_link: geometry collision mesh filename=file:///home/boyang/student_projects_ws/src/sampling_based_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; visual mesh filename=file:///home/boyang/student_projects_ws/src/sampling_based_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
