Commit message: added panda_grasp_finger_edge grasping frame to panda hand

File: mppi_examples/mppi_manipulation/data/panda.urdf.xacro (robot description, xacro)
@@ -88,4 +88,20 @@
             <origin xyz="0 0 0.1" rpy="0 0 0"/>
         </joint>
+        <link name="panda_grasp_finger"/>
+          <joint name="panda_grasp__finger_joint" type="fixed">
+            <parent link="panda_hand"/>
+            <child link="panda_grasp_finger"/>
+            <axis xyz="0 1 0"/>
+            <origin rpy="0 0 0" xyz="0 0.025 0.125"/>
+            <!-- 0.106-->
+          </joint>
+          <link name="panda_grasp_finger_edge"/>
+          <joint name="panda_grasp__finger_edge_joint" type="fixed">
+            <parent link="panda_hand"/>
+            <child link="panda_grasp_finger_edge"/>
+            <axis xyz="0 1 0"/>
+            <origin rpy="0 0 0" xyz="0 0.04 0.15"/>
+            <!-- 0.106-->
+          </joint>
     </xacro:if>
 </robot>
