Commit message: in fixed mode need to be manually changed to the true pose

File: mppi_examples/mppi_manipulation/data/panda_mobile.urdf.xacro (robot description, xacro)
@@ -19,4 +19,5 @@
             <parent link="world"/>
             <child link="base_link"/>
+            <origin xyz="0.004 1.087 0.000" rpy="0.000 0.000 -1.500"/>
         </joint>
     </xacro:if>

Commit message: shiftin slightly back the grasp frame

File: mppi_examples/mppi_manipulation/data/panda_mobile.urdf.xacro (robot description, xacro)
@@ -40,5 +40,5 @@
             <child link="panda_grasp"/>
             <axis xyz="0 1 0"/>
-            <origin xyz="0 0 0.1" rpy="0 0 0"/>
+            <origin xyz="0 0 0.085" rpy="0 0 0"/>
         </joint>
     </xacro:if>

Commit message: local changes

File: mppi_examples/mppi_manipulation/data/panda_mobile.urdf.xacro (robot description, xacro)
@@ -19,5 +19,5 @@
             <parent link="world"/>
             <child link="base_link"/>
-            <origin xyz="-0.2667636086710243 0.7114964305976865 0.0" rpy="0.000 0.000 -1.5898602011730607"/>
+             <origin xyz="0.016562803523970236 0.536778652875357 0.0" rpy="0.000 0.000 -1.5943151411055445"/>
         </joint>
     </xacro:if>
@@ -40,5 +40,5 @@
             <child link="panda_grasp"/>
             <axis xyz="0 1 0"/>
-            <origin xyz="0 0 0.085" rpy="0 0 0"/>
+            <origin xyz="0 0 0.10" rpy="0 0 0"/>
         </joint>
     </xacro:if>

Commit message: calibrated panda offset

File: mppi_examples/mppi_manipulation/data/panda_mobile.urdf.xacro (robot description, xacro)
@@ -29,5 +29,5 @@
         <child link="franka_mount_link"/>
         <!--        <origin xyz="$(optenv RIDGEBACK_FRANKA_XYZ 0.21 0.0 0.2)" rpy="$(optenv RIDGEBACK_FRANKA_RPY 0 0 0)"/>-->
-        <origin xyz="0.30 0.0 0.445" rpy="0 0 0"/>
+        <origin xyz="0.295 0.005 0.445" rpy="0 0 0"/>
     </joint>
     <link name="franka_mount_link"/>

Commit message: random changes here and there

File: mppi_examples/mppi_manipulation/data/panda_mobile.urdf.xacro (robot description, xacro)
@@ -37,8 +37,8 @@
         <link name="panda_grasp"/>
         <joint name="panda_grasp_joint" type="fixed">
-            <parent link="panda_hand"/>
+            <parent link="panda_rightfinger"/>
             <child link="panda_grasp"/>
             <axis xyz="0 1 0"/>
-            <origin xyz="0 0 0.095" rpy="0 0 0"/> <!-- 0.106-->
+            <origin xyz="0 -0.005 0.045" rpy="0 0 0"/> <!--origin xyz="0 0 0.095" rpy="0 0 0"/-->
         </joint>
     </xacro:if>

Commit message: change to debug on robot

File: mppi_examples/mppi_manipulation/data/panda_mobile.urdf.xacro (robot description, xacro)
@@ -37,8 +37,8 @@
         <link name="panda_grasp"/>
         <joint name="panda_grasp_joint" type="fixed">
-            <parent link="panda_hand"/>
+            <parent link="panda_leftfinger"/>
             <child link="panda_grasp"/>
             <axis xyz="0 1 0"/>
-            <origin xyz="0 0 0.095" rpy="0 0 0"/> <!-- 0.106-->
+            <origin xyz="0 0 0.045" rpy="0 0 0"/> <!-- offset panda_hand xyz="0 0 0.095" rpy="0 0 0"-->
         </joint>
     </xacro:if>

Commit message: moving grasp frame

File: mppi_examples/mppi_manipulation/data/panda_mobile.urdf.xacro (robot description, xacro)
@@ -40,5 +40,5 @@
             <child link="panda_grasp"/>
             <axis xyz="0 1 0"/>
-            <origin xyz="0 0 0.045" rpy="0 0 0"/> <!-- offset panda_hand xyz="0 0 0.095" rpy="0 0 0"-->
+            <origin xyz="0 -0.02 0.035" rpy="0 0 0"/> <!-- 0 0 0.45 offset panda_hand xyz="0 0 0.095" rpy="0 0 0"-->
         </joint>
     </xacro:if>

Commit message: bugfix for new frame and added connect_controller param in the launch file for security and debugging

File: mppi_examples/mppi_manipulation/data/panda_mobile.urdf.xacro (robot description, xacro)
@@ -42,4 +42,20 @@
             <origin xyz="0 0 0.095" rpy="0 0 0"/> <!-- 0.106-->
         </joint>
+        <link name="panda_grasp_finger"/>
+          <joint name="panda_grasp__finger_joint" type="fixed">
+            <parent link="panda_hand"/>
+            <child link="panda_grasp_finger"/>
+            <axis xyz="0 1 0"/>
+            <origin rpy="0 0 0" xyz="0 0.025 0.125"/>
+            <!-- 0.106-->
+          </joint>
+          <link name="panda_grasp_finger_edge"/>
+          <joint name="panda_grasp__finger_edge_joint" type="fixed">
+            <parent link="panda_hand"/>
+            <child link="panda_grasp_finger_edge"/>
+            <axis xyz="0 1 0"/>
+            <origin rpy="0 0 0" xyz="0 0.04 0.15"/>
+            <!-- 0.106-->
+          </joint>
     </xacro:if>
 </robot>
