Commit message: shelf working in simulation

File: mppi_examples/mppi_manipulation/data/objects/shelf.urdf (robot description, URDF)
Before this commit: robot shelf, 6 links, 5 joints
Links:
- added link door_hinge
- link door: mass None -> 5.8
Joints:
- added joint door_hinge_joint: type fixed, parent shelf, child door_hinge, origin xyz=0 -0.3 0.45
- joint articulation_joint: origin xyz=0 -0.3 0.45 -> xyz=0 0 0; parent shelf -> door_hinge
- joint fixed: origin xyz=0.5 0 0 rpy=0 0 3.14159 -> xyz=0.6 0 0 rpy=0 0 3.14159

File: mppi_examples/mppi_manipulation/data/objects/shelf.urdf.xacro (robot description, xacro)
@@ -1,4 +1,4 @@
 <?xml version="1.0" ?>
-<robot name="shelf" xmlns:xacro="http://www.ros.org/wiki/xacro" >
+<robot name="shelf" xmlns:xacro="http://www.ros.org/wiki/xacro">
     <xacro:arg name="height" default="0.0"/>
     <xacro:property name="height" default="$(arg height)"/>
@@ -9,12 +9,25 @@
     <xacro:property name="handle_length" default="0.16"/>
     <xacro:property name="handle_offset" default="0.25"/>
+    <xacro:macro name="box_inertia" params="m x y z">
+        <inertial>
+            <origin rpy="0 0 0" xyz="0 0 0"/>
+            <mass value="${m}"/>
+            <inertia ixx="${0.0833 * m * (y**2 + z**2)}"
+                     ixy="0"
+                     ixz="0"
+                     iyy="${0.0833 * m * (x**2 + z**2)}"
+                     iyz="0"
+                     izz="${0.0833 * m * (z**2 + y**2)}"/>
+        </inertial>
+    </xacro:macro>
     <link name="world"/>
     <joint name="fixed" type="fixed">
         <parent link="world"/>
         <child link="shelf"/>
-        <origin xyz="1.5 0 ${height}" rpy="0 0 3.14159"/>
+        <origin xyz="0 0 ${height}" rpy="0 0 3.14159"/>
     </joint>
     <link name="shelf"/>
     <link name="door">
+        <xacro:box_inertia m="5.8" x="${door_width}" y="${door_length}" z="${door_height}"/>
         <visual>
             <origin rpy="0 0 0" xyz="0 ${door_length/2} 0"/>
@@ -48,5 +61,5 @@
         <limit effort="100" lower="0" upper="1.57" velocity="10.0"/>
     </joint>
-    <link name="handle">
+    <link name="handle_link">
         <inertial>
             <origin rpy="0 0 0" xyz="0 0 0"/>
@@ -116,14 +129,15 @@
     <joint name="handle_joint" type="fixed">
         <parent link="door"/>
-        <child link="handle"/>
-        <origin xyz="${handle_height + door_width/2} ${handle_offset} 0" rpy="0 0 0"/> <!-- height handle + half the width door, 0.30 minus some offset -->
+        <child link="handle_link"/>
+        <origin xyz="${handle_height + door_width/2} ${handle_offset} 0"
+                rpy="0 0 0"/> <!-- height handle + half the width door, 0.30 minus some offset -->
     </joint>
     <joint name="handle_support_left_joint" type="fixed">
-        <parent link="handle"/>
+        <parent link="handle_link"/>
         <child link="handle_support_left"/>
         <origin xyz="-${handle_height/2} 0 ${handle_length/2}" rpy="0 0 0"/>
     </joint>
     <joint name="handle_support_right_joint" type="fixed">
-        <parent link="handle"/>
+        <parent link="handle_link"/>
         <child link="handle_support_right"/>
         <origin xyz="-${handle_height/2} 0 -${handle_length/2}" rpy="0 0 0"/>

File: mppi_examples/mppi_manipulation/data/panda.urdf (robot description, URDF)
Before this commit: robot panda, 13 links, 12 joints
Links:
- link panda_hand: geometry collision box size=0.035 0.19 0.065; visual mesh filename=/home/giuseppe/catkin_ws/src/sampling_based_control/mppi_ex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
- link panda_leftfinger: geometry collision box size=0.02 0.02 0.05; visual mesh filename=/home/giuseppe/catkin_ws/src/sampling_based_control/mppi_ex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
- link panda_link0: geometry collision mesh filename=/home/giuseppe/catkin_ws/src/sampling_based_control/mppi_ex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; visual mesh filename=/home/giuseppe/catkin_ws/src/sampling_based_control/mppi_ex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
- link panda_link1: geometry collision mesh filename=/home/giuseppe/catkin_ws/src/sampling_based_control/mppi_ex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; visual mesh filename=/home/giuseppe/catkin_ws/src/sampling_based_control/mppi_ex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
- link panda_link2: geometry collision mesh filename=/home/giuseppe/catkin_ws/src/sampling_based_control/mppi_ex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; visual mesh filename=/home/giuseppe/catkin_ws/src/sampling_based_control/mppi_ex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
- link panda_link3: geometry collision mesh filename=/home/giuseppe/catkin_ws/src/sampling_based_control/mppi_ex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; visual mesh filename=/home/giuseppe/catkin_ws/src/sampling_based_control/mppi_ex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
- link panda_link4: geometry collision mesh filename=/home/giuseppe/catkin_ws/src/sampling_based_control/mppi_ex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; visual mesh filename=/home/giuseppe/catkin_ws/src/sampling_based_control/mppi_ex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
- link panda_link5: geometry collision mesh filename=/home/giuseppe/catkin_ws/src/sampling_based_control/mppi_ex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; visual mesh filename=/home/giuseppe/catkin_ws/src/sampling_based_control/mppi_ex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
- link panda_link6: geometry collision mesh filename=/home/giuseppe/catkin_ws/src/sampling_based_control/mppi_ex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; visual mesh filename=/home/giuseppe/catkin_ws/src/sampling_based_control/mppi_ex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
- link panda_link7: geometry collision mesh filename=/home/giuseppe/catkin_ws/src/sampling_based_control/mppi_ex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; visual mesh filename=/home/giuseppe/catkin_ws/src/sampling_based_control/mppi_ex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
- link panda_rightfinger: geometry collision box size=0.02 0.02 0.05; visual mesh filename=/home/giuseppe/catkin_ws/src/sampling_based_control/mppi_ex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
