Commit message: changes from tuesday tests

File: mppi_examples/mppi_manipulation/data/objects/box.urdf.xacro (robot description, xacro)
@@ -19,5 +19,5 @@
             <origin rpy="0 0 0" xyz="0 0 0"/>
             <geometry>
-                <box size="${obstacle_size} ${obstacle_size} ${obstacle_size}"/>
+                <box size="0.4 0.6 0.34"/>
             </geometry>
             <material name="box_material">
@@ -28,5 +28,5 @@
             <origin rpy="0 0 0" xyz="0 0 0"/>
             <geometry>
-                <box size="${obstacle_size} ${obstacle_size} ${obstacle_size}"/>
+                <box size="0.4 0.6 0.34"/>
             </geometry>
         </collision>

File: mppi_examples/mppi_manipulation/data/objects/shelf.urdf.xacro (robot description, xacro)
@@ -10,6 +10,6 @@
     <xacro:property name="handle_length" default="0.16"/>
     <xacro:property name="handle_offset" default="0.27"/>
-    <xacro:property name="shelf_x" default="0.959"/>
-    <xacro:property name="shelf_y" default="-1.05"/>
+    <xacro:property name="shelf_x" default="0.943"/>
+    <xacro:property name="shelf_y" default="-0.952"/>
     <xacro:property name="shelf_z" default="0.903"/>
     <xacro:macro name="box_inertia" params="m x y z">
@@ -30,5 +30,5 @@
             <parent link="world"/>
             <child link="shelf"/>
-            <origin xyz="${shelf_x} ${shelf_y} ${shelf_z}" rpy="-0.019 0.002 -3.090"/>
+            <origin xyz="${shelf_x} ${shelf_y} ${shelf_z}" rpy="-0.008 -0.001 -3.085"/>
         </joint>
     </xacro:if>

File: mppi_examples/mppi_manipulation/data/panda_mobile.urdf.xacro (robot description, xacro)
@@ -40,5 +40,5 @@
             <child link="panda_grasp"/>
             <axis xyz="0 1 0"/>
-            <origin xyz="0 0 0.098" rpy="0 0 0"/> <!-- 0.106-->
+            <origin xyz="0 0 0.095" rpy="0 0 0"/> <!-- 0.106-->
         </joint>
     </xacro:if>
