Commit message: parameter and minor changes

File: mppi_examples/mppi_manipulation/data/objects/drawer.urdf.xacro (robot description, xacro)
@@ -7,5 +7,5 @@
         <parent link="world"/>
         <child link="drawer_frame"/>
-        <origin xyz="1.0 0.3 ${height + 0.01}" rpy="0 0 3.14"/>
+        <origin xyz="1.5 0.3 ${height + 0.01}" rpy="0 0 3.14"/>
     </joint>
     <link name="drawer_frame">
@@ -78,5 +78,5 @@
         <origin xyz="0.046 0 0"/>
         <axis xyz="1 0 0"/>
-        <limit effort="100" lower="0" upper="0.5" velocity="10.0"/>
+        <limit effort="100" lower="0" upper="0.55" velocity="10.0"/>
     </joint>
     <link name="handle_link">
@@ -100,4 +100,7 @@
                 <cylinder radius="0.005" length="0.010"/>
             </geometry>
+            <material name="">
+                <contact name="steel"/>
+            </material>
         </collision>
     </link>

Commit message: fix collision mesh

File: mppi_examples/mppi_manipulation/data/objects/drawer.urdf.xacro (robot description, xacro)
@@ -98,5 +98,5 @@
             <origin rpy="0 0 0" xyz="0 0 0"/>
             <geometry>
-                <cylinder radius="0.005" length="0.010"/>
+                <cylinder radius="0.005" length="0.10"/>
             </geometry>
             <material name="">

File: mppi_examples/mppi_manipulation/data/objects/microwave.urdf.xacro (robot description, xacro)
@@ -74,5 +74,5 @@
             <origin rpy="0 0 0" xyz="0 0 0"/>
             <geometry>
-                <cylinder radius="0.005" length="0.010"/>
+                <cylinder radius="0.005" length="0.10"/>
             </geometry>
         </collision>
