Commit message: separate observer node

File: mppi_examples/mppi_manipulation/data/objects/shelf.urdf.xacro (robot description, xacro)
@@ -1,4 +1,5 @@
 <?xml version="1.0" ?>
 <robot name="shelf" xmlns:xacro="http://www.ros.org/wiki/xacro">
+    <xacro:arg name="fixed" default="true"/>
     <xacro:arg name="height" default="0.0"/>
     <xacro:property name="height" default="$(arg height)"/>
@@ -21,10 +22,12 @@
         </inertial>
     </xacro:macro>
-    <link name="world"/>
-    <joint name="fixed" type="fixed">
-        <parent link="world"/>
-        <child link="shelf"/>
-        <origin xyz="0 0 ${height}" rpy="0 0 3.14159"/>
-    </joint>
+    <xacro:if value="$(arg fixed)">
+        <link name="world"/>
+        <joint name="fixed" type="fixed">
+            <parent link="world"/>
+            <child link="shelf"/>
+            <origin xyz="0 0 ${height}" rpy="0 0 3.14159"/>
+        </joint>
+    </xacro:if>
     <link name="shelf"/>
     <link name="door">

Commit message: separate observer node and tuned urdf in vicon room

File: mppi_examples/mppi_manipulation/data/objects/shelf.urdf.xacro (robot description, xacro)
@@ -133,5 +133,5 @@
         <parent link="door"/>
         <child link="handle_link"/>
-        <origin xyz="${handle_height + door_width/2} ${handle_offset} 0"
+        <origin xyz="${handle_height + door_width/2} ${handle_offset} -0.15"
                 rpy="0 0 0"/> <!-- height handle + half the width door, 0.30 minus some offset -->
     </joint>

File: mppi_examples/mppi_manipulation/data/panda_mobile.urdf.xacro (robot description, xacro)
@@ -18,5 +18,6 @@
         <parent link="mid_mount"/>
         <child link="franka_mount_link"/>
-        <origin xyz="$(optenv RIDGEBACK_FRANKA_XYZ 0.21 0.0 0.2)" rpy="$(optenv RIDGEBACK_FRANKA_RPY 0 0 0)"/>
+<!--        <origin xyz="$(optenv RIDGEBACK_FRANKA_XYZ 0.21 0.0 0.2)" rpy="$(optenv RIDGEBACK_FRANKA_RPY 0 0 0)"/>-->
+        <origin xyz="$(optenv RIDGEBACK_FRANKA_XYZ 0.30 0.0 0.445)" rpy="$(optenv RIDGEBACK_FRANKA_RPY 0 0 0)"/>
     </joint>
     <link name="franka_mount_link"/>

File: mppi_examples/mppi_manipulation/data/ridgeback.urdf.xacro (robot description, xacro)
@@ -16,4 +16,10 @@
             <child link="ridgeback_sensor_mount_link"/>
         </joint>
+        <link name="reference_link"/>
+        <joint name="reference_link_joint" type="fixed">
+            <origin xyz="-0.343 0 0.77" rpy="0 0 0"/>
+            <parent link="mid_mount"/>
+            <child link="reference_link"/>
+        </joint>
     </xacro:macro>
 </robot>

Commit message: urdf restructuring for gazebo simulation

File: mppi_examples/mppi_manipulation/data/objects/shelf.urdf.xacro (robot description, xacro)
@@ -27,5 +27,5 @@
             <parent link="world"/>
             <child link="shelf"/>
-            <origin xyz="1.0 0 ${height}" rpy="0 0 3.14159"/>
+            <origin xyz="10.0 2.0 ${height}" rpy="0 0 3.14159"/>
         </joint>
     </xacro:if>

File: mppi_examples/mppi_manipulation/data/ridgeback.urdf.xacro (robot description, xacro)
@@ -7,5 +7,5 @@
             <visual>
                 <geometry>
-                    <mesh filename="package://mppi_manipulation/data/meshes/ridgeback_sensor_mount.dae"/>
+                    <mesh filename="${resources_prefix}$(find mppi_manipulation)/data/meshes/ridgeback_sensor_mount.dae"/>
                 </geometry>
             </visual>
@@ -22,18 +22,4 @@
             <child link="reference_link"/>
         </joint>
-<!--        Just an hack to get the reference pose from gazebo: using a movable joint does not cause collapse of the model-->
-        <link name="reference_link_gazebo">
-            <inertial>
-                <mass value="0.001"/>
-                <origin xyz="0 0 0" rpy="0 0 0"/>
-                <inertia ixx="${dummy_inertia}" ixy="0.0" ixz="0.0" iyy="${dummy_inertia}" iyz="0.0" izz="${dummy_inertia}"/>
-            </inertial>
-        </link>
-        <joint name="reference_link_gazeb_joint" type="revolute">
-            <origin xyz="-0.343 0 0.77" rpy="0 0 0"/>
-            <parent link="mid_mount"/>
-            <child link="reference_link_gazebo"/>
-            <limit upper="0.0" lower="0.0" effort="0.0" velocity="0.0"/>
-        </joint>
     </xacro:macro>
 </robot>

File: mppi_examples/mppi_manipulation/data/ridgeback.xacro (robot description, xacro)
@@ -48,5 +48,5 @@
             <origin xyz="0 0 0" rpy="0 0 0" />
             <geometry>
-                <mesh filename="package://ridgeback_description/meshes/body.stl"/>
+                <mesh filename="${resources_prefix}$(find ridgeback_description)/meshes/body.stl"/>
             </geometry>
             <material name="black" />
@@ -75,5 +75,5 @@
             <origin xyz="0 0 0" rpy="0 0 ${PI}" />
             <geometry>
-                <mesh filename="package://ridgeback_description/meshes/side-cover.stl"/>
+                <mesh filename="${resources_prefix}$(find ridgeback_description)/meshes/side-cover.stl"/>
             </geometry>
             <material name="yellow" />
@@ -84,5 +84,5 @@
             <origin xyz="0 0 0" rpy="0 0 0" />
             <geometry>
-                <mesh filename="package://ridgeback_description/meshes/side-cover.stl"/>
+                <mesh filename="${resources_prefix}$(find ridgeback_description)/meshes/side-cover.stl"/>
             </geometry>
             <material name="yellow" />
@@ -98,5 +98,5 @@
             <origin xyz="0 0 0" rpy="0 0 0" />
             <geometry>
-                <mesh filename="package://ridgeback_description/meshes/end-cover.stl" />
+                <mesh filename="${resources_prefix}$(find ridgeback_description)/meshes/end-cover.stl" />
             </geometry>
             <material name="black" />
@@ -112,5 +112,5 @@
             <origin xyz="0 0 0" rpy="0 0 ${PI}" />
             <geometry>
-                <mesh filename="package://ridgeback_description/meshes/end-cover.stl" />
+                <mesh filename="${resources_prefix}$(find ridgeback_description)/meshes/end-cover.stl" />
             </geometry>
             <material name="black" />
@@ -131,5 +131,5 @@
             <origin xyz="0 0 0" rpy="0 0 0" />
             <geometry>
-                <mesh filename="package://ridgeback_description/meshes/lights.stl" />
+                <mesh filename="${resources_prefix}$(find ridgeback_description)/meshes/lights.stl" />
             </geometry>
             <material name="white" />
@@ -140,5 +140,5 @@
             <origin xyz="0 0 0" rpy="0 0 ${PI}" />
             <geometry>
-                <mesh filename="package://ridgeback_description/meshes/lights.stl" />
+                <mesh filename="${resources_prefix}$(find ridgeback_description)/meshes/lights.stl" />
             </geometry>
             <material name="red" />
@@ -154,5 +154,5 @@
             <origin xyz="0 0 0" rpy="0 0 0" />
             <geometry>
-                <mesh filename="package://ridgeback_description/meshes/top.stl" />
+                <mesh filename="${resources_prefix}$(find ridgeback_description)/meshes/top.stl" />
             </geometry>
             <material name="black" />
@@ -168,5 +168,5 @@
             <origin xyz="0 0 0" rpy="0 ${PI/2} 0" />
             <geometry>
-                <mesh filename="package://ridgeback_description/meshes/axle.stl" />
+                <mesh filename="${resources_prefix}$(find ridgeback_description)/meshes/axle.stl" />
             </geometry>
             <material name="black" />

File: mppi_examples/mppi_manipulation/data/ridgeback_gazebo.urdf.xacro (robot description, xacro)
@@ -12,5 +12,5 @@
                 <origin xyz="0 0 0" rpy="${PI/2} 0 0"/>
                 <geometry>
-                    <mesh filename="package://ridgeback_description/meshes/wheel.stl"/>
+                    <mesh filename="${resources_prefix}$(find ridgeback_description)/meshes/wheel.stl"/>
                 </geometry>
                 <material name="black"/>
@@ -46,4 +46,12 @@
             </actuator>
         </transmission>
+<!--        <gazebo reference="${prefix}_${side}_wheel_link">-->
+<!--            <mu1 value="50.0"/>-->
+<!--            <mu2 value="100.0"/>-->
+<!--            <kp>1000000.0</kp>-->
+<!--            <kd>100.0</kd>-->
+<!--            <minDepth>0.001</minDepth>-->
+<!--            <maxVel>1.0</maxVel>-->
+<!--        </gazebo>-->
     </xacro:macro>
     <xacro:macro name="rocker" params="prefix joint_type location *joint_limits">
@@ -52,5 +60,5 @@
                 <origin xyz="0 0 0" rpy="${PI/2} 0 ${PI/2}"/>
                 <geometry>
-                    <mesh filename="package://ridgeback_description/meshes/rocker.stl"/>
+                    <mesh filename="${resources_prefix}$(find ridgeback_description)/meshes/rocker.stl"/>
                 </geometry>
                 <material name="black"/>
@@ -85,4 +93,18 @@
         <limit effort="0" velocity="0"/>
     </xacro:rocker>
+    <!--        Just an hack to get the reference pose from gazebo: using a movable joint does not cause collapse of the model-->
+    <link name="reference_link_gazebo">
+        <inertial>
+            <mass value="0.001"/>
+            <origin xyz="0 0 0" rpy="0 0 0"/>
+            <inertia ixx="${dummy_inertia}" ixy="0.0" ixz="0.0" iyy="${dummy_inertia}" iyz="0.0" izz="${dummy_inertia}"/>
+        </inertial>
+    </link>
+    <joint name="reference_link_gazebo_joint" type="revolute">
+        <origin xyz="-0.343 0 0.77" rpy="0 0 0"/>
+        <parent link="mid_mount"/>
+        <child link="reference_link_gazebo"/>
+        <limit upper="0.0" lower="0.0" effort="0.0" velocity="0.0"/>
+    </joint>
     <!-- Bring in simulation data for Gazebo. -->
     <xacro:include filename="$(find mppi_manipulation)/data/ridgeback_plugins.xacro"/>

Commit message: changin urfd as for vicon setup

File: mppi_examples/mppi_manipulation/data/objects/shelf.urdf.xacro (robot description, xacro)
@@ -27,5 +27,5 @@
             <parent link="world"/>
             <child link="shelf"/>
-            <origin xyz="10.0 2.0 ${height}" rpy="0 0 3.14159"/>
+            <origin xyz="-0.318 -0.510 0.904" rpy="-0.007 0.002 1.5999"/>
         </joint>
     </xacro:if>

File: mppi_examples/mppi_manipulation/data/panda_mobile.urdf.xacro (robot description, xacro)
@@ -19,5 +19,5 @@
             <parent link="world"/>
             <child link="base_link"/>
-            <origin xyz="0.004 1.087 0.000" rpy="0.000 0.000 -1.500"/>
+            <origin xyz="-0.2667636086710243 0.7114964305976865 0.0" rpy="0.000 0.000 -1.5898602011730607"/>
         </joint>
     </xacro:if>

Commit message: shelf urdf change

File: mppi_examples/mppi_manipulation/data/objects/shelf.urdf.xacro (robot description, xacro)
@@ -4,8 +4,8 @@
     <xacro:arg name="height" default="0.0"/>
     <xacro:property name="height" default="$(arg height)"/>
-    <xacro:property name="door_length" default="0.30"/>
+    <xacro:property name="door_length" default="0.295"/>
     <xacro:property name="door_height" default="0.90"/>
-    <xacro:property name="door_width" default="0.02"/>
-    <xacro:property name="handle_height" default="0.036"/>
+    <xacro:property name="door_width" default="0.01"/>
+    <xacro:property name="handle_height" default="0.026"/> <!-- 0.036-->
     <xacro:property name="handle_length" default="0.16"/>
     <xacro:property name="handle_offset" default="0.25"/>

Commit message: tuned urdf

File: mppi_examples/mppi_manipulation/data/objects/shelf.urdf.xacro (robot description, xacro)
@@ -6,6 +6,6 @@
     <xacro:property name="door_length" default="0.30"/>
     <xacro:property name="door_height" default="0.90"/>
-    <xacro:property name="door_width" default="0.02"/>
-    <xacro:property name="handle_height" default="0.036"/>
+    <xacro:property name="door_width" default="0.016"/>
+    <xacro:property name="handle_height" default="0.026"/>
     <xacro:property name="handle_length" default="0.16"/>
     <xacro:property name="handle_offset" default="0.25"/>
@@ -146,3 +146,9 @@
         <origin xyz="-${handle_height/2} 0 -${handle_length/2}" rpy="0 0 0"/>
     </joint>
+    <link name="measured_joint_link"/>
+    <joint name="measured_joint_handle_joint" type="fixed">
+        <parent link="handle_link"/>
+        <child link="measured_joint_link"/>
+        <origin xyz="-0.038456463645002395 -0.24676779774627114 0.0" rpy="0 0 0"/>
+    </joint>
 </robot>

Commit message: wrong handle offset

File: mppi_examples/mppi_manipulation/data/objects/shelf.urdf.xacro (robot description, xacro)
@@ -9,5 +9,5 @@
     <xacro:property name="handle_height" default="0.026"/>
     <xacro:property name="handle_length" default="0.16"/>
-    <xacro:property name="handle_offset" default="0.25"/>
+    <xacro:property name="handle_offset" default="0.27"/>
     <xacro:macro name="box_inertia" params="m x y z">
         <inertial>

Commit message: correct (hopefully) axis

File: mppi_examples/mppi_manipulation/data/objects/shelf.urdf.xacro (robot description, xacro)
@@ -58,9 +58,14 @@
     <joint name="articulation_joint" type="revolute">
         <parent link="door_hinge"/>
-        <child link="door"/>
+        <child link="measured_joint_link"/>
         <dynamics damping="2.0" friction="4.0"/>
-        <origin xyz="0 0 0"/>
+        <origin xyz=" -0.004 0.023 -0.150"/>
         <axis xyz="0 0 -1"/>
         <limit effort="100" lower="0" upper="1.57" velocity="10.0"/>
+    </joint>
+    <joint name="door_link" type="fixed">
+        <parent link="measured_joint_link"/>
+        <child link="door"/>
+        <origin xyz="0.004 -0.023 0.150"/>
     </joint>
     <link name="handle_link">
@@ -147,8 +152,8 @@
     </joint>
     <link name="measured_joint_link"/>
-    <joint name="measured_joint_handle_joint" type="fixed">
+<!--     <joint name="measured_joint_handle_joint" type="fixed">
         <parent link="handle_link"/>
         <child link="measured_joint_link"/>
         <origin xyz="-0.038456463645002395 -0.24676779774627114 0.0" rpy="0 0 0"/>
-    </joint>
+    </joint> -->
 </robot>

Commit message: changing dynamics

File: mppi_examples/mppi_manipulation/data/objects/shelf.urdf.xacro (robot description, xacro)
@@ -89,4 +89,7 @@
                 <box size="0.01 0.01 ${handle_length+0.01}"/>
             </geometry>
+            <material name="">
+                <contact name="steel"/>
+            </material>
         </collision>
     </link>
@@ -111,4 +114,7 @@
                 <box size="${handle_height} 0.01 0.01"/>
             </geometry>
+            <material name="">
+                <contact name="steel"/>
+            </material>
         </collision>
     </link>
@@ -133,4 +139,7 @@
                 <box size="${handle_height} 0.01 0.01"/>
             </geometry>
+            <material name="">
+                <contact name="steel"/>
+            </material>
         </collision>
     </link>

File: mppi_examples/mppi_panda/resources/panda/panda.urdf.xacro (robot description, xacro)
@@ -490,5 +490,8 @@
                             <box size="0.0222 0.015 0.02"/>
                         </geometry>
-                    </collision>
+                         <material name="">
+                            <contact name="steel"/>
+                        </material>
+                   </collision>
                     <collision>
                         <origin rpy="${3.14 * 30 / 180.0} 0 0.0" xyz="0 0.017 0.027"/>
@@ -496,4 +499,7 @@
                             <box size="0.0222 0.007 0.025"/>
                         </geometry>
+                        <material name="">
+                            <contact name="steel"/>
+                        </material>
                     </collision>
                     <collision>
@@ -502,4 +508,7 @@
                             <box size="0.0222 0.0145 0.018"/>
                         </geometry>
+                        <material name="">
+                            <contact name="steel"/>
+                        </material>
                     </collision>
                 </xacro:if>
@@ -527,4 +536,7 @@
                             <box size="0.0222 0.015 0.02"/>
                         </geometry>
+                        <material name="">
+                            <contact name="steel"/>
+                        </material>
                     </collision>
                     <collision>
@@ -533,4 +545,7 @@
                             <box size="0.0222 0.007 0.025"/>
                         </geometry>
+                        <material name="">
+                            <contact name="steel"/>
+                        </material>
                     </collision>
                     <collision>
@@ -539,4 +554,7 @@
                             <box size="0.0222 0.0145 0.018"/>
                         </geometry>
+                        <material name="">
+                            <contact name="steel"/>
+                        </material>
                     </collision>
                 </xacro:if>

Commit message: shelf origin

File: mppi_examples/mppi_manipulation/data/objects/shelf.urdf.xacro (robot description, xacro)
@@ -27,5 +27,5 @@
             <parent link="world"/>
             <child link="shelf"/>
-            <origin xyz="-0.318 -0.510 0.904" rpy="-0.007 0.002 1.5999"/>
+            <origin xyz="-0.011 -0.431 0.905" rpy="-0.006 0.001 1.585"/>
         </joint>
     </xacro:if>
