Commit message: new custom fingers

File: mppi_examples/mppi_manipulation/data/objects/shelf.urdf.xacro (robot description, xacro)
@@ -7,5 +7,5 @@
     <xacro:property name="door_height" default="0.90"/>
     <xacro:property name="door_width" default="0.016"/>
-    <xacro:property name="handle_height" default="0.026"/>
+    <xacro:property name="handle_height" default="0.05"/> <!-- 0.026 -->
     <xacro:property name="handle_length" default="0.16"/>
     <xacro:property name="handle_offset" default="0.27"/>

File: mppi_examples/mppi_panda/resources/panda/panda.urdf.xacro (robot description, xacro)
@@ -7,4 +7,5 @@
     <xacro:arg name="collision_hand" default="true"/>
     <xacro:arg name="collision_finger" default="true"/>
+    <xacro:arg name="custom_fingers" default="false"/>
     <xacro:arg name="no_position_limits" default="true"/>
     <xacro:arg name="add_finger" default="false"/>
@@ -17,4 +18,5 @@
     <xacro:property name="no_position_limits" value="$(arg no_position_limits)"/>
     <xacro:property name="add_finger" value="$(arg add_finger)"/>
+    <xacro:include filename="$(find mppi_panda)/resources/panda/custom_fingers.urdf"/>
     <xacro:macro name="panda_robot" params="parent_link:='world' robot_description:=''">
         <joint name="panda_joint_${parent_link}" type="fixed">
@@ -468,96 +470,101 @@
                 </actuator>
             </transmission>
-            <link name="panda_leftfinger">
-                <inertial>
-                    <mass value="0.1"/>
-                    <origin rpy="0 0 0" xyz="0 0.0145644 0.0227941"/>
-                    <inertia ixx="3.01220925051e-05" ixy="0.0" ixz="0.0" iyy="2.95873808038e-05" iyz="0.0"
-                             izz="6.95125211657e-06"/>
-                </inertial>
-                <visual>
-                    <origin rpy="0 0 0" xyz="0 0 0"/>
-                    <geometry>
-                        <mesh filename="${resources_prefix}${resources_directory}/resources/panda/meshes/visual/finger.dae"/>
-                    </geometry>
-                    <material name="">
-                        <color rgba="1 1 1 1"/>
-                    </material>
-                </visual>
-                <xacro:if value="${collision_finger}">
-                    <collision>
-                        <origin rpy="0.0 0 0.0" xyz="0 0.018 0.01"/>
+            <xacro:if value="$(arg custom_fingers)">
+              <xacro:custom_fingers/>
+            </xacro:if>
+            <xacro:unless value="$(arg custom_fingers)">
+                <link name="panda_leftfinger">
+                    <inertial>
+                        <mass value="0.1"/>
+                        <origin rpy="0 0 0" xyz="0 0.0145644 0.0227941"/>
+                        <inertia ixx="3.01220925051e-05" ixy="0.0" ixz="0.0" iyy="2.95873808038e-05" iyz="0.0"
+                                 izz="6.95125211657e-06"/>
+                    </inertial>
+                    <visual>
+                        <origin rpy="0 0 0" xyz="0 0 0"/>
                         <geometry>
-                            <box size="0.0222 0.015 0.02"/>
-                        </geometry>
-                         <material name="">
-                            <contact name="steel"/>
-                        </material>
-                   </collision>
-                    <collision>
-                        <origin rpy="${3.14 * 30 / 180.0} 0 0.0" xyz="0 0.017 0.027"/>
-                        <geometry>
-                            <box size="0.0222 0.007 0.025"/>
+                            <mesh filename="${resources_prefix}${resources_directory}/resources/panda/meshes/visual/finger.dae"/>
                         </geometry>
                         <material name="">
-                            <contact name="steel"/>
+                            <color rgba="1 1 1 1"/>
                         </material>
-                    </collision>
-                    <collision>
-                        <origin rpy="0.0 0 0.0" xyz="0 0.007 0.045"/>
+                    </visual>
+                    <xacro:if value="${collision_finger}">
+                        <collision>
+                            <origin rpy="0.0 0 0.0" xyz="0 0.018 0.01"/>
+                            <geometry>
+                                <box size="0.0222 0.015 0.02"/>
+                            </geometry>
+                             <material name="">
+                                <contact name="steel"/>
+                            </material>
+                       </collision>
+                        <collision>
+                            <origin rpy="${3.14 * 30 / 180.0} 0 0.0" xyz="0 0.017 0.027"/>
+                            <geometry>
+                                <box size="0.0222 0.007 0.025"/>
+                            </geometry>
+                            <material name="">
+                                <contact name="steel"/>
+                            </material>
+                        </collision>
+                        <collision>
+                            <origin rpy="0.0 0 0.0" xyz="0 0.007 0.045"/>
+                            <geometry>
+                                <box size="0.0222 0.0145 0.018"/>
+                            </geometry>
+                            <material name="">
+                                <contact name="steel"/>
+                            </material>
+                        </collision>
+                    </xacro:if>
+                </link>
+                <link name="panda_rightfinger">
+                    <inertial>
+                        <mass value="0.1"/>
+                        <origin rpy="0 0 3.14159265359" xyz="0 0.0145644 0.0227941"/>
+                        <inertia ixx="3.01220925051e-05" ixy="0.0" ixz="0.0" iyy="2.95873808038e-05" iyz="0.0"
+                                 izz="6.95125211657e-06"/>
+                    </inertial>
+                    <visual>
+                        <origin rpy="0 0 3.14159265359" xyz="0 0 0"/>
                         <geometry>
-                            <box size="0.0222 0.0145 0.018"/>
+                            <mesh filename="${resources_prefix}${resources_directory}/resources/panda/meshes/visual/finger.dae"/>
                         </geometry>
                         <material name="">
-                            <contact name="steel"/>
+                            <color rgba="1 1 1 1"/>
                         </material>
-                    </collision>
-                </xacro:if>
-            </link>
-            <link name="panda_rightfinger">
-                <inertial>
-                    <mass value="0.1"/>
-                    <origin rpy="0 0 3.14159265359" xyz="0 0.0145644 0.0227941"/>
-                    <inertia ixx="3.01220925051e-05" ixy="0.0" ixz="0.0" iyy="2.95873808038e-05" iyz="0.0"
-                             izz="6.95125211657e-06"/>
-                </inertial>
-                <visual>
-                    <origin rpy="0 0 3.14159265359" xyz="0 0 0"/>
-                    <geometry>
-                        <mesh filename="${resources_prefix}${resources_directory}/resources/panda/meshes/visual/finger.dae"/>
-                    </geometry>
-                    <material name="">
-                        <color rgba="1 1 1 1"/>
-                    </material>
-                </visual>
-                <xacro:if value="${collision_finger}">
-                    <collision>
-                        <origin rpy="0.0 0 0.0" xyz="0 -0.018 0.01"/>
-                        <geometry>
-                            <box size="0.0222 0.015 0.02"/>
-                        </geometry>
-                        <material name="">
-                            <contact name="steel"/>
-                        </material>
-                    </collision>
-                    <collision>
-                        <origin rpy="${-3.14 * 30 / 180.0} 0 0.0" xyz="0 -0.017 0.027"/>
-                        <geometry>
-                            <box size="0.0222 0.007 0.025"/>
-                        </geometry>
-                        <material name="">
-                            <contact name="steel"/>
-                        </material>
-                    </collision>
-                    <collision>
-                        <origin rpy="0.0 0 0.0" xyz="0 -0.007 0.045"/>
-                        <geometry>
-                            <box size="0.0222 0.0145 0.018"/>
-                        </geometry>
-                        <material name="">
-                            <contact name="steel"/>
-                        </material>
-                    </collision>
-                </xacro:if>
-            </link>
+                    </visual>
+                    <xacro:if value="${collision_finger}">
+                        <collision>
+                            <origin rpy="0.0 0 0.0" xyz="0 -0.018 0.01"/>
+                            <geometry>
+                                <box size="0.0222 0.015 0.02"/>
+                            </geometry>
+                            <material name="">
+                                <contact name="steel"/>
+                            </material>
+                        </collision>
+                        <collision>
+                            <origin rpy="${-3.14 * 30 / 180.0} 0 0.0" xyz="0 -0.017 0.027"/>
+                            <geometry>
+                                <box size="0.0222 0.007 0.025"/>
+                            </geometry>
+                            <material name="">
+                                <contact name="steel"/>
+                            </material>
+                        </collision>
+                        <collision>
+                            <origin rpy="0.0 0 0.0" xyz="0 -0.007 0.045"/>
+                            <geometry>
+                                <box size="0.0222 0.0145 0.018"/>
+                            </geometry>
+                            <material name="">
+                                <contact name="steel"/>
+                            </material>
+                        </collision>
+                    </xacro:if>
+                </link>
+            </xacro:unless>
             <joint name="panda_finger_joint1" type="prismatic">
                 <parent link="panda_hand"/>

Commit message: adding shelf base to avoid base collisions

File: mppi_examples/mppi_manipulation/data/objects/shelf.urdf.xacro (robot description, xacro)
@@ -10,4 +10,7 @@
     <xacro:property name="handle_length" default="0.16"/>
     <xacro:property name="handle_offset" default="0.27"/>
+    <xacro:property name="shelf_x" default="-0.011"/>
+    <xacro:property name="shelf_y" default="-0.431"/>
+    <xacro:property name="shelf_z" default="0.905"/>
     <xacro:macro name="box_inertia" params="m x y z">
         <inertial>
@@ -27,8 +30,25 @@
             <parent link="world"/>
             <child link="shelf"/>
-            <origin xyz="-0.011 -0.431 0.905" rpy="-0.006 0.001 1.585"/>
+            <origin xyz="${shelf_x} ${shelf_y} ${shelf_z}" rpy="-0.006 0.001 1.585"/>
         </joint>
     </xacro:if>
-    <link name="shelf"/>
+    <link name="shelf">
+        <xacro:box_inertia m="5" x="${door_width}" y="${door_length}" z="${shelf_z}"/>
+        <visual>
+            <origin rpy="0 0 0" xyz="0 -${door_length/2} ${-shelf_z/2}"/>
+            <geometry>
+                <box size="${door_width} ${door_length} ${shelf_z}"/>
+            </geometry>
+            <material name="shelf_material">
+                <color rgba="0.0 1.0 1.0 1"/>
+            </material>
+        </visual>
+        <collision>
+            <origin rpy="0 0 0" xyz="0 -${door_length/2} ${-shelf_z/2}"/>
+            <geometry>
+                <box size="${door_width} ${door_length} ${shelf_z}"/>
+            </geometry>
+        </collision>
+    </link>
     <link name="door">
         <xacro:box_inertia m="5.8" x="${door_width}" y="${door_length}" z="${door_height}"/>

Commit message: calibrated revolute joint and fixed observer bug (not using axis as reference)

File: mppi_examples/mppi_manipulation/data/objects/shelf.urdf.xacro (robot description, xacro)
@@ -7,10 +7,10 @@
     <xacro:property name="door_height" default="0.90"/>
     <xacro:property name="door_width" default="0.016"/>
-    <xacro:property name="handle_height" default="0.05"/> <!-- 0.026 -->
+    <xacro:property name="handle_height" default="0.056"/> <!-- 0.026 -->
     <xacro:property name="handle_length" default="0.16"/>
     <xacro:property name="handle_offset" default="0.27"/>
-    <xacro:property name="shelf_x" default="-0.011"/>
-    <xacro:property name="shelf_y" default="-0.431"/>
-    <xacro:property name="shelf_z" default="0.905"/>
+    <xacro:property name="shelf_x" default="0.012"/>
+    <xacro:property name="shelf_y" default="-0.410"/>
+    <xacro:property name="shelf_z" default="0.903"/>
     <xacro:macro name="box_inertia" params="m x y z">
         <inertial>
@@ -30,5 +30,5 @@
             <parent link="world"/>
             <child link="shelf"/>
-            <origin xyz="${shelf_x} ${shelf_y} ${shelf_z}" rpy="-0.006 0.001 1.585"/>
+            <origin xyz="${shelf_x} ${shelf_y} ${shelf_z}" rpy="-0.012 0.003 1.583"/>
         </joint>
     </xacro:if>
@@ -76,9 +76,15 @@
         <origin xyz="0 -${door_length} ${door_height/2}"/>
     </joint>
+    <link name="axis_link"/>
+    <joint name="axis_joint" type="fixed">
+        <parent link="door_hinge"/>
+        <child link="axis_link"/>
+        <origin xyz="0.004 0.027 -0.150"/>
+    </joint>
     <joint name="articulation_joint" type="revolute">
-        <parent link="door_hinge"/>
+        <parent link="axis_link"/>
         <child link="measured_joint_link"/>
         <dynamics damping="2.0" friction="4.0"/>
-        <origin xyz=" -0.004 0.023 -0.150"/>
+        <origin xyz="0 0 0"/>
         <axis xyz="0 0 -1"/>
         <limit effort="100" lower="0" upper="1.57" velocity="10.0"/>
@@ -87,5 +93,5 @@
         <parent link="measured_joint_link"/>
         <child link="door"/>
-        <origin xyz="0.004 -0.023 0.150"/>
+        <origin xyz="-0.004 -0.027 0.150"/>
     </joint>
     <link name="handle_link">
@@ -181,8 +187,9 @@
     </joint>
     <link name="measured_joint_link"/>
-<!--     <joint name="measured_joint_handle_joint" type="fixed">
+    <link name="measured_joint_link_test"/>
+    <joint name="measured_test_handle_joint" type="fixed">
         <parent link="handle_link"/>
-        <child link="measured_joint_link"/>
-        <origin xyz="-0.038456463645002395 -0.24676779774627114 0.0" rpy="0 0 0"/>
-    </joint> -->
+        <child link="measured_joint_link_test"/>
+        <origin xyz="-0.06 -0.243 0.0" rpy="0 0 0"/>
+    </joint>
 </robot>

File: mppi_examples/mppi_manipulation/data/panda_mobile.urdf.xacro (robot description, xacro)
@@ -19,5 +19,5 @@
             <parent link="world"/>
             <child link="base_link"/>
-             <origin xyz="0.016562803523970236 0.536778652875357 0.0" rpy="0.000 0.000 -1.5943151411055445"/>
+             <origin xyz="0.01085080249015791 0.6237166552544203 0.0" rpy="0.000 0.000 -1.6091077199502668"/>
         </joint>
     </xacro:if>
@@ -29,5 +29,5 @@
         <child link="franka_mount_link"/>
         <!--        <origin xyz="$(optenv RIDGEBACK_FRANKA_XYZ 0.21 0.0 0.2)" rpy="$(optenv RIDGEBACK_FRANKA_RPY 0 0 0)"/>-->
-        <origin xyz="$(optenv RIDGEBACK_FRANKA_XYZ 0.30 0.0 0.445)" rpy="$(optenv RIDGEBACK_FRANKA_RPY 0 0 0)"/>
+        <origin xyz="0.30 0.0 0.445" rpy="0 0 0"/>
     </joint>
     <link name="franka_mount_link"/>
@@ -40,5 +40,5 @@
             <child link="panda_grasp"/>
             <axis xyz="0 1 0"/>
-            <origin xyz="0 0 0.10" rpy="0 0 0"/>
+            <origin xyz="0 0 0.106" rpy="0 0 0"/> <!-- 0.106-->
         </joint>
     </xacro:if>

Commit message: vicon tuning

File: mppi_examples/mppi_manipulation/data/objects/shelf.urdf.xacro (robot description, xacro)
@@ -10,6 +10,6 @@
     <xacro:property name="handle_length" default="0.16"/>
     <xacro:property name="handle_offset" default="0.27"/>
-    <xacro:property name="shelf_x" default="0.012"/>
-    <xacro:property name="shelf_y" default="-0.410"/>
+    <xacro:property name="shelf_x" default="0.469"/>
+    <xacro:property name="shelf_y" default="-0.358"/>
     <xacro:property name="shelf_z" default="0.903"/>
     <xacro:macro name="box_inertia" params="m x y z">
@@ -30,5 +30,5 @@
             <parent link="world"/>
             <child link="shelf"/>
-            <origin xyz="${shelf_x} ${shelf_y} ${shelf_z}" rpy="-0.012 0.003 1.583"/>
+            <origin xyz="${shelf_x} ${shelf_y} ${shelf_z}" rpy="-0.008 0.007 -3.104"/>
         </joint>
     </xacro:if>
@@ -73,5 +73,5 @@
         <parent link="shelf"/>
         <child link="door_hinge"/>
-        <dynamics damping="2.0" friction="4.0"/>
+        <dynamics damping="2.0" friction="8.0"/>
         <origin xyz="0 -${door_length} ${door_height/2}"/>
     </joint>

File: mppi_examples/mppi_manipulation/data/panda_mobile.urdf.xacro (robot description, xacro)
@@ -19,5 +19,5 @@
             <parent link="world"/>
             <child link="base_link"/>
-             <origin xyz="0.01085080249015791 0.6237166552544203 0.0" rpy="0.000 0.000 -1.6091077199502668"/>
+             <origin xyz="-0.5265965085817698 -0.2806388380571893 0.0" rpy="0.000 0.000 -0.04332860681335808"/>
         </joint>
     </xacro:if>
@@ -40,5 +40,5 @@
             <child link="panda_grasp"/>
             <axis xyz="0 1 0"/>
-            <origin xyz="0 0 0.106" rpy="0 0 0"/> <!-- 0.106-->
+            <origin xyz="0 0 0.098" rpy="0 0 0"/> <!-- 0.106-->
         </joint>
     </xacro:if>

Commit message: recording rate and plots

File: mppi_examples/mppi_manipulation/data/objects/shelf.urdf.xacro (robot description, xacro)
@@ -10,5 +10,5 @@
     <xacro:property name="handle_length" default="0.16"/>
     <xacro:property name="handle_offset" default="0.27"/>
-    <xacro:property name="shelf_x" default="0.469"/>
+    <xacro:property name="shelf_x" default="1.469"/>
     <xacro:property name="shelf_y" default="-0.358"/>
     <xacro:property name="shelf_z" default="0.903"/>

Commit message: experiment tuning

File: mppi_examples/mppi_manipulation/data/objects/shelf.urdf.xacro (robot description, xacro)
@@ -10,6 +10,6 @@
     <xacro:property name="handle_length" default="0.16"/>
     <xacro:property name="handle_offset" default="0.27"/>
-    <xacro:property name="shelf_x" default="0.469"/>
-    <xacro:property name="shelf_y" default="-0.358"/>
+    <xacro:property name="shelf_x" default="0.959"/>
+    <xacro:property name="shelf_y" default="-1.05"/>
     <xacro:property name="shelf_z" default="0.903"/>
     <xacro:macro name="box_inertia" params="m x y z">
@@ -30,5 +30,5 @@
             <parent link="world"/>
             <child link="shelf"/>
-            <origin xyz="${shelf_x} ${shelf_y} ${shelf_z}" rpy="-0.008 0.007 -3.104"/>
+            <origin xyz="${shelf_x} ${shelf_y} ${shelf_z}" rpy="-0.019 0.002 -3.090"/>
         </joint>
     </xacro:if>

Commit message: flexible urdf model for simulation

File: mppi_examples/mppi_manipulation/data/objects/shelf.urdf.xacro (robot description, xacro)
@@ -3,5 +3,15 @@
     <xacro:arg name="fixed" default="true"/>
     <xacro:arg name="height" default="0.0"/>
+    <xacro:arg name="shelf_x" default="0.943"/>
+    <xacro:arg name="shelf_y" default="-0.952"/>
+    <xacro:arg name="shelf_z" default="0.903"/>
+    <xacro:arg name="hinge_offset_x" default="0.004"/>
+    <xacro:arg name="hinge_offset_y" default="0.027"/>
+    <xacro:property name="shelf_x" default="$(arg shelf_x)"/>
+    <xacro:property name="shelf_y" default="$(arg shelf_y)"/>
+    <xacro:property name="shelf_z" default="$(arg shelf_z)"/>
     <xacro:property name="height" default="$(arg height)"/>
+    <xacro:property name="hinge_offset_x" default="$(arg hinge_offset_x)"/>
+    <xacro:property name="hinge_offset_y" default="$(arg hinge_offset_y)"/>
     <xacro:property name="door_length" default="0.295"/>
     <xacro:property name="door_height" default="0.90"/>
@@ -10,7 +20,4 @@
     <xacro:property name="handle_length" default="0.16"/>
     <xacro:property name="handle_offset" default="0.27"/>
-    <xacro:property name="shelf_x" default="0.943"/>
-    <xacro:property name="shelf_y" default="-0.952"/>
-    <xacro:property name="shelf_z" default="0.903"/>
     <xacro:macro name="box_inertia" params="m x y z">
         <inertial>
@@ -80,5 +87,5 @@
         <parent link="door_hinge"/>
         <child link="axis_link"/>
-        <origin xyz="0.004 0.027 -0.150"/>
+        <origin xyz="${hinge_offset_x} ${hinge_offset_y} -0.150"/>
     </joint>
     <joint name="articulation_joint" type="revolute">
@@ -93,5 +100,5 @@
         <parent link="measured_joint_link"/>
         <child link="door"/>
-        <origin xyz="-0.004 -0.027 0.150"/>
+        <origin xyz="-${hinge_offset_x} -${hinge_offset_y} 0.150"/>
     </joint>
     <link name="handle_link">
