Commit message: experiments with and without filter

File: mppi_examples/mppi_manipulation/data/objects/shelf.urdf.xacro (robot description, xacro)
@@ -1,4 +1,5 @@
 <?xml version="1.0" ?>
 <robot name="shelf" xmlns:xacro="http://www.ros.org/wiki/xacro">
+    <xacro:arg name="prefix" default=""/>
     <xacro:arg name="fixed" default="true"/>
     <xacro:arg name="height" default="0.0"/>
@@ -6,6 +7,8 @@
     <xacro:arg name="shelf_y" default="-0.952"/>
     <xacro:arg name="shelf_z" default="0.903"/>
+    <xacro:arg name="articulation_mismatch_offset" default="0.0"/>
     <xacro:arg name="hinge_offset_x" default="0.004"/>
     <xacro:arg name="hinge_offset_y" default="0.027"/>
+    <xacro:property name="prefix" default="$(arg prefix)"/>
     <xacro:property name="shelf_x" default="$(arg shelf_x)"/>
     <xacro:property name="shelf_y" default="$(arg shelf_y)"/>
@@ -14,4 +17,5 @@
     <xacro:property name="hinge_offset_x" default="$(arg hinge_offset_x)"/>
     <xacro:property name="hinge_offset_y" default="$(arg hinge_offset_y)"/>
+    <xacro:property name="articulation_mismatch_offset" default="$(arg articulation_mismatch_offset)"/>
     <xacro:property name="door_length" default="0.295"/>
     <xacro:property name="door_height" default="0.90"/>
@@ -29,5 +33,5 @@
                      iyy="${0.0833 * m * (x**2 + z**2)}"
                      iyz="0"
-                     izz="${0.0833 * m * (z**2 + y**2)}"/>
+                     izz="${0.0833 * m * (x**2 + y**2)}"/>
         </inertial>
     </xacro:macro>
@@ -36,10 +40,10 @@
         <joint name="fixed" type="fixed">
             <parent link="world"/>
-            <child link="shelf"/>
+            <child link="${prefix}shelf"/>
             <origin xyz="${shelf_x} ${shelf_y} ${shelf_z}" rpy="-0.008 -0.001 -3.085"/>
         </joint>
     </xacro:if>
-    <link name="shelf">
-        <xacro:box_inertia m="5" x="${door_width}" y="${door_length}" z="${shelf_z}"/>
+    <link name="${prefix}shelf">
+        <xacro:box_inertia m="4" x="${door_width}" y="${door_length}" z="${shelf_z}"/>
         <visual>
             <origin rpy="0 0 0" xyz="0 -${door_length/2} ${-shelf_z/2}"/>
@@ -58,5 +62,5 @@
         </collision>
     </link>
-    <link name="door">
+    <link name="${prefix}door">
         <xacro:box_inertia m="5.8" x="${door_width}" y="${door_length}" z="${door_height}"/>
         <visual>
@@ -76,20 +80,20 @@
         </collision>
     </link>
-    <link name="door_hinge"/>
-    <joint name="door_hinge_joint" type="fixed">
-        <parent link="shelf"/>
-        <child link="door_hinge"/>
+    <link name="${prefix}door_hinge"/>
+    <joint name="${prefix}door_hinge_joint" type="fixed">
+        <parent link="${prefix}shelf"/>
+        <child link="${prefix}door_hinge"/>
         <dynamics damping="2.0" friction="8.0"/>
         <origin xyz="0 -${door_length} ${door_height/2}"/>
     </joint>
-    <link name="axis_link"/>
-    <joint name="axis_joint" type="fixed">
-        <parent link="door_hinge"/>
-        <child link="axis_link"/>
-        <origin xyz="${hinge_offset_x} ${hinge_offset_y} -0.150"/>
+    <link name="${prefix}axis_link"/>
+    <joint name="${prefix}axis_joint" type="fixed">
+        <parent link="${prefix}door_hinge"/>
+        <child link="${prefix}axis_link"/>
+        <origin xyz="${hinge_offset_x} ${hinge_offset_y + articulation_mismatch_offset} -0.150"/>
     </joint>
     <joint name="articulation_joint" type="revolute">
-        <parent link="axis_link"/>
-        <child link="measured_joint_link"/>
+        <parent link="${prefix}axis_link"/>
+        <child link="${prefix}measured_joint_link"/>
         <dynamics damping="2.0" friction="4.0"/>
         <origin xyz="0 0 0"/>
@@ -97,10 +101,10 @@
         <limit effort="100" lower="0" upper="1.57" velocity="10.0"/>
     </joint>
-    <joint name="door_link" type="fixed">
-        <parent link="measured_joint_link"/>
-        <child link="door"/>
-        <origin xyz="-${hinge_offset_x} -${hinge_offset_y} 0.150"/>
-    </joint>
-    <link name="handle_link">
+    <joint name="${prefix}door_link" type="fixed">
+        <parent link="${prefix}measured_joint_link"/>
+        <child link="${prefix}door"/>
+        <origin xyz="-${hinge_offset_x} -${hinge_offset_y + articulation_mismatch_offset} 0.150"/>
+    </joint>
+    <link name="${prefix}handle_link">
         <inertial>
             <origin rpy="0 0 0" xyz="0 0 0"/>
@@ -127,5 +131,5 @@
         </collision>
     </link>
-    <link name="handle_support_left">
+    <link name="${prefix}handle_support_left">
         <inertial>
             <origin rpy="0 0 0" xyz="0 0 0"/>
@@ -152,5 +156,5 @@
         </collision>
     </link>
-    <link name="handle_support_right">
+    <link name="${prefix}handle_support_right">
         <inertial>
             <origin rpy="0 0 0" xyz="0 0 0"/>
@@ -177,25 +181,25 @@
         </collision>
     </link>
-    <joint name="handle_joint" type="fixed">
-        <parent link="door"/>
-        <child link="handle_link"/>
+    <joint name="${prefix}handle_joint" type="fixed">
+        <parent link="${prefix}door"/>
+        <child link="${prefix}handle_link"/>
         <origin xyz="${handle_height + door_width/2} ${handle_offset} -0.15"
                 rpy="0 0 0"/> <!-- height handle + half the width door, 0.30 minus some offset -->
     </joint>
-    <joint name="handle_support_left_joint" type="fixed">
-        <parent link="handle_link"/>
-        <child link="handle_support_left"/>
+    <joint name="${prefix}handle_support_left_joint" type="fixed">
+        <parent link="${prefix}handle_link"/>
+        <child link="${prefix}handle_support_left"/>
         <origin xyz="-${handle_height/2} 0 ${handle_length/2}" rpy="0 0 0"/>
     </joint>
-    <joint name="handle_support_right_joint" type="fixed">
-        <parent link="handle_link"/>
-        <child link="handle_support_right"/>
+    <joint name="${prefix}handle_support_right_joint" type="fixed">
+        <parent link="${prefix}handle_link"/>
+        <child link="${prefix}handle_support_right"/>
         <origin xyz="-${handle_height/2} 0 -${handle_length/2}" rpy="0 0 0"/>
     </joint>
-    <link name="measured_joint_link"/>
-    <link name="measured_joint_link_test"/>
-    <joint name="measured_test_handle_joint" type="fixed">
-        <parent link="handle_link"/>
-        <child link="measured_joint_link_test"/>
+    <link name="${prefix}measured_joint_link"/>
+    <link name="${prefix}measured_joint_link_test"/>
+    <joint name="${prefix}measured_test_handle_joint" type="fixed">
+        <parent link="${prefix}handle_link"/>
+        <child link="${prefix}measured_joint_link_test"/>
         <origin xyz="-0.06 -0.243 0.0" rpy="0 0 0"/>
     </joint>
