Commit message: urdf refactoring and ros controller

File: mppi_examples/mppi_manipulation/data/objects/door.urdf.xacro (robot description, xacro)
@@ -1,9 +1,11 @@
 <?xml version="1.0" ?>
-<robot name="door">
+<robot name="door" xmlns:xacro="http://www.ros.org/wiki/xacro" >
+    <xacro:arg name="height" default="0.0"/>
+    <xacro:property name="height" default="$(arg height)"/>
     <link name="world"/>
     <joint name="fixed" type="fixed">
         <parent link="world"/>
         <child link="door_frame"/>
-        <origin xyz="0.65 0.3 0.01" rpy="0 0 3.14"/>
+        <origin xyz="0.65 0.3 ${height + 0.01}" rpy="0 0 3.14"/>
     </joint>
     <link name="door_frame">

File: mppi_examples/mppi_manipulation/data/objects/drawer.urdf.xacro (robot description, xacro)
@@ -1,9 +1,11 @@
 <?xml version="1.0" ?>
-<robot name="door">
+<robot name="drawer"  xmlns:xacro="http://www.ros.org/wiki/xacro" >
+    <xacro:arg name="height" default="0.0"/>
+    <xacro:property name="height" default="$(arg height)"/>
     <link name="world"/>
     <joint name="fixed" type="fixed">
         <parent link="world"/>
         <child link="drawer_frame"/>
-        <origin xyz="0.65 0.3 0.01" rpy="0 0 3.14"/>
+        <origin xyz="0.65 0.3 ${height + 0.01}" rpy="0 0 3.14"/>
     </joint>
     <link name="drawer_frame">

File: mppi_examples/mppi_manipulation/data/objects/microwave.urdf.xacro (robot description, xacro)
@@ -1,9 +1,11 @@
 <?xml version="1.0" ?>
-<robot name="door">
+<robot name="microwave"  xmlns:xacro="http://www.ros.org/wiki/xacro" >
+    <xacro:arg name="height" default="0.0"/>
+    <xacro:property name="height" default="$(arg height)"/>
     <link name="world"/>
     <joint name="fixed" type="fixed">
         <parent link="world"/>
         <child link="door_frame"/>
-        <origin xyz="0.65 -0.3 0.3" rpy="1.57 0 3.14"/>
+        <origin xyz="0.65 -0.3 ${height + 0.3}" rpy="1.57 0 3.14"/>
     </joint>
     <link name="door_frame">

File: mppi_examples/mppi_manipulation/data/objects/shelf.urdf.xacro (robot description, xacro)
@@ -1,4 +1,6 @@
 <?xml version="1.0" ?>
 <robot name="shelf" xmlns:xacro="http://www.ros.org/wiki/xacro" >
+    <xacro:arg name="height" default="0.0"/>
+    <xacro:property name="height" default="$(arg height)"/>
     <xacro:property name="door_length" default="0.30"/>
     <xacro:property name="door_height" default="0.90"/>
@@ -11,5 +13,5 @@
         <parent link="world"/>
         <child link="shelf"/>
-        <origin xyz="0.5 0 0" rpy="0 0 3.14159"/>
+        <origin xyz="1.5 0 ${height}" rpy="0 0 3.14159"/>
     </joint>
     <link name="shelf"/>

File: mppi_examples/mppi_manipulation/data/objects/valve.urdf.xacro (robot description, xacro)
@@ -3,9 +3,11 @@
     <xacro:arg name="resource_prefix" default=""/>
     <xacro:arg name="resource_directory" default="$(find mppi_manipulation)/data/meshes"/>
+    <xacro:arg name="height" default="0.0"/>
+    <xacro:property name="height" default="$(arg height)"/>
     <link name="world"/>
     <joint name="fixed" type="fixed">
         <parent link="world"/>
         <child link="valve_base"/>
-        <origin xyz="0.5 0.0 0.335" rpy="1.57 0 0"/>
+        <origin xyz="0.5 0.0 ${height + 0.335}" rpy="1.57 0 0"/>
     </joint>
     <link name="valve_base"/>

Commit message: launch refactoring and same description for fixed and moving base

File: mppi_examples/mppi_manipulation/data/objects/door.urdf.xacro (robot description, xacro)
@@ -7,5 +7,5 @@
         <parent link="world"/>
         <child link="door_frame"/>
-        <origin xyz="0.65 0.3 ${height + 0.01}" rpy="0 0 3.14"/>
+        <origin xyz="1.0 0.3 ${height + 0.01}" rpy="0 0 3.14"/>
     </joint>
     <link name="door_frame">

File: mppi_examples/mppi_manipulation/data/objects/drawer.urdf.xacro (robot description, xacro)
@@ -7,5 +7,5 @@
         <parent link="world"/>
         <child link="drawer_frame"/>
-        <origin xyz="0.65 0.3 ${height + 0.01}" rpy="0 0 3.14"/>
+        <origin xyz="1.0 0.3 ${height + 0.01}" rpy="0 0 3.14"/>
     </joint>
     <link name="drawer_frame">

File: mppi_examples/mppi_manipulation/data/objects/microwave.urdf.xacro (robot description, xacro)
@@ -7,5 +7,5 @@
         <parent link="world"/>
         <child link="door_frame"/>
-        <origin xyz="0.65 -0.3 ${height + 0.3}" rpy="1.57 0 3.14"/>
+        <origin xyz="1.0 -0.3 ${height + 0.3}" rpy="1.57 0 3.14"/>
     </joint>
     <link name="door_frame">

File: mppi_examples/mppi_manipulation/data/objects/shelf.urdf.xacro (robot description, xacro)
@@ -27,5 +27,5 @@
             <parent link="world"/>
             <child link="shelf"/>
-            <origin xyz="0 0 ${height}" rpy="0 0 3.14159"/>
+            <origin xyz="1.0 0 ${height}" rpy="0 0 3.14159"/>
         </joint>
     </xacro:if>

File: mppi_examples/mppi_manipulation/data/objects/valve.urdf.xacro (robot description, xacro)
@@ -9,5 +9,5 @@
         <parent link="world"/>
         <child link="valve_base"/>
-        <origin xyz="0.5 0.0 ${height + 0.335}" rpy="1.57 0 0"/>
+        <origin xyz="1.0 0.0 ${height + 0.335}" rpy="1.57 0 0"/>
     </joint>
     <link name="valve_base"/>

File: mppi_examples/mppi_manipulation/data/panda_mobile.urdf.xacro (robot description, xacro)
@@ -1,4 +1,5 @@
 <?xml version="1.0"?>
 <robot xmlns:xacro="http://www.ros.org/wiki/xacro" name="panda">
+    <xacro:arg name="fixed_base" default="false"/>
     <xacro:include filename="$(find mppi_panda)/resources/panda/panda.urdf.xacro"/>
     <xacro:include filename="$(find mppi_manipulation)/data/planar_base.urdf.xacro"/>
@@ -6,10 +7,18 @@
     <!--    Root world link-->
     <link name="world"/>
-    <joint name="world_joint" type="fixed">
-        <parent link="world"/>
-        <child link="omni_base_root_link"/>
-    </joint>
     <!--    Omnidirectional base-->
-    <xacro:planar_base connect_to="base_link"/>
+    <xacro:unless value="$(arg fixed_base)">
+        <joint name="world_joint" type="fixed">
+            <parent link="world"/>
+            <child link="omni_base_root_link"/>
+        </joint>
+        <xacro:planar_base connect_to="base_link"/>
+    </xacro:unless>
+    <xacro:if value="$(arg fixed_base)">
+        <joint name="world_joint" type="fixed">
+            <parent link="world"/>
+            <child link="base_link"/>
+        </joint>
+    </xacro:if>
     <!--   Ridgeback base: for collision and appearance -->
     <xacro:ridgeback/>
@@ -18,5 +27,5 @@
         <parent link="mid_mount"/>
         <child link="franka_mount_link"/>
-<!--        <origin xyz="$(optenv RIDGEBACK_FRANKA_XYZ 0.21 0.0 0.2)" rpy="$(optenv RIDGEBACK_FRANKA_RPY 0 0 0)"/>-->
+        <!--        <origin xyz="$(optenv RIDGEBACK_FRANKA_XYZ 0.21 0.0 0.2)" rpy="$(optenv RIDGEBACK_FRANKA_RPY 0 0 0)"/>-->
         <origin xyz="$(optenv RIDGEBACK_FRANKA_XYZ 0.30 0.0 0.445)" rpy="$(optenv RIDGEBACK_FRANKA_RPY 0 0 0)"/>
     </joint>

Commit message: fix to collision mesh

File: mppi_examples/mppi_manipulation/data/objects/door.urdf.xacro (robot description, xacro)
@@ -98,5 +98,5 @@
             <origin rpy="0 0 0" xyz="0 0 0"/>
             <geometry>
-                <cylinder radius="0.005" length="0.010"/>
+                <cylinder radius="0.005" length="0.10"/>
             </geometry>
         </collision>

Commit message: evaluation wip

File: mppi_examples/mppi_manipulation/data/objects/door.urdf.xacro (robot description, xacro)
@@ -1,13 +1,19 @@
 <?xml version="1.0" ?>
 <robot name="door" xmlns:xacro="http://www.ros.org/wiki/xacro" >
+    <xacro:arg name="prefix" default=""/>
     <xacro:arg name="height" default="0.0"/>
+    <xacro:arg name="door_x" default="1.0"/>
+    <xacro:arg name="articulation_mismatch_offset" default="0.0"/>
+    <xacro:property name="prefix" default="$(arg prefix)"/>
+    <xacro:property name="door_x" default="$(arg door_x)"/>
+    <xacro:property name="articulation_mismatch_offset" default="$(arg articulation_mismatch_offset)"/>
     <xacro:property name="height" default="$(arg height)"/>
     <link name="world"/>
     <joint name="fixed" type="fixed">
         <parent link="world"/>
-        <child link="door_frame"/>
-        <origin xyz="1.0 0.3 ${height + 0.01}" rpy="0 0 3.14"/>
+        <child link="${prefix}door_frame"/>
+        <origin xyz="${door_x} 0.3 ${height + 0.01}" rpy="0 0 3.14"/>
     </joint>
-    <link name="door_frame">
+    <link name="${prefix}door_frame">
         <visual>
             <origin rpy="0 0 0" xyz="0 0 0.25"/>
@@ -50,12 +56,12 @@
         <axis xyz="0 1 0"/>
     </joint-->
-    <link name="door_link">
+    <link name="${prefix}door_link">
         <inertial>
-            <origin rpy="0 0 0" xyz="0 0 0.25"/>
+            <origin rpy="0 0 0" xyz="0 0 ${0.25 - articulation_mismatch_offset}"/>
             <mass value="1.0"/>
             <inertia ixx="0.048966669" ixy="0" ixz="0" iyy="0.046466667" iyz="0" izz="0.0041666669"/>
         </inertial>
         <visual>
-            <origin rpy="0 0 0" xyz="0 0 0.25"/>
+            <origin rpy="0 0 0" xyz="0 0 ${0.25 - articulation_mismatch_offset}"/>
             <geometry>
                 <box size="0.02 0.6 0.5"/>
@@ -66,5 +72,5 @@
         </visual>
         <collision>
-            <origin rpy="0 0 0" xyz="0 0 0.25"/>
+            <origin rpy="0 0 0" xyz="0 0 ${0.25 - articulation_mismatch_offset}"/>
             <geometry>
                 <box size="0.02 0.6 0.5"/>
@@ -73,12 +79,12 @@
     </link>
     <joint name="articulation_joint" type="revolute">
-        <parent link="door_frame"/>
-        <child link="door_link"/>
+        <parent link="${prefix}door_frame"/>
+        <child link="${prefix}door_link"/>
         <dynamics damping="1.0" friction="4.0"/>
-        <origin xyz="0.046 0 0"/>
+        <origin xyz="0.046 0.0 ${articulation_mismatch_offset}"/>
         <axis xyz="0 1 0"/>
         <limit effort="100" lower="0" upper="1.57" velocity="10.0"/>
     </joint>
-    <link name="handle_link">
+    <link name="${prefix}handle_link">
         <inertial>
             <origin rpy="0 0 0" xyz="0 0 0"/>
@@ -98,12 +104,12 @@
             <origin rpy="0 0 0" xyz="0 0 0"/>
             <geometry>
-                <cylinder radius="0.005" length="0.010"/>
+                <cylinder radius="0.005" length="0.10"/>
             </geometry>
         </collision>
     </link>
-    <joint name="handle_joint" type="fixed">
-        <parent link="door_link"/>
-        <child link="handle_link"/>
-        <origin xyz="0.055 0 0.47" rpy="1.5708 0 0"/>
+    <joint name="${prefix}handle_joint" type="fixed">
+        <parent link="${prefix}door_link"/>
+        <child link="${prefix}handle_link"/>
+        <origin xyz="0.055 0 ${0.47 - articulation_mismatch_offset}" rpy="1.5708 0 0"/>
         <dynamics damping="1.0" friction="2.0"/>
         <axis xyz="0 1 0"/>

Commit message: before adding integral to sim

File: mppi_examples/mppi_manipulation/data/objects/door.urdf.xacro (robot description, xacro)
@@ -3,8 +3,8 @@
     <xacro:arg name="prefix" default=""/>
     <xacro:arg name="height" default="0.0"/>
-    <xacro:arg name="door_x" default="1.0"/>
+    <xacro:arg name="origin_x" default="1.0"/>
     <xacro:arg name="articulation_mismatch_offset" default="0.0"/>
     <xacro:property name="prefix" default="$(arg prefix)"/>
-    <xacro:property name="door_x" default="$(arg door_x)"/>
+    <xacro:property name="origin_x" default="$(arg origin_x)"/>
     <xacro:property name="articulation_mismatch_offset" default="$(arg articulation_mismatch_offset)"/>
     <xacro:property name="height" default="$(arg height)"/>
@@ -13,5 +13,5 @@
         <parent link="world"/>
         <child link="${prefix}door_frame"/>
-        <origin xyz="${door_x} 0.3 ${height + 0.01}" rpy="0 0 3.14"/>
+        <origin xyz="${origin_x} 0.3 ${height + 0.01}" rpy="0 0 3.14"/>
     </joint>
     <link name="${prefix}door_frame">
@@ -32,28 +32,4 @@
         </collision>
     </link>
-    <!--link name="door_frame_step">
-        <visual>
-            <origin rpy="0 0 0" xyz="0 0 0.25"/>
-            <geometry>
-                <box size="0.081 0.6 0.10"/>
-            </geometry>
-            <material name="frame_material">
-                <color rgba="0.5 0.0 0.0 1" />
-            </material>
-        </visual>
-        <collision>
-            <origin rpy="0 0 0" xyz="0 0 0.25"/>
-            <geometry>
-                <box size="0.081 0.6 0.10"/>
-            </geometry>
-        </collision>
-    </link>
-    <joint name="step_joint" type="fixed">
-        <parent link="door_frame"/>
-        <child link="door_frame_step"/>
-        <origin xyz="0.0155 0 0.31" rpy="0 0 0"/>
-        <dynamics damping="1.0" friction="2.0"/>
-        <axis xyz="0 1 0"/>
-    </joint-->
     <link name="${prefix}door_link">
         <inertial>

File: mppi_examples/mppi_manipulation/data/objects/drawer.urdf.xacro (robot description, xacro)
@@ -2,12 +2,18 @@
 <robot name="drawer"  xmlns:xacro="http://www.ros.org/wiki/xacro" >
     <xacro:arg name="height" default="0.0"/>
+    <xacro:arg name="prefix" default=""/>
+    <xacro:arg name="origin_x" default="1.0"/>
+    <xacro:arg name="articulation_mismatch_offset" default="0.0"/>
+    <xacro:property name="origin_x" default="$(arg origin_x)"/>
+    <xacro:property name="prefix" default="$(arg prefix)"/>
+    <xacro:property name="articulation_mismatch_offset" default="$(arg articulation_mismatch_offset)"/>
     <xacro:property name="height" default="$(arg height)"/>
     <link name="world"/>
     <joint name="fixed" type="fixed">
         <parent link="world"/>
-        <child link="drawer_frame"/>
-        <origin xyz="1.5 0.3 ${height + 0.01}" rpy="0 0 3.14"/>
+        <child link="${prefix}drawer_frame"/>
+        <origin xyz="${origin_x} 0.3 ${height + 0.01}" rpy="0 0 3.14"/>
     </joint>
-    <link name="drawer_frame">
+    <link name="${prefix}drawer_frame">
         <visual>
             <origin rpy="0 0 0" xyz="0 0 0.25"/>
@@ -26,29 +32,5 @@
         </collision>
     </link>
-    <!--link name="door_frame_step">
-        <visual>
-            <origin rpy="0 0 0" xyz="0 0 0.25"/>
-            <geometry>
-                <box size="0.081 0.6 0.10"/>
-            </geometry>
-            <material name="frame_material">
-                <color rgba="0.5 0.0 0.0 1" />
-            </material>
-        </visual>
-        <collision>
-            <origin rpy="0 0 0" xyz="0 0 0.25"/>
-            <geometry>
-                <box size="0.081 0.6 0.10"/>
-            </geometry>
-        </collision>
-    </link>
-    <joint name="step_joint" type="fixed">
-        <parent link="door_frame"/>
-        <child link="door_frame_step"/>
-        <origin xyz="0.0155 0 0.31" rpy="0 0 0"/>
-        <dynamics damping="1.0" friction="2.0"/>
-        <axis xyz="0 1 0"/>
-    </joint-->
-    <link name="drawer_link">
+    <link name="${prefix}drawer_link">
         <inertial>
             <origin rpy="0 0 0" xyz="0 0 0.25"/>
@@ -73,6 +55,6 @@
     </link>
     <joint name="articulation_joint" type="prismatic">
-        <parent link="drawer_frame"/>
-        <child link="drawer_link"/>
+        <parent link="${prefix}drawer_frame"/>
+        <child link="${prefix}drawer_link"/>
         <dynamics damping="2.0" friction="4.0"/>
         <origin xyz="0.046 0 0"/>
@@ -80,5 +62,5 @@
         <limit effort="100" lower="0" upper="0.55" velocity="10.0"/>
     </joint>
-    <link name="handle_link">
+    <link name="${prefix}handle_link">
         <inertial>
             <origin rpy="0 0 0" xyz="0 0 0"/>
@@ -105,7 +87,7 @@
         </collision>
     </link>
-    <joint name="handle_joint" type="fixed">
-        <parent link="drawer_link"/>
-        <child link="handle_link"/>
+    <joint name="${prefix}handle_joint" type="fixed">
+        <parent link="${prefix}drawer_link"/>
+        <child link="${prefix}handle_link"/>
         <origin xyz="0.055 0 0.47" rpy="1.5708 0 0"/>
         <dynamics damping="1.0" friction="2.0"/>

File: mppi_examples/mppi_manipulation/data/objects/microwave.urdf.xacro (robot description, xacro)
@@ -2,12 +2,18 @@
 <robot name="microwave"  xmlns:xacro="http://www.ros.org/wiki/xacro" >
     <xacro:arg name="height" default="0.0"/>
+    <xacro:arg name="origin_x" default="1.0"/>
+    <xacro:arg name="prefix" default=""/>
+    <xacro:arg name="articulation_mismatch_offset" default="0.0"/>
     <xacro:property name="height" default="$(arg height)"/>
+    <xacro:property name="origin_x" default="$(arg origin_x)"/>
+    <xacro:property name="prefix" default="$(arg prefix)"/>
+    <xacro:property name="articulation_mismatch_offset" default="$(arg articulation_mismatch_offset)"/>
     <link name="world"/>
     <joint name="fixed" type="fixed">
         <parent link="world"/>
-        <child link="door_frame"/>
-        <origin xyz="1.0 -0.3 ${height + 0.3}" rpy="1.57 0 3.14"/>
+        <child link="${prefix}door_frame"/>
+        <origin xyz="${origin_x} -0.3 1.0" rpy="1.57 0 3.14"/> <!-- ${height + 0.3} -->
     </joint>
-    <link name="door_frame">
+    <link name="${prefix}door_frame">
         <visual>
             <origin rpy="0 0 0" xyz="0 0 0.2"/>
@@ -26,5 +32,5 @@
         </collision>
     </link>
-    <link name="door_link">
+    <link name="${prefix}door_link">
         <inertial>
             <origin rpy="0 0 0" xyz="0 0 0.2"/>
@@ -49,6 +55,6 @@
     </link>
     <joint name="articulation_joint" type="revolute">
-        <parent link="door_frame"/>
-        <child link="door_link"/>
+        <parent link="${prefix}door_frame"/>
+        <child link="${prefix}door_link"/>
         <dynamics damping="1.0" friction="4.0"/>
         <origin xyz="0.046 0 0"/>
@@ -56,5 +62,5 @@
         <limit effort="100" lower="0" upper="1.57" velocity="10.0"/>
     </joint>
-    <link name="handle_link">
+    <link name="${prefix}handle_link">
         <inertial>
             <origin rpy="0 0 0" xyz="0 0 0"/>
@@ -78,7 +84,7 @@
         </collision>
     </link>
-    <joint name="handle_joint" type="fixed">
-        <parent link="door_link"/>
-        <child link="handle_link"/>
+    <joint name="${prefix}handle_joint" type="fixed">
+        <parent link="${prefix}door_link"/>
+        <child link="${prefix}handle_link"/>
         <origin xyz="0.055 0 0.4" rpy="1.5708 0 0"/>
         <dynamics damping="1.0" friction="2.0"/>

File: mppi_examples/mppi_manipulation/data/objects/shelf.urdf (robot description, URDF)
Before this commit: robot shelf, 7 links, 6 joints
Links:
- link shelf: geometry visual cylinder length=0.01 radius=0.10

File: mppi_examples/mppi_manipulation/data/objects/shelf.urdf.xacro (robot description, xacro)
@@ -4,5 +4,5 @@
     <xacro:arg name="fixed" default="true"/>
     <xacro:arg name="height" default="0.0"/>
-    <xacro:arg name="shelf_x" default="0.943"/>
+    <xacro:arg name="origin_x" default="0.943"/>
     <xacro:arg name="shelf_y" default="-0.952"/>
     <xacro:arg name="shelf_z" default="0.903"/>
@@ -11,5 +11,5 @@
     <xacro:arg name="hinge_offset_y" default="0.027"/>
     <xacro:property name="prefix" default="$(arg prefix)"/>
-    <xacro:property name="shelf_x" default="$(arg shelf_x)"/>
+    <xacro:property name="origin_x" default="$(arg origin_x)"/>
     <xacro:property name="shelf_y" default="$(arg shelf_y)"/>
     <xacro:property name="shelf_z" default="$(arg shelf_z)"/>
@@ -41,5 +41,5 @@
             <parent link="world"/>
             <child link="${prefix}shelf"/>
-            <origin xyz="${shelf_x} ${shelf_y} ${shelf_z}" rpy="-0.008 -0.001 -3.085"/>
+            <origin xyz="${origin_x} ${shelf_y} ${shelf_z}" rpy="-0.008 -0.001 -3.085"/>
         </joint>
     </xacro:if>
@@ -53,4 +53,13 @@
             <material name="shelf_material">
                 <color rgba="0.0 1.0 1.0 1"/>
+            </material>
+        </visual>
+        <visual>
+            <origin xyz="0 0 ${-shelf_z}" rpy="0 0 0" />
+            <geometry>
+                <cylinder radius="0.35" length="0.01"/>
+            </geometry>
+            <material name="Cyan">
+                <color rgba="0 1.0 1.0 0.3"/>
             </material>
         </visual>

File: mppi_examples/mppi_manipulation/data/ridgeback.xacro (robot description, xacro)
@@ -28,4 +28,13 @@
             <inertia ixx="0.048966669" ixy="0" ixz="0" iyy="0.046466667" iyz="0" izz="0.0041666669"/>
         </inertial>
+        <visual>
+            <origin xyz="0 0 0" rpy="0 0 0" />
+            <geometry>
+               <cylinder radius="0.53" length="0.01"/>
+            </geometry>
+            <material name="Cyan">
+               <color rgba="0 1.0 1.0 0.3"/>
+            </material>
+        </visual>
 <!--        <collision>-->
 <!--            <origin rpy="0 0 0" xyz="0 0 0.25"/>-->

File: mppi_examples/mppi_panda/resources/panda/panda.urdf.xacro (robot description, xacro)
@@ -501,4 +501,16 @@
                         </material>
                     </visual>
+                    <!-- <xacro:if value="${collision_finger}">
+                        <collision>
+                            <origin rpy="0 0 0" xyz="0 0 0"/>
+                            <geometry>
+                                <mesh filename="${resources_prefix}${resources_directory}/resources/panda/meshes/collision/finger.obj"/>
+                            </geometry>
+                            <material name="">
+                                <contact name="steel"/>
+                            </material>
+                        </collision>
+                    </xacro:if>
+ -->
                     <xacro:if value="${collision_finger}">
                         <collision>
@@ -547,4 +559,15 @@
                         </material>
                     </visual>
+                    <!-- <xacro:if value="${collision_finger}">
+                        <collision>
+                            <origin rpy="0 0 3.14159265359" xyz="0 0 0"/>
+                            <geometry>
+                                <mesh filename="${resources_prefix}${resources_directory}/resources/panda/meshes/collision/finger.obj"/>
+                            </geometry>
+                            <material name="">
+                                <contact name="steel"/>
+                            </material>
+                        </collision>
+                    </xacro:if> -->
                     <xacro:if value="${collision_finger}">
                         <collision>
