Commit message: mppi_manipulation working and nice tuning

File: mppi_examples/mppi_manipulation/data/objects/door.urdf.xacro (robot description, xacro)
@@ -82,4 +82,7 @@
                 <cylinder radius="0.005" length="0.10"/>
             </geometry>
+            <material name="">
+                <contact name="steel"/>
+            </material>
         </collision>
     </link>

File: mppi_examples/mppi_manipulation/data/objects/microwave.urdf.xacro (robot description, xacro)
@@ -82,4 +82,7 @@
                 <cylinder radius="0.005" length="0.10"/>
             </geometry>
+            <material name="">
+                <contact name="steel"/>
+            </material>
         </collision>
     </link>

File: mppi_examples/mppi_manipulation/data/planar_base.urdf.xacro (robot description, xacro)
@@ -18,5 +18,5 @@
             <inertial>
                 <origin rpy="0 0 0" xyz="0.0 0.0 0.0"/>
-                <mass value="0.01"/>
+                <mass value="5.0"/>
                 <inertia ixx="0.01" ixy="0.0" ixz="0.0" iyy="0.01" iyz="0.0" izz="0.01"/>
             </inertial>
@@ -25,5 +25,5 @@
             <inertial>
                 <origin rpy="0 0 0" xyz="0.0 0.0 0.0"/>
-                <mass value="0.01"/>
+                <mass value="5.0"/>
                 <inertia ixx="0.01" ixy="0.0" ixz="0.0" iyy="0.01" iyz="0.0" izz="0.01"/>
             </inertial>
@@ -33,5 +33,5 @@
                 <origin rpy="0 0 0" xyz="0.0 0.0 0.0"/>
                 <mass value="0.01"/>
-                <inertia ixx="0.01" ixy="0.0" ixz="0.0" iyy="0.01" iyz="0.0" izz="0.01"/>
+                <inertia ixx="5.0" ixy="0.0" ixz="0.0" iyy="0.01" iyz="0.0" izz="0.01"/>
             </inertial>
         </link>
@@ -42,5 +42,5 @@
             <axis xyz="1 0 0"/>
             <limit effort="1000.0" lower="-10" upper="10" velocity="1.0"/>
-            <dynamics damping="0.0" friction="10"/>
+            <dynamics damping="1.0" friction="0.0"/>
         </joint>
         <xacro:add_transmission joint_name="x_base_joint"/>
@@ -51,5 +51,5 @@
             <axis xyz="0 1 0"/>
             <limit effort="1000.0" lower="-10" upper="10" velocity="1.0"/>
-            <dynamics damping="0.0" friction="10"/>
+            <dynamics damping="1.0" friction="0.0"/>
         </joint>
         <xacro:add_transmission joint_name="y_base_joint"/>
@@ -60,5 +60,5 @@
             <axis xyz="0 0 1"/>
             <limit effort="1000.0" velocity="1.0" upper="10.0" lower="-10.0"/>
-            <dynamics damping="0.0" friction="10"/>
+            <dynamics damping="1.0" friction="0.0"/>
         </joint>
         <xacro:add_transmission joint_name="pivot_joint"/>
