Commit message: fix urdf

File: mppi_examples/mppi_manipulation/data/objects/new_shelf.urdf.xacro (robot description, xacro)
@@ -1,6 +1,8 @@
 <?xml version="1.0" ?>
-<robot name="shelf_new" xmlns:xacro="http://www.ros.org/wiki/xacro">
+<robot name="shelf" xmlns:xacro="http://www.ros.org/wiki/xacro">
     <xacro:arg name="fixed" default="true"/>
     <xacro:arg name="height" default="0.0"/>
+    <xacro:arg name="prefix" default=""/>
+    <xacro:property name="prefix" default="$(arg prefix)"/>
     <xacro:property name="height" default="$(arg height)"/>
     <xacro:property name="door_length" default="0.359"/>
@@ -20,5 +22,5 @@
     <xacro:macro name="box_inertia" params="m x y z">
         <inertial>
-            <origin rpy="0 0 0" xyz="0 0 0"/>
+            <origin rpy="0 0 0" xyz="0 ${-y/2} 0"/>
             <mass value="${m}"/>
             <inertia ixx="${0.0833 * m * (y**2 + z**2)}"
@@ -27,5 +29,5 @@
                      iyy="${0.0833 * m * (x**2 + z**2)}"
                      iyz="0"
-                     izz="${0.0833 * m * (z**2 + y**2)}"/>
+                     izz="${0.0833 * m * (x**2 + y**2)}"/>
         </inertial>
     </xacro:macro>
@@ -34,15 +36,9 @@
         <joint name="fixed" type="fixed">
             <parent link="world"/>
-            <child link="shelf"/>
-            <origin xyz="${shelf_x} ${shelf_y} ${shelf_z}" rpy="0.009 0.001 1.645"/>
+            <child link="${prefix}shelf"/>
+            <origin xyz="${shelf_x} ${shelf_y} ${shelf_z}" rpy="0.0 0.0 1.645"/>
         </joint>
     </xacro:if>
-    <gazebo>
-        <plugin name="gazebo_ros_control" filename="libgazebo_ros_control.so">
-            <robotNamespace>/shelf</robotNamespace>
-            <robotParam>urdf_object </robotParam>
-        </plugin>
-    </gazebo>
-    <link name="shelf">
+    <link name="${prefix}shelf">
         <xacro:box_inertia m="5" x="${corpus_width}" y="${corpus_length}" z="${shelf_z}"/>
         <visual>
@@ -56,6 +52,6 @@
         </visual>
     </link>
-    <link name="door">
-        <xacro:box_inertia m="5.8" x="${door_width}" y="${door_length}" z="${door_height}"/>
+    <link name="${prefix}door">
+        <xacro:box_inertia m="3.0" x="${door_width}" y="${door_length}" z="${door_height}"/>
         <visual>
             <origin rpy="0 0 0" xyz="${-door_width/2} ${door_length/2} 0"/>
@@ -77,5 +73,5 @@
         </collision>
     </link>
-    <link name="door_hinge">
+    <link name="${prefix}door_hinge">
         <inertial>
             <mass value="0.01"/>
@@ -84,35 +80,35 @@
         </inertial>
     </link>
-    <joint name="door_hinge_joint" type="fixed">
-        <parent link="shelf"/>
-        <child link="door_hinge"/>
+    <joint name="${prefix}door_hinge_joint" type="fixed">
+        <parent link="${prefix}shelf"/>
+        <child link="${prefix}door_hinge"/>
         <origin xyz="${door_width/2+0.012} -${door_length + corpus_width +corpus_door_gap} ${door_height/2}"/>
     </joint>
-    <link name="axis_link">
-        <inertial>
-            <mass value="0.01"/>
-            <origin rpy="0 0 0" xyz="0 0 0"/>
-            <inertia ixx="0.0" ixy="0.0" ixz="0.0" iyy="0.0" iyz="0.0" izz="0.0"/>
-        </inertial>
-    </link>
-    <joint name="axis_joint" type="fixed">
-        <parent link="door_hinge"/>
-        <child link="axis_link"/>
+    <link name="${prefix}axis_link">
+        <inertial>
+            <mass value="0.01"/>
+            <origin rpy="0 0 0" xyz="0 0 0"/>
+            <inertia ixx="0.0" ixy="0.0" ixz="0.0" iyy="0.0" iyz="0.0" izz="0.0"/>
+        </inertial>
+    </link>
+    <joint name="${prefix}axis_joint" type="fixed">
+        <parent link="${prefix}door_hinge"/>
+        <child link="${prefix}axis_link"/>
         <origin xyz="0.0 0.0 0.0"/>
     </joint>
     <joint name="articulation_joint" type="revolute">
-        <parent link="axis_link"/>
-        <child link="measured_joint_link"/>
-        <dynamics damping="5.0" friction="10.0"/>
+        <parent link="${prefix}axis_link"/>
+        <child link="${prefix}measured_joint_link"/>
+        <dynamics damping="0.0" friction="0.0"/>
         <origin xyz="0 0 0"/>
         <axis xyz="0 0 -1"/>
-        <limit effort="100" lower="0" upper="1.57" velocity="10.0"/>
-    </joint>
-    <joint name="door_link" type="fixed">
-        <parent link="measured_joint_link"/>
-        <child link="door"/>
+        <limit effort="100" lower="0" upper="1.75" velocity="10.0"/>
+    </joint>
+    <joint name="${prefix}door_link" type="fixed">
+        <parent link="${prefix}measured_joint_link"/>
+        <child link="${prefix}door"/>
         <origin xyz="0.0 0.0 0.0"/>
     </joint>
-    <link name="handle_link">
+    <link name="${prefix}handle_link">
         <inertial>
             <origin rpy="0 0 0" xyz="0 0 0"/>
@@ -135,9 +131,9 @@
             </geometry>
             <material name="">
-                <contact name="rubber"/>
-            </material>
-        </collision>
-    </link>
-    <link name="handle_support_left">
+                <contact name="steel"/>
+            </material>
+        </collision>
+    </link>
+    <link name="${prefix}handle_support_left">
         <inertial>
             <origin rpy="0 0 0" xyz="0 0 0"/>
@@ -164,5 +160,5 @@
         </collision>
     </link>
-    <link name="handle_support_right">
+    <link name="${prefix}handle_support_right">
         <inertial>
             <origin rpy="0 0 0" xyz="0 0 0"/>
@@ -189,61 +185,51 @@
         </collision>
     </link>
-    <joint name="handle_joint" type="fixed">
-        <parent link="door"/>
-        <child link="handle_link"/>
+    <joint name="${prefix}handle_joint" type="fixed">
+        <parent link="${prefix}door"/>
+        <child link="${prefix}handle_link"/>
         <origin xyz="${handle_height + 0.012} ${handle_offset_y} ${handle_offset_z}"
                 rpy="0 0 0"/> <!-- height handle + half the width door, 0.30 minus some offset -->
     </joint>
-    <joint name="handle_ref" type="fixed">
-        <parent link="handle_link"/>
-        <child link="handle_ref"/>
-        <origin xyz="${-handle_height/2} 0 0"
+    <joint name="${prefix}handle_ref" type="fixed">
+        <parent link="${prefix}handle_link"/>
+        <child link="${prefix}handle_ref"/>
+        <origin xyz="${-handle_height/2-0.012} 0 0"
                 rpy="0 0 0"/> <!-- height handle + half the width door, 0.30 minus some offset -->
     </joint>
-    <link name="handle_ref">
-        <inertial>
-            <mass value="0.01"/>
-            <origin rpy="0 0 0" xyz="0 0 0"/>
-            <inertia ixx="0.0" ixy="0.0" ixz="0.0" iyy="0.0" iyz="0.0" izz="0.0"/>
-        </inertial>
-    </link>
-    <joint name="handle_support_left_joint" type="fixed">
-        <parent link="handle_link"/>
-        <child link="handle_support_left"/>
+    <link name="${prefix}handle_ref">
+        <inertial>
+            <mass value="0.01"/>
+            <origin rpy="0 0 0" xyz="0 0 0"/>
+            <inertia ixx="0.0" ixy="0.0" ixz="0.0" iyy="0.0" iyz="0.0" izz="0.0"/>
+        </inertial>
+    </link>
+    <joint name="${prefix}handle_support_left_joint" type="fixed">
+        <parent link="${prefix}handle_link"/>
+        <child link="${prefix}handle_support_left"/>
         <origin xyz="-${handle_height/2} 0 -${handle_length/2}" rpy="0 0 0"/>
     </joint>
-    <joint name="handle_support_right_joint" type="fixed">
-        <parent link="handle_link"/>
-        <child link="handle_support_right"/>
+    <joint name="${prefix}handle_support_right_joint" type="fixed">
+        <parent link="${prefix}handle_link"/>
+        <child link="${prefix}handle_support_right"/>
         <origin xyz="-${handle_height/2} 0 ${handle_length/2}" rpy="0 0 0"/>
     </joint>
-    <link name="measured_joint_link">
-        <inertial>
-            <mass value="0.01"/>
-            <origin rpy="0 0 0" xyz="0 0 0"/>
-            <inertia ixx="0.0" ixy="0.0" ixz="0.0" iyy="0.0" iyz="0.0" izz="0.0"/>
-        </inertial>
-    </link>
-    <link name="measured_joint_link_test">
-        <inertial>
-            <mass value="0.01"/>
-            <origin rpy="0 0 0" xyz="0 0 0"/>
-            <inertia ixx="0.0" ixy="0.0" ixz="0.0" iyy="0.0" iyz="0.0" izz="0.0"/>
-        </inertial>
-    </link>
-    <joint name="measured_test_handle_joint" type="fixed">
-        <parent link="handle_link"/>
-        <child link="measured_joint_link_test"/>
+    <link name="${prefix}measured_joint_link">
+        <inertial>
+            <mass value="0.01"/>
+            <origin rpy="0 0 0" xyz="0 0 0"/>
+            <inertia ixx="0.0" ixy="0.0" ixz="0.0" iyy="0.0" iyz="0.0" izz="0.0"/>
+        </inertial>
+    </link>
+    <link name="${prefix}measured_joint_link_test">
+        <inertial>
+            <mass value="0.01"/>
+            <origin rpy="0 0 0" xyz="0 0 0"/>
+            <inertia ixx="0.0" ixy="0.0" ixz="0.0" iyy="0.0" iyz="0.0" izz="0.0"/>
+        </inertial>
+    </link>
+    <joint name="${prefix}measured_test_handle_joint" type="fixed">
+        <parent link="${prefix}handle_link"/>
+        <child link="${prefix}measured_joint_link_test"/>
         <origin xyz="-0.06 -0.243 0.0" rpy="0 0 0"/>
     </joint>
-    <transmission name="hinge">
-        <type>transmission_interface/SimpleTransmission</type>
-        <joint name="articulation_joint">
-            <hardwareInterface>EffortJointInterface</hardwareInterface>
-        </joint>
-        <actuator name="motor1">
-            <hardwareInterface>EffortJointInterface</hardwareInterface>
-            <mechanicalReduction>1</mechanicalReduction>
-        </actuator>
-    </transmission>
 </robot>

Commit message: urdf tuning

File: mppi_examples/mppi_manipulation/data/objects/new_shelf.urdf.xacro (robot description, xacro)
@@ -2,9 +2,7 @@
 <robot name="shelf" xmlns:xacro="http://www.ros.org/wiki/xacro">
     <xacro:arg name="fixed" default="true"/>
-    <xacro:arg name="height" default="0.0"/>
     <xacro:arg name="prefix" default=""/>
     <xacro:property name="prefix" default="$(arg prefix)"/>
-    <xacro:property name="height" default="$(arg height)"/>
-    <xacro:property name="door_length" default="0.359"/>
+    <xacro:property name="door_length" default="0.363"/>
     <xacro:property name="door_height" default="0.748"/>
     <xacro:property name="door_width" default="0.018"/>
@@ -12,12 +10,12 @@
     <xacro:property name="corpus_length" default="0.4"/>
     <xacro:property name="corpus_height" default="0.827"/>
-    <xacro:property name="corpus_width" default="0.018"/>
-    <xacro:property name="handle_height" default="0.057"/> <!-- 0.026 -->
+    <xacro:property name="corpus_width" default="0.016"/>
+    <xacro:property name="handle_height" default="0.056"/>
     <xacro:property name="handle_length" default="0.16"/>
-    <xacro:property name="handle_offset_y" default="0.338"/>
+    <xacro:property name="handle_offset_y" default="0.335"/> <!-- 0.338 -->
     <xacro:property name="handle_offset_z" default="-0.024"/>
-    <xacro:property name="shelf_x" default="-0.242"/>
-    <xacro:property name="shelf_y" default="-0.595"/>
-    <xacro:property name="shelf_z" default="0.834"/>
+    <xacro:property name="shelf_x" default="0.268466"/>
+    <xacro:property name="shelf_y" default="-0.407"/>
+    <xacro:property name="shelf_z" default="0.8299"/>
     <xacro:macro name="box_inertia" params="m x y z">
         <inertial>
@@ -37,5 +35,5 @@
             <parent link="world"/>
             <child link="${prefix}shelf"/>
-            <origin xyz="${shelf_x} ${shelf_y} ${shelf_z}" rpy="0.0 0.0 1.645"/>
+            <origin xyz="-0.366084 -0.0270533   0.833161" rpy="3.1396  3.13991 -1.57152"/>
         </joint>
     </xacro:if>
@@ -83,5 +81,5 @@
         <parent link="${prefix}shelf"/>
         <child link="${prefix}door_hinge"/>
-        <origin xyz="${door_width/2+0.012} -${door_length + corpus_width +corpus_door_gap} ${door_height/2}"/>
+        <origin xyz="${door_width/2} -${door_length + corpus_width +corpus_door_gap} ${door_height/2}"/>
     </joint>
     <link name="${prefix}axis_link">
@@ -188,20 +186,7 @@
         <parent link="${prefix}door"/>
         <child link="${prefix}handle_link"/>
-        <origin xyz="${handle_height + 0.012} ${handle_offset_y} ${handle_offset_z}"
+        <origin xyz="${handle_height} ${handle_offset_y} ${handle_offset_z}"
                 rpy="0 0 0"/> <!-- height handle + half the width door, 0.30 minus some offset -->
     </joint>
-    <joint name="${prefix}handle_ref" type="fixed">
-        <parent link="${prefix}handle_link"/>
-        <child link="${prefix}handle_ref"/>
-        <origin xyz="${-handle_height/2-0.012} 0 0"
-                rpy="0 0 0"/> <!-- height handle + half the width door, 0.30 minus some offset -->
-    </joint>
-    <link name="${prefix}handle_ref">
-        <inertial>
-            <mass value="0.01"/>
-            <origin rpy="0 0 0" xyz="0 0 0"/>
-            <inertia ixx="0.0" ixy="0.0" ixz="0.0" iyy="0.0" iyz="0.0" izz="0.0"/>
-        </inertial>
-    </link>
     <joint name="${prefix}handle_support_left_joint" type="fixed">
         <parent link="${prefix}handle_link"/>
@@ -221,15 +206,3 @@
         </inertial>
     </link>
-    <link name="${prefix}measured_joint_link_test">
-        <inertial>
-            <mass value="0.01"/>
-            <origin rpy="0 0 0" xyz="0 0 0"/>
-            <inertia ixx="0.0" ixy="0.0" ixz="0.0" iyy="0.0" iyz="0.0" izz="0.0"/>
-        </inertial>
-    </link>
-    <joint name="${prefix}measured_test_handle_joint" type="fixed">
-        <parent link="${prefix}handle_link"/>
-        <child link="${prefix}measured_joint_link_test"/>
-        <origin xyz="-0.06 -0.243 0.0" rpy="0 0 0"/>
-    </joint>
 </robot>

File: mppi_examples/mppi_manipulation/data/panda_mobile.urdf.xacro (robot description, xacro)
@@ -29,5 +29,5 @@
         <child link="franka_mount_link"/>
         <!--        <origin xyz="$(optenv RIDGEBACK_FRANKA_XYZ 0.21 0.0 0.2)" rpy="$(optenv RIDGEBACK_FRANKA_RPY 0 0 0)"/>-->
-        <origin xyz="0.295 0.005 0.445" rpy="0 0 0"/>
+        <origin xyz="0.282 0.005 0.442" rpy="0 0 0"/>
     </joint>
     <link name="franka_mount_link"/>

File: mppi_examples/mppi_manipulation/data/ridgeback.urdf.xacro (robot description, xacro)
@@ -5,9 +5,9 @@
         <!-- Sensor mount -->
         <link name="ridgeback_sensor_mount_link">
-<!--             <visual>
+            <visual>
                 <geometry>
                     <mesh filename="package://mppi_manipulation/data/meshes/ridgeback_sensor_mount.dae"/>
                 </geometry>
-            </visual> -->
+            </visual>
         </link>
         <joint name="ridgeback_sensor_mount_joint" type="fixed">
@@ -18,6 +18,6 @@
         <link name="reference_link"/>
         <joint name="reference_link_joint" type="fixed">
-            <origin xyz="-0.343 0 0.77" rpy="0 0 0"/>
-            <parent link="mid_mount"/>
+            <origin xyz="-0.01 0.0 0.018" rpy="0 0 0"/>
+            <parent link="franka_mount_link"/>
             <child link="reference_link"/>
         </joint>

File: mppi_examples/mppi_manipulation/data/ridgeback.xacro (robot description, xacro)
@@ -9,5 +9,5 @@
     <xacro:property name="chassis_width" value="0.793" />
     <xacro:property name="chassis_height" value="0.216" />
-    <xacro:property name="deck_height" value="0.280" />
+    <xacro:property name="deck_height" value="0.292" />
     <xacro:property name="axle_offset" value="0.0500" />
     <xacro:property name="dummy_inertia" value="1e-09"/>

Commit message: more urdf calibration

File: mppi_examples/mppi_manipulation/data/objects/new_shelf.urdf.xacro (robot description, xacro)
@@ -35,5 +35,5 @@
             <parent link="world"/>
             <child link="${prefix}shelf"/>
-            <origin xyz="-0.366084 -0.0270533   0.833161" rpy="3.1396  3.13991 -1.57152"/>
+            <origin xyz="-1.02326 0.270515  0.83613" rpy="3.14127   3.141 -1.5944"/>
         </joint>
     </xacro:if>

Commit message: debugging changes

File: mppi_examples/mppi_manipulation/data/objects/new_shelf.urdf.xacro (robot description, xacro)
@@ -35,5 +35,5 @@
             <parent link="world"/>
             <child link="${prefix}shelf"/>
-            <origin xyz="-1.02326 0.270515  0.83613" rpy="3.14127   3.141 -1.5944"/>
+            <origin xyz="1.95786 0.0978068  0.823227" rpy="0.00415786 0.00520789   -3.09487"/>
         </joint>
     </xacro:if>

Commit message: working on the robot

File: mppi_examples/mppi_manipulation/data/objects/new_shelf.urdf.xacro (robot description, xacro)
@@ -35,5 +35,5 @@
             <parent link="world"/>
             <child link="${prefix}shelf"/>
-            <origin xyz="1.95786 0.0978068  0.823227" rpy="0.00415786 0.00520789   -3.09487"/>
+            <origin xyz="100 100 0" rpy="0.00415786 0.00520789   -3.09487"/>
         </joint>
     </xacro:if>

Commit message: pose deadband

File: mppi_examples/mppi_manipulation/data/objects/new_shelf.urdf.xacro (robot description, xacro)
@@ -35,5 +35,5 @@
             <parent link="world"/>
             <child link="${prefix}shelf"/>
-            <origin xyz="100 100 0" rpy="0.00415786 0.00520789   -3.09487"/>
+            <origin xyz="-0.0184082  -0.00688391  0.831371" rpy="3.13934 -3.14112 -1.60109"/>
         </joint>
     </xacro:if>

Commit message: tuning and swapping finger

File: mppi_examples/mppi_manipulation/data/objects/new_shelf.urdf.xacro (robot description, xacro)
@@ -98,6 +98,6 @@
         <parent link="${prefix}axis_link"/>
         <child link="${prefix}measured_joint_link"/>
-        <dynamics damping="0.0" friction="0.0"/>
         <origin xyz="0 0 0"/>
+        <dynamics damping="2.0" friction="4.0"/>
         <axis xyz="0 0 -1"/>
         <limit effort="100" lower="0" upper="1.75" velocity="10.0"/>

Commit message: changes from tests

File: mppi_examples/mppi_manipulation/data/objects/new_shelf.urdf.xacro (robot description, xacro)
@@ -35,5 +35,5 @@
             <parent link="world"/>
             <child link="${prefix}shelf"/>
-            <origin xyz="-0.0184082  -0.00688391  0.831371" rpy="3.13934 -3.14112 -1.60109"/>
+            <origin xyz="-0.0133671 -0.01902 0.831604" rpy=" 3.14067 -3.14135 -1.59462"/>
         </joint>
     </xacro:if>

Commit message: tests from friday

File: mppi_examples/mppi_manipulation/data/objects/new_shelf.urdf.xacro (robot description, xacro)
@@ -34,6 +34,6 @@
         <joint name="fixed" type="fixed">
             <parent link="world"/>
-            <child link="${prefix}shelf"/>
-            <origin xyz="-0.0133671 -0.01902 0.831604" rpy=" 3.14067 -3.14135 -1.59462"/>
+            <child link="${prefix}shelf"/> 0
+            <origin xyz=".272902 -0.0944762   0.830376" rpy="0.000710616 0.000859919  1.51977"/>
         </joint>
     </xacro:if>

Commit message: playing with zbf and sampling

File: mppi_examples/mppi_manipulation/data/objects/new_shelf.urdf.xacro (robot description, xacro)
@@ -35,5 +35,5 @@
             <parent link="world"/>
             <child link="${prefix}shelf"/> 0
-            <origin xyz=".272902 -0.0944762   0.830376" rpy="0.000710616 0.000859919  1.51977"/>
+            <origin xyz="100.272902 -0.0944762   0.830376" rpy="0.000710616 0.000859919  1.51977"/>
         </joint>
     </xacro:if>

File: mppi_examples/mppi_manipulation/data/panda_mobile.urdf.xacro (robot description, xacro)
@@ -7,4 +7,26 @@
     <!--    Root world link-->
     <link name="world"/>
+    <!-- Obstacle link -->
+    <link name="obstacle_link">
+        <inertial>
+                <origin rpy="0 0 0" xyz="0.0 0.0 0.0"/>
+                <mass value="0.01"/>
+                <inertia ixx="0.01" ixy="0.0" ixz="0.0" iyy="0.01" iyz="0.0" izz="0.01"/>
+            </inertial>
+        <visual>
+            <origin xyz="0 0 0" rpy="0 0 0" />
+            <geometry>
+               <sphere radius="0.5"/>
+            </geometry>
+            <material name="Cyan">
+               <color rgba="0 1.0 1.0 0.3"/>
+            </material>
+        </visual>
+    </link>
+    <joint name="obstacle_joint" type="fixed">
+      <parent link="omni_base_root_link"/>
+      <child link="obstacle_link"/>
+      <origin xyz="0.0 0.0 1.0" rpy="0 0 0"/>
+    </joint>
     <!--    Omnidirectional base-->
     <xacro:unless value="$(arg fixed_base)">

Commit message: experiments 26_10_21

File: mppi_examples/mppi_manipulation/data/objects/new_shelf.urdf.xacro (robot description, xacro)
@@ -34,6 +34,6 @@
         <joint name="fixed" type="fixed">
             <parent link="world"/>
-            <child link="${prefix}shelf"/> 0
-            <origin xyz=".272902 -0.0944762   0.830376" rpy="0.000710616 0.000859919  1.51977"/>
+            <child link="${prefix}shelf"/>
+            <origin xyz="0.0104058 -0.0257724   0.831197" rpy="3.14083  3.14073 -1.60941"/>
         </joint>
     </xacro:if>

File: mppi_examples/mppi_manipulation/data/panda_mobile.urdf.xacro (robot description, xacro)
@@ -29,5 +29,5 @@
         <child link="franka_mount_link"/>
         <!--        <origin xyz="$(optenv RIDGEBACK_FRANKA_XYZ 0.21 0.0 0.2)" rpy="$(optenv RIDGEBACK_FRANKA_RPY 0 0 0)"/>-->
-        <origin xyz="0.282 0.005 0.442" rpy="0 0 0"/>
+        <origin xyz="0.282 0.005 0.447" rpy="0 0 0"/>
     </joint>
     <link name="franka_mount_link"/>
@@ -43,3 +43,10 @@
         </joint>
     </xacro:if>
+    <!-- The position of the frame published by Vicon -->
+    <link name="reference_link"/>
+    <joint name="reference_link_joint" type="fixed">
+        <origin xyz="-0.015 0.0 0.01" rpy="0 0 0"/>
+        <parent link="franka_mount_link"/>
+        <child link="reference_link"/>
+    </joint>
 </robot>

File: mppi_examples/mppi_manipulation/data/ridgeback.urdf.xacro (robot description, xacro)
@@ -16,10 +16,4 @@
             <child link="ridgeback_sensor_mount_link"/>
         </joint>
-        <link name="reference_link"/>
-        <joint name="reference_link_joint" type="fixed">
-            <origin xyz="-0.01 0.0 0.018" rpy="0 0 0"/>
-            <parent link="franka_mount_link"/>
-            <child link="reference_link"/>
-        </joint>
     </xacro:macro>
 </robot>

File: mppi_examples/mppi_manipulation/data/ridgeback.xacro (robot description, xacro)
@@ -9,5 +9,5 @@
     <xacro:property name="chassis_width" value="0.793" />
     <xacro:property name="chassis_height" value="0.216" />
-    <xacro:property name="deck_height" value="0.292" />
+    <xacro:property name="deck_height" value="0.293" />
     <xacro:property name="axle_offset" value="0.0500" />
     <xacro:property name="dummy_inertia" value="1e-09"/>
