Commit message: bunch of stuff for obstacle avoidance experiment in simulation

File: mppi_examples/mppi_manipulation/data/objects/new_shelf.urdf.xacro (robot description, xacro)
@@ -34,11 +34,6 @@
         <joint name="fixed" type="fixed">
             <parent link="world"/>
-<<<<<<< HEAD
             <child link="${prefix}shelf"/> 0
             <origin xyz="100.272902 -0.0944762   0.830376" rpy="0.000710616 0.000859919  1.51977"/>
-=======
-            <child link="${prefix}shelf"/>
-            <origin xyz="0.0104058 -0.0257724   0.831197" rpy="3.14083  3.14073 -1.60941"/>
->>>>>>> robot_experiments
         </joint>
     </xacro:if>

File: mppi_examples/mppi_manipulation/data/panda_mobile.urdf.xacro (robot description, xacro)
@@ -17,8 +17,8 @@
             <origin xyz="0 0 0" rpy="0 0 0" />
             <geometry>
-               <sphere radius="0.5"/>
+               <sphere radius="0.4"/>
             </geometry>
             <material name="Cyan">
-               <color rgba="0 1.0 1.0 0.3"/>
+               <color rgba="0 1.0 1.0 0.1"/>
             </material>
         </visual>
@@ -27,5 +27,38 @@
       <parent link="omni_base_root_link"/>
       <child link="obstacle_link"/>
-      <origin xyz="0.0 0.0 1.0" rpy="0 0 0"/>
+      <origin xyz="0.0 0.0 1.2" rpy="0 0 0"/>
+    </joint>
+    <!-- Base limits link -->
+    <link name="base_limit_left">
+        <visual>
+            <origin xyz="0 ${0.4 + 0.5/2 + 0.35} 0" rpy="0 0 0" /> <!-- width_robot/2 + wight_box_marker/2 + clearance -->
+            <geometry>
+               <box size="20 0.5 0.2"/>
+            </geometry>
+            <material name="Red">
+               <color rgba="1.0 0.0 0.0 0.5"/>
+            </material>
+        </visual>
+    </link>
+    <joint name="base_limit_left_joint" type="fixed">
+      <parent link="omni_base_root_link"/>
+      <child link="base_limit_left"/>
+      <origin xyz="0.0 0.0 0.0" rpy="0 0 0"/>
+    </joint>
+    <link name="base_limit_right">
+        <visual>
+            <origin xyz="0 -${0.4 + 0.5/2 + 0.35} 0" rpy="0 0 0" /> <!-- width_robot/2 + wight_box_marker/2 + clearance -->
+            <geometry>
+               <box size="20 0.5 0.2"/>
+            </geometry>
+            <material name="Red">
+               <color rgba="1.0 0.0 0.0 0.5"/>
+            </material>
+        </visual>
+    </link>
+    <joint name="base_limit_right_joint" type="fixed">
+      <parent link="omni_base_root_link"/>
+      <child link="base_limit_right"/>
+      <origin xyz="0.0 0.0 0.0" rpy="0 0 0"/>
     </joint>
     <!--    Omnidirectional base-->

File: mppi_examples/mppi_manipulation/data/ridgeback.urdf.xacro (robot description, xacro)
@@ -5,9 +5,9 @@
         <!-- Sensor mount -->
         <link name="ridgeback_sensor_mount_link">
-            <visual>
+<!--             <visual>
                 <geometry>
                     <mesh filename="package://mppi_manipulation/data/meshes/ridgeback_sensor_mount.dae"/>
                 </geometry>
-            </visual>
+            </visual> -->
         </link>
         <joint name="ridgeback_sensor_mount_joint" type="fixed">
