Commit message: Restructuring, optimizations.

File: mppi_examples/mppi_manipulation/data/objects/valve_gazebo.urdf.xacro (robot description, xacro)
@@ -3,6 +3,6 @@
     <xacro:arg name="resource_prefix" default=""/>
     <xacro:arg name="resource_directory" default="$(find mppi_manipulation)/data/meshes"/>
-    <xacro:arg name="height" default="0.0"/>
-    <xacro:property name="height" default="$(arg height)"/>
+    <xacro:property name="base_position_x" default="1.0"/>
+    <xacro:property name="base_position_y" default="0.0"/>
     <xacro:property name="base_length" default="0.2"/>
     <xacro:property name="base_height" default="0.5"/>
@@ -20,15 +20,9 @@
         </inertial>
     </xacro:macro>
-    <gazebo>
-        <plugin name="gazebo_ros_control" filename="libgazebo_ros_control.so">
-            <robotNamespace>/valve</robotNamespace>
-            <robotParam>urdf_object </robotParam>
-        </plugin>
-    </gazebo>
     <link name="world"/>
     <joint name="fixed" type="fixed">
         <parent link="world"/>
         <child link="valve_base"/>
-        <origin xyz="1.0 0.0 ${base_height/2.0}" rpy="0.0 0 0"/>
+        <origin xyz="${base_position_x} ${base_position_y} ${base_height/2.0}" rpy="0.0 0 0"/>
     </joint>
     <link name="valve_base">
@@ -43,13 +37,10 @@
             </material>
         </visual>
-        <!-- <collision>
+        <collision>
             <origin rpy="0 0 0" xyz="0 0 0"/>
             <geometry>
-                <box size="${base_width} ${base_length} ${base_height}"/>
+                <box size="${base_width} ${base_length} ${base_height-0.1}"/>
             </geometry>
-            <material name="">
-                <contact name="rubber"/>
-            </material>
-        </collision> -->
+        </collision>
     </link>
     <link name="handle_link">
@@ -78,6 +69,12 @@
         <dynamics damping="0.0" friction="0.0"/>
         <axis xyz="0 1 0"/>
-        <limit upper="3.14" lower="-3.14" effort="100" velocity="1.0"/>
+        <limit upper="300.14" lower="-300.14" effort="100" velocity="1.0"/>
     </joint>
+    <gazebo>
+        <plugin name="gazebo_ros_control" filename="libgazebo_ros_control.so">
+            <robotNamespace>/valve</robotNamespace>
+            <robotParam>urdf_object </robotParam>
+        </plugin>
+    </gazebo>
     <transmission name="hinge">
         <type>transmission_interface/SimpleTransmission</type>

File: mppi_examples/mppi_manipulation/data/objects/valve_rviz.urdf.xacro (robot description, xacro)
@@ -8,7 +8,16 @@
     <xacro:property name="base_height" default="0.5"/>
     <xacro:property name="base_width" default="0.2"/>
-    <!--
-    <xacro:arg name="height" default="0.0"/>
-    <xacro:property name="height" default="$(arg height)"/> -->
+    <xacro:macro name="box_inertia" params="m x y z">
+        <inertial>
+            <origin rpy="0 0 0" xyz="0 0 0"/>
+            <mass value="${m}"/>
+            <inertia ixx="${0.0833 * m * (y**2 + z**2)}"
+                     ixy="0"
+                     ixz="0"
+                     iyy="${0.0833 * m * (x**2 + z**2)}"
+                     iyz="0"
+                     izz="${0.0833 * m * (x**2 + y**2)}"/>
+        </inertial>
+    </xacro:macro>
     <link name="world"/>
     <joint name="fixed" type="fixed">
@@ -18,4 +27,20 @@
     </joint>
     <link name="valve_base">
+        <xacro:box_inertia m="100" x="${base_width}" y="${base_length}" z="${base_height}"/>
+        <visual>
+            <origin rpy="0 0 0" xyz="0 0 0"/>
+            <geometry>
+                <box size="${base_width} ${base_length} ${base_height}"/>
+            </geometry>
+            <material name="base_material">
+                <color rgba="1.0 1.0 1.0 1"/>
+            </material>
+        </visual>
+        <collision>
+            <origin rpy="0 0 0" xyz="0 0 0"/>
+            <geometry>
+                <box size="${base_width} ${base_length} ${base_height-0.1}"/>
+            </geometry>
+        </collision>
     </link>
     <link name="handle_link">
@@ -28,11 +53,11 @@
             <origin rpy="0 0 0" xyz="0 0 0"/>
             <geometry>
-                <mesh filename="$(arg resource_prefix)$(arg resource_directory)/valve_visual.obj"/>
+                <mesh filename="file://$(arg resource_directory)/valve_visual.obj"/>
             </geometry>
         </visual>
         <collision>
             <origin rpy="0 0 0" xyz="0 0 0"/>
-	    <geometry>
-                <mesh  filename="$(arg resource_prefix)$(arg resource_directory)/valve_collision.obj"/>
+        <geometry>
+                <mesh  filename="file://$(arg resource_directory)/valve_collision.obj"/>
             </geometry>
         </collision>

Commit message: Updates to valve description.

File: mppi_examples/mppi_manipulation/data/objects/valve_gazebo.urdf.xacro (robot description, xacro)
@@ -69,5 +69,5 @@
         <origin xyz="0 0 ${base_height/2.0+0.2}" rpy="0 0 0"/> <!-- 1.5708 0 0 -->
         <dynamics damping="0.0" friction="0.002"/>
-        <axis xyz="0 1 0"/>
+        <axis xyz="0 0 1"/>
         <limit upper="300.14" lower="-300.14" effort="100" velocity="1.0"/>
     </joint>

File: mppi_examples/mppi_manipulation/data/objects/valve_rviz.urdf.xacro (robot description, xacro)
@@ -47,5 +47,5 @@
         <origin xyz="$(arg object_position)" rpy="$(arg object_rpy)"/>
         <dynamics damping="0.0" friction="0.0"/>
-        <axis xyz="0 1 0"/>
+        <axis xyz="0 0 1"/>
         <limit upper="300.14" lower="-300.14" effort="100" velocity="1.0"/>
     </joint>

Commit message: Updates to gazebo valve position/orientation.

File: mppi_examples/mppi_manipulation/data/objects/valve_gazebo.urdf.xacro (robot description, xacro)
@@ -3,4 +3,6 @@
     <xacro:arg name="resource_prefix" default=""/>
     <xacro:arg name="resource_directory" default="$(find mppi_manipulation)/data/meshes"/>
+    <xacro:arg name="object_position" default="-1 0 1"/>
+    <xacro:arg name="object_rpy" default="1.5708 0 0"/>
     <xacro:property name="base_position_x" default="1.0"/>
     <xacro:property name="base_position_y" default="0.0"/>
@@ -65,9 +67,10 @@
     </link>
     <joint name="articulation_joint" type="revolute">
-        <parent link="valve_base"/>
+        <parent link="world"/>
         <child link="handle_link"/>
-        <origin xyz="0 0 ${base_height/2.0+0.2}" rpy="0 0 0"/> <!-- 1.5708 0 0 -->
+        <!--<origin xyz="0 0 ${base_height/2.0+0.2}" rpy="1.5708 0 0"/> <!- 1.5708 0 0 -->
+        <origin xyz="$(arg object_position)" rpy="$(arg object_rpy)"/>
         <dynamics damping="0.0" friction="0.002"/>
-        <axis xyz="0 1 0"/>
+        <axis xyz="0 0 1"/>
         <limit upper="300.14" lower="-300.14" effort="100" velocity="1.0"/>
     </joint>
