Commit message: Fixed urdfs, added rviz config.

File: mppi_examples/mppi_manipulation/data/objects/valve.urdf.xacro (robot description, xacro)
@@ -21,5 +21,6 @@
             <origin rpy="0 0 0" xyz="0 0 0"/>
             <geometry>
-                <mesh filename="$(arg resource_prefix)$(arg resource_directory)/valve_visual.obj"/>
+                <!-- <mesh filename="$(arg resource_prefix)$(arg resource_directory)/valve_visual.obj"/> -->
+                <mesh filename="file://$(arg resource_directory)/valve_visual.obj"/>
             </geometry>
         </visual>
@@ -27,5 +28,6 @@
             <origin rpy="0 0 0" xyz="0 0 0"/>
 	    <geometry>
-                <mesh  filename="$(arg resource_prefix)$(arg resource_directory)/valve_collision.obj"/>
+                <!-- <mesh  filename="$(arg resource_prefix)$(arg resource_directory)/valve_collision.obj"/> -->
+                <mesh  filename="file://$(arg resource_directory)/valve_collision.obj"/>
             </geometry>
         </collision>

File: mppi_examples/mppi_omav_interaction/data/omav_pinocchio_hook.urdf.xacro (robot description, xacro)
@@ -6,8 +6,8 @@
     <xacro:property name="tool_length" value="0.05"/>         <!-- [m] -->
     <xacro:property name="tool_radius" value="0.0075"/>         <!-- [m] -->
-    <xacro:property name="mass_ouzel" value="5.0"/>
-    <xacro:property name="ixx_ouzel" value="0.12"/>
-    <xacro:property name="iyy_ouzel" value="0.14"/>
-    <xacro:property name="izz_ouzel" value="0.18"/>
+    <xacro:property name="mass_ouzel" value="4.337"/>
+    <xacro:property name="ixx_ouzel" value="0.078359"/>
+    <xacro:property name="iyy_ouzel" value="0.081797"/>
+    <xacro:property name="izz_ouzel" value="0.153355"/>
     <xacro:property name="radius_ouzel" value="0.2"/>
     <xacro:property name="height_ouzel" value="0.3"/>

Commit message: Publishing rviz markers for hook position. Added cost update for valve (set ref angle as current+0.5rad). Added common cost header file. Vectorized costs. Parameterized frames in cost computation. Renamed topics.

File: mppi_examples/mppi_manipulation/data/objects/valve.urdf.xacro (robot description, xacro)
@@ -28,11 +28,11 @@
             <origin rpy="0 0 0" xyz="0 0 0"/>
             <geometry>
-                <mesh filename="$(arg resource_prefix)$(arg resource_directory)/valve_visual.obj"/>
+                <mesh filename="$(arg resource_prefix)$(arg resource_directory)/valve_visual.obj" scale="1 1 1"/>
             </geometry>
         </visual>
         <collision>
             <origin rpy="0 0 0" xyz="0 0 0"/>
-	    <geometry>
-                <mesh  filename="$(arg resource_prefix)$(arg resource_directory)/valve_collision.obj"/>
+	       <geometry>
+                <mesh  filename="$(arg resource_prefix)$(arg resource_directory)/valve_collision.obj" scale="1 1 1"/>
             </geometry>
         </collision>
@@ -42,5 +42,5 @@
         <child link="handle_link"/>
         <origin xyz="0 0 ${base_height/2.0+0.1}" rpy="1.5708 0 0"/>
-        <dynamics damping="0.0" friction="0.0"/>
+        <dynamics damping="0.0" friction="0.002"/>
         <axis xyz="0 1 0"/>
         <limit upper="300.14" lower="-300.14" effort="100" velocity="1.0"/>

File: mppi_examples/mppi_manipulation/data/objects/valve_gazebo.urdf.xacro (robot description, xacro)
@@ -53,5 +53,5 @@
             <origin rpy="0 0 0" xyz="0 0 0"/>
             <geometry>
-                <mesh filename="$(arg resource_prefix)$(arg resource_directory)/valve_visual.obj"/>
+                <mesh filename="$(arg resource_prefix)$(arg resource_directory)/valve_visual.obj" scale="1 1 1"/>
             </geometry>
         </visual>
@@ -59,5 +59,5 @@
             <origin rpy="0 0 0" xyz="0 0 0"/>
 	    <geometry>
-                <mesh  filename="$(arg resource_prefix)$(arg resource_directory)/valve_collision.obj"/>
+                <mesh  filename="$(arg resource_prefix)$(arg resource_directory)/valve_collision.obj" scale="1 1 1"/>
             </geometry>
         </collision>
@@ -67,5 +67,5 @@
         <child link="handle_link"/>
         <origin xyz="0 0 ${base_height/2.0+0.1}" rpy="1.5708 0 0"/>
-        <dynamics damping="0.0" friction="0.0"/>
+        <dynamics damping="0.0" friction="0.002"/>
         <axis xyz="0 1 0"/>
         <limit upper="300.14" lower="-300.14" effort="100" velocity="1.0"/>

File: mppi_examples/mppi_manipulation/data/objects/valve_rviz.urdf.xacro (robot description, xacro)
@@ -53,5 +53,5 @@
             <origin rpy="0 0 0" xyz="0 0 0"/>
             <geometry>
-                <mesh filename="file://$(arg resource_directory)/valve_visual.obj"/>
+                <mesh filename="file://$(arg resource_directory)/valve_visual.obj" scale="1 1 1"/>
             </geometry>
         </visual>
@@ -59,5 +59,5 @@
             <origin rpy="0 0 0" xyz="0 0 0"/>
         <geometry>
-                <mesh  filename="file://$(arg resource_directory)/valve_collision.obj"/>
+                <mesh  filename="file://$(arg resource_directory)/valve_collision.obj" scale="1 1 1"/>
             </geometry>
         </collision>

Commit message: Added LEE version of the valve.

File: mppi_examples/mppi_manipulation/data/objects/valve.urdf.xacro (robot description, xacro)
@@ -8,4 +8,5 @@
     <xacro:property name="base_height" default="0.5"/>
     <xacro:property name="base_width" default="0.2"/>
+    <xacro:property name="valve_type" default="lee_"/>
     <!--
     <xacro:arg name="height" default="0.0"/>
@@ -28,5 +29,5 @@
             <origin rpy="0 0 0" xyz="0 0 0"/>
             <geometry>
-                <mesh filename="$(arg resource_prefix)$(arg resource_directory)/valve_visual.obj" scale="1 1 1"/>
+                <mesh filename="$(arg resource_prefix)$(arg resource_directory)/valve_${valve_type}visual.obj" scale="1 1 1"/>
             </geometry>
         </visual>
@@ -34,5 +35,5 @@
             <origin rpy="0 0 0" xyz="0 0 0"/>
 	       <geometry>
-                <mesh  filename="$(arg resource_prefix)$(arg resource_directory)/valve_collision.obj" scale="1 1 1"/>
+                <mesh  filename="$(arg resource_prefix)$(arg resource_directory)/valve_${valve_type}collision.obj" scale="1 1 1"/>
             </geometry>
         </collision>
@@ -41,5 +42,5 @@
         <parent link="valve_base"/>
         <child link="handle_link"/>
-        <origin xyz="0 0 ${base_height/2.0+0.1}" rpy="1.5708 0 0"/>
+        <origin xyz="0 0 ${base_height/2.0+0.2}" rpy="0 0 0"/> <!-- 1.5708 0 0 -->
         <dynamics damping="0.0" friction="0.002"/>
         <axis xyz="0 1 0"/>

File: mppi_examples/mppi_manipulation/data/objects/valve_gazebo.urdf.xacro (robot description, xacro)
@@ -8,4 +8,5 @@
     <xacro:property name="base_height" default="0.5"/>
     <xacro:property name="base_width" default="0.2"/>
+    <xacro:property name="valve_type" default="lee_"/>
     <xacro:macro name="box_inertia" params="m x y z">
         <inertial>
@@ -53,5 +54,5 @@
             <origin rpy="0 0 0" xyz="0 0 0"/>
             <geometry>
-                <mesh filename="$(arg resource_prefix)$(arg resource_directory)/valve_visual.obj" scale="1 1 1"/>
+                <mesh filename="$(arg resource_prefix)$(arg resource_directory)/valve_${valve_type}visual.obj" scale="1 1 1"/>
             </geometry>
         </visual>
@@ -59,5 +60,5 @@
             <origin rpy="0 0 0" xyz="0 0 0"/>
 	    <geometry>
-                <mesh  filename="$(arg resource_prefix)$(arg resource_directory)/valve_collision.obj" scale="1 1 1"/>
+                <mesh  filename="$(arg resource_prefix)$(arg resource_directory)/valve_${valve_type}collision.obj" scale="1 1 1"/>
             </geometry>
         </collision>
@@ -66,5 +67,5 @@
         <parent link="valve_base"/>
         <child link="handle_link"/>
-        <origin xyz="0 0 ${base_height/2.0+0.1}" rpy="1.5708 0 0"/>
+        <origin xyz="0 0 ${base_height/2.0+0.2}" rpy="0 0 0"/> <!-- 1.5708 0 0 -->
         <dynamics damping="0.0" friction="0.002"/>
         <axis xyz="0 1 0"/>

File: mppi_examples/mppi_manipulation/data/objects/valve_rviz.urdf.xacro (robot description, xacro)
@@ -8,4 +8,5 @@
     <xacro:property name="base_height" default="0.5"/>
     <xacro:property name="base_width" default="0.2"/>
+    <xacro:property name="valve_type" default="lee_"/>
     <xacro:macro name="box_inertia" params="m x y z">
         <inertial>
@@ -53,5 +54,5 @@
             <origin rpy="0 0 0" xyz="0 0 0"/>
             <geometry>
-                <mesh filename="file://$(arg resource_directory)/valve_visual.obj" scale="1 1 1"/>
+                <mesh filename="file://$(arg resource_directory)/valve_${valve_type}visual.obj" scale="1 1 1"/>
             </geometry>
         </visual>
@@ -59,5 +60,5 @@
             <origin rpy="0 0 0" xyz="0 0 0"/>
         <geometry>
-                <mesh  filename="file://$(arg resource_directory)/valve_collision.obj" scale="1 1 1"/>
+                <mesh  filename="file://$(arg resource_directory)/valve_${valve_type}collision.obj" scale="1 1 1"/>
             </geometry>
         </collision>
@@ -66,5 +67,5 @@
         <parent link="valve_base"/>
         <child link="handle_link"/>
-        <origin xyz="0 0 ${base_height/2.0+0.1}" rpy="1.5708 0 0"/>
+        <origin xyz="0 0 ${base_height/2.0+0.2}" rpy="0 0 0"/> <!-- 1.5708 0 0 -->
         <dynamics damping="0.0" friction="0.0"/>
         <axis xyz="0 1 0"/>

Commit message: Updates to valve obj valves (reoriented s.t. z axis is aligned with rotation axis), updates to xacro files for more consistency.

File: mppi_examples/mppi_manipulation/data/objects/valve.urdf.xacro (robot description, xacro)
@@ -3,4 +3,6 @@
     <xacro:arg name="resource_prefix" default=""/>
     <xacro:arg name="resource_directory" default="$(find mppi_manipulation)/data/meshes"/>
+    <xacro:arg name="object_position" default="-1 0 1"/>
+    <xacro:arg name="object_rpy" default="1.5708 0 0"/>
     <xacro:property name="base_position_x" default="1.0"/>
     <xacro:property name="base_position_y" default="0.0"/>
@@ -9,12 +11,10 @@
     <xacro:property name="base_width" default="0.2"/>
     <xacro:property name="valve_type" default="lee_"/>
-    <!--
-    <xacro:arg name="height" default="0.0"/>
-    <xacro:property name="height" default="$(arg height)"/> -->
     <link name="world"/>
     <joint name="fixed" type="fixed">
         <parent link="world"/>
         <child link="valve_base"/>
-        <origin xyz="${base_position_x} ${base_position_y} ${base_height/2.0}" rpy="0.0 0 0"/>
+        <!-- <origin xyz="${base_position_x} ${base_position_y} ${base_height/2.0}" rpy="0 0 0"/> -->
+        <origin xyz="0 0 0" rpy="0 0 0"/>
     </joint>
     <link name="valve_base">
@@ -42,7 +42,8 @@
         <parent link="valve_base"/>
         <child link="handle_link"/>
-        <origin xyz="0 0 ${base_height/2.0+0.2}" rpy="0 0 0"/> <!-- 1.5708 0 0 -->
+        <!--<origin xyz="0 0 ${base_height/2.0+0.2}" rpy="0 0 0"/> <!- 1.5708 0 0 -->
+        <origin xyz="$(arg object_position)" rpy="$(arg object_rpy)"/>
         <dynamics damping="0.0" friction="0.002"/>
-        <axis xyz="0 1 0"/>
+        <axis xyz="0 0 1"/>
         <limit upper="300.14" lower="-300.14" effort="100" velocity="1.0"/>
     </joint>

File: mppi_examples/mppi_manipulation/data/objects/valve_rviz.urdf.xacro (robot description, xacro)
@@ -1,6 +1,7 @@
 <?xml version="1.0" encoding="utf-8"?>
 <robot name="valve" xmlns:xacro="http://www.ros.org/wiki/xacro">
-    <xacro:arg name="resource_prefix" default=""/>
     <xacro:arg name="resource_directory" default="$(find mppi_manipulation)/data/meshes"/>
+    <xacro:arg name="object_position" default="-1 0 1"/>
+    <xacro:arg name="object_rpy" default="1.5708 0 0"/>
     <xacro:property name="base_position_x" default="1.0"/>
     <xacro:property name="base_position_y" default="0.0"/>
@@ -9,16 +10,4 @@
     <xacro:property name="base_width" default="0.2"/>
     <xacro:property name="valve_type" default="lee_"/>
-    <xacro:macro name="box_inertia" params="m x y z">
-        <inertial>
-            <origin rpy="0 0 0" xyz="0 0 0"/>
-            <mass value="${m}"/>
-            <inertia ixx="${0.0833 * m * (y**2 + z**2)}"
-                     ixy="0"
-                     ixz="0"
-                     iyy="${0.0833 * m * (x**2 + z**2)}"
-                     iyz="0"
-                     izz="${0.0833 * m * (x**2 + y**2)}"/>
-        </inertial>
-    </xacro:macro>
     <link name="world"/>
     <joint name="fixed" type="fixed">
@@ -28,5 +17,4 @@
     </joint>
     <link name="valve_base">
-        <xacro:box_inertia m="100" x="${base_width}" y="${base_length}" z="${base_height}"/>
         <visual>
             <origin rpy="0 0 0" xyz="0 0 0"/>
@@ -38,17 +26,6 @@
             </material>
         </visual>
-        <collision>
-            <origin rpy="0 0 0" xyz="0 0 0"/>
-            <geometry>
-                <box size="${base_width} ${base_length} ${base_height-0.1}"/>
-            </geometry>
-        </collision>
     </link>
     <link name="handle_link">
-        <inertial>
-            <origin rpy="0 0 0" xyz="0 0 0"/>
-            <mass value="0.1"/>
-            <inertia ixx="0.001" ixy="0" ixz="0" iyy="0.001" iyz="0" izz="0.001"/>
-        </inertial>
         <visual>
             <origin rpy="0 0 0" xyz="0 0 0"/>
@@ -65,7 +42,8 @@
     </link>
     <joint name="articulation_joint" type="revolute">
-        <parent link="valve_base"/>
+        <parent link="world"/>
         <child link="handle_link"/>
-        <origin xyz="0 0 ${base_height/2.0+0.2}" rpy="0 0 0"/> <!-- 1.5708 0 0 -->
+        <!--<origin xyz="0 0 ${base_height/2.0+0.2}" rpy="1.5708 0 0"/> <!- 1.5708 0 0 -->
+        <origin xyz="$(arg object_position)" rpy="$(arg object_rpy)"/>
         <dynamics damping="0.0" friction="0.0"/>
         <axis xyz="0 1 0"/>

Commit message: Updates during experiments.

File: mppi_examples/mppi_manipulation/data/objects/valve.urdf.xacro (robot description, xacro)
@@ -5,4 +5,5 @@
     <xacro:arg name="object_position" default="-1 0 1"/>
     <xacro:arg name="object_rpy" default="1.5708 0 0"/>
+    <xacro:arg name="host_name" default="kea"/>
     <xacro:property name="base_position_x" default="1.0"/>
     <xacro:property name="base_position_y" default="0.0"/>
@@ -26,14 +27,15 @@
             <inertia ixx="0.001" ixy="0" ixz="0" iyy="0.001" iyz="0" izz="0.001"/>
         </inertial>
-        <visual>
+        <!-- <visual>
             <origin rpy="0 0 0" xyz="0 0 0"/>
             <geometry>
                 <mesh filename="$(arg resource_prefix)$(arg resource_directory)/valve_${valve_type}visual.obj" scale="1 1 1"/>
             </geometry>
-        </visual>
+        </visual> -->
         <collision>
             <origin rpy="0 0 0" xyz="0 0 0"/>
 	       <geometry>
-                <mesh  filename="$(arg resource_prefix)$(arg resource_directory)/valve_${valve_type}collision.obj" scale="1 1 1"/>
+                <!-- <mesh  filename="$(arg resource_prefix)$(arg resource_directory)/valve_${valve_type}collision.obj" scale="1 1 1"/> -->
+                <mesh  filename="/home/$(arg host_name)/catkin_ws/src/sampling_based_control/mppi_examples/mppi_manipulation/data/meshes/valve_${valve_type}collision.obj" scale="1 1 1"/>
             </geometry>
         </collision>

File: mppi_examples/mppi_manipulation/data/objects/valve_rviz.urdf.xacro (robot description, xacro)
@@ -11,5 +11,5 @@
     <xacro:property name="valve_type" default="lee_"/>
     <link name="world"/>
-    <joint name="fixed" type="fixed">
+    <!-- <joint name="fixed" type="fixed">
         <parent link="world"/>
         <child link="valve_base"/>
@@ -26,5 +26,5 @@
             </material>
         </visual>
-    </link>
+    </link> -->
     <link name="handle_link">
         <visual>

File: mppi_examples/mppi_omav_interaction/data/omav_hook_visualization.urdf.xacro (robot description, xacro)
@@ -2,5 +2,5 @@
 <robot xmlns:xacro="http://www.ros.org/wiki/xacro" name="omav_hook_visualization">
     <!-- Properties -->
-    <xacro:property name="manipulator_length" value="0.62"/>   <!-- [m] -->
+    <xacro:property name="manipulator_length" value="0.605"/>   <!-- [m] -->
     <xacro:property name="manipulator_radius" value="0.0075"/>  <!-- [m] -->
     <xacro:property name="tool_length" value="0.05"/>         <!-- [m] -->
@@ -12,7 +12,7 @@
     <xacro:property name="radius_ouzel" value="0.2"/>
     <xacro:property name="height_ouzel" value="0.3"/>
-    <link name="odom_omav"/>
-    <joint name="odom_omav_to_omav_base" type="fixed">
-        <parent link="odom_omav"/>
+    <link name="state"/>
+    <joint name="state_to_omav_base" type="fixed">
+        <parent link="state"/>
         <child link="omav_base"/>
         <origin rpy="0 0 0" xyz="0.0 0.0 0.0"/>

File: mppi_examples/mppi_omav_interaction/data/omav_pinocchio_hook.urdf.xacro (robot description, xacro)
@@ -2,5 +2,5 @@
 <robot xmlns:xacro="http://www.ros.org/wiki/xacro" name="omav_pinocchio_hook">
     <!-- Properties -->
-    <xacro:property name="manipulator_length" value="0.62"/>   <!-- [m] -->
+    <xacro:property name="manipulator_length" value="0.605"/>   <!-- [m] -->
     <xacro:property name="manipulator_radius" value="0.0075"/>  <!-- [m] -->
     <xacro:property name="tool_length" value="0.05"/>         <!-- [m] -->

File: mppi_examples/mppi_omav_interaction/data/omav_raisim_hook.urdf.xacro (robot description, xacro)
@@ -2,5 +2,5 @@
 <robot xmlns:xacro="http://www.ros.org/wiki/xacro" name="omav_raisim_hook">
     <!-- Properties -->
-    <xacro:property name="manipulator_length" value="0.62"/>   <!-- [m] -->
+    <xacro:property name="manipulator_length" value="0.605"/>   <!-- [m] -->
     <xacro:property name="manipulator_radius" value="0.0075"/>  <!-- [m] -->
     <xacro:property name="tool_length" value="0.05"/>         <!-- [m] -->

Commit message: Parameterized hook length, reduced and paramterized debug publishing rate and observer rate.

File: mppi_examples/mppi_manipulation/data/objects/valve.urdf.xacro (robot description, xacro)
@@ -5,5 +5,5 @@
     <xacro:arg name="object_position" default="-1 0 1"/>
     <xacro:arg name="object_rpy" default="1.5708 0 0"/>
-    <xacro:arg name="host_name" default="kea"/>
+    <xacro:arg name="host_name" default="$(arg host_name)"/>
     <xacro:property name="base_position_x" default="1.0"/>
     <xacro:property name="base_position_y" default="0.0"/>

File: mppi_examples/mppi_omav_interaction/data/omav_hook_visualization.urdf.xacro (robot description, xacro)
@@ -2,12 +2,8 @@
 <robot xmlns:xacro="http://www.ros.org/wiki/xacro" name="omav_hook_visualization">
     <!-- Properties -->
-    <xacro:property name="manipulator_length" value="0.605"/>   <!-- [m] -->
+    <xacro:property name="manipulator_length" value="$(arg manipulator_length)"/>   <!-- [m] -->
     <xacro:property name="manipulator_radius" value="0.0075"/>  <!-- [m] -->
     <xacro:property name="tool_length" value="0.05"/>         <!-- [m] -->
     <xacro:property name="tool_radius" value="0.0075"/>         <!-- [m] -->
-    <xacro:property name="mass_ouzel" value="5.0"/>
-    <xacro:property name="ixx_ouzel" value="0.12"/>
-    <xacro:property name="iyy_ouzel" value="0.14"/>
-    <xacro:property name="izz_ouzel" value="0.18"/>
     <xacro:property name="radius_ouzel" value="0.2"/>
     <xacro:property name="height_ouzel" value="0.3"/>

File: mppi_examples/mppi_omav_interaction/data/omav_pinocchio_hook.urdf.xacro (robot description, xacro)
@@ -2,5 +2,5 @@
 <robot xmlns:xacro="http://www.ros.org/wiki/xacro" name="omav_pinocchio_hook">
     <!-- Properties -->
-    <xacro:property name="manipulator_length" value="0.605"/>   <!-- [m] -->
+    <xacro:property name="manipulator_length" value="$(arg manipulator_length)"/>   <!-- [m] -->
     <xacro:property name="manipulator_radius" value="0.0075"/>  <!-- [m] -->
     <xacro:property name="tool_length" value="0.05"/>         <!-- [m] -->
@@ -35,5 +35,5 @@
             </geometry>
         </collision>
-        <visual>
+        <!-- <visual>
             <origin rpy="0 0 0" xyz="0 0 0"/>
             <geometry>
@@ -43,5 +43,5 @@
                 <color rgba="1 1 1 1"/>
             </material>
-        </visual>
+        </visual> -->
     </link>
     <joint name="omav_to_rod" type="fixed">
@@ -60,5 +60,5 @@
             </material>
         </collision>
-        <visual>
+        <!-- <visual>
             <origin rpy="0 1.5708 0" xyz="0 0 0"/>
             <geometry>
@@ -68,5 +68,5 @@
                 <color rgba="1 1 1 1"/>
             </material>
-        </visual>
+        </visual> -->
     </link>
     <joint name="rod_to_tip" type="fixed">
@@ -85,5 +85,5 @@
             </material>
         </collision>
-        <visual>
+        <!-- <visual>
             <origin rpy="0 0 0" xyz="0 0.0 0"/>
             <geometry>
@@ -93,5 +93,5 @@
                 <color rgba="1 1 1 1"/>
             </material>
-        </visual>
+        </visual> -->
     </link>
     <joint name="tip_to_hook" type="fixed">
@@ -110,5 +110,5 @@
             </material>
         </collision>
-        <visual>
+        <!-- <visual>
             <origin rpy="0 0 0" xyz="0 0 0"/>
             <geometry>
@@ -118,5 +118,5 @@
                 <color rgba="1 1 1 1"/>
             </material>
-        </visual>
+        </visual> -->
     </link>
 </robot>

File: mppi_examples/mppi_omav_interaction/data/omav_raisim_hook.urdf.xacro (robot description, xacro)
@@ -2,5 +2,5 @@
 <robot xmlns:xacro="http://www.ros.org/wiki/xacro" name="omav_raisim_hook">
     <!-- Properties -->
-    <xacro:property name="manipulator_length" value="0.605"/>   <!-- [m] -->
+    <xacro:property name="manipulator_length" value="$(arg manipulator_length)"/>   <!-- [m] -->
     <xacro:property name="manipulator_radius" value="0.0075"/>  <!-- [m] -->
     <xacro:property name="tool_length" value="0.05"/>         <!-- [m] -->

Commit message: Added publishing of object state and reference to optimal rollout.

File: mppi_examples/mppi_manipulation/data/objects/valve.urdf.xacro (robot description, xacro)
@@ -6,9 +6,4 @@
     <xacro:arg name="object_rpy" default="1.5708 0 0"/>
     <xacro:arg name="host_name" default="$(arg host_name)"/>
-    <xacro:property name="base_position_x" default="1.0"/>
-    <xacro:property name="base_position_y" default="0.0"/>
-    <xacro:property name="base_length" default="0.2"/>
-    <xacro:property name="base_height" default="0.5"/>
-    <xacro:property name="base_width" default="0.2"/>
     <xacro:property name="valve_type" default="lee_"/>
     <link name="world"/>
@@ -46,5 +41,5 @@
         <!--<origin xyz="0 0 ${base_height/2.0+0.2}" rpy="0 0 0"/> <!- 1.5708 0 0 -->
         <origin xyz="$(arg object_position)" rpy="$(arg object_rpy)"/>
-        <dynamics damping="0.0" friction="0.002"/>
+        <dynamics damping="0.1" friction="0.1"/>
         <axis xyz="0 0 1"/>
         <limit upper="300.14" lower="-300.14" effort="100" velocity="1.0"/>
