Commit message: Added thin valve collision model.

File: mppi_examples/mppi_manipulation/data/objects/valve.urdf.xacro (robot description, xacro)
@@ -6,5 +6,5 @@
     <xacro:arg name="object_rpy" default="1.5708 0 0"/>
     <xacro:arg name="host_name" default="$(arg host_name)"/>
-    <xacro:property name="valve_type" default="lee_"/>
+    <xacro:arg name="valve_type" default="lee_thin_"/>
     <link name="world"/>
     <joint name="fixed" type="fixed">
@@ -32,5 +32,5 @@
 	       <geometry>
                 <!-- <mesh  filename="$(arg resource_prefix)$(arg resource_directory)/valve_${valve_type}collision.obj" scale="1 1 1"/> -->
-                <mesh  filename="/home/$(arg host_name)/catkin_ws/src/sampling_based_control/mppi_examples/mppi_manipulation/data/meshes/valve_${valve_type}collision.obj" scale="1 1 1"/>
+                <mesh  filename="/home/$(arg host_name)/catkin_ws/src/sampling_based_control/mppi_examples/mppi_manipulation/data/meshes/valve_$(arg valve_type)collision.obj" scale="1 1 1"/>
             </geometry>
         </collision>

Commit message: Updated models (removed 'tip', parameterized collision-visual difference, added material 'steel' properties). Updated material property in raisim to lower bounciness and lower friction. Updated thin valve collision model.

File: mppi_examples/mppi_manipulation/data/objects/valve.urdf.xacro (robot description, xacro)
@@ -6,5 +6,5 @@
     <xacro:arg name="object_rpy" default="1.5708 0 0"/>
     <xacro:arg name="host_name" default="$(arg host_name)"/>
-    <xacro:arg name="valve_type" default="lee_thin_"/>
+    <xacro:arg name="valve_type" default="lee_thin"/>
     <link name="world"/>
     <joint name="fixed" type="fixed">
@@ -32,6 +32,9 @@
 	       <geometry>
                 <!-- <mesh  filename="$(arg resource_prefix)$(arg resource_directory)/valve_${valve_type}collision.obj" scale="1 1 1"/> -->
-                <mesh  filename="/home/$(arg host_name)/catkin_ws/src/sampling_based_control/mppi_examples/mppi_manipulation/data/meshes/valve_$(arg valve_type)collision.obj" scale="1 1 1"/>
+                <mesh  filename="/home/$(arg host_name)/catkin_ws/src/sampling_based_control/mppi_examples/mppi_manipulation/data/meshes/valve_$(arg valve_type)_collision.obj" scale="1 1 1"/>
             </geometry>
+            <material name="">
+                <contact name="steel"/>
+            </material>
         </collision>
     </link>
@@ -41,5 +44,5 @@
         <!--<origin xyz="0 0 ${base_height/2.0+0.2}" rpy="0 0 0"/> <!- 1.5708 0 0 -->
         <origin xyz="$(arg object_position)" rpy="$(arg object_rpy)"/>
-        <dynamics damping="0.1" friction="0.1"/>
+        <dynamics damping="1" friction="2"/>
         <axis xyz="0 0 1"/>
         <limit upper="300.14" lower="-300.14" effort="100" velocity="1.0"/>

File: mppi_examples/mppi_manipulation/data/objects/valve_gazebo.urdf.xacro (robot description, xacro)
@@ -5,4 +5,5 @@
     <xacro:arg name="object_position" default="-1 0 1"/>
     <xacro:arg name="object_rpy" default="1.5708 0 0"/>
+    <xacro:arg name="valve_type" default="lee"/>
     <xacro:property name="base_position_x" default="1.0"/>
     <xacro:property name="base_position_y" default="0.0"/>
@@ -10,5 +11,4 @@
     <xacro:property name="base_height" default="0.5"/>
     <xacro:property name="base_width" default="0.2"/>
-    <xacro:property name="valve_type" default="lee_"/>
     <xacro:macro name="box_inertia" params="m x y z">
         <inertial>
@@ -56,5 +56,5 @@
             <origin rpy="0 0 0" xyz="0 0 0"/>
             <geometry>
-                <mesh filename="$(arg resource_prefix)$(arg resource_directory)/valve_${valve_type}visual.obj" scale="1 1 1"/>
+                <mesh filename="$(arg resource_prefix)$(arg resource_directory)/valve_$(arg valve_type)_visual.obj" scale="1 1 1"/>
             </geometry>
         </visual>
@@ -62,5 +62,5 @@
             <origin rpy="0 0 0" xyz="0 0 0"/>
 	    <geometry>
-                <mesh  filename="$(arg resource_prefix)$(arg resource_directory)/valve_${valve_type}collision.obj" scale="1 1 1"/>
+                <mesh  filename="$(arg resource_prefix)$(arg resource_directory)/valve_$(arg valve_type)_collision.obj" scale="1 1 1"/>
             </geometry>
         </collision>
@@ -78,5 +78,5 @@
         <plugin name="gazebo_ros_control" filename="libgazebo_ros_control.so">
             <robotNamespace>/valve</robotNamespace>
-            <robotParam>urdf_object </robotParam>
+            <robotParam>urdf_gazebo</robotParam>
         </plugin>
     </gazebo>

File: mppi_examples/mppi_manipulation/data/objects/valve_rviz.urdf.xacro (robot description, xacro)
@@ -4,4 +4,5 @@
     <xacro:arg name="object_position" default="-1 0 1"/>
     <xacro:arg name="object_rpy" default="1.5708 0 0"/>
+    <xacro:arg name="valve_type" default="lee"/>
     <xacro:property name="base_position_x" default="1.0"/>
     <xacro:property name="base_position_y" default="0.0"/>
@@ -9,5 +10,4 @@
     <xacro:property name="base_height" default="0.5"/>
     <xacro:property name="base_width" default="0.2"/>
-    <xacro:property name="valve_type" default="lee_"/>
     <link name="world"/>
     <!-- <joint name="fixed" type="fixed">
@@ -31,5 +31,5 @@
             <origin rpy="0 0 0" xyz="0 0 0"/>
             <geometry>
-                <mesh filename="file://$(arg resource_directory)/valve_${valve_type}visual.obj" scale="1 1 1"/>
+                <mesh filename="file://$(arg resource_directory)/valve_$(arg valve_type)_visual.obj" scale="1 1 1"/>
             </geometry>
         </visual>
@@ -37,5 +37,5 @@
             <origin rpy="0 0 0" xyz="0 0 0"/>
         <geometry>
-                <mesh  filename="file://$(arg resource_directory)/valve_${valve_type}collision.obj" scale="1 1 1"/>
+                <mesh  filename="file://$(arg resource_directory)/valve_$(arg valve_type)_collision.obj" scale="1 1 1"/>
             </geometry>
         </collision>

File: mppi_examples/mppi_omav_interaction/data/omav_hook_visualization.urdf.xacro (robot description, xacro)
@@ -41,4 +41,5 @@
             <geometry>
                 <cylinder radius="${manipulator_radius}" length="${manipulator_length}"/>
+                <!-- <box size="${manipulator_radius*2} ${manipulator_radius*2} ${manipulator_length}"/> -->
             </geometry>
         </collision>
@@ -47,4 +48,5 @@
             <geometry>
                 <cylinder radius="${manipulator_radius}" length="${manipulator_length}"/>
+                <!-- <box size="${manipulator_radius*2} ${manipulator_radius*2} ${manipulator_length}"/> -->
             </geometry>
             <material name="">
@@ -53,8 +55,8 @@
         </visual>
     </link>
-    <joint name="rod_to_tip" type="fixed">
+    <joint name="rod_to_hook" type="fixed">
         <parent link="rod"/>
-        <child link="tip"/>
-        <origin rpy="0 0 0" xyz="${manipulator_length/2} 0.0 0.0"/>
+        <child link="hook"/>
+        <origin rpy="0 0 0" xyz="${manipulator_length/2} 0.0 -${tool_length/2}"/>
     </joint>
     <!--
@@ -85,5 +87,5 @@
         </link>
 -->
-        <link name="tip">
+        <!-- <link name="tip">
             <collision>
                 <origin rpy="0 0 0" xyz="0 0 0"/>
@@ -104,10 +106,10 @@
                 </material>
             </visual>
-        </link>
-        <joint name="tip_to_hook" type="fixed">
+        </link> -->
+        <!-- <joint name="tip_to_hook" type="fixed">
             <parent link="tip"/>
             <child link="hook"/>
             <origin rpy="0 0 0" xyz="0.0 0.0 -${tool_length/2}"/>
-        </joint>
+        </joint> -->
         <link name="hook">
             <collision>
@@ -124,4 +126,5 @@
                 <geometry>
                     <cylinder radius="${tool_radius}" length="${tool_length}"/>
+                    <!-- <box size="${tool_radius*2} ${tool_radius*2} ${tool_length}"/> -->
                 </geometry>
                 <material name="">

File: mppi_examples/mppi_omav_interaction/data/omav_raisim_hook.urdf.xacro (robot description, xacro)
@@ -80,7 +80,8 @@
             <geometry>
                 <cylinder radius="${manipulator_radius}" length="${manipulator_length}"/>
+                <!-- <box size="${manipulator_radius*2} ${manipulator_radius*2} ${manipulator_length}"/> -->
             </geometry>
             <material name="">
-                <contact name="rubber"/>
+                <contact name="steel"/>
             </material>
         </collision>
@@ -89,4 +90,5 @@
             <geometry>
                 <cylinder radius="${manipulator_radius}" length="${manipulator_length}"/>
+                <!-- <box size="${manipulator_radius*2} ${manipulator_radius*2} ${manipulator_length}"/> -->
             </geometry>
             <material name="">
@@ -95,10 +97,10 @@
         </visual>
     </link>
-    <joint name="rod_to_tip" type="fixed">
+    <joint name="rod_to_hook" type="fixed">
         <parent link="rod"/>
-        <child link="tip"/>
-        <origin rpy="0 0 0" xyz="${manipulator_length/2} 0.0 0.0"/>
+        <child link="hook"/>
+        <origin rpy="0 0 0" xyz="${manipulator_length/2} 0.0 -${tool_length/2}"/>
     </joint>
-    <link name="tip">
+    <!-- <link name="tip">
         <collision>
             <origin rpy="0 0 0" xyz="0 0 0"/>
@@ -107,5 +109,5 @@
             </geometry>
             <material name="">
-                <contact name="rubber"/>
+                <contact name="steel"/>
             </material>
         </collision>
@@ -119,5 +121,5 @@
             </material>
         </visual>
-    </link>
+    </link> -->
 <!--
     <joint name="tip_to_thick" type="fixed">
@@ -133,5 +135,5 @@
             </geometry>
             <material name="">
-                <contact name="rubber"/>
+                <contact name="steel"/>
             </material>
         </collision>
@@ -147,9 +149,9 @@
     </link>
 -->
-    <joint name="tip_to_hook" type="fixed">
+    <!-- <joint name="tip_to_hook" type="fixed">
         <parent link="tip"/>
         <child link="hook"/>
         <origin rpy="0 0 0" xyz="0.0 0.0 -${tool_length/2}"/>
-    </joint>
+    </joint> -->
     <link name="hook">
         <collision>
@@ -157,7 +159,8 @@
             <geometry>
                 <cylinder radius="${tool_radius}" length="${tool_length}"/>
+                <!-- <box size="${tool_radius*2} ${tool_radius*2} ${tool_length}"/> -->
             </geometry>
             <material name="">
-                <contact name="rubber"/>
+                <contact name="steel"/>
             </material>
         </collision>
@@ -166,4 +169,5 @@
             <geometry>
                 <cylinder radius="${tool_radius}" length="${tool_length}"/>
+                <!-- <box size="${tool_radius*2} ${tool_radius*2} ${tool_length}"/> -->
             </geometry>
             <material name="">

Commit message: Reverted raisim simulation params, added lee81 collision obj.

File: mppi_examples/mppi_manipulation/data/objects/valve.urdf.xacro (robot description, xacro)
@@ -44,5 +44,5 @@
         <!--<origin xyz="0 0 ${base_height/2.0+0.2}" rpy="0 0 0"/> <!- 1.5708 0 0 -->
         <origin xyz="$(arg object_position)" rpy="$(arg object_rpy)"/>
-        <dynamics damping="1" friction="2"/>
+        <dynamics damping="0" friction="0.002"/>
         <axis xyz="0 0 1"/>
         <limit upper="300.14" lower="-300.14" effort="100" velocity="1.0"/>

Commit message: fix: use correct path for valve mesh files

File: mppi_examples/mppi_manipulation/data/objects/valve.urdf.xacro (robot description, xacro)
@@ -5,5 +5,4 @@
     <xacro:arg name="object_position" default="-1 0 1"/>
     <xacro:arg name="object_rpy" default="1.5708 0 0"/>
-    <xacro:arg name="host_name" default="$(arg host_name)"/>
     <xacro:arg name="valve_type" default="lee_thin"/>
     <link name="world"/>
@@ -32,5 +31,5 @@
 	       <geometry>
                 <!-- <mesh  filename="$(arg resource_prefix)$(arg resource_directory)/valve_${valve_type}collision.obj" scale="1 1 1"/> -->
-                <mesh  filename="/home/$(arg host_name)/catkin_ws/src/sampling_based_control/mppi_examples/mppi_manipulation/data/meshes/valve_$(arg valve_type)_collision.obj" scale="1 1 1"/>
+                <mesh  filename="$(arg resource_directory)/valve_$(arg valve_type)_collision.obj" scale="1 1 1"/>
             </geometry>
             <material name="">
