Commit message: Cleanup and attitude cost in code. Added rotation of the forces from body to worldframe. Very bad behavior of the controller.

File: mppi_examples/mppi_omav_raisim/data/omav.urdf (robot description, URDF)
Before this commit: robot omav, 4 links, 3 joints
Links:
- added link goal, mass 1.0; visual box size=0.2 0.2 0.2
- added link omav_rotation_x, mass 1.0; visual box size=0.03 0.03 0.03
- added link omav_rotation_y, mass 1.0; visual box size=0.03 0.03 0.03
- added link omav_rotation_z, mass 1.0; visual box size=0.3 0.3 0.3
- link omav_z: geometry visual box size=0.03 0.03 0.03
Joints:
- added joint fixed: type fixed, parent odom, child goal, origin xyz=5.0 5.0 5.0 rpy=0 0 0
- added joint omav_rot_x: type continuous, parent omav_z, child omav_rotation_x, origin xyz=0 0 0 rpy=0 0 0, axis 1 0 0, limit effort=1000 velocity=1000.0
- added joint omav_rot_y: type continuous, parent omav_rotation_x, child omav_rotation_y, origin xyz=0 0 0 rpy=0 0 0, axis 0 1 0, limit effort=1000 velocity=1000.0
- added joint omav_rot_z: type continuous, parent omav_rotation_y, child omav_rotation_z, origin xyz=0 0 0 rpy=0 0 0, axis 0 0 1, limit effort=1000 velocity=1000.0
- joint omav_pos_x: limit lower=-30.14 upper=30.14 effort=1000 velocity=2.0 -> lower=-1000.0 upper=1000.0 effort=1000 velocity=1000.0
- joint omav_pos_y: limit lower=-30.14 upper=30.14 effort=1000 velocity=2.0 -> lower=-1000.0 upper=1000.0 effort=1000 velocity=1000.0
- joint omav_pos_z: limit lower=-30.14 upper=30.14 effort=1000 velocity=2.0 -> lower=-1000.0 upper=1000.0 effort=1000 velocity=1000.0
