Commit message: Applied comments by Giuseppe. As well as some cleanup.

File: mppi_examples/mppi_omav_raisim/data/omav_raisim.urdf.xacro (robot description, xacro)
@@ -7,7 +7,4 @@
     <xacro:property name="radius_ouzel" value="0.5"/>
     <xacro:property name="height_ouzel" value="0.3"/>
-    <link name="odom">
-        <origin rpy="0 0 0" xyz="0 0 0"/>
-    </link>
     <link name="ouzel">
         <inertial>
@@ -32,8 +29,3 @@
         </visual>
     </link>
-    <joint name="odom_drone" type="fixed">
-        <origin xyz="0 0 0" rpy="0 0 0"/>
-        <parent link="odom"/>
-        <child link="ouzel"/>
-    </joint>
 </robot>
