Commit message: Implemented reconsidering.

File: mppi_examples/mppi_omav_interaction/data/omav_raisim_rod.urdf.xacro (robot description, xacro)
@@ -5,5 +5,5 @@
     <xacro:property name="iyy_ouzel" value="0.14"/>
     <xacro:property name="izz_ouzel" value="0.18"/>
-    <xacro:property name="radius_ouzel" value="0.25"/>
+    <xacro:property name="radius_ouzel" value="0.2"/>
     <xacro:property name="height_ouzel" value="0.3"/>
     <link name="world"/>
@@ -68,5 +68,5 @@
         <parent link="omav"/>
         <child link="rod"/>
-        <origin rpy="0 0 0" xyz="0.5 0.0 0.0"/>
+        <origin rpy="0 0 0" xyz="0.275 0.0 0.0"/>
     </joint>
     <link name="rod">
@@ -74,5 +74,5 @@
             <origin rpy="0 1.5708 0" xyz="0 0 0"/>
             <geometry>
-                <cylinder radius="0.05" length="0.7"/>
+                <cylinder radius="0.015" length="0.54"/>
             </geometry>
         </collision>
@@ -80,5 +80,5 @@
             <origin rpy="0 1.5708 0" xyz="0 0 0"/>
             <geometry>
-                <cylinder radius="0.05" length="0.7"/>
+                <cylinder radius="0.015" length="0.54"/>
             </geometry>
             <material name="">
@@ -90,5 +90,5 @@
         <parent link="rod"/>
         <child link="tip"/>
-        <origin rpy="0 0 0" xyz="0.35 0.0 0.0"/>
+        <origin rpy="0 0 0" xyz="0.27 0.0 0.0"/>
     </joint>
     <link name="tip">
@@ -96,5 +96,5 @@
             <origin rpy="0 0 0" xyz="0 0 0"/>
             <geometry>
-                <sphere radius="0.05"/>
+                <sphere radius="0.015"/>
             </geometry>
         </collision>
@@ -102,5 +102,5 @@
             <origin rpy="0 0 0" xyz="0 0.0 0"/>
             <geometry>
-                <sphere radius="0.05"/>
+                <sphere radius="0.015"/>
             </geometry>
             <material name="">
