Commit message: Added material properties to have more realistic contact behaviour.

File: mppi_examples/mppi_omav_interaction/data/button.urdf.xacro (robot description, xacro)
@@ -16,5 +16,5 @@
         <axis xyz="1 0 0"/>
         <limit effort="1000.0" velocity="5.0" lower="-100" upper="100"/>
-        <dynamics spring_mount="0 0 0" stiffness="1.0" damping="1"/>
+        <dynamics spring_mount="0 0 0" stiffness="10.0" damping="1"/>
     </joint>
     <link name="button_x">
@@ -29,4 +29,7 @@
                 <box size="${dimension_cube} ${dimension_cube} ${dimension_cube}"/>
             </geometry>
+            <material name="">
+                <contact name="rubber"/>
+            </material>
         </collision>
         <visual>

File: mppi_examples/mppi_omav_interaction/data/omav_raisim_rod.urdf.xacro (robot description, xacro)
@@ -98,4 +98,7 @@
                 <sphere radius="0.015"/>
             </geometry>
+            <material name="">
+                <contact name="rubber"/>
+            </material>
         </collision>
         <visual>

Commit message: New examples for opening drawer and door.

File: mppi_examples/mppi_omav_interaction/data/button.urdf.xacro (robot description, xacro)
@@ -4,12 +4,12 @@
     <xacro:property name="dimension_cube" value="0.3"/>
     <link name="world"/>
-    <link name="odom"/>
     <joint name="odom_to_world" type="fixed">
         <parent link="world"/>
-        <child link="odom"/>
+        <child link="odom_button"/>
         <origin rpy="0 0 0" xyz="2.0 0.0 1.0"/>
     </joint>
-    <joint name="odom_to_button_x" type="prismatic">
-        <parent link="odom"/>
+    <link name="odom_button"/>
+    <joint name="articulation_joint" type="prismatic">
+        <parent link="odom_button"/>
         <child link="button_x"/>
         <origin rpy="0 0 0" xyz="0.0 0.0 0.0"/>

File: mppi_examples/mppi_omav_interaction/data/omav_hook_visualization.urdf.xacro (robot description, xacro)
@@ -1,4 +1,4 @@
 <?xml version="1.0"?>
-<robot xmlns:xacro="http://www.ros.org/wiki/xacro" name="ouzel_raisim">
+<robot xmlns:xacro="http://www.ros.org/wiki/xacro" name="ouzel">
     <xacro:property name="mass_ouzel" value="5.0"/>
     <xacro:property name="ixx_ouzel" value="0.12"/>
@@ -7,46 +7,11 @@
     <xacro:property name="radius_ouzel" value="0.2"/>
     <xacro:property name="height_ouzel" value="0.3"/>
-    <link name="world"/>
     <link name="odom_omav"/>
-    <joint name="odom_to_world" type="fixed">
-        <parent link="world"/>
-        <child link="odom_omav"/>
+    <joint name="odom_omav_to_omav_base" type="fixed">
+        <parent link="odom_omav"/>
+        <child link="omav_base"/>
+        <origin rpy="0 0 0" xyz="0.0 0.0 0.0"/>
     </joint>
-    <joint name="odom_to_omav_x" type="prismatic">
-        <parent link="odom_omav"/>
-        <child link="omav_x"/>
-        <origin rpy="0 0 0" xyz="0.0 0.0 0.0"/>
-        <axis xyz="1 0 0"/>
-        <limit effort="1000.0" velocity="5.0" lower="-100" upper="100"/>
-    </joint>
-    <link name="omav_x"/>
-    <joint name="omav_x_to_omav_y" type="prismatic">
-        <parent link="omav_x"/>
-        <child link="omav_y"/>
-        <origin rpy="0 0 0" xyz="0.0 0.0 0.0"/>
-        <axis xyz="0 1 0"/>
-        <limit effort="1000.0" velocity="5.0" lower="-100" upper="100"/>
-    </joint>
-    <link name="omav_y"/>
-    <joint name="omav_y_to_omav_z" type="prismatic">
-        <parent link="omav_y"/>
-        <child link="omav_z"/>
-        <origin rpy="0 0 0" xyz="0.0 0.0 0.0"/>
-        <axis xyz="0 0 1"/>
-        <limit effort="1000.0" velocity="5.0" lower="-100" upper="100"/>
-    </joint>
-    <link name="omav_z"/>
-    <joint name="omav_z_to_omav" type="spherical">
-        <parent link="omav_z"/>
-        <child link="omav"/>
-        <origin rpy="0 0 0" xyz="0.0 0.0 0.0"/>
-        <axis xyz="0 1 0"/>
-    </joint>
-    <link name="omav">
-        <inertial>
-            <mass value="${mass_ouzel}"/>
-            <origin rpy="0 0 0" xyz="0 0 0"/>
-            <inertia ixx="${ixx_ouzel}" ixy="0" ixz="0" iyy="${iyy_ouzel}" iyz="0" izz="${izz_ouzel}"/>
-        </inertial>
+    <link name="omav_base">
         <collision>
             <origin rpy="0 0 0" xyz="0 0 0"/>
@@ -61,10 +26,10 @@
             </geometry>
             <material name="">
-                <color rgba="1 1 1 1"/>
+                <color rgba="1 1 1 0.0"/>
             </material>
         </visual>
     </link>
     <joint name="omav_to_rod" type="fixed">
-        <parent link="omav"/>
+        <parent link="omav_base"/>
         <child link="rod"/>
         <origin rpy="0 0 0" xyz="0.275 0.0 0.0"/>
@@ -112,3 +77,28 @@
         </visual>
     </link>
+    <joint name="tip_to_hook" type="fixed">
+        <parent link="tip"/>
+        <child link="hook"/>
+        <origin rpy="0 0 0" xyz="0.0 0.0 -0.025"/>
+    </joint>
+    <link name="hook">
+        <collision>
+            <origin rpy="0 0 0" xyz="0 0 0"/>
+            <geometry>
+                <cylinder radius="0.015" length="0.05"/>
+            </geometry>
+            <material name="">
+                <contact name="rubber"/>
+            </material>
+        </collision>
+        <visual>
+            <origin rpy="0 0 0" xyz="0 0 0"/>
+            <geometry>
+                <cylinder radius="0.015" length="0.05"/>
+            </geometry>
+            <material name="">
+                <color rgba="1 1 1 1"/>
+            </material>
+        </visual>
+    </link>
 </robot>

File: mppi_examples/mppi_omav_interaction/data/omav_raisim_hook.urdf.xacro (robot description, xacro)
@@ -8,11 +8,11 @@
     <xacro:property name="height_ouzel" value="0.3"/>
     <link name="world"/>
-    <link name="odom_omav"/>
+    <link name="odom"/>
     <joint name="odom_to_world" type="fixed">
         <parent link="world"/>
-        <child link="odom_omav"/>
+        <child link="odom"/>
     </joint>
     <joint name="odom_to_omav_x" type="prismatic">
-        <parent link="odom_omav"/>
+        <parent link="odom"/>
         <child link="omav_x"/>
         <origin rpy="0 0 0" xyz="0.0 0.0 0.0"/>
@@ -76,4 +76,7 @@
                 <cylinder radius="0.015" length="0.54"/>
             </geometry>
+            <material name="">
+                <contact name="rubber"/>
+            </material>
         </collision>
         <visual>
@@ -112,3 +115,28 @@
         </visual>
     </link>
+    <joint name="tip_to_hook" type="fixed">
+        <parent link="tip"/>
+        <child link="hook"/>
+        <origin rpy="0 0 0" xyz="0.0 0.0 -0.025"/>
+    </joint>
+    <link name="hook">
+        <collision>
+            <origin rpy="0 0 0" xyz="0 0 0"/>
+            <geometry>
+                <cylinder radius="0.015" length="0.05"/>
+            </geometry>
+            <material name="">
+                <contact name="rubber"/>
+            </material>
+        </collision>
+        <visual>
+            <origin rpy="0 0 0" xyz="0 0 0"/>
+            <geometry>
+                <cylinder radius="0.015" length="0.05"/>
+            </geometry>
+            <material name="">
+                <color rgba="1 1 1 1"/>
+            </material>
+        </visual>
+    </link>
 </robot>
