Commit message: Added initial state to the debug publish.

File: mppi_examples/mppi_omav_interaction/data/omav_raisim_hook.urdf.xacro (robot description, xacro)
@@ -7,7 +7,7 @@
     <xacro:property name="tool_radius" value="0.0075"/>         <!-- [m] -->
     <xacro:property name="mass_ouzel" value="4.337"/>
-    <xacro:property name="ixx_ouzel" value="0.12"/>
-    <xacro:property name="iyy_ouzel" value="0.14"/>
-    <xacro:property name="izz_ouzel" value="0.18"/>
+    <xacro:property name="ixx_ouzel" value="0.078359"/>
+    <xacro:property name="iyy_ouzel" value="0.081797"/>
+    <xacro:property name="izz_ouzel" value="0.153355"/>
     <xacro:property name="radius_ouzel" value="0.2"/>
     <xacro:property name="height_ouzel" value="0.3"/>
