Commit message: Added a node for the vicon observer.

File: mppi_examples/mppi_omav_interaction/data/omav_hook_visualization.urdf.xacro (robot description, xacro)
@@ -57,4 +57,29 @@
         <origin rpy="0 0 0" xyz="0.27 0.0 0.0"/>
     </joint>
+    <joint name="tip_to_thick" type="fixed">
+        <parent link="tip"/>
+        <child link="thick"/>
+        <origin rpy="0 0 0" xyz="-0.025 0.0 0.0"/>
+    </joint>
+    <link name="thick">
+        <collision>
+            <origin rpy="0 1.5708 0" xyz="0 0 0"/>
+            <geometry>
+                <cylinder radius="0.015" length="0.05"/>
+            </geometry>
+            <material name="">
+                <contact name="rubber"/>
+            </material>
+        </collision>
+        <visual>
+            <origin rpy="0 1.5708 0" xyz="0 0 0"/>
+            <geometry>
+                <cylinder radius="0.015" length="0.05"/>
+            </geometry>
+            <material name="">
+                <color rgba="1 1 1 1"/>
+            </material>
+        </visual>
+    </link>
     <link name="tip">
         <collision>

File: mppi_examples/mppi_omav_interaction/data/omav_raisim_hook.urdf.xacro (robot description, xacro)
@@ -115,4 +115,29 @@
         </visual>
     </link>
+    <joint name="tip_to_thick" type="fixed">
+        <parent link="tip"/>
+        <child link="thick"/>
+        <origin rpy="0 0 0" xyz="-0.025 0.0 0.0"/>
+    </joint>
+    <link name="thick">
+        <collision>
+            <origin rpy="0 1.5708 0" xyz="0 0 0"/>
+            <geometry>
+                <cylinder radius="0.015" length="0.05"/>
+            </geometry>
+            <material name="">
+                <contact name="rubber"/>
+            </material>
+        </collision>
+        <visual>
+            <origin rpy="0 1.5708 0" xyz="0 0 0"/>
+            <geometry>
+                <cylinder radius="0.015" length="0.05"/>
+            </geometry>
+            <material name="">
+                <color rgba="1 1 1 1"/>
+            </material>
+        </visual>
+    </link>
     <joint name="tip_to_hook" type="fixed">
         <parent link="tip"/>

Commit message: Slightly changed urdf, to more realistic values.

File: mppi_examples/mppi_omav_interaction/data/omav_hook_visualization.urdf.xacro (robot description, xacro)
@@ -60,5 +60,5 @@
         <parent link="tip"/>
         <child link="thick"/>
-        <origin rpy="0 0 0" xyz="-0.025 0.0 0.0"/>
+        <origin rpy="0 0 0" xyz="-0.0175 0.0 0.0"/>
     </joint>
     <link name="thick">

File: mppi_examples/mppi_omav_interaction/data/omav_raisim_hook.urdf.xacro (robot description, xacro)
@@ -118,5 +118,5 @@
         <parent link="tip"/>
         <child link="thick"/>
-        <origin rpy="0 0 0" xyz="-0.025 0.0 0.0"/>
+        <origin rpy="0 0 0" xyz="-0.0175 0.0 0.0"/>
     </joint>
     <link name="thick">

Commit message: Slightly updated parameters.

File: mppi_examples/mppi_omav_interaction/data/omav_hook_visualization.urdf.xacro (robot description, xacro)
@@ -60,5 +60,5 @@
         <parent link="tip"/>
         <child link="thick"/>
-        <origin rpy="0 0 0" xyz="-0.0175 0.0 0.0"/>
+        <origin rpy="0 0 0" xyz="-0.02 0.0 0.0"/>
     </joint>
     <link name="thick">
@@ -66,5 +66,5 @@
             <origin rpy="0 1.5708 0" xyz="0 0 0"/>
             <geometry>
-                <cylinder radius="0.015" length="0.05"/>
+                <cylinder radius="0.015" length="0.055"/>
             </geometry>
             <material name="">
@@ -75,5 +75,5 @@
             <origin rpy="0 1.5708 0" xyz="0 0 0"/>
             <geometry>
-                <cylinder radius="0.015" length="0.05"/>
+                <cylinder radius="0.015" length="0.055"/>
             </geometry>
             <material name="">

File: mppi_examples/mppi_omav_interaction/data/omav_raisim_hook.urdf.xacro (robot description, xacro)
@@ -118,5 +118,5 @@
         <parent link="tip"/>
         <child link="thick"/>
-        <origin rpy="0 0 0" xyz="-0.0175 0.0 0.0"/>
+        <origin rpy="0 0 0" xyz="-0.02 0.0 0.0"/>
     </joint>
     <link name="thick">
@@ -124,5 +124,5 @@
             <origin rpy="0 1.5708 0" xyz="0 0 0"/>
             <geometry>
-                <cylinder radius="0.015" length="0.05"/>
+                <cylinder radius="0.015" length="0.055"/>
             </geometry>
             <material name="">
@@ -133,5 +133,5 @@
             <origin rpy="0 1.5708 0" xyz="0 0 0"/>
             <geometry>
-                <cylinder radius="0.015" length="0.05"/>
+                <cylinder radius="0.015" length="0.055"/>
             </geometry>
             <material name="">

Commit message: Working version, added multiple improvements.

File: mppi_examples/mppi_omav_interaction/data/omav_hook_visualization.urdf.xacro (robot description, xacro)
@@ -1,4 +1,9 @@
 <?xml version="1.0"?>
 <robot xmlns:xacro="http://www.ros.org/wiki/xacro" name="omav_hook_visualization">
+    <!-- Properties -->
+    <xacro:property name="manipulator_length" value="0.62"/>   <!-- [m] -->
+    <xacro:property name="manipulator_radius" value="0.0075"/>  <!-- [m] -->
+    <xacro:property name="tool_length" value="0.05"/>         <!-- [m] -->
+    <xacro:property name="tool_radius" value="0.0075"/>         <!-- [m] -->
     <xacro:property name="mass_ouzel" value="5.0"/>
     <xacro:property name="ixx_ouzel" value="0.12"/>
@@ -26,5 +31,5 @@
             </geometry>
             <material name="">
-                <color rgba="1 1 1 0.0"/>
+                <color rgba="1 1 1 1.0"/>
             </material>
         </visual>
@@ -33,5 +38,5 @@
         <parent link="omav_base"/>
         <child link="rod"/>
-        <origin rpy="0 0 0" xyz="0.31 0.0 0.0"/>
+        <origin rpy="0 0 0" xyz="${manipulator_length/2} 0.0 0.0"/>
     </joint>
     <link name="rod">
@@ -39,5 +44,5 @@
             <origin rpy="0 1.5708 0" xyz="0 0 0"/>
             <geometry>
-                <cylinder radius="0.0075" length="0.62"/>
+                <cylinder radius="${manipulator_radius}" length="${manipulator_length}"/>
             </geometry>
         </collision>
@@ -45,5 +50,5 @@
             <origin rpy="0 1.5708 0" xyz="0 0 0"/>
             <geometry>
-                <cylinder radius="0.0075" length="0.62"/>
+                <cylinder radius="${manipulator_radius}" length="${manipulator_length}"/>
             </geometry>
             <material name="">
@@ -55,5 +60,5 @@
         <parent link="rod"/>
         <child link="tip"/>
-        <origin rpy="0 0 0" xyz="0.31 0.0 0.0"/>
+        <origin rpy="0 0 0" xyz="${manipulator_length/2} 0.0 0.0"/>
     </joint>
     <joint name="tip_to_thick" type="fixed">
@@ -86,5 +91,5 @@
             <origin rpy="0 0 0" xyz="0 0 0"/>
             <geometry>
-                <sphere radius="0.015"/>
+                <sphere radius="${tool_radius}"/>
             </geometry>
             <material name="">
@@ -95,5 +100,5 @@
             <origin rpy="0 0 0" xyz="0 0.0 0"/>
             <geometry>
-                <sphere radius="0.0075"/>
+                <sphere radius="${tool_radius}"/>
             </geometry>
             <material name="">
@@ -105,5 +110,5 @@
         <parent link="tip"/>
         <child link="hook"/>
-        <origin rpy="0 0 0" xyz="0.0 0.0 -0.025"/>
+        <origin rpy="0 0 0" xyz="0.0 0.0 -${tool_length/2}"/>
     </joint>
     <link name="hook">
@@ -111,5 +116,5 @@
             <origin rpy="0 0 0" xyz="0 0 0"/>
             <geometry>
-                <cylinder radius="0.0075" length="0.05"/>
+                <cylinder radius="${tool_radius}" length="${tool_length}"/>
             </geometry>
             <material name="">
@@ -120,5 +125,5 @@
             <origin rpy="0 0 0" xyz="0 0 0"/>
             <geometry>
-                <cylinder radius="0.0075" length="0.05"/>
+                <cylinder radius="${tool_radius}" length="${tool_length}"/>
             </geometry>
             <material name="">

File: mppi_examples/mppi_omav_interaction/data/omav_pinocchio_hook.urdf.xacro (robot description, xacro)
@@ -1,4 +1,9 @@
 <?xml version="1.0"?>
 <robot xmlns:xacro="http://www.ros.org/wiki/xacro" name="omav_pinocchio_hook">
+    <!-- Properties -->
+    <xacro:property name="manipulator_length" value="0.62"/>   <!-- [m] -->
+    <xacro:property name="manipulator_radius" value="0.0075"/>  <!-- [m] -->
+    <xacro:property name="tool_length" value="0.05"/>         <!-- [m] -->
+    <xacro:property name="tool_radius" value="0.0075"/>         <!-- [m] -->
     <xacro:property name="mass_ouzel" value="5.0"/>
     <xacro:property name="ixx_ouzel" value="0.12"/>
@@ -43,5 +48,5 @@
         <parent link="omav"/>
         <child link="rod"/>
-        <origin rpy="0 0 0" xyz="0.31 0.0 0.0"/>
+        <origin rpy="0 0 0" xyz="${manipulator_length/2} 0.0 0.0"/>
     </joint>
     <link name="rod">
@@ -49,5 +54,5 @@
             <origin rpy="0 1.5708 0" xyz="0 0 0"/>
             <geometry>
-                <cylinder radius="0.015" length="0.62"/>
+                <cylinder radius="${manipulator_radius}" length="${manipulator_length}"/>
             </geometry>
             <material name="">
@@ -58,5 +63,5 @@
             <origin rpy="0 1.5708 0" xyz="0 0 0"/>
             <geometry>
-                <cylinder radius="0.015" length="0.62"/>
+                <cylinder radius="${manipulator_radius}" length="${manipulator_length}"/>
             </geometry>
             <material name="">
@@ -68,5 +73,5 @@
         <parent link="rod"/>
         <child link="tip"/>
-        <origin rpy="0 0 0" xyz="0.31 0.0 0.0"/>
+        <origin rpy="0 0 0" xyz="${manipulator_length/2} 0.0 0.0"/>
     </joint>
     <link name="tip">
@@ -74,5 +79,5 @@
             <origin rpy="0 0 0" xyz="0 0 0"/>
             <geometry>
-                <sphere radius="0.015"/>
+                <sphere radius="${manipulator_radius}"/>
             </geometry>
             <material name="">
@@ -83,5 +88,5 @@
             <origin rpy="0 0 0" xyz="0 0.0 0"/>
             <geometry>
-                <sphere radius="0.015"/>
+                <sphere radius="${manipulator_radius}"/>
             </geometry>
             <material name="">
@@ -93,5 +98,5 @@
         <parent link="tip"/>
         <child link="hook"/>
-        <origin rpy="0 0 0" xyz="0.0 0.0 -0.025"/>
+        <origin rpy="0 0 0" xyz="0.0 0.0 -${tool_length/2}"/>
     </joint>
     <link name="hook">
@@ -99,5 +104,5 @@
             <origin rpy="0 0 0" xyz="0 0 0"/>
             <geometry>
-                <cylinder radius="0.015" length="0.05"/>
+                <cylinder radius="${tool_radius}" length="${tool_length}"/>
             </geometry>
             <material name="">
@@ -108,5 +113,5 @@
             <origin rpy="0 0 0" xyz="0 0 0"/>
             <geometry>
-                <cylinder radius="0.015" length="0.05"/>
+                <cylinder radius="${tool_radius}" length="${tool_length}"/>
             </geometry>
             <material name="">

File: mppi_examples/mppi_omav_interaction/data/omav_raisim_hook.urdf.xacro (robot description, xacro)
@@ -1,4 +1,9 @@
 <?xml version="1.0"?>
 <robot xmlns:xacro="http://www.ros.org/wiki/xacro" name="omav_raisim_hook">
+    <!-- Properties -->
+    <xacro:property name="manipulator_length" value="0.62"/>   <!-- [m] -->
+    <xacro:property name="manipulator_radius" value="0.0075"/>  <!-- [m] -->
+    <xacro:property name="tool_length" value="0.05"/>         <!-- [m] -->
+    <xacro:property name="tool_radius" value="0.0075"/>         <!-- [m] -->
     <xacro:property name="mass_ouzel" value="5.0"/>
     <xacro:property name="ixx_ouzel" value="0.12"/>
@@ -68,5 +73,5 @@
         <parent link="omav"/>
         <child link="rod"/>
-        <origin rpy="0 0 0" xyz="0.31 0.0 0.0"/>
+        <origin rpy="0 0 0" xyz="${manipulator_length/2} 0.0 0.0"/>
     </joint>
     <link name="rod">
@@ -74,5 +79,5 @@
             <origin rpy="0 1.5708 0" xyz="0 0 0"/>
             <geometry>
-                <cylinder radius="0.0075" length="0.62"/>
+                <cylinder radius="${manipulator_radius}" length="${manipulator_length}"/>
             </geometry>
             <material name="">
@@ -83,5 +88,5 @@
             <origin rpy="0 1.5708 0" xyz="0 0 0"/>
             <geometry>
-                <cylinder radius="0.0075" length="0.62"/>
+                <cylinder radius="${manipulator_radius}" length="${manipulator_length}"/>
             </geometry>
             <material name="">
@@ -93,5 +98,5 @@
         <parent link="rod"/>
         <child link="tip"/>
-        <origin rpy="0 0 0" xyz="0.31 0.0 0.0"/>
+        <origin rpy="0 0 0" xyz="${manipulator_length/2} 0.0 0.0"/>
     </joint>
     <link name="tip">
@@ -99,5 +104,5 @@
             <origin rpy="0 0 0" xyz="0 0 0"/>
             <geometry>
-                <sphere radius="0.0075"/>
+                <sphere radius="${tool_radius}"/>
             </geometry>
             <material name="">
@@ -108,5 +113,5 @@
             <origin rpy="0 0 0" xyz="0 0.0 0"/>
             <geometry>
-                <sphere radius="0.0075"/>
+                <sphere radius="${tool_radius}"/>
             </geometry>
             <material name="">
@@ -143,5 +148,5 @@
         <parent link="tip"/>
         <child link="hook"/>
-        <origin rpy="0 0 0" xyz="0.0 0.0 -0.025"/>
+        <origin rpy="0 0 0" xyz="0.0 0.0 -${tool_length/2}"/>
     </joint>
     <link name="hook">
@@ -149,5 +154,5 @@
             <origin rpy="0 0 0" xyz="0 0 0"/>
             <geometry>
-                <cylinder radius="0.0075" length="0.05"/>
+                <cylinder radius="${tool_radius}" length="${tool_length}"/>
             </geometry>
             <material name="">
@@ -158,5 +163,5 @@
             <origin rpy="0 0 0" xyz="0 0 0"/>
             <geometry>
-                <cylinder radius="0.0075" length="0.05"/>
+                <cylinder radius="${tool_radius}" length="${tool_length}"/>
             </geometry>
             <material name="">

Commit message: Improved warmstarting and added force cost.

File: mppi_examples/mppi_omav_interaction/data/omav_hook_visualization.urdf.xacro (robot description, xacro)
@@ -38,5 +38,5 @@
         <parent link="omav_base"/>
         <child link="rod"/>
-        <origin rpy="0 0 0" xyz="${manipulator_length/2} 0.0 0.0"/>
+        <origin rpy="-1.5708 0 0" xyz="${manipulator_length/2} 0.0 0.0"/>
     </joint>
     <link name="rod">

File: mppi_examples/mppi_omav_interaction/data/omav_pinocchio_hook.urdf.xacro (robot description, xacro)
@@ -48,5 +48,5 @@
         <parent link="omav"/>
         <child link="rod"/>
-        <origin rpy="0 0 0" xyz="${manipulator_length/2} 0.0 0.0"/>
+        <origin rpy="-1.5708 0 0" xyz="${manipulator_length/2} 0.0 0.0"/>
     </joint>
     <link name="rod">

File: mppi_examples/mppi_omav_interaction/data/omav_raisim_hook.urdf.xacro (robot description, xacro)
@@ -73,5 +73,5 @@
         <parent link="omav"/>
         <child link="rod"/>
-        <origin rpy="0 0 0" xyz="${manipulator_length/2} 0.0 0.0"/>
+        <origin rpy="-1.5708 0 0" xyz="${manipulator_length/2} 0.0 0.0"/>
     </joint>
     <link name="rod">

Commit message: Parameterized rod angles.

File: mppi_examples/mppi_omav_interaction/data/omav_hook_visualization.urdf.xacro (robot description, xacro)
@@ -38,5 +38,5 @@
         <parent link="omav_base"/>
         <child link="rod"/>
-        <origin rpy="-1.5708 0 0" xyz="${manipulator_length/2} 0.0 0.0"/>
+        <origin rpy="$(arg omav_to_rod_angle) 0 0" xyz="${manipulator_length/2} 0.0 0.0"/>
     </joint>
     <link name="rod">

File: mppi_examples/mppi_omav_interaction/data/omav_pinocchio_hook.urdf.xacro (robot description, xacro)
@@ -48,5 +48,5 @@
         <parent link="omav"/>
         <child link="rod"/>
-        <origin rpy="-1.5708 0 0" xyz="${manipulator_length/2} 0.0 0.0"/>
+        <origin rpy="$(arg omav_to_rod_angle) 0 0" xyz="${manipulator_length/2} 0.0 0.0"/>
     </joint>
     <link name="rod">

File: mppi_examples/mppi_omav_interaction/data/omav_raisim_hook.urdf.xacro (robot description, xacro)
@@ -73,5 +73,5 @@
         <parent link="omav"/>
         <child link="rod"/>
-        <origin rpy="-1.5708 0 0" xyz="${manipulator_length/2} 0.0 0.0"/>
+        <origin rpy="$(arg omav_to_rod_angle) 0 0" xyz="${manipulator_length/2} 0.0 0.0"/>
     </joint>
     <link name="rod">

Commit message: Fixed hook length.

File: mppi_examples/mppi_omav_interaction/data/omav_hook_visualization.urdf.xacro (robot description, xacro)
@@ -4,5 +4,5 @@
     <xacro:property name="manipulator_length" value="$(arg manipulator_length)"/>   <!-- [m] -->
     <xacro:property name="manipulator_radius" value="0.0075"/>  <!-- [m] -->
-    <xacro:property name="tool_length" value="0.05"/>         <!-- [m] -->
+    <xacro:property name="tool_length" value="0.065"/>         <!-- [m] -->
     <xacro:property name="tool_radius" value="0.0075"/>         <!-- [m] -->
     <xacro:property name="radius_ouzel" value="0.2"/>

File: mppi_examples/mppi_omav_interaction/data/omav_pinocchio_hook.urdf.xacro (robot description, xacro)
@@ -4,5 +4,5 @@
     <xacro:property name="manipulator_length" value="$(arg manipulator_length)"/>   <!-- [m] -->
     <xacro:property name="manipulator_radius" value="0.0075"/>  <!-- [m] -->
-    <xacro:property name="tool_length" value="0.05"/>         <!-- [m] -->
+    <xacro:property name="tool_length" value="0.065"/>         <!-- [m] -->
     <xacro:property name="tool_radius" value="0.0075"/>         <!-- [m] -->
     <xacro:property name="mass_ouzel" value="4.337"/>

File: mppi_examples/mppi_omav_interaction/data/omav_raisim_hook.urdf.xacro (robot description, xacro)
@@ -4,5 +4,5 @@
     <xacro:property name="manipulator_length" value="$(arg manipulator_length)"/>   <!-- [m] -->
     <xacro:property name="manipulator_radius" value="0.0075"/>  <!-- [m] -->
-    <xacro:property name="tool_length" value="0.05"/>         <!-- [m] -->
+    <xacro:property name="tool_length" value="0.065"/>         <!-- [m] -->
     <xacro:property name="tool_radius" value="0.0075"/>         <!-- [m] -->
     <xacro:property name="mass_ouzel" value="4.337"/>

Commit message: Updates during experiments.

File: mppi_examples/mppi_omav_interaction/data/omav_hook_visualization.urdf.xacro (robot description, xacro)
@@ -4,5 +4,5 @@
     <xacro:property name="manipulator_length" value="$(arg manipulator_length)"/>   <!-- [m] -->
     <xacro:property name="manipulator_radius" value="0.0075"/>  <!-- [m] -->
-    <xacro:property name="tool_length" value="0.065"/>         <!-- [m] -->
+    <xacro:property name="tool_length" value="0.04"/>         <!-- [m] -->
     <xacro:property name="tool_radius" value="0.0075"/>         <!-- [m] -->
     <xacro:property name="radius_ouzel" value="0.2"/>

File: mppi_examples/mppi_omav_interaction/data/omav_pinocchio_hook.urdf.xacro (robot description, xacro)
@@ -4,5 +4,5 @@
     <xacro:property name="manipulator_length" value="$(arg manipulator_length)"/>   <!-- [m] -->
     <xacro:property name="manipulator_radius" value="0.0075"/>  <!-- [m] -->
-    <xacro:property name="tool_length" value="0.065"/>         <!-- [m] -->
+    <xacro:property name="tool_length" value="0.04"/>         <!-- [m] -->
     <xacro:property name="tool_radius" value="0.0075"/>         <!-- [m] -->
     <xacro:property name="mass_ouzel" value="4.337"/>

File: mppi_examples/mppi_omav_interaction/data/omav_raisim_hook.urdf.xacro (robot description, xacro)
@@ -4,5 +4,5 @@
     <xacro:property name="manipulator_length" value="$(arg manipulator_length)"/>   <!-- [m] -->
     <xacro:property name="manipulator_radius" value="0.0075"/>  <!-- [m] -->
-    <xacro:property name="tool_length" value="0.065"/>         <!-- [m] -->
+    <xacro:property name="tool_length" value="0.04"/>         <!-- [m] -->
     <xacro:property name="tool_radius" value="0.0075"/>         <!-- [m] -->
     <xacro:property name="mass_ouzel" value="4.337"/>
