Commit message: updated urdf

File: mppi_examples/mppi_omav_interaction/data/omav_hook_visualization.urdf.xacro (robot description, xacro)
@@ -2,61 +2,65 @@
 <robot xmlns:xacro="http://www.ros.org/wiki/xacro" name="omav_hook_visualization">
     <!-- Properties -->
-    <xacro:property name="manipulator_length" value="$(arg manipulator_length)"/>   <!-- [m] -->
-    <xacro:property name="manipulator_radius" value="0.0075"/>  <!-- [m] -->
-    <xacro:property name="tool_length" value="0.04"/>         <!-- [m] -->
-    <xacro:property name="tool_radius" value="0.0075"/>         <!-- [m] -->
-    <xacro:property name="radius_ouzel" value="0.2"/>
-    <xacro:property name="height_ouzel" value="0.3"/>
-    <link name="state"/>
+    <xacro:property name="manipulator_length" value="$(arg manipulator_length)" />
+    <!-- [m] -->
+    <xacro:property name="manipulator_radius" value="0.0075" />
+    <!-- [m] -->
+    <xacro:property name="tool_length" value="0.04" />
+    <!-- [m] -->
+    <xacro:property name="tool_radius" value="0.0075" />
+    <!-- [m] -->
+    <xacro:property name="radius_ouzel" value="0.48" />
+    <xacro:property name="height_ouzel" value="0.3" />
+    <link name="state" />
     <joint name="state_to_omav_base" type="fixed">
-        <parent link="state"/>
-        <child link="omav_base"/>
-        <origin rpy="0 0 0" xyz="0.0 0.0 0.0"/>
+        <parent link="state" />
+        <child link="omav_base" />
+        <origin rpy="0 0 0" xyz="0.0 0.0 0.0" />
     </joint>
     <link name="omav_base">
         <collision>
-            <origin rpy="0 0 0" xyz="0 0 0"/>
+            <origin rpy="0 0 0" xyz="0 0 0" />
             <geometry>
-                <cylinder radius="${radius_ouzel}" length="${height_ouzel}"/>
+                <cylinder radius="${radius_ouzel}" length="${height_ouzel}" />
             </geometry>
         </collision>
         <visual>
-            <origin rpy="0 0 0" xyz="0 0 0"/>
+            <origin rpy="0 0 0" xyz="0 0 0" />
             <geometry>
-                <cylinder radius="${radius_ouzel}" length="${height_ouzel}"/>
+                <cylinder radius="${radius_ouzel}" length="${height_ouzel}" />
             </geometry>
             <material name="">
-                <color rgba="1 1 1 1.0"/>
+                <color rgba="1 1 1 1.0" />
             </material>
         </visual>
     </link>
     <joint name="omav_to_rod" type="fixed">
-        <parent link="omav_base"/>
-        <child link="rod"/>
-        <origin rpy="$(arg omav_to_rod_angle) 0 0" xyz="${manipulator_length/2} 0.0 0.0"/>
+        <parent link="omav_base" />
+        <child link="rod" />
+        <origin rpy="$(arg omav_to_rod_angle) 0 0" xyz="${manipulator_length/2} 0.0 0.0" />
     </joint>
     <link name="rod">
         <collision>
-            <origin rpy="0 1.5708 0" xyz="0 0 0"/>
+            <origin rpy="0 1.5708 0" xyz="0 0 0" />
             <geometry>
-                <cylinder radius="${manipulator_radius}" length="${manipulator_length}"/>
+                <cylinder radius="${manipulator_radius}" length="${manipulator_length}" />
                 <!-- <box size="${manipulator_radius*2} ${manipulator_radius*2} ${manipulator_length}"/> -->
             </geometry>
         </collision>
         <visual>
-            <origin rpy="0 1.5708 0" xyz="0 0 0"/>
+            <origin rpy="0 1.5708 0" xyz="0 0 0" />
             <geometry>
-                <cylinder radius="${manipulator_radius}" length="${manipulator_length}"/>
+                <cylinder radius="${manipulator_radius}" length="${manipulator_length}" />
                 <!-- <box size="${manipulator_radius*2} ${manipulator_radius*2} ${manipulator_length}"/> -->
             </geometry>
             <material name="">
-                <color rgba="1 1 1 1"/>
+                <color rgba="1 1 1 1" />
             </material>
         </visual>
     </link>
     <joint name="rod_to_hook" type="fixed">
-        <parent link="rod"/>
-        <child link="hook"/>
-        <origin rpy="0 0 0" xyz="${manipulator_length/2} 0.0 -${tool_length/2}"/>
+        <parent link="rod" />
+        <child link="hook" />
+        <origin rpy="0 0 0" xyz="${manipulator_length/2} 0.0 -${tool_length/2}" />
     </joint>
     <!--
@@ -87,5 +91,5 @@
         </link>
 -->
-        <!-- <link name="tip">
+    <!-- <link name="tip">
             <collision>
                 <origin rpy="0 0 0" xyz="0 0 0"/>
@@ -107,29 +111,29 @@
             </visual>
         </link> -->
-        <!-- <joint name="tip_to_hook" type="fixed">
+    <!-- <joint name="tip_to_hook" type="fixed">
             <parent link="tip"/>
             <child link="hook"/>
             <origin rpy="0 0 0" xyz="0.0 0.0 -${tool_length/2}"/>
         </joint> -->
-        <link name="hook">
-            <collision>
-                <origin rpy="0 0 0" xyz="0 0 0"/>
-                <geometry>
-                    <cylinder radius="${tool_radius}" length="${tool_length}"/>
-                </geometry>
-                <material name="">
-                    <contact name="rubber"/>
-                </material>
-            </collision>
-            <visual>
-                <origin rpy="0 0 0" xyz="0 0 0"/>
-                <geometry>
-                    <cylinder radius="${tool_radius}" length="${tool_length}"/>
-                    <!-- <box size="${tool_radius*2} ${tool_radius*2} ${tool_length}"/> -->
-                </geometry>
-                <material name="">
-                    <color rgba="1 1 1 1"/>
-                </material>
-            </visual>
-        </link>
-    </robot>
+    <link name="hook">
+        <collision>
+            <origin rpy="0 0 0" xyz="0 0 0" />
+            <geometry>
+                <cylinder radius="${tool_radius}" length="${tool_length}" />
+            </geometry>
+            <material name="">
+                <contact name="rubber" />
+            </material>
+        </collision>
+        <visual>
+            <origin rpy="0 0 0" xyz="0 0 0" />
+            <geometry>
+                <cylinder radius="${tool_radius}" length="${tool_length}" />
+                <!-- <box size="${tool_radius*2} ${tool_radius*2} ${tool_length}"/> -->
+            </geometry>
+            <material name="">
+                <color rgba="1 1 1 1" />
+            </material>
+        </visual>
+    </link>
+</robot>

File: mppi_examples/mppi_omav_interaction/data/omav_pinocchio_hook.urdf.xacro (robot description, xacro)
@@ -2,35 +2,39 @@
 <robot xmlns:xacro="http://www.ros.org/wiki/xacro" name="omav_pinocchio_hook">
     <!-- Properties -->
-    <xacro:property name="manipulator_length" value="$(arg manipulator_length)"/>   <!-- [m] -->
-    <xacro:property name="manipulator_radius" value="0.0075"/>  <!-- [m] -->
-    <xacro:property name="tool_length" value="0.04"/>         <!-- [m] -->
-    <xacro:property name="tool_radius" value="0.0075"/>         <!-- [m] -->
-    <xacro:property name="mass_ouzel" value="4.337"/>
-    <xacro:property name="ixx_ouzel" value="0.078359"/>
-    <xacro:property name="iyy_ouzel" value="0.081797"/>
-    <xacro:property name="izz_ouzel" value="0.153355"/>
-    <xacro:property name="radius_ouzel" value="0.2"/>
-    <xacro:property name="height_ouzel" value="0.3"/>
-    <link name="world"/>
-    <link name="odom"/>
+    <xacro:property name="manipulator_length" value="$(arg manipulator_length)" />
+    <!-- [m] -->
+    <xacro:property name="manipulator_radius" value="0.0075" />
+    <!-- [m] -->
+    <xacro:property name="tool_length" value="0.04" />
+    <!-- [m] -->
+    <xacro:property name="tool_radius" value="0.0075" />
+    <!-- [m] -->
+    <xacro:property name="mass_ouzel" value="5.54" />
+    <xacro:property name="ixx_ouzel" value="0.1712" />
+    <xacro:property name="iyy_ouzel" value="0.1866" />
+    <xacro:property name="izz_ouzel" value="0.3253" />
+    <xacro:property name="radius_ouzel" value="0.48" />
+    <xacro:property name="height_ouzel" value="0.3" />
+    <link name="world" />
+    <link name="odom" />
     <joint name="odom_to_world" type="fixed">
-        <parent link="world"/>
-        <child link="odom"/>
+        <parent link="world" />
+        <child link="odom" />
     </joint>
     <joint name="odom_to_omav" type="floating">
-        <parent link="odom"/>
-        <child link="omav"/>
-        <origin rpy="0 0 0" xyz="0.0 0.0 0.0"/>
+        <parent link="odom" />
+        <child link="omav" />
+        <origin rpy="0 0 0" xyz="0.0 0.0 0.0" />
     </joint>
     <link name="omav">
         <inertial>
-            <mass value="${mass_ouzel}"/>
-            <origin rpy="0 0 0" xyz="0 0 0"/>
-            <inertia ixx="${ixx_ouzel}" ixy="0" ixz="0" iyy="${iyy_ouzel}" iyz="0" izz="${izz_ouzel}"/>
+            <mass value="${mass_ouzel}" />
+            <origin rpy="0 0 0" xyz="0 0 0" />
+            <inertia ixx="${ixx_ouzel}" ixy="0" ixz="0" iyy="${iyy_ouzel}" iyz="0" izz="${izz_ouzel}" />
         </inertial>
         <collision>
-            <origin rpy="0 0 0" xyz="0 0 0"/>
+            <origin rpy="0 0 0" xyz="0 0 0" />
             <geometry>
-                <cylinder radius="${radius_ouzel}" length="${height_ouzel}"/>
+                <cylinder radius="${radius_ouzel}" length="${height_ouzel}" />
             </geometry>
         </collision>
@@ -46,16 +50,16 @@
     </link>
     <joint name="omav_to_rod" type="fixed">
-        <parent link="omav"/>
-        <child link="rod"/>
-        <origin rpy="$(arg omav_to_rod_angle) 0 0" xyz="${manipulator_length/2} 0.0 0.0"/>
+        <parent link="omav" />
+        <child link="rod" />
+        <origin rpy="$(arg omav_to_rod_angle) 0 0" xyz="${manipulator_length/2} 0.0 0.0" />
     </joint>
     <link name="rod">
         <collision>
-            <origin rpy="0 1.5708 0" xyz="0 0 0"/>
+            <origin rpy="0 1.5708 0" xyz="0 0 0" />
             <geometry>
-                <cylinder radius="${manipulator_radius}" length="${manipulator_length}"/>
+                <cylinder radius="${manipulator_radius}" length="${manipulator_length}" />
             </geometry>
             <material name="">
-                <contact name="rubber"/>
+                <contact name="rubber" />
             </material>
         </collision>
@@ -71,16 +75,16 @@
     </link>
     <joint name="rod_to_tip" type="fixed">
-        <parent link="rod"/>
-        <child link="tip"/>
-        <origin rpy="0 0 0" xyz="${manipulator_length/2} 0.0 0.0"/>
+        <parent link="rod" />
+        <child link="tip" />
+        <origin rpy="0 0 0" xyz="${manipulator_length/2} 0.0 0.0" />
     </joint>
     <link name="tip">
         <collision>
-            <origin rpy="0 0 0" xyz="0 0 0"/>
+            <origin rpy="0 0 0" xyz="0 0 0" />
             <geometry>
-                <sphere radius="${manipulator_radius}"/>
+                <sphere radius="${manipulator_radius}" />
             </geometry>
             <material name="">
-                <contact name="rubber"/>
+                <contact name="rubber" />
             </material>
         </collision>
@@ -96,16 +100,16 @@
     </link>
     <joint name="tip_to_hook" type="fixed">
-        <parent link="tip"/>
-        <child link="hook"/>
-        <origin rpy="0 0 0" xyz="0.0 0.0 -${tool_length/2}"/>
+        <parent link="tip" />
+        <child link="hook" />
+        <origin rpy="0 0 0" xyz="0.0 0.0 -${tool_length/2}" />
     </joint>
     <link name="hook">
         <collision>
-            <origin rpy="0 0 0" xyz="0 0 0"/>
+            <origin rpy="0 0 0" xyz="0 0 0" />
             <geometry>
-                <cylinder radius="${tool_radius}" length="${tool_length}"/>
+                <cylinder radius="${tool_radius}" length="${tool_length}" />
             </geometry>
             <material name="">
-                <contact name="rubber"/>
+                <contact name="rubber" />
             </material>
         </collision>

File: mppi_examples/mppi_omav_interaction/data/omav_raisim_hook.urdf.xacro (robot description, xacro)
@@ -2,103 +2,107 @@
 <robot xmlns:xacro="http://www.ros.org/wiki/xacro" name="omav_raisim_hook">
     <!-- Properties -->
-    <xacro:property name="manipulator_length" value="$(arg manipulator_length)"/>   <!-- [m] -->
-    <xacro:property name="manipulator_radius" value="0.0075"/>  <!-- [m] -->
-    <xacro:property name="tool_length" value="0.04"/>         <!-- [m] -->
-    <xacro:property name="tool_radius" value="0.0075"/>         <!-- [m] -->
-    <xacro:property name="mass_ouzel" value="4.337"/>
-    <xacro:property name="ixx_ouzel" value="0.078359"/>
-    <xacro:property name="iyy_ouzel" value="0.081797"/>
-    <xacro:property name="izz_ouzel" value="0.153355"/>
-    <xacro:property name="radius_ouzel" value="0.2"/>
-    <xacro:property name="height_ouzel" value="0.3"/>
-    <link name="world"/>
-    <link name="odom"/>
+    <xacro:property name="manipulator_length" value="$(arg manipulator_length)" />
+    <!-- [m] -->
+    <xacro:property name="manipulator_radius" value="0.0075" />
+    <!-- [m] -->
+    <xacro:property name="tool_length" value="0.04" />
+    <!-- [m] -->
+    <xacro:property name="tool_radius" value="0.0075" />
+    <!-- [m] -->
+    <xacro:property name="mass_ouzel" value="5.54" />
+    <xacro:property name="ixx_ouzel" value="0.1712" />
+    <xacro:property name="iyy_ouzel" value="0.1866" />
+    <xacro:property name="izz_ouzel" value="0.3253" />
+    <xacro:property name="radius_ouzel" value="0.48" />
+    <xacro:property name="height_ouzel" value="0.3" />
+    <link name="world" />
+    <link name="odom" />
     <joint name="odom_to_world" type="fixed">
-        <parent link="world"/>
-        <child link="odom"/>
+        <parent link="world" />
+        <child link="odom" />
     </joint>
     <joint name="odom_to_omav_x" type="prismatic">
-        <parent link="odom"/>
-        <child link="omav_x"/>
-        <origin rpy="0 0 0" xyz="0.0 0.0 0.0"/>
-        <axis xyz="1 0 0"/>
-        <limit effort="1000.0" velocity="5.0" lower="-100" upper="100"/>
+        <parent link="odom" />
+        <child link="omav_x" />
+        <origin rpy="0 0 0" xyz="0.0 0.0 0.0" />
+        <axis xyz="1 0 0" />
+        <limit effort="1000.0" velocity="5.0" lower="-100" upper="100" />
     </joint>
-    <link name="omav_x"/>
+    <link name="omav_x" />
     <joint name="omav_x_to_omav_y" type="prismatic">
-        <parent link="omav_x"/>
-        <child link="omav_y"/>
-        <origin rpy="0 0 0" xyz="0.0 0.0 0.0"/>
-        <axis xyz="0 1 0"/>
-        <limit effort="1000.0" velocity="5.0" lower="-100" upper="100"/>
+        <parent link="omav_x" />
+        <child link="omav_y" />
+        <origin rpy="0 0 0" xyz="0.0 0.0 0.0" />
+        <axis xyz="0 1 0" />
+        <limit effort="1000.0" velocity="5.0" lower="-100" upper="100" />
     </joint>
-    <link name="omav_y"/>
+    <link name="omav_y" />
     <joint name="omav_y_to_omav_z" type="prismatic">
-        <parent link="omav_y"/>
-        <child link="omav_z"/>
-        <origin rpy="0 0 0" xyz="0.0 0.0 0.0"/>
-        <axis xyz="0 0 1"/>
-        <limit effort="1000.0" velocity="5.0" lower="-100" upper="100"/>
+        <parent link="omav_y" />
+        <child link="omav_z" />
+        <origin rpy="0 0 0" xyz="0.0 0.0 0.0" />
+        <axis xyz="0 0 1" />
+        <limit effort="1000.0" velocity="5.0" lower="-100" upper="100" />
     </joint>
-    <link name="omav_z"/>
+    <link name="omav_z" />
     <joint name="omav_z_to_omav" type="spherical">
-        <parent link="omav_z"/>
-        <child link="omav"/>
-        <origin rpy="0 0 0" xyz="0.0 0.0 0.0"/>
-        <axis xyz="0 1 0"/>
+        <parent link="omav_z" />
+        <child link="omav" />
+        <origin rpy="0 0 0" xyz="0.0 0.0 0.0" />
+        <axis xyz="0 1 0" />
     </joint>
     <link name="omav">
         <inertial>
-            <mass value="${mass_ouzel}"/>
-            <origin rpy="0 0 0" xyz="0 0 0"/>
-            <inertia ixx="${ixx_ouzel}" ixy="0" ixz="0" iyy="${iyy_ouzel}" iyz="0" izz="${izz_ouzel}"/>
+            <mass value="${mass_ouzel}" />
+            <origin rpy="0 0 0" xyz="0 0 0" />
+            <inertia ixx="${ixx_ouzel}" ixy="0" ixz="0" iyy="${iyy_ouzel}" iyz="0" izz="${izz_ouzel}" />
         </inertial>
         <collision>
-            <origin rpy="0 0 0" xyz="0 0 0"/>
+            <origin rpy="0 0 0" xyz="0 0 0" />
             <geometry>
-                <cylinder radius="${radius_ouzel}" length="${height_ouzel}"/>
+                <cylinder radius="${radius_ouzel}" length="${height_ouzel}" />
             </geometry>
         </collision>
         <visual>
-            <origin rpy="0 0 0" xyz="0 0 0"/>
+            <origin rpy="0 0 0" xyz="0 0 0" />
             <geometry>
-                <cylinder radius="${radius_ouzel}" length="${height_ouzel}"/>
+                <cylinder radius="${radius_ouzel}" length="${height_ouzel}" />
             </geometry>
             <material name="">
-                <color rgba="1 1 1 1"/>
+                <color rgba="1 1 1 1" />
             </material>
         </visual>
     </link>
     <joint name="omav_to_rod" type="fixed">
-        <parent link="omav"/>
-        <child link="rod"/>
-        <origin rpy="$(arg omav_to_rod_angle) 0 0" xyz="${manipulator_length/2} 0.0 0.0"/>
+        <parent link="omav" />
+        <child link="rod" />
+        <origin rpy="$(arg omav_to_rod_angle) 0 0" xyz="${manipulator_length/2} 0.0 0.0" />
     </joint>
     <link name="rod">
         <collision>
-            <origin rpy="0 1.5708 0" xyz="0 0 0"/>
+            <origin rpy="0 1.5708 0" xyz="0 0 0" />
             <geometry>
-                <cylinder radius="${manipulator_radius}" length="${manipulator_length}"/>
+                <cylinder radius="${manipulator_radius}" length="${manipulator_length}" />
                 <!-- <box size="${manipulator_radius*2} ${manipulator_radius*2} ${manipulator_length}"/> -->
             </geometry>
             <material name="">
-                <contact name="steel"/>
+                <contact name="steel" />
             </material>
         </collision>
         <visual>
-            <origin rpy="0 1.5708 0" xyz="0 0 0"/>
+            <origin rpy="0 1.5708 0" xyz="0 0 0" />
             <geometry>
-                <cylinder radius="${manipulator_radius}" length="${manipulator_length}"/>
+                <cylinder radius="${manipulator_radius}" length="${manipulator_length}" />
                 <!-- <box size="${manipulator_radius*2} ${manipulator_radius*2} ${manipulator_length}"/> -->
             </geometry>
             <material name="">
-                <color rgba="1 1 1 1"/>
+                <color rgba="1 1 1 1" />
             </material>
         </visual>
     </link>
     <joint name="rod_to_hook" type="fixed">
-        <parent link="rod"/>
-        <child link="hook"/>
-        <origin rpy="0 0 0" xyz="${manipulator_length/2} 0.0 -${tool_length/2}"/>
+        <parent link="rod" />
+        <child link="hook" />
+        <origin rpy="0 0 0" xyz="${manipulator_length/2} 0.0 -${tool_length/2}" />
     </joint>
     <!-- <link name="tip">
@@ -122,5 +126,5 @@
         </visual>
     </link> -->
-<!--
+    <!--
     <joint name="tip_to_thick" type="fixed">
         <parent link="tip"/>
@@ -156,21 +160,21 @@
     <link name="hook">
         <collision>
-            <origin rpy="0 0 0" xyz="0 0 0"/>
+            <origin rpy="0 0 0" xyz="0 0 0" />
             <geometry>
-                <cylinder radius="${tool_radius}" length="${tool_length}"/>
+                <cylinder radius="${tool_radius}" length="${tool_length}" />
                 <!-- <box size="${tool_radius*2} ${tool_radius*2} ${tool_length}"/> -->
             </geometry>
             <material name="">
-                <contact name="steel"/>
+                <contact name="steel" />
             </material>
         </collision>
         <visual>
-            <origin rpy="0 0 0" xyz="0 0 0"/>
+            <origin rpy="0 0 0" xyz="0 0 0" />
             <geometry>
-                <cylinder radius="${tool_radius}" length="${tool_length}"/>
+                <cylinder radius="${tool_radius}" length="${tool_length}" />
                 <!-- <box size="${tool_radius*2} ${tool_radius*2} ${tool_length}"/> -->
             </geometry>
             <material name="">
-                <color rgba="1 1 1 1"/>
+                <color rgba="1 1 1 1" />
             </material>
         </visual>
