Commit message: fix: update all vehicle parameters to values of real drone

File: mppi_examples/mppi_omav_interaction/data/omav_hook_visualization.urdf.xacro (robot description, xacro)
@@ -6,5 +6,5 @@
     <xacro:property name="manipulator_radius" value="0.0075" />
     <!-- [m] -->
-    <xacro:property name="tool_length" value="0.04" />
+    <xacro:property name="tool_length" value="0.05" />
     <!-- [m] -->
     <xacro:property name="tool_radius" value="0.0075" />
@@ -38,5 +38,5 @@
         <parent link="omav_base" />
         <child link="rod" />
-        <origin rpy="$(arg omav_to_rod_angle) 0 0" xyz="${manipulator_length/2} 0.0 0.0" />
+        <origin rpy="$(arg omav_to_rod_angle) 0 0" xyz="${manipulator_length/2} -0.02 0.11" />
     </joint>
     <link name="rod">

File: mppi_examples/mppi_omav_interaction/data/omav_pinocchio_hook.urdf.xacro (robot description, xacro)
@@ -6,12 +6,12 @@
     <xacro:property name="manipulator_radius" value="0.0075" />
     <!-- [m] -->
-    <xacro:property name="tool_length" value="0.04" />
+    <xacro:property name="tool_length" value="0.05" />
     <!-- [m] -->
     <xacro:property name="tool_radius" value="0.0075" />
     <!-- [m] -->
-    <xacro:property name="mass_ouzel" value="5.54" />
-    <xacro:property name="ixx_ouzel" value="0.1712" />
-    <xacro:property name="iyy_ouzel" value="0.1866" />
-    <xacro:property name="izz_ouzel" value="0.3253" />
+    <xacro:property name="mass_ouzel" value="5.459" />
+    <xacro:property name="ixx_ouzel" value="0.18" />
+    <xacro:property name="iyy_ouzel" value="0.18" />
+    <xacro:property name="izz_ouzel" value="0.27945" />
     <xacro:property name="radius_ouzel" value="0.48" />
     <xacro:property name="height_ouzel" value="0.3" />
@@ -52,5 +52,5 @@
         <parent link="omav" />
         <child link="rod" />
-        <origin rpy="$(arg omav_to_rod_angle) 0 0" xyz="${manipulator_length/2} 0.0 0.0" />
+        <origin rpy="$(arg omav_to_rod_angle) 0 0" xyz="${manipulator_length/2} -0.02 0.11" />
     </joint>
     <link name="rod">

File: mppi_examples/mppi_omav_interaction/data/omav_raisim_hook.urdf.xacro (robot description, xacro)
@@ -6,12 +6,12 @@
     <xacro:property name="manipulator_radius" value="0.0075" />
     <!-- [m] -->
-    <xacro:property name="tool_length" value="0.04" />
+    <xacro:property name="tool_length" value="0.05" />
     <!-- [m] -->
     <xacro:property name="tool_radius" value="0.0075" />
     <!-- [m] -->
-    <xacro:property name="mass_ouzel" value="5.54" />
-    <xacro:property name="ixx_ouzel" value="0.1712" />
-    <xacro:property name="iyy_ouzel" value="0.1866" />
-    <xacro:property name="izz_ouzel" value="0.3253" />
+    <xacro:property name="mass_ouzel" value="5.459" />
+    <xacro:property name="ixx_ouzel" value="0.18" />
+    <xacro:property name="iyy_ouzel" value="0.18" />
+    <xacro:property name="izz_ouzel" value="0.27945" />
     <xacro:property name="radius_ouzel" value="0.48" />
     <xacro:property name="height_ouzel" value="0.3" />
@@ -77,5 +77,5 @@
         <parent link="omav" />
         <child link="rod" />
-        <origin rpy="$(arg omav_to_rod_angle) 0 0" xyz="${manipulator_length/2} 0.0 0.0" />
+        <origin rpy="$(arg omav_to_rod_angle) 0 0" xyz="${manipulator_length/2} -0.02 0.11" />
     </joint>
     <link name="rod">
