Commit message: Velocity and Forces added in the cost function.

File: mppi_examples/mppi_omav_interaction/data/objects/linear_drawer.urdf.xacro (robot description, xacro)
@@ -114,5 +114,5 @@
         <axis xyz="1 0 0"/>
         <limit effort="1000.0" velocity="5.0" lower="-0.5" upper="0.0"/>
-        <dynamics spring_mount="0 0 0" stiffness="0.0" damping="0.5"/>
+        <dynamics damping="2.0" friction="4.0"/>
     </joint>
     <link name="drawer">
@@ -141,5 +141,5 @@
         <parent link="drawer"/>
         <child link="handle"/>
-        <origin rpy="1.5708 0 0" xyz="-0.3 0.0 0.0"/>
+        <origin rpy="0 0 0" xyz="-0.3 0.0 0.0"/>
     </joint>
     <link name="handle">
