Commit message: New Costfunctin, torque and efficiency penalized. Tunable using rqt_reconfigure.

File: mppi_examples/mppi_omav_interaction/data/objects/door.urdf.xacro (robot description, xacro)
@@ -25,6 +25,6 @@
         <origin rpy="0 0 0" xyz="0 0.25 0.0"/>
         <axis xyz="0 0 1"/>
-        <limit effort="100.0" velocity="1.5" lower="-1.57" upper="0.1"/>
-        <dynamics damping="1.0" friction="4.0"/>
+        <limit effort="100.0" velocity="1.5" lower="-2" upper="0.0"/>
+        <dynamics damping="4.0" friction="1.0"/>
     </joint>
     <link name="hinge"/>

Commit message: Finalized new more physical cost functions. Jumps in torque that need to be fixed still.

File: mppi_examples/mppi_omav_interaction/data/objects/door.urdf.xacro (robot description, xacro)
@@ -2,5 +2,5 @@
 <robot xmlns:xacro="http://www.ros.org/wiki/xacro" name="cube">
     <xacro:property name="mass_cube" value="0.5"/>
-    <xacro:property name="dimension_cube" value="0.3"/>
+    <xacro:property name="door_handle_distance" value="-0.1"/>
     <link name="world"/>
     <joint name="world_wall" type="fixed">
@@ -56,8 +56,8 @@
         </visual>
     </link>
-    <joint name="drawer_handle" type="fixed">
+    <joint name="door_handle" type="fixed">
         <parent link="door"/>
         <child link="handle"/>
-        <origin rpy="0 0 0" xyz="-0.1 0.0 0.0"/>
+        <origin rpy="0 0 0" xyz="${door_handle_distance} -0.15 0.0"/>
     </joint>
     <link name="handle">
@@ -81,4 +81,10 @@
         </visual>
     </link>
+    <joint name="handle_ref" type="fixed">
+        <parent link="handle"/>
+        <child link="handle_ref"/>
+        <origin rpy="0 0 0" xyz="${-door_handle_distance/2} 0.0 0.0"/>
+    </joint>
+    <link name="handle_ref" />
     <joint name="handle_left" type="fixed">
         <parent link="handle"/>
