Commit message: Working version for opening the door on the omav framework.

File: mppi_examples/mppi_omav_interaction/data/objects/button.urdf.xacro (robot description, xacro)
@@ -9,5 +9,11 @@
         <origin rpy="0 0 0" xyz="2.0 0.0 1.0"/>
     </joint>
-    <link name="odom_button"/>
+    <link name="odom_button">
+        <inertial>
+            <mass value="${mass_cube}"/>
+            <origin rpy="0 0 0" xyz="0 0 0"/>
+            <inertia ixx="0.12" ixy="0" ixz="0" iyy="0.14" iyz="0" izz="0.18"/>
+        </inertial>
+    </link>
     <joint name="articulation_joint" type="prismatic">
         <parent link="odom_button"/>

File: mppi_examples/mppi_omav_interaction/data/objects/shelf.urdf.xacro (robot description, xacro)
@@ -33,4 +33,10 @@
         </joint>
     </xacro:if>
+    <gazebo>
+        <plugin name="gazebo_ros_control" filename="libgazebo_ros_control.so">
+            <robotNamespace>/shelf</robotNamespace>
+            <robotParam>urdf_object </robotParam>
+        </plugin>
+    </gazebo>
     <link name="shelf">
         <xacro:box_inertia m="5" x="${door_width}" y="${door_length}" z="${shelf_z}"/>
@@ -44,10 +50,4 @@
             </material>
         </visual>
-        <collision>
-            <origin rpy="0 0 0" xyz="0 -${door_length/2} ${-shelf_z/2}"/>
-            <geometry>
-                <box size="${door_width} ${door_length} ${shelf_z}"/>
-            </geometry>
-        </collision>
     </link>
     <link name="door">
@@ -72,12 +72,23 @@
         </collision>
     </link>
-    <link name="door_hinge"/>
+    <link name="door_hinge">
+        <inertial>
+            <mass value="0.01"/>
+            <origin rpy="0 0 0" xyz="0 0 0"/>
+            <inertia ixx="0.0" ixy="0.0" ixz="0.0" iyy="0.0" iyz="0.0" izz="0.0"/>
+        </inertial>
+    </link>
     <joint name="door_hinge_joint" type="fixed">
         <parent link="shelf"/>
         <child link="door_hinge"/>
-        <dynamics damping="2.0" friction="8.0"/>
         <origin xyz="0 -${door_length} ${door_height/2}"/>
     </joint>
-    <link name="axis_link"/>
+    <link name="axis_link">
+        <inertial>
+            <mass value="0.01"/>
+            <origin rpy="0 0 0" xyz="0 0 0"/>
+            <inertia ixx="0.0" ixy="0.0" ixz="0.0" iyy="0.0" iyz="0.0" izz="0.0"/>
+        </inertial>
+    </link>
     <joint name="axis_joint" type="fixed">
         <parent link="door_hinge"/>
@@ -88,5 +99,5 @@
         <parent link="axis_link"/>
         <child link="measured_joint_link"/>
-        <dynamics damping="2.0" friction="4.0"/>
+        <dynamics damping="2.0" friction="0.5"/>
         <origin xyz="0 0 0"/>
         <axis xyz="0 0 -1"/>
@@ -105,5 +116,5 @@
         </inertial>
         <visual>
-            <origin rpy="1.57 0 0" xyz="0 0 0"/>
+            <origin rpy="0 0 0" xyz="0 0 0"/>
             <geometry>
                 <box size="0.01 0.01 ${handle_length+0.01}"/>
@@ -114,5 +125,5 @@
         </visual>
         <collision>
-            <origin rpy="1.57 0 0" xyz="0 0 0"/>
+            <origin rpy="0 0 0" xyz="0 0 0"/>
             <geometry>
                 <box size="0.01 0.01 ${handle_length+0.01}"/>
@@ -138,5 +149,4 @@
             </material>
         </visual>
-        <!--
         <collision>
             <origin rpy="0 0 0" xyz="0 0 0"/>
@@ -148,5 +158,4 @@
             </material>
         </collision>
-        -->
     </link>
     <link name="handle_support_right">
@@ -165,5 +174,4 @@
             </material>
         </visual>
-        <!--
         <collision>
             <origin rpy="0 0 0" xyz="0 0 0"/>
@@ -175,5 +183,4 @@
             </material>
         </collision>
-        -->
     </link>
     <joint name="handle_joint" type="fixed">
@@ -189,17 +196,35 @@
                 rpy="0 0 0"/> <!-- height handle + half the width door, 0.30 minus some offset -->
     </joint>
-    <link name="handle_ref"/>
+    <link name="handle_ref">
+        <inertial>
+            <mass value="0.01"/>
+            <origin rpy="0 0 0" xyz="0 0 0"/>
+            <inertia ixx="0.0" ixy="0.0" ixz="0.0" iyy="0.0" iyz="0.0" izz="0.0"/>
+        </inertial>
+    </link>
     <joint name="handle_support_left_joint" type="fixed">
         <parent link="handle_link"/>
         <child link="handle_support_left"/>
-        <origin xyz="-${handle_height/2} -${handle_length/2} 0" rpy="0 0 0"/>
+        <origin xyz="-${handle_height/2} 0 -${handle_length/2}" rpy="0 0 0"/>
     </joint>
     <joint name="handle_support_right_joint" type="fixed">
         <parent link="handle_link"/>
         <child link="handle_support_right"/>
-        <origin xyz="-${handle_height/2} ${handle_length/2} 0" rpy="0 0 0"/>
-    </joint>
-    <link name="measured_joint_link"/>
-    <link name="measured_joint_link_test"/>
+        <origin xyz="-${handle_height/2} 0 ${handle_length/2}" rpy="0 0 0"/>
+    </joint>
+    <link name="measured_joint_link">
+        <inertial>
+            <mass value="0.01"/>
+            <origin rpy="0 0 0" xyz="0 0 0"/>
+            <inertia ixx="0.0" ixy="0.0" ixz="0.0" iyy="0.0" iyz="0.0" izz="0.0"/>
+        </inertial>
+    </link>
+    <link name="measured_joint_link_test">
+        <inertial>
+            <mass value="0.01"/>
+            <origin rpy="0 0 0" xyz="0 0 0"/>
+            <inertia ixx="0.0" ixy="0.0" ixz="0.0" iyy="0.0" iyz="0.0" izz="0.0"/>
+        </inertial>
+    </link>
     <joint name="measured_test_handle_joint" type="fixed">
         <parent link="handle_link"/>
@@ -207,3 +232,13 @@
         <origin xyz="-0.06 -0.243 0.0" rpy="0 0 0"/>
     </joint>
+    <transmission name="hinge">
+        <type>transmission_interface/SimpleTransmission</type>
+        <joint name="articulation_joint">
+            <hardwareInterface>EffortJointInterface</hardwareInterface>
+        </joint>
+        <actuator name="motor1">
+            <hardwareInterface>EffortJointInterface</hardwareInterface>
+            <mechanicalReduction>1</mechanicalReduction>
+        </actuator>
+    </transmission>
 </robot>

File: mppi_examples/mppi_omav_interaction/data/omav_hook_visualization.urdf.xacro (robot description, xacro)
@@ -1,4 +1,4 @@
 <?xml version="1.0"?>
-<robot xmlns:xacro="http://www.ros.org/wiki/xacro" name="ouzel">
+<robot xmlns:xacro="http://www.ros.org/wiki/xacro" name="omav_hook_visualization">
     <xacro:property name="mass_ouzel" value="5.0"/>
     <xacro:property name="ixx_ouzel" value="0.12"/>
@@ -39,5 +39,5 @@
             <origin rpy="0 1.5708 0" xyz="0 0 0"/>
             <geometry>
-                <cylinder radius="0.015" length="0.54"/>
+                <cylinder radius="0.0075" length="0.54"/>
             </geometry>
         </collision>
@@ -45,5 +45,5 @@
             <origin rpy="0 1.5708 0" xyz="0 0 0"/>
             <geometry>
-                <cylinder radius="0.015" length="0.54"/>
+                <cylinder radius="0.0075" length="0.54"/>
             </geometry>
             <material name="">
@@ -70,5 +70,5 @@
             <origin rpy="0 0 0" xyz="0 0.0 0"/>
             <geometry>
-                <sphere radius="0.015"/>
+                <sphere radius="0.0075"/>
             </geometry>
             <material name="">
@@ -86,5 +86,5 @@
             <origin rpy="0 0 0" xyz="0 0 0"/>
             <geometry>
-                <cylinder radius="0.015" length="0.05"/>
+                <cylinder radius="0.0075" length="0.05"/>
             </geometry>
             <material name="">
@@ -95,5 +95,5 @@
             <origin rpy="0 0 0" xyz="0 0 0"/>
             <geometry>
-                <cylinder radius="0.015" length="0.05"/>
+                <cylinder radius="0.0075" length="0.05"/>
             </geometry>
             <material name="">

File: mppi_examples/mppi_omav_interaction/data/omav_pinocchio_hook.urdf.xacro (robot description, xacro)
@@ -1,4 +1,4 @@
 <?xml version="1.0"?>
-<robot xmlns:xacro="http://www.ros.org/wiki/xacro" name="ouzel_raisim">
+<robot xmlns:xacro="http://www.ros.org/wiki/xacro" name="omav_pinocchio_hook">
     <xacro:property name="mass_ouzel" value="5.0"/>
     <xacro:property name="ixx_ouzel" value="0.12"/>

File: mppi_examples/mppi_omav_interaction/data/omav_raisim_hook.urdf.xacro (robot description, xacro)
@@ -1,4 +1,4 @@
 <?xml version="1.0"?>
-<robot xmlns:xacro="http://www.ros.org/wiki/xacro" name="ouzel_raisim">
+<robot xmlns:xacro="http://www.ros.org/wiki/xacro" name="omav_raisim_hook">
     <xacro:property name="mass_ouzel" value="5.0"/>
     <xacro:property name="ixx_ouzel" value="0.12"/>
@@ -74,5 +74,5 @@
             <origin rpy="0 1.5708 0" xyz="0 0 0"/>
             <geometry>
-                <cylinder radius="0.015" length="0.54"/>
+                <cylinder radius="0.0075" length="0.54"/>
             </geometry>
             <material name="">
@@ -83,5 +83,5 @@
             <origin rpy="0 1.5708 0" xyz="0 0 0"/>
             <geometry>
-                <cylinder radius="0.015" length="0.54"/>
+                <cylinder radius="0.0075" length="0.54"/>
             </geometry>
             <material name="">
@@ -99,5 +99,5 @@
             <origin rpy="0 0 0" xyz="0 0 0"/>
             <geometry>
-                <sphere radius="0.015"/>
+                <sphere radius="0.0075"/>
             </geometry>
             <material name="">
@@ -108,5 +108,5 @@
             <origin rpy="0 0 0" xyz="0 0.0 0"/>
             <geometry>
-                <sphere radius="0.015"/>
+                <sphere radius="0.0075"/>
             </geometry>
             <material name="">
@@ -124,5 +124,5 @@
             <origin rpy="0 0 0" xyz="0 0 0"/>
             <geometry>
-                <cylinder radius="0.015" length="0.05"/>
+                <cylinder radius="0.0075" length="0.05"/>
             </geometry>
             <material name="">
@@ -133,5 +133,5 @@
             <origin rpy="0 0 0" xyz="0 0 0"/>
             <geometry>
-                <cylinder radius="0.015" length="0.05"/>
+                <cylinder radius="0.0075" length="0.05"/>
             </geometry>
             <material name="">
