Commit message: Working version with double integrator and smooth trajectories.

File: mppi_examples/mppi_omav_interaction/data/objects/shelf.urdf.xacro (robot description, xacro)
@@ -99,5 +99,5 @@
         <parent link="axis_link"/>
         <child link="measured_joint_link"/>
-        <dynamics damping="2.0" friction="10.0"/>
+        <dynamics damping="5.0" friction="10.0"/>
         <origin xyz="0 0 0"/>
         <axis xyz="0 0 -1"/>
@@ -155,5 +155,5 @@
             </geometry>
             <material name="">
-                <contact name="steel"/>
+                <contact name="rubber"/>
             </material>
         </collision>
@@ -180,5 +180,5 @@
             </geometry>
             <material name="">
-                <contact name="steel"/>
+                <contact name="rubber"/>
             </material>
         </collision>

File: mppi_examples/mppi_omav_interaction/data/omav_hook_visualization.urdf.xacro (robot description, xacro)
@@ -62,73 +62,75 @@
         <origin rpy="0 0 0" xyz="${manipulator_length/2} 0.0 0.0"/>
     </joint>
-    <joint name="tip_to_thick" type="fixed">
-        <parent link="tip"/>
-        <child link="thick"/>
-        <origin rpy="0 0 0" xyz="-0.02 0.0 0.0"/>
-    </joint>
-    <link name="thick">
-        <collision>
-            <origin rpy="0 1.5708 0" xyz="0 0 0"/>
-            <geometry>
-                <cylinder radius="0.015" length="0.055"/>
-            </geometry>
-            <material name="">
-                <contact name="rubber"/>
-            </material>
-        </collision>
-        <visual>
-            <origin rpy="0 1.5708 0" xyz="0 0 0"/>
-            <geometry>
-                <cylinder radius="0.015" length="0.055"/>
-            </geometry>
-            <material name="">
-                <color rgba="1 1 1 1"/>
-            </material>
-        </visual>
-    </link>
-    <link name="tip">
-        <collision>
-            <origin rpy="0 0 0" xyz="0 0 0"/>
-            <geometry>
-                <sphere radius="${tool_radius}"/>
-            </geometry>
-            <material name="">
-                <contact name="rubber"/>
-            </material>
-        </collision>
-        <visual>
-            <origin rpy="0 0 0" xyz="0 0.0 0"/>
-            <geometry>
-                <sphere radius="${tool_radius}"/>
-            </geometry>
-            <material name="">
-                <color rgba="1 1 1 1"/>
-            </material>
-        </visual>
-    </link>
-    <joint name="tip_to_hook" type="fixed">
-        <parent link="tip"/>
-        <child link="hook"/>
-        <origin rpy="0 0 0" xyz="0.0 0.0 -${tool_length/2}"/>
-    </joint>
-    <link name="hook">
-        <collision>
-            <origin rpy="0 0 0" xyz="0 0 0"/>
-            <geometry>
-                <cylinder radius="${tool_radius}" length="${tool_length}"/>
-            </geometry>
-            <material name="">
-                <contact name="rubber"/>
-            </material>
-        </collision>
-        <visual>
-            <origin rpy="0 0 0" xyz="0 0 0"/>
-            <geometry>
-                <cylinder radius="${tool_radius}" length="${tool_length}"/>
-            </geometry>
-            <material name="">
-                <color rgba="1 1 1 1"/>
-            </material>
-        </visual>
-    </link>
-</robot>
+    <!--
+        <joint name="tip_to_thick" type="fixed">
+            <parent link="tip"/>
+            <child link="thick"/>
+            <origin rpy="0 0 0" xyz="-0.04 0.0 0.0"/>
+        </joint>
+        <link name="thick">
+            <collision>
+                <origin rpy="0 1.5708 0" xyz="0 0 0"/>
+                <geometry>
+                    <cylinder radius="0.015" length="0.095"/>
+                </geometry>
+                <material name="">
+                    <contact name="rubber"/>
+                </material>
+            </collision>
+            <visual>
+                <origin rpy="0 1.5708 0" xyz="0 0 0"/>
+                <geometry>
+                    <cylinder radius="0.015" length="0.095"/>
+                </geometry>
+                <material name="">
+                    <color rgba="1 1 1 1"/>
+                </material>
+            </visual>
+        </link>
+-->
+        <link name="tip">
+            <collision>
+                <origin rpy="0 0 0" xyz="0 0 0"/>
+                <geometry>
+                    <sphere radius="${tool_radius}"/>
+                </geometry>
+                <material name="">
+                    <contact name="rubber"/>
+                </material>
+            </collision>
+            <visual>
+                <origin rpy="0 0 0" xyz="0 0.0 0"/>
+                <geometry>
+                    <sphere radius="${tool_radius}"/>
+                </geometry>
+                <material name="">
+                    <color rgba="1 1 1 1"/>
+                </material>
+            </visual>
+        </link>
+        <joint name="tip_to_hook" type="fixed">
+            <parent link="tip"/>
+            <child link="hook"/>
+            <origin rpy="0 0 0" xyz="0.0 0.0 -${tool_length/2}"/>
+        </joint>
+        <link name="hook">
+            <collision>
+                <origin rpy="0 0 0" xyz="0 0 0"/>
+                <geometry>
+                    <cylinder radius="${tool_radius}" length="${tool_length}"/>
+                </geometry>
+                <material name="">
+                    <contact name="rubber"/>
+                </material>
+            </collision>
+            <visual>
+                <origin rpy="0 0 0" xyz="0 0 0"/>
+                <geometry>
+                    <cylinder radius="${tool_radius}" length="${tool_length}"/>
+                </geometry>
+                <material name="">
+                    <color rgba="1 1 1 1"/>
+                </material>
+            </visual>
+        </link>
+    </robot>

File: mppi_examples/mppi_omav_interaction/data/omav_raisim_hook.urdf.xacro (robot description, xacro)
@@ -120,8 +120,9 @@
         </visual>
     </link>
+<!--
     <joint name="tip_to_thick" type="fixed">
         <parent link="tip"/>
         <child link="thick"/>
-        <origin rpy="0 0 0" xyz="-0.02 0.0 0.0"/>
+        <origin rpy="0 0 0" xyz="-0.04 0.0 0.0"/>
     </joint>
     <link name="thick">
@@ -129,5 +130,5 @@
             <origin rpy="0 1.5708 0" xyz="0 0 0"/>
             <geometry>
-                <cylinder radius="0.015" length="0.055"/>
+                <cylinder radius="0.015" length="0.095"/>
             </geometry>
             <material name="">
@@ -138,5 +139,5 @@
             <origin rpy="0 1.5708 0" xyz="0 0 0"/>
             <geometry>
-                <cylinder radius="0.015" length="0.055"/>
+                <cylinder radius="0.015" length="0.095"/>
             </geometry>
             <material name="">
@@ -145,4 +146,5 @@
         </visual>
     </link>
+-->
     <joint name="tip_to_hook" type="fixed">
         <parent link="tip"/>

Commit message: Beginning to improve a better shift of the inputs in order to fix acceleration reset.

File: mppi_examples/mppi_omav_interaction/data/objects/shelf.urdf.xacro (robot description, xacro)
@@ -104,5 +104,5 @@
         <parent link="axis_link"/>
         <child link="measured_joint_link"/>
-        <dynamics damping="5.0" friction="10.0"/>
+        <dynamics damping="0.1" friction="1.0"/>
         <origin xyz="0 0 0"/>
         <axis xyz="0 0 -1"/>

Commit message: Slight change in cost function, at force cost.

File: mppi_examples/mppi_omav_interaction/data/objects/shelf.urdf.xacro (robot description, xacro)
@@ -35,5 +35,5 @@
             <parent link="world"/>
             <child link="shelf"/>
-            <origin xyz="${shelf_x} ${shelf_y} ${shelf_z}" rpy="0.009 0.001 1.645"/>
+            <origin xyz="${shelf_x} ${shelf_y} ${shelf_z}" rpy="-0.009 0.0 1.645"/>
         </joint>
     </xacro:if>

Commit message: Added feedforward terms and quadratic Cost on force. Additionally changed shelf parameters.

File: mppi_examples/mppi_omav_interaction/data/objects/shelf.urdf.xacro (robot description, xacro)
@@ -20,5 +20,5 @@
     <xacro:macro name="box_inertia" params="m x y z">
         <inertial>
-            <origin rpy="0 0 0" xyz="0 0 0"/>
+            <origin rpy="0 0 0" xyz="0 ${-y/2} 0"/>
             <mass value="${m}"/>
             <inertia ixx="${0.0833 * m * (y**2 + z**2)}"
@@ -27,5 +27,5 @@
                      iyy="${0.0833 * m * (x**2 + z**2)}"
                      iyz="0"
-                     izz="${0.0833 * m * (z**2 + y**2)}"/>
+                     izz="${0.0833 * m * (x**2 + y**2)}"/>
         </inertial>
     </xacro:macro>
@@ -35,5 +35,5 @@
             <parent link="world"/>
             <child link="shelf"/>
-            <origin xyz="${shelf_x} ${shelf_y} ${shelf_z}" rpy="-0.009 0.0 1.645"/>
+            <origin xyz="${shelf_x} ${shelf_y} ${shelf_z}" rpy="0.0 0.0 1.645"/>
         </joint>
     </xacro:if>
@@ -57,5 +57,5 @@
     </link>
     <link name="door">
-        <xacro:box_inertia m="5.8" x="${door_width}" y="${door_length}" z="${door_height}"/>
+        <xacro:box_inertia m="3.0" x="${door_width}" y="${door_length}" z="${door_height}"/>
         <visual>
             <origin rpy="0 0 0" xyz="${-door_width/2} ${door_length/2} 0"/>
@@ -104,8 +104,8 @@
         <parent link="axis_link"/>
         <child link="measured_joint_link"/>
-        <dynamics damping="0.1" friction="1.0"/>
+        <dynamics damping="0.0" friction="0.0"/>
         <origin xyz="0 0 0"/>
         <axis xyz="0 0 -1"/>
-        <limit effort="100" lower="0" upper="1.57" velocity="10.0"/>
+        <limit effort="100" lower="0" upper="1.75" velocity="10.0"/>
     </joint>
     <joint name="door_link" type="fixed">

File: mppi_examples/mppi_omav_interaction/data/objects/shelf_gazebo.urdf.xacro (robot description, xacro)
@@ -20,5 +20,5 @@
     <xacro:macro name="box_inertia" params="m x y z">
         <inertial>
-            <origin rpy="0 0 0" xyz="0 0 0"/>
+            <origin rpy="0 0 0" xyz="0 ${-y/2} 0"/>
             <mass value="${m}"/>
             <inertia ixx="${0.0833 * m * (y**2 + z**2)}"
@@ -27,5 +27,5 @@
                      iyy="${0.0833 * m * (x**2 + z**2)}"
                      iyz="0"
-                     izz="${0.0833 * m * (z**2 + y**2)}"/>
+                     izz="${0.0833 * m * (x**2 + y**2)}"/>
         </inertial>
     </xacro:macro>
@@ -35,5 +35,5 @@
             <parent link="world"/>
             <child link="shelf"/>
-            <origin xyz="${shelf_x} ${shelf_y} ${shelf_z}" rpy="0.009 0.001 1.645"/>
+            <origin xyz="${shelf_x} ${shelf_y} ${shelf_z}" rpy="0.0 0.0 1.645"/>
         </joint>
     </xacro:if>
@@ -57,5 +57,5 @@
     </link>
     <link name="door">
-        <xacro:box_inertia m="5.8" x="${door_width}" y="${door_length}" z="${door_height}"/>
+        <xacro:box_inertia m="3.0" x="${door_width}" y="${door_length}" z="${door_height}"/>
         <visual>
             <origin rpy="0 0 0" xyz="${-door_width/2} ${door_length/2} 0"/>
@@ -104,8 +104,8 @@
         <parent link="axis_link"/>
         <child link="measured_joint_link"/>
-        <dynamics damping="1.5" friction="0.1"/>
+        <dynamics damping="0.0" friction="0.0"/>
         <origin xyz="0 0 0"/>
         <axis xyz="0 0 -1"/>
-        <limit effort="100" lower="0" upper="1.57" velocity="10.0"/>
+        <limit effort="100" lower="0" upper="1.8" velocity="10.0"/>
     </joint>
     <joint name="door_link" type="fixed">

File: mppi_examples/mppi_omav_interaction/data/omav_raisim_hook.urdf.xacro (robot description, xacro)
@@ -6,5 +6,5 @@
     <xacro:property name="tool_length" value="0.05"/>         <!-- [m] -->
     <xacro:property name="tool_radius" value="0.0075"/>         <!-- [m] -->
-    <xacro:property name="mass_ouzel" value="5.0"/>
+    <xacro:property name="mass_ouzel" value="4.337"/>
     <xacro:property name="ixx_ouzel" value="0.12"/>
     <xacro:property name="iyy_ouzel" value="0.14"/>

Commit message: refactor: set same shelf pose from launch file for all three shelf descriptions

File: mppi_examples/mppi_omav_interaction/data/objects/shelf.urdf.xacro (robot description, xacro)
@@ -3,4 +3,8 @@
     <xacro:arg name="fixed" default="true"/>
     <xacro:arg name="height" default="0.0"/>
+    <xacro:arg name="shelf_x" default="-0.242"/>
+    <xacro:arg name="shelf_y" default="-0.595"/>
+    <xacro:arg name="shelf_z" default="0.834"/>
+    <xacro:arg name="shelf_orientation" default="0.0 0.0 1.645"/>
     <xacro:property name="height" default="$(arg height)"/>
     <xacro:property name="door_length" default="0.359"/>
@@ -15,7 +19,8 @@
     <xacro:property name="handle_offset_y" default="0.338"/>
     <xacro:property name="handle_offset_z" default="-0.024"/>
-    <xacro:property name="shelf_x" default="-0.242"/>
-    <xacro:property name="shelf_y" default="-0.595"/>
-    <xacro:property name="shelf_z" default="0.834"/>
+    <xacro:property name="shelf_x" default="$(arg shelf_x)"/>
+    <xacro:property name="shelf_y" default="$(arg shelf_y)"/>
+    <xacro:property name="shelf_z" default="$(arg shelf_z)"/>
+    <xacro:property name="shelf_orientation" default="$(arg shelf_orientation)"/>
     <xacro:macro name="box_inertia" params="m x y z">
         <inertial>
@@ -35,5 +40,5 @@
             <parent link="world"/>
             <child link="shelf"/>
-            <origin xyz="${shelf_x} ${shelf_y} ${shelf_z}" rpy="0.0 0.0 1.645"/>
+            <origin xyz="${shelf_x} ${shelf_y} ${shelf_z}" rpy="${shelf_orientation}"/>
         </joint>
     </xacro:if>

File: mppi_examples/mppi_omav_interaction/data/objects/shelf_gazebo.urdf.xacro (robot description, xacro)
@@ -3,4 +3,8 @@
     <xacro:arg name="fixed" default="true"/>
     <xacro:arg name="height" default="0.0"/>
+    <xacro:arg name="shelf_x" default="-0.242"/>
+    <xacro:arg name="shelf_y" default="-0.595"/>
+    <xacro:arg name="shelf_z" default="0.834"/>
+    <xacro:arg name="shelf_orientation" default="0.0 0.0 1.645"/>
     <xacro:property name="height" default="$(arg height)"/>
     <xacro:property name="door_length" default="0.359"/>
@@ -15,7 +19,8 @@
     <xacro:property name="handle_offset_y" default="0.338"/>
     <xacro:property name="handle_offset_z" default="-0.024"/>
-    <xacro:property name="shelf_x" default="-0.242"/>
-    <xacro:property name="shelf_y" default="-0.595"/>
-    <xacro:property name="shelf_z" default="0.834"/>
+    <xacro:property name="shelf_x" default="$(arg shelf_x)"/>
+    <xacro:property name="shelf_y" default="$(arg shelf_y)"/>
+    <xacro:property name="shelf_z" default="$(arg shelf_z)"/>
+    <xacro:property name="shelf_orientation" default="$(arg shelf_orientation)"/>
     <xacro:macro name="box_inertia" params="m x y z">
         <inertial>
@@ -35,5 +40,5 @@
             <parent link="world"/>
             <child link="shelf"/>
-            <origin xyz="${shelf_x} ${shelf_y} ${shelf_z}" rpy="0.0 0.0 1.645"/>
+            <origin xyz="${shelf_x} ${shelf_y} ${shelf_z}" rpy="${shelf_orientation}"/>
         </joint>
     </xacro:if>

File: mppi_examples/mppi_omav_interaction/data/objects/shelf_rviz.urdf.xacro (robot description, xacro)
@@ -3,4 +3,8 @@
     <xacro:arg name="fixed" default="true"/>
     <xacro:arg name="height" default="0.0"/>
+    <xacro:arg name="shelf_x" default="-0.242"/>
+    <xacro:arg name="shelf_y" default="-0.595"/>
+    <xacro:arg name="shelf_z" default="0.834"/>
+    <xacro:arg name="shelf_orientation" default="0.0 0.0 1.645"/>
     <xacro:property name="height" default="$(arg height)"/>
     <xacro:property name="door_length" default="0.359"/>
@@ -15,7 +19,8 @@
     <xacro:property name="handle_offset_y" default="0.338"/>
     <xacro:property name="handle_offset_z" default="-0.024"/>
-    <xacro:property name="shelf_x" default="-0.242"/>
-    <xacro:property name="shelf_y" default="-0.595"/>
-    <xacro:property name="shelf_z" default="0.834"/>
+    <xacro:property name="shelf_x" default="$(arg shelf_x)"/>
+    <xacro:property name="shelf_y" default="$(arg shelf_y)"/>
+    <xacro:property name="shelf_z" default="$(arg shelf_z)"/>
+    <xacro:property name="shelf_orientation" default="$(arg shelf_orientation)"/>
     <xacro:macro name="box_inertia" params="m x y z">
         <inertial>
@@ -35,5 +40,5 @@
             <parent link="world"/>
             <child link="shelf"/>
-            <origin xyz="${shelf_x} ${shelf_y} ${shelf_z}" rpy="0.009 0.001 1.645"/>
+            <origin xyz="${shelf_x} ${shelf_y} ${shelf_z}" rpy="${shelf_orientation}"/>
         </joint>
     </xacro:if>

Commit message: fix: append hardwareinterface in urdf to remove deprecation warning

File: mppi_examples/mppi_omav_interaction/data/objects/shelf.urdf.xacro (robot description, xacro)
@@ -245,8 +245,8 @@
         <type>transmission_interface/SimpleTransmission</type>
         <joint name="articulation_joint">
-            <hardwareInterface>EffortJointInterface</hardwareInterface>
+            <hardwareInterface>hardware_interface/EffortJointInterface</hardwareInterface>
         </joint>
         <actuator name="motor1">
-            <hardwareInterface>EffortJointInterface</hardwareInterface>
+            <hardwareInterface>hardware_interface/EffortJointInterface</hardwareInterface>
             <mechanicalReduction>1</mechanicalReduction>
         </actuator>

File: mppi_examples/mppi_omav_interaction/data/objects/shelf_gazebo.urdf.xacro (robot description, xacro)
@@ -245,8 +245,8 @@
         <type>transmission_interface/SimpleTransmission</type>
         <joint name="articulation_joint">
-            <hardwareInterface>EffortJointInterface</hardwareInterface>
+            <hardwareInterface>hardware_interface/EffortJointInterface</hardwareInterface>
         </joint>
         <actuator name="motor1">
-            <hardwareInterface>EffortJointInterface</hardwareInterface>
+            <hardwareInterface>hardware_interface/EffortJointInterface</hardwareInterface>
             <mechanicalReduction>1</mechanicalReduction>
         </actuator>

File: mppi_examples/mppi_omav_interaction/data/objects/shelf_rviz.urdf.xacro (robot description, xacro)
@@ -245,8 +245,8 @@
         <type>transmission_interface/SimpleTransmission</type>
         <joint name="articulation_joint">
-            <hardwareInterface>EffortJointInterface</hardwareInterface>
+            <hardwareInterface>hardware_interface/EffortJointInterface</hardwareInterface>
         </joint>
         <actuator name="motor1">
-            <hardwareInterface>EffortJointInterface</hardwareInterface>
+            <hardwareInterface>hardware_interface/EffortJointInterface</hardwareInterface>
             <mechanicalReduction>1</mechanicalReduction>
         </actuator>

File: mppi_examples/mppi_omav_interaction/data/objects/valve.urdf.xacro (robot description, xacro)
@@ -9,5 +9,4 @@
         <parent link="world"/>
         <child link="valve_base"/>
-        <!-- <origin xyz="${base_position_x} ${base_position_y} ${base_height/2.0}" rpy="0 0 0"/> -->
         <origin xyz="0 0 0" rpy="0 0 0"/>
     </joint>
@@ -20,10 +19,4 @@
             <inertia ixx="0.001" ixy="0" ixz="0" iyy="0.001" iyz="0" izz="0.001"/>
         </inertial>
-        <!-- <visual>
-            <origin rpy="0 0 0" xyz="0 0 0"/>
-            <geometry>
-                <mesh filename="$(arg resource_directory)/valve_${valve_type}visual.obj" scale="1 1 1"/>
-            </geometry>
-        </visual> -->
         <collision>
             <origin rpy="0 0 0" xyz="0 0 0"/>
@@ -39,5 +32,4 @@
         <parent link="valve_base"/>
         <child link="handle_link"/>
-        <!--<origin xyz="0 0 ${base_height/2.0+0.2}" rpy="0 0 0"/> <!- 1.5708 0 0 -->
         <origin xyz="$(arg object_position)" rpy="$(arg object_rpy)"/>
         <dynamics damping="0" friction="0.002"/>

File: mppi_examples/mppi_omav_interaction/data/objects/valve_gazebo.urdf.xacro (robot description, xacro)
@@ -68,5 +68,4 @@
         <parent link="world"/>
         <child link="handle_link"/>
-        <!--<origin xyz="0 0 ${base_height/2.0+0.2}" rpy="1.5708 0 0"/> <!- 1.5708 0 0 -->
         <origin xyz="$(arg object_position)" rpy="$(arg object_rpy)"/>
         <dynamics damping="0.0" friction="0.002"/>
@@ -83,8 +82,8 @@
         <type>transmission_interface/SimpleTransmission</type>
         <joint name="articulation_joint">
-            <hardwareInterface>EffortJointInterface</hardwareInterface>
+            <hardwareInterface>hardware_interface/EffortJointInterface</hardwareInterface>
         </joint>
         <actuator name="motor1">
-            <hardwareInterface>EffortJointInterface</hardwareInterface>
+            <hardwareInterface>hardware_interface/EffortJointInterface</hardwareInterface>
             <mechanicalReduction>1</mechanicalReduction>
         </actuator>

File: mppi_examples/mppi_omav_interaction/data/objects/valve_rviz.urdf.xacro (robot description, xacro)
@@ -44,5 +44,4 @@
         <parent link="world"/>
         <child link="handle_link"/>
-        <!--<origin xyz="0 0 ${base_height/2.0+0.2}" rpy="1.5708 0 0"/> <!- 1.5708 0 0 -->
         <origin xyz="$(arg object_position)" rpy="$(arg object_rpy)"/>
         <dynamics damping="0.0" friction="0.0"/>
