Commit message: Added real values to the drone urdf.

File: mppi_examples/mppi_omav_interaction/data/objects/shelf_gazebo.urdf.xacro (robot description, xacro)
@@ -99,5 +99,5 @@
         <parent link="axis_link"/>
         <child link="measured_joint_link"/>
-        <dynamics damping="2.0" friction="10.0"/>
+        <dynamics damping="0.5" friction="0.1"/>
         <origin xyz="0 0 0"/>
         <axis xyz="0 0 -1"/>

File: mppi_examples/mppi_omav_interaction/data/omav_hook_visualization.urdf.xacro (robot description, xacro)
@@ -33,5 +33,5 @@
         <parent link="omav_base"/>
         <child link="rod"/>
-        <origin rpy="0 0 0" xyz="0.275 0.0 0.0"/>
+        <origin rpy="0 0 0" xyz="0.31 0.0 0.0"/>
     </joint>
     <link name="rod">
@@ -39,5 +39,5 @@
             <origin rpy="0 1.5708 0" xyz="0 0 0"/>
             <geometry>
-                <cylinder radius="0.0075" length="0.54"/>
+                <cylinder radius="0.0075" length="0.62"/>
             </geometry>
         </collision>
@@ -45,5 +45,5 @@
             <origin rpy="0 1.5708 0" xyz="0 0 0"/>
             <geometry>
-                <cylinder radius="0.0075" length="0.54"/>
+                <cylinder radius="0.0075" length="0.62"/>
             </geometry>
             <material name="">
@@ -55,5 +55,5 @@
         <parent link="rod"/>
         <child link="tip"/>
-        <origin rpy="0 0 0" xyz="0.27 0.0 0.0"/>
+        <origin rpy="0 0 0" xyz="0.31 0.0 0.0"/>
     </joint>
     <joint name="tip_to_thick" type="fixed">

File: mppi_examples/mppi_omav_interaction/data/omav_pinocchio_hook.urdf.xacro (robot description, xacro)
@@ -43,5 +43,5 @@
         <parent link="omav"/>
         <child link="rod"/>
-        <origin rpy="0 0 0" xyz="0.275 0.0 0.0"/>
+        <origin rpy="0 0 0" xyz="0.31 0.0 0.0"/>
     </joint>
     <link name="rod">
@@ -49,5 +49,5 @@
             <origin rpy="0 1.5708 0" xyz="0 0 0"/>
             <geometry>
-                <cylinder radius="0.015" length="0.54"/>
+                <cylinder radius="0.015" length="0.62"/>
             </geometry>
             <material name="">
@@ -58,5 +58,5 @@
             <origin rpy="0 1.5708 0" xyz="0 0 0"/>
             <geometry>
-                <cylinder radius="0.015" length="0.54"/>
+                <cylinder radius="0.015" length="0.62"/>
             </geometry>
             <material name="">
@@ -68,5 +68,5 @@
         <parent link="rod"/>
         <child link="tip"/>
-        <origin rpy="0 0 0" xyz="0.27 0.0 0.0"/>
+        <origin rpy="0 0 0" xyz="0.31 0.0 0.0"/>
     </joint>
     <link name="tip">

File: mppi_examples/mppi_omav_interaction/data/omav_raisim_hook.urdf.xacro (robot description, xacro)
@@ -68,5 +68,5 @@
         <parent link="omav"/>
         <child link="rod"/>
-        <origin rpy="0 0 0" xyz="0.275 0.0 0.0"/>
+        <origin rpy="0 0 0" xyz="0.31 0.0 0.0"/>
     </joint>
     <link name="rod">
@@ -74,5 +74,5 @@
             <origin rpy="0 1.5708 0" xyz="0 0 0"/>
             <geometry>
-                <cylinder radius="0.0075" length="0.54"/>
+                <cylinder radius="0.0075" length="0.62"/>
             </geometry>
             <material name="">
@@ -83,5 +83,5 @@
             <origin rpy="0 1.5708 0" xyz="0 0 0"/>
             <geometry>
-                <cylinder radius="0.0075" length="0.54"/>
+                <cylinder radius="0.0075" length="0.62"/>
             </geometry>
             <material name="">
@@ -93,5 +93,5 @@
         <parent link="rod"/>
         <child link="tip"/>
-        <origin rpy="0 0 0" xyz="0.27 0.0 0.0"/>
+        <origin rpy="0 0 0" xyz="0.31 0.0 0.0"/>
     </joint>
     <link name="tip">

Commit message: Working verstion for flight tests.

File: mppi_examples/mppi_omav_interaction/data/objects/shelf_gazebo.urdf.xacro (robot description, xacro)
@@ -4,13 +4,18 @@
     <xacro:arg name="height" default="0.0"/>
     <xacro:property name="height" default="$(arg height)"/>
-    <xacro:property name="door_length" default="0.295"/>
-    <xacro:property name="door_height" default="0.90"/>
-    <xacro:property name="door_width" default="0.016"/>
-    <xacro:property name="handle_height" default="0.056"/> <!-- 0.026 -->
+    <xacro:property name="door_length" default="0.359"/>
+    <xacro:property name="door_height" default="0.748"/>
+    <xacro:property name="door_width" default="0.018"/>
+    <xacro:property name="corpus_door_gap" default="0.004"/>
+    <xacro:property name="corpus_length" default="0.4"/>
+    <xacro:property name="corpus_height" default="0.827"/>
+    <xacro:property name="corpus_width" default="0.018"/>
+    <xacro:property name="handle_height" default="0.057"/> <!-- 0.026 -->
     <xacro:property name="handle_length" default="0.16"/>
-    <xacro:property name="handle_offset" default="0.27"/>
-    <xacro:property name="shelf_x" default="0.943"/>
-    <xacro:property name="shelf_y" default="-0.952"/>
-    <xacro:property name="shelf_z" default="0.903"/>
+    <xacro:property name="handle_offset_y" default="0.338"/>
+    <xacro:property name="handle_offset_z" default="-0.024"/>
+    <xacro:property name="shelf_x" default="-0.242"/>
+    <xacro:property name="shelf_y" default="-0.595"/>
+    <xacro:property name="shelf_z" default="0.834"/>
     <xacro:macro name="box_inertia" params="m x y z">
         <inertial>
@@ -30,5 +35,5 @@
             <parent link="world"/>
             <child link="shelf"/>
-            <origin xyz="${shelf_x} ${shelf_y} ${shelf_z}" rpy="-0.008 -0.001 -3.085"/>
+            <origin xyz="${shelf_x} ${shelf_y} ${shelf_z}" rpy="0.009 0.001 1.645"/>
         </joint>
     </xacro:if>
@@ -40,9 +45,9 @@
     </gazebo>
     <link name="shelf">
-        <xacro:box_inertia m="5" x="${door_width}" y="${door_length}" z="${shelf_z}"/>
-        <visual>
-            <origin rpy="0 0 0" xyz="0 -${door_length/2} ${-shelf_z/2}"/>
-            <geometry>
-                <box size="${door_width} ${door_length} ${shelf_z}"/>
+        <xacro:box_inertia m="5" x="${corpus_width}" y="${corpus_length}" z="${shelf_z}"/>
+        <visual>
+            <origin rpy="0 0 0" xyz="0 -${corpus_length/2} ${-shelf_z/2}"/>
+            <geometry>
+                <box size="${corpus_width} ${corpus_length} ${shelf_z}"/>
             </geometry>
             <material name="shelf_material">
@@ -54,5 +59,5 @@
         <xacro:box_inertia m="5.8" x="${door_width}" y="${door_length}" z="${door_height}"/>
         <visual>
-            <origin rpy="0 0 0" xyz="0 ${door_length/2} 0"/>
+            <origin rpy="0 0 0" xyz="${-door_width/2} ${door_length/2} 0"/>
             <geometry>
                 <box size="${door_width} ${door_length} ${door_height}"/>
@@ -75,5 +80,5 @@
         <inertial>
             <mass value="0.01"/>
-            <origin rpy="0 0 0" xyz="0 0 0"/>
+            <origin rpy="0 0 0" xyz="0.0 0 0"/>
             <inertia ixx="0.0" ixy="0.0" ixz="0.0" iyy="0.0" iyz="0.0" izz="0.0"/>
         </inertial>
@@ -82,5 +87,5 @@
         <parent link="shelf"/>
         <child link="door_hinge"/>
-        <origin xyz="0 -${door_length} ${door_height/2}"/>
+        <origin xyz="${door_width/2+0.012} -${door_length + corpus_width +corpus_door_gap} ${door_height/2}"/>
     </joint>
     <link name="axis_link">
@@ -94,10 +99,10 @@
         <parent link="door_hinge"/>
         <child link="axis_link"/>
-        <origin xyz="0.004 0.027 -0.150"/>
+        <origin xyz="0.0 0.0 0.0"/>
     </joint>
     <joint name="articulation_joint" type="revolute">
         <parent link="axis_link"/>
         <child link="measured_joint_link"/>
-        <dynamics damping="0.5" friction="0.1"/>
+        <dynamics damping="1.5" friction="0.1"/>
         <origin xyz="0 0 0"/>
         <axis xyz="0 0 -1"/>
@@ -107,5 +112,5 @@
         <parent link="measured_joint_link"/>
         <child link="door"/>
-        <origin xyz="-0.004 -0.027 0.150"/>
+        <origin xyz="0.0 0.0 0.0"/>
     </joint>
     <link name="handle_link">
@@ -155,5 +160,5 @@
             </geometry>
             <material name="">
-                <contact name="steel"/>
+                <contact name="rubber"/>
             </material>
         </collision>
@@ -180,5 +185,5 @@
             </geometry>
             <material name="">
-                <contact name="steel"/>
+                <contact name="rubber"/>
             </material>
         </collision>
@@ -187,5 +192,5 @@
         <parent link="door"/>
         <child link="handle_link"/>
-        <origin xyz="${handle_height + door_width/2} ${handle_offset} -0.15"
+        <origin xyz="${handle_height + 0.012} ${handle_offset_y} ${handle_offset_z}"
                 rpy="0 0 0"/> <!-- height handle + half the width door, 0.30 minus some offset -->
     </joint>

File: mppi_examples/mppi_omav_interaction/data/objects/shelf_new.urdf.xacro (robot description, xacro)
@@ -1,4 +1,4 @@
 <?xml version="1.0" ?>
-<robot name="shelf" xmlns:xacro="http://www.ros.org/wiki/xacro">
+<robot name="shelf_new" xmlns:xacro="http://www.ros.org/wiki/xacro">
     <xacro:arg name="fixed" default="true"/>
     <xacro:arg name="height" default="0.0"/>
@@ -198,5 +198,5 @@
         <parent link="handle_link"/>
         <child link="handle_ref"/>
-        <origin xyz="${-handle_height/2-0.012} 0 0"
+        <origin xyz="${-handle_height/2} 0 0"
                 rpy="0 0 0"/> <!-- height handle + half the width door, 0.30 minus some offset -->
     </joint>

Commit message: Updates for shelf simulation and observer.

File: mppi_examples/mppi_omav_interaction/data/objects/shelf_gazebo.urdf.xacro (robot description, xacro)
@@ -38,10 +38,4 @@
         </joint>
     </xacro:if>
-    <gazebo>
-        <plugin name="gazebo_ros_control" filename="libgazebo_ros_control.so">
-            <robotNamespace>/shelf</robotNamespace>
-            <robotParam>urdf_object </robotParam>
-        </plugin>
-    </gazebo>
     <link name="shelf">
         <xacro:box_inertia m="5" x="${corpus_width}" y="${corpus_length}" z="${shelf_z}"/>
@@ -237,4 +231,10 @@
         <origin xyz="-0.06 -0.243 0.0" rpy="0 0 0"/>
     </joint>
+    <gazebo>
+        <plugin name="gazebo_ros_control" filename="libgazebo_ros_control.so">
+            <robotNamespace>/shelf</robotNamespace>
+            <robotParam>urdf_gazebo</robotParam>
+        </plugin>
+    </gazebo>
     <transmission name="hinge">
         <type>transmission_interface/SimpleTransmission</type>

File: mppi_examples/mppi_omav_interaction/data/objects/shelf_new_2021_11.urdf.xacro (robot description, xacro)
@@ -34,5 +34,5 @@
         <joint name="fixed" type="fixed">
             <parent link="world"/>
-            <child link="${prefix}shelf"/> 0
+            <child link="${prefix}shelf"/>
             <origin xyz="100.272902 -0.0944762   0.830376" rpy="0.000710616 0.000859919  1.51977"/>
         </joint>
