Commit message: fix: revert floating base for raisim shelf object

File: mppi_examples/mppi_omav_interaction/data/objects/shelf_raisim.urdf.xacro (robot description, xacro)
@@ -35,34 +35,8 @@
     </xacro:macro>
     <link name="world"/>
-    <link name="shelf_x" />
-    <link name="shelf_y" />
-    <link name="shelf_z" />
-    <joint name="world_to_shelf_x" type="prismatic">
+    <joint name="fixed" type="fixed">
         <parent link="world"/>
-        <child link="shelf_x"/>
-        <origin rpy="0 0 0" xyz="0.0 0.0 0.0"/>
-        <axis xyz="1 0 0"/>
-        <limit effort="1000.0" velocity="0.0" lower="-100" upper="100"/>
-    </joint>
-    <joint name="shelf_x_to_shelf_y" type="prismatic">
-        <parent link="shelf_x"/>
-        <child link="shelf_y"/>
-        <origin rpy="0 0 0" xyz="0.0 0.0 0.0"/>
-        <axis xyz="0 1 0"/>
-        <limit effort="1000.0" velocity="0.0" lower="-100" upper="100"/>
-    </joint>
-    <joint name="shelf_y_to_shelf_z" type="prismatic">
-        <parent link="shelf_y"/>
-        <child link="shelf_z"/>
-        <origin rpy="0 0 0" xyz="0.0 0.0 0.0"/>
-        <axis xyz="0 0 1"/>
-        <limit effort="1000.0" velocity="0.0" lower="-100" upper="100"/>
-    </joint>
-    <joint name="shelf_z_to_shelf" type="spherical">
-        <parent link="shelf_z"/>
         <child link="shelf"/>
-        <origin rpy="0 0 0" xyz="0.0 0.0 0.0"/>
-        <axis xyz="1 0 0"/>
-        <limit effort="1000.0" velocity="0.0" lower="0" upper="10" />
+        <origin xyz="0 0 0" rpy="0 0 0"/>
     </joint>
     <link name="shelf">

Commit message: refactor: clean up object pose updating for raisim

File: mppi_examples/mppi_omav_interaction/data/objects/shelf_raisim.urdf.xacro (robot description, xacro)
@@ -35,10 +35,10 @@
     </xacro:macro>
     <link name="world"/>
-    <joint name="fixed" type="fixed">
+    <joint name="base" type="fixed">
         <parent link="world"/>
-        <child link="shelf"/>
+        <child link="base"/>
         <origin xyz="0 0 0" rpy="0 0 0"/>
     </joint>
-    <link name="shelf">
+    <link name="base">
         <xacro:box_inertia m="5" x="${corpus_width}" y="${corpus_length}" z="${shelf_z}"/>
         <visual>
@@ -81,5 +81,5 @@
     </link>
     <joint name="door_hinge_joint" type="fixed">
-        <parent link="shelf"/>
+        <parent link="base"/>
         <child link="door_hinge"/>
         <origin xyz="${door_width/2+0.012} -${door_length + corpus_width +corpus_door_gap} ${door_height/2}"/>

Commit message: fix: spawn shelf far away from drone during startup

File: mppi_examples/mppi_omav_interaction/data/objects/shelf_raisim.urdf.xacro (robot description, xacro)
@@ -38,5 +38,5 @@
         <parent link="world"/>
         <child link="base"/>
-        <origin xyz="0 0 0" rpy="0 0 0"/>
+        <origin xyz="10 10 0" rpy="0 0 0"/>
     </joint>
     <link name="base">
