Commit message: adapting state to be the same as dishwasher benchmark

File: mppi_examples/mppi_panda_mobile/resources/panda/base.urdf.xacro (robot description, xacro)
@@ -2,4 +2,34 @@
 <robot name="panda_mobile" xmlns:xacro="http://www.ros.org/wiki/xacro">
     <xacro:macro name="panda_base" params="base_link:='base'">
+        <link name="world"/>
+        <link name="x_link"/>
+        <joint name="x_velocity_joint" type="prismatic">
+            <origin rpy="0 0 0" xyz="0 0 0"/>
+            <axis xyz="1 0 0"/>
+            <parent link="world"/>
+            <child link="x_link"/>
+            <limit lower="-10" upper="10" effort="200" velocity="2"/>
+        </joint>
+        <link name="xy_link"/>
+        <joint name="y_velocity_joint" type="prismatic">
+            <origin rpy="0 0 0" xyz="0 0 0"/>
+            <axis xyz="0 1 0"/>
+            <parent link="x_link"/>
+            <child link="xy_link"/>
+            <limit lower="-10" upper="10" effort="200" velocity="2"/>
+        </joint>
+        <link name="xyw_link"/>
+        <joint name="w_velocity_joint" type="revolute">
+            <origin rpy="0 0 0" xyz="0 0 0"/>
+            <axis xyz="0 0 1"/>
+            <parent link="xy_link"/>
+            <child link="xyw_link"/>
+            <limit effort="200" velocity="2" upper="-30" lower="30"/>
+        </joint>
+        <joint name="base_link_joint" type="fixed">
+            <origin rpy="0 0 0" xyz="0 0 0"/>
+            <parent link="xyw_link"/>
+            <child link="${base_link}"/>
+        </joint>
         <link name="${base_link}">
             <collision>

File: mppi_examples/mppi_panda_mobile/resources/panda/panda_mobile.urdf (robot description, URDF)
Before this commit: robot panda, 11 links, 10 joints
Links:
- added link world
- added link x_link
- added link xy_link
- added link xyw_link
Joints:
- added joint base_link_joint: type fixed, parent xyw_link, child base, origin xyz=0 0 0 rpy=0 0 0
- added joint w_velocity_joint: type continuous, parent xy_link, child xyw_link, origin xyz=0 0 0 rpy=0 0 0, axis 0 0 1, limit effort=200 velocity=2
- added joint x_velocity_joint: type prismatic, parent world, child x_link, origin xyz=0 0 0 rpy=0 0 0, axis 1 0 0, limit lower=-10 upper=10 effort=200 velocity=2
- added joint y_velocity_joint: type prismatic, parent x_link, child xy_link, origin xyz=0 0 0 rpy=0 0 0, axis 0 1 0, limit lower=-10 upper=10 effort=200 velocity=2

Commit message: integration of safety filter

File: mppi_examples/mppi_panda_mobile/resources/panda/base.urdf.xacro (robot description, xacro)
@@ -2,4 +2,40 @@
 <robot name="panda_mobile" xmlns:xacro="http://www.ros.org/wiki/xacro">
     <xacro:macro name="panda_base" params="base_link:='base'">
+        <link name="world"/>
+        <link name="x_link">
+            <inertial>
+                <origin xyz="0 0 0" rpy="0 0 0" />
+                <mass value="3.06"/>
+                <inertia ixx="0.3" ixy="0.0" ixz="0.0" iyy="0.3" iyz="0.0" izz="0.3" />
+            </inertial>
+        </link>
+        <joint name="x_base_joint" type="prismatic">
+            <origin rpy="0 0 0" xyz="0 0 0"/>
+            <axis xyz="1 0 0"/>
+            <parent link="world"/>
+            <child link="x_link"/>
+            <limit lower="-10" upper="10" effort="200" velocity="2"/>
+        </joint>
+        <link name="y_link">
+            <inertial>
+                <origin xyz="0 0 0" rpy="0 0 0" />
+                <mass value="3.06"/>
+                <inertia ixx="0.3" ixy="0.0" ixz="0.0" iyy="0.3" iyz="0.0" izz="0.3" />
+            </inertial>
+        </link>
+        <joint name="y_base_joint" type="prismatic">
+            <origin rpy="0 0 0" xyz="0 0 0"/>
+            <axis xyz="0 1 0"/>
+            <parent link="x_link"/>
+            <child link="y_link"/>
+            <limit lower="-10" upper="10" effort="200" velocity="2"/>
+        </joint>
+        <joint name="w_base_joint" type="revolute">
+            <origin rpy="0 0 0" xyz="0 0 0"/>
+            <axis xyz="0 0 1"/>
+            <parent link="y_link"/>
+            <child link="${base_link}"/>
+            <limit effort="200" velocity="2" upper="30" lower="-30"/>
+        </joint>
         <link name="${base_link}">
             <collision>
@@ -14,5 +50,4 @@
                     <box size="0.5 0.5 0.25"/>
                 </geometry>
-                <material name="green"/>
             </visual>
         </link>
