Commit message: Works now with obstacle, very hack implementation.

File: mppi_examples/mppi_pathfinder/resources/pathfinder.urdf (robot description, URDF)
Before this commit: robot pathfinder, 2 links, 1 joints
Links:
- added link cart_link2, mass 1.0; visual box size=0.3 0.3 0.3
- added link obstacle, mass 1.0; visual box size=1 1 1
- link cart_link: geometry visual box size=0.03 0.03 0.03
Joints:
- removed joint cart
- added joint cart_x: type prismatic, parent odom, child cart_link, origin xyz=0 0 0 rpy=0 0 0, axis 1 0 0, limit lower=-30.14 upper=30.14 effort=1000 velocity=2.0
- added joint cart_y: type prismatic, parent cart_link, child cart_link2, origin xyz=0 0 0 rpy=0 0 0, axis 0 1 0, limit lower=-30.14 upper=30.14 effort=1000 velocity=2.0
- added joint fixed: type fixed, parent odom, child obstacle, origin xyz=14.0 2.0 0.0 rpy=0 0 0

Commit message: Cleanup and working fine.

File: mppi_examples/mppi_pathfinder/resources/pathfinder.urdf (robot description, URDF)
Before this commit: robot pathfinder, 4 links, 3 joints
Links:
- added link cart_link3, mass 1.0; visual box size=0.3 0.3 0.3
- link cart_link2: geometry visual box size=0.03 0.03 0.03
- link obstacle: geometry visual cylinder length=2 radius=2
Joints:
- added joint cart_theta: type continuous, parent cart_link2, child cart_link3, origin xyz=0 0 0 rpy=0 0 0, axis 0 0 1, limit effort=1000 velocity=1.0

Commit message: Minor fixes to different examples

File: mppi_examples/mppi_pathfinder/resources/pathfinder.urdf (robot description, URDF)
Before this commit: robot pathfinder, 5 links, 4 joints
Links:
- removed link cart_link2
- removed link cart_link3
- removed link obstacle
- link cart_link: geometry visual box size=0.3 0.3 0.3
Joints:
- removed joint cart_theta
- removed joint cart_y
- removed joint fixed
