Commit message: calibrated urdf

File: mppi_examples/mppi_panda/resources/bota/urdf/BFT_SENS_SER_M8.urdf.xacro (robot description, xacro)
@@ -32,5 +32,5 @@
         <geometry>
           <mesh
-            filename="package://moma_description/sensors/bota/meshes/BFT_SENS_SER_M8/mounting.STL" />
+            filename="package://mppi_panda/resources/bota/meshes/BFT_SENS_SER_M8/mounting.STL" />
         </geometry>
         <material
@@ -46,5 +46,5 @@
         <geometry>
           <mesh
-            filename="package://moma_description/sensors/bota/meshes/BFT_SENS_SER_M8/mounting.STL" />
+            filename="package://mppi_panda/resources/bota/meshes/BFT_SENS_SER_M8/mounting.STL" />
         </geometry>
       </collision> -->
@@ -72,5 +72,5 @@
         <geometry>
           <mesh
-            filename="package://moma_description/sensors/bota/meshes/BFT_SENS_SER_M8/wrench.STL" />
+            filename="package://mppi_panda/resources/bota/meshes/BFT_SENS_SER_M8/wrench.STL" />
         </geometry>
         <material
@@ -86,5 +86,5 @@
         <geometry>
           <mesh
-            filename="package://moma_description/sensors/bota/meshes/BFT_SENS_SER_M8/wrench.STL" />
+            filename="package://mppi_panda/resources/bota/meshes/BFT_SENS_SER_M8/wrench.STL" />
         </geometry>
       </collision> -->

File: mppi_examples/mppi_panda/resources/panda/panda.urdf.xacro (robot description, xacro)
@@ -25,5 +25,5 @@
     <xacro:property name="add_wrench_sensor" default="$(arg add_wrench_sensor)"/>
     <xacro:include filename="$(find mppi_panda)/resources/panda/custom_fingers.urdf"/>
-    <xacro:include filename="$(find mppi_panda)/sensors/bota/urdf/BFT_SENS_SER_M8.urdf.xacro"/>
+    <xacro:include filename="$(find mppi_panda)/resources/bota/urdf/BFT_SENS_SER_M8.urdf.xacro"/>
     <xacro:macro name="panda_robot" params="parent_link:='world' robot_description:=''">
         <joint name="panda_joint_${parent_link}" type="fixed">
@@ -437,10 +437,10 @@
             </xacro:BFT_SENS_SER_M8>
             <joint name="hand_flange_joint" type="fixed">
-                <origin xyz="0 0 0" rpy="0 0 0"/>
+                <origin xyz="0 0 0" rpy="0 0 -2.355"/>
                 <parent link="ft_sensor0_wrench"/>
                 <child link="hand_flange"/>
             </joint>
         </xacro:if>
-        <xacro:unless>
+        <xacro:unless value="${add_wrench_sensor}">
             <joint name="hand_flange_joint" type="fixed">
                 <origin xyz="0 0 0" rpy="0 0 -0.785398163397"/>
