Commit message: cylinder replacement finish

File: mppi_examples/mppi_sliding/data/objects/cylinder_t.urdf (robot description, URDF)
Before this commit: robot cylinder, 1 links, 0 joints
Links:
- removed link cylinder_frame
- added link cylinder_t_frame, mass 10; collision cylinder length=0.2 radius=0.04; visual cylinder length=0.2 radius=0.04

File: mppi_examples/mppi_sliding/data/objects/table.urdf (robot description, URDF)
Before this commit: robot cylinder, 1 links, 0 joints
Links:
- removed link cylinder_frame
- added link table_frame, mass 10; collision box size=3 3 0.2; visual box size=3 3 0.2
