Commit message: mug into the loop and model updater added

File: mppi_examples/mppi_sliding/data/objects/cylinder.urdf (robot description, URDF)
Before this commit: robot cylinder, 1 links, 0 joints
Links:
- link cylinder_frame: geometry collision cylinder length=0.1 radius=0.05; visual cylinder length=0.1 radius=0.05

File: mppi_examples/mppi_sliding/data/objects/cylinder_t.urdf (robot description, URDF)
Before this commit: robot cylinder_t, 1 links, 0 joints
Links:
- link cylinder_t_frame: geometry collision cylinder length=0.1 radius=0.05; visual cylinder length=0.1 radius=0.05

File: mppi_examples/mppi_sliding/data/objects/mug_dynamic.urdf (robot description, URDF)
Before this commit: robot mug, 2 links, 1 joints
Links:
- link base_inertia: mass 0.3 -> 1

File: mppi_examples/mppi_sliding/data/objects/mug_vis.urdf (robot description, URDF)
Before this commit: robot mug, 2 links, 1 joints
Links:
- link base_inertia: mass 0.3 -> 1

Commit message: Add Raisim Cylinder update

File: mppi_examples/mppi_sliding/data/objects/cylinder.urdf (robot description, URDF)
Before this commit: robot cylinder, 1 links, 0 joints
Links:
- link cylinder_frame: geometry collision cylinder length=0.1 radius=0.03; visual cylinder length=0.1 radius=0.03
