Commit message: add mug obj and vis in Rviz

File: mppi_examples/mppi_sliding/data/objects/mug_dynamic.urdf (robot description, URDF)
Before this commit: robot mug, 2 links, 1 joints
Links:
- removed link world
- added link mug_frame; collision mesh filename=/home/boyang/catkin_ws/src/sampling_based_control/mppi_exam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 scale=0.05 0.05 0.05; visual mesh filename=/home/boyang/catkin_ws/src/sampling_based_control/mppi_exam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 scale=0.05 0.05 0.05
- link base_inertia: mass 16.793507758 -> 1.0
Joints:
- joint base_to_base_inertia: parent world -> mug_frame

File: mppi_examples/mppi_sliding/data/objects/mug_vis.urdf (robot description, URDF)
Before this commit: robot mug, 2 links, 1 joints
Links:
- removed link world
- added link mug_frame; collision mesh filename=file:///home/boyang/catkin_ws/src/sampling_based_control/mp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 scale=0.05 0.05 0.05; visual mesh filename=file:///home/boyang/catkin_ws/src/sampling_based_control/mp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 scale=0.05 0.05 0.05
- link base_inertia: mass 16.793507758 -> 1
Joints:
- joint base_to_base_inertia: parent world -> mug_frame

Commit message: add mug in sim loop

File: mppi_examples/mppi_sliding/data/objects/mug_dynamic.urdf (robot description, URDF)
Before this commit: robot mug, 2 links, 1 joints
Links:
- link base_inertia: mass 1.0 -> 1

Commit message: mug into the loop finish

File: mppi_examples/mppi_sliding/data/objects/mug_dynamic.urdf (robot description, URDF)
Before this commit: robot mug, 2 links, 1 joints
Links:
- link base_inertia: mass 1 -> 0.3

File: mppi_examples/mppi_sliding/data/objects/mug_vis.urdf (robot description, URDF)
Before this commit: robot mug, 2 links, 1 joints
Links:
- link base_inertia: mass 1 -> 0.3

Commit message: Adapt to ASL PC

File: mppi_examples/mppi_sliding/data/objects/mug_dynamic.urdf (robot description, URDF)
Before this commit: robot mug, 2 links, 1 joints
Links:
- link mug_frame: geometry collision mesh filename=/home/user/catkin_ws/src/sampling_based_control/mppi_exampl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 scale=0.05 0.05 0.05; visual mesh filename=/home/user/catkin_ws/src/sampling_based_control/mppi_exampl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 scale=0.05 0.05 0.05

File: mppi_examples/mppi_sliding/data/objects/mug_vis.urdf (robot description, URDF)
Before this commit: robot mug, 2 links, 1 joints
Links:
- link mug_frame: geometry collision mesh filename=file:///home/user/catkin_ws/src/sampling_based_control/mppi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 scale=0.05 0.05 0.05; visual mesh filename=file:///home/user/catkin_ws/src/sampling_based_control/mppi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 scale=0.05 0.05 0.05

File: mppi_examples/object_modeling_playground/data/objects/mug.urdf (robot description, URDF)
Before this commit: robot mug, 2 links, 1 joints
Links:
- link mug_frame: geometry collision mesh filename=file:///home/user/catkin_ws/src/sampling_based_control/mppi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 scale=0.1 0.1 0.1; visual mesh filename=file:///home/user/catkin_ws/src/sampling_based_control/mppi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 scale=0.1 0.1 0.1

Commit message: Sync Panda and ASL_PC

File: mppi_examples/mppi_sliding/data/objects/mug_dynamic.urdf (robot description, URDF)
Before this commit: robot mug, 2 links, 1 joints
Joints:
- joint base_to_base_inertia: origin xyz=0 0 0 rpy=0 0 0 -> xyz=0 0 0.0 rpy=0 0 0

File: mppi_examples/mppi_sliding/data/objects/table.urdf (robot description, URDF)
Before this commit: robot table, 1 links, 0 joints
Links:
- link table_frame: geometry collision box size=2 2 0.1; visual box size=2 2 0.1
