Commit message: Clean up, lightning structure

File: mppi_examples/mppi_sliding/data/objects/mug_1_vis.urdf (robot description, URDF)
Before this commit: robot mug_2, 1 links, 0 joints
Links:
- link mug_frame: geometry collision mesh filename=file:///home/user/catkin_ws/src/sampling_based_control/mppi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 scale=1.0 1.0 1.0; visual mesh filename=file:///home/user/catkin_ws/src/sampling_based_control/mppi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 scale=0.05 0.05 0.05
