Commit message: Add second mug, but not in the raisim yet

File: mppi_examples/mppi_sliding/data/objects/mug_0_dynamics.urdf (robot description, URDF)
Before this commit: robot mug_2, 1 links, 0 joints
Links:
- removed link mug_frame
- added link mug_frame_0, mass 0.1; collision mesh filename=/home/user/catkin_ws/src/sampling_based_control/mppi_exampl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 scale=1.0 1.0 1.0; visual mesh filename=/home/user/catkin_ws/src/sampling_based_control/mppi_exampl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 scale=0.05 0.05 0.05

File: mppi_examples/mppi_sliding/data/objects/mug_0_vis.urdf (robot description, URDF)
Before this commit: robot mug_2, 1 links, 0 joints
Links:
- removed link mug_frame
- added link mug_frame_0, mass 0.1; collision mesh filename=file:///home/user/catkin_ws/src/sampling_based_control/mppi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 scale=1.0 1.0 1.0; visual mesh filename=file:///home/user/catkin_ws/src/sampling_based_control/mppi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 scale=0.05 0.05 0.05

File: mppi_examples/mppi_sliding/data/objects/mug_1_dynamics.urdf (robot description, URDF)
Before this commit: robot mug_1, 1 links, 0 joints
Links:
- removed link mug_frame
- added link mug_frame_1, mass 0.1; collision mesh filename=/home/user/catkin_ws/src/sampling_based_control/mppi_exampl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 scale=1.0 1.0 1.0; visual mesh filename=/home/user/catkin_ws/src/sampling_based_control/mppi_exampl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 scale=0.05 0.05 0.05

File: mppi_examples/mppi_sliding/data/objects/mug_1_vis.urdf (robot description, URDF)
Before this commit: robot mug_1, 1 links, 0 joints
Links:
- removed link mug_frame
- added link mug_frame_1, mass 0.1; collision mesh filename=file:///home/user/catkin_ws/src/sampling_based_control/mppi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 scale=1.0 1.0 1.0; visual mesh filename=file:///home/user/catkin_ws/src/sampling_based_control/mppi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 scale=0.05 0.05 0.05
