Commit message: Change cost from quad to linear, tune a sliding example

File: mppi_examples/mppi_sliding/data/objects/table.urdf (robot description, URDF)
Before this commit: robot table, 1 links, 0 joints
Links:
- link table_frame: geometry collision box size=1.5 1.5 0.1; visual box size=1.5 1.5 0.1

Commit message: Important: A working example of pushing, need to be this setup and params

File: mppi_examples/mppi_sliding/data/objects/table.urdf (robot description, URDF)
Before this commit: robot table, 1 links, 0 joints
Links:
- link table_frame: geometry collision box size=2 2 0.1; visual box size=2 2 0.1
