Commit message: add mug and kp

File: mppi_examples/object_modeling_playground/data/objects/mug.urdf (robot description, URDF)
Before this commit: robot mug, 1 links, 0 joints
Links:
- link mug_frame: geometry collision mesh filename=file:///home/boyang/catkin_ws/src/sampling_based_control/mp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 scale=0.1 0.1 0.1; visual mesh filename=file:///home/boyang/catkin_ws/src/sampling_based_control/mp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 scale=0.1 0.1 0.1

Commit message: Modify URDF

File: mppi_examples/object_modeling_playground/data/objects/mug.urdf (robot description, URDF)
Before this commit: robot mug, 2 links, 1 joints
Links:
- removed link world
- added link mug_frame; collision mesh filename=file:///home/boyang/catkin_ws/src/sampling_based_control/mp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 scale=0.1 0.1 0.1; visual mesh filename=file:///home/boyang/catkin_ws/src/sampling_based_control/mp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 scale=0.1 0.1 0.1
Joints:
- joint base_to_base_inertia: parent world -> mug_frame
