Commit message: Add real_controller.cpp for panda control test

File: mppi_examples/mppi_sliding/data/panda.urdf.xacro (robot description, xacro)
@@ -50,5 +50,5 @@
             </inertial>
         </link>
-        <joint name="x_base_joint" type="prismatic">
+        <joint name="x_base_joint" type="fixed">
             <parent link="odom"/>
             <child link="x_slider"/>
@@ -59,5 +59,5 @@
         </joint>
         <xacro:add_transmission joint_name="x_base_joint"/>
-        <joint name="y_base_joint" type="prismatic">
+        <joint name="y_base_joint" type="fixed">
             <parent link="x_slider"/>
             <child link="y_slider"/>
@@ -68,5 +68,5 @@
         </joint>
         <xacro:add_transmission joint_name="y_base_joint"/>
-        <joint name="pivot_joint" type="revolute">
+        <joint name="pivot_joint" type="fixed">
             <parent link="y_slider"/>
             <child link="pivot"/>
