Commit message: Comment out update, system works

File: mppi_examples/mppi_sliding/data/panda.urdf (robot description, URDF)
Before this commit: robot panda, 13 links, 12 joints
Links:
- link panda_hand: geometry collision box size=0.035 0.19 0.065; visual mesh filename=/home/franka/boyang_ws/src/sampling_based_control/mppi_exam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
- link panda_leftfinger: geometry collision box size=0.02 0.02 0.05; visual mesh filename=/home/franka/boyang_ws/src/sampling_based_control/mppi_exam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
- link panda_link0: geometry collision mesh filename=/home/franka/boyang_ws/src/sampling_based_control/mppi_exam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; visual mesh filename=/home/franka/boyang_ws/src/sampling_based_control/mppi_exam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
- link panda_link1: geometry collision mesh filename=/home/franka/boyang_ws/src/sampling_based_control/mppi_exam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; visual mesh filename=/home/franka/boyang_ws/src/sampling_based_control/mppi_exam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
- link panda_link2: geometry collision mesh filename=/home/franka/boyang_ws/src/sampling_based_control/mppi_exam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; visual mesh filename=/home/franka/boyang_ws/src/sampling_based_control/mppi_exam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
- link panda_link3: geometry collision mesh filename=/home/franka/boyang_ws/src/sampling_based_control/mppi_exam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; visual mesh filename=/home/franka/boyang_ws/src/sampling_based_control/mppi_exam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
- link panda_link4: geometry collision mesh filename=/home/franka/boyang_ws/src/sampling_based_control/mppi_exam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; visual mesh filename=/home/franka/boyang_ws/src/sampling_based_control/mppi_exam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
- link panda_link5: geometry collision mesh filename=/home/franka/boyang_ws/src/sampling_based_control/mppi_exam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; visual mesh filename=/home/franka/boyang_ws/src/sampling_based_control/mppi_exam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
- link panda_link6: geometry collision mesh filename=/home/franka/boyang_ws/src/sampling_based_control/mppi_exam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; visual mesh filename=/home/franka/boyang_ws/src/sampling_based_control/mppi_exam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
- link panda_link7: geometry collision mesh filename=/home/franka/boyang_ws/src/sampling_based_control/mppi_exam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; visual mesh filename=/home/franka/boyang_ws/src/sampling_based_control/mppi_exam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
- link panda_rightfinger: geometry collision box size=0.02 0.02 0.05; visual mesh filename=/home/franka/boyang_ws/src/sampling_based_control/mppi_exam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
