Commit message: consolidated launch files, results of experiments from apr 11

File: mppi_examples/mppi_manipulation/data/objects/11826_mppi/mobility.urdf.xacro (robot description, xacro)
@@ -3,5 +3,9 @@
 <robot name="11826" xmlns:xacro="http://www.ros.org/wiki/xacro" >
   <xacro:arg name="prefix" default=""/>
+  <xacro:arg name="resources_directory" default=""/>
+  <xacro:arg name="resources_prefix" default=""/>
   <xacro:property name="prefix" default="$(arg prefix)"/>
+  <xacro:property name="resources_directory" default="$(arg resources_directory)"/>
+  <xacro:property name="resources_prefix" default="$(arg resources_prefix)"/>
   <link name="world"/>
   <link name="base"/>
@@ -15,5 +19,5 @@
     <visual>
       <geometry>
-        <mesh filename="textured_objs/original-4.obj" scale="0.4538303702144554 0.4538303702144554 0.4538303702144554"/>
+        <mesh filename="${resources_directory}${resources_prefix}textured_objs/original-4.obj" scale="0.4538303702144554 0.4538303702144554 0.4538303702144554"/>
       </geometry>
       <origin xyz="0.23330056661655543 0.2226204113200439 -0.19163586347627987" rpy="0.0 -0.0 0.0"/>
@@ -21,5 +25,5 @@
     <visual>
       <geometry>
-        <mesh filename="textured_objs/original-3.obj" scale="0.4538303702144554 0.4538303702144554 0.4538303702144554"/>
+        <mesh filename="${resources_directory}${resources_prefix}textured_objs/original-3.obj" scale="0.4538303702144554 0.4538303702144554 0.4538303702144554"/>
       </geometry>
       <origin xyz="0.23330056661655543 0.2226204113200439 -0.19163586347627987" rpy="0.0 -0.0 0.0"/>
@@ -27,5 +31,5 @@
     <visual>
       <geometry>
-        <mesh filename="textured_objs/original-2.obj" scale="0.4538303702144554 0.4538303702144554 0.4538303702144554"/>
+        <mesh filename="${resources_directory}${resources_prefix}textured_objs/original-2.obj" scale="0.4538303702144554 0.4538303702144554 0.4538303702144554"/>
       </geometry>
       <origin xyz="0.23330056661655543 0.2226204113200439 -0.19163586347627987" rpy="0.0 -0.0 0.0"/>
@@ -33,5 +37,5 @@
     <collision>
       <geometry>
-        <mesh filename="consolidated_collision_meshes/link_2.obj" scale="0.4538303702144554 0.4538303702144554 0.4538303702144554"/>
+        <mesh filename="${resources_directory}${resources_prefix}consolidated_collision_meshes/link_2.obj" scale="0.4538303702144554 0.4538303702144554 0.4538303702144554"/>
       </geometry>
       <origin xyz="0.0 0.0 0.0" rpy="0.0 -0.0 0.0"/>
@@ -41,5 +45,5 @@
     <visual>
       <geometry>
-        <mesh filename="consolidated_collision_meshes/link_3.obj" scale="0.4538303702144554 0.4538303702144554 0.4538303702144554"/>
+        <mesh filename="${resources_directory}${resources_prefix}consolidated_collision_meshes/link_3.obj" scale="0.4538303702144554 0.4538303702144554 0.4538303702144554"/>
       </geometry>
       <origin xyz="0.0 0.0 0.0" rpy="0.0 -0.0 0.0"/>
@@ -47,5 +51,5 @@
     <collision>
       <geometry>
-        <mesh filename="consolidated_collision_meshes/link_3.obj" scale="0.4538303702144554 0.4538303702144554 0.4538303702144554"/>
+        <mesh filename="${resources_directory}${resources_prefix}consolidated_collision_meshes/link_3.obj" scale="0.4538303702144554 0.4538303702144554 0.4538303702144554"/>
       </geometry>
       <origin xyz="0.0 0.0 0.0" rpy="0.0 -0.0 0.0"/>
