Commit message: print mppi cost components

File: mppi_examples/mppi_manipulation/data/objects/11826_mppi/mobility.urdf (robot description, URDF)
Before this commit: robot partnet_b5ca6cded4b23f2455b2aedb5bd199c6, 5 links, 4 joints
Joints:
- joint fixed: origin xyz=0.0 -0.07044640523565884 0.7743112142292514 rpy=0.0 -0.0 0.0 -> xyz=1.5 0. 0.85 rpy=0.0 -0.0 0.0

File: mppi_examples/mppi_manipulation/data/objects/11826_mppi/mobility.urdf.xacro (robot description, xacro)
@@ -59,5 +59,5 @@
     <parent link="world"/>
     <child link="base"/>
-    <origin xyz="0.0 -0.07044640523565884 0.7743112142292514" rpy="0.0 -0.0 0.0"/>
+    <origin xyz="1.5 0. 0.85" rpy="0.0 -0.0 0.0"/>
     <axis xyz="1.0 0.0 0.0"/>
   </joint>

Commit message: new standard oven position

File: mppi_examples/mppi_manipulation/data/objects/11826_mppi/mobility.urdf (robot description, URDF)
Before this commit: robot partnet_b5ca6cded4b23f2455b2aedb5bd199c6, 5 links, 4 joints
Joints:
- joint fixed: origin xyz=1.5 0. 0.85 rpy=0.0 -0.0 0.0 -> xyz=1.5 0.5 0.85 rpy=0.0 -0.0 0.0

File: mppi_examples/mppi_manipulation/data/objects/11826_mppi/mobility.urdf.xacro (robot description, xacro)
@@ -59,5 +59,5 @@
     <parent link="world"/>
     <child link="base"/>
-    <origin xyz="1.5 0. 0.85" rpy="0.0 -0.0 0.0"/>
+    <origin xyz="1.5 0.5 0.85" rpy="0.0 -0.0 0.0"/>
     <axis xyz="1.0 0.0 0.0"/>
   </joint>
