Commit message: tuning from testing on apr 20th

File: mppi_examples/mppi_manipulation/data/objects/zanussi/mobility.urdf.xacro (robot description, xacro)
@@ -48,5 +48,5 @@
     <child link="base"/>
     <!--<origin xyz="-1.156 1.46 1.01" rpy="0.0 0.0 1.57"/>-->
-    <origin xyz="-0.73 1.16 1.01" rpy="0.0 0.0 2.496"/>
+    <origin xyz="-0.727 1.18 1.005" rpy="0.0 0.0 2.525"/>
     <axis xyz="1.0 0.0 0.0"/>
   </joint>

File: mppi_examples/mppi_manipulation/data/rd_raisim_cylinder.urdf (robot description, URDF)
Before this commit: robot panda, 35 links, 34 joints
Links:
- link panda_leftfinger: geometry collision cylinder length=0.04 radius=0.004; visual cylinder length=0.07 radius=0.008

File: mppi_examples/mppi_panda/resources/panda/panda.urdf.xacro (robot description, xacro)
@@ -493,12 +493,13 @@
                     </inertial>
                     <visual>
-                        <origin rpy="0 0 0" xyz="0 0 0"/>
-                        <geometry>
-                            <mesh filename="${resources_prefix}${resources_directory}/resources/panda/meshes/visual/finger.dae"/>
-                        </geometry>
-                        <material name="">
-                            <color rgba="1 1 1 1"/>
-                        </material>
-                    </visual>
+      <origin rpy="0.0 0 3.14159265359" xyz="0 0.022 0.039"/>
+      <geometry>
+        <cylinder radius="0.008" length="0.07"/>
+        <!--<box size="0.021 0.009 0.070"/>-->
+      </geometry>
+      <material name="steel">
+        <color rgba="1 0 0 1"/>
+      </material>
+    </visual>
                     <!-- <xacro:if value="${collision_finger}">
                         <collision>

Commit message: new zanussi model with boxes instead of meshes for the handle

File: mppi_examples/mppi_manipulation/data/objects/zanussi/mobility.urdf.xacro (robot description, xacro)
@@ -19,13 +19,49 @@
     <visual>
       <geometry>
-        <mesh filename="${resources_directory}${resources_prefix}consolidated_collision_meshes/door_mesh.obj" scale="1 1 1"/>
+        <mesh filename="${resources_directory}${resources_prefix}consolidated_collision_meshes/door_mesh_2.obj" scale="1 1 1"/>
       </geometry>
       <origin xyz="0 0 0" rpy="0.0 0.0 0.0"/>
     </visual>
+    <visual>
+      <geometry>
+        <box size="0.40 0.02 0.02"/>
+      </geometry>
+      <origin xyz="0.297 0.428 0.051" rpy="0.0 0.0 0.0"/>
+    </visual>
+    <visual>
+      <geometry>
+        <box size="0.05 0.02 0.045"/>
+      </geometry>
+      <origin xyz="0.072 0.428 0.040" rpy="0.0 0.0 0.0"/>
+    </visual>
+    <visual>
+      <geometry>
+        <box size="0.05 0.02 0.045"/>
+      </geometry>
+      <origin xyz="0.52 0.428 0.040" rpy="0.0 0.0 0.0"/>
+    </visual>
     <collision>
       <geometry>
-        <mesh filename="${resources_directory}${resources_prefix}consolidated_collision_meshes/door_mesh.obj" scale="1 1 1"/>
+        <mesh filename="${resources_directory}${resources_prefix}consolidated_collision_meshes/door_mesh_2.obj" scale="1 1 1"/>
       </geometry>
       <origin xyz="0.0 0.0 0.0" rpy="0.0 0.0 0.0"/>
+    </collision>
+    <collision>
+      <geometry>
+        <box size="0.40 0.02 0.02"/>
+      </geometry>
+      <origin xyz="0.297 0.428 0.051" rpy="0.0 0.0 0.0"/>
+    </collision>
+    <collision>
+      <geometry>
+        <box size="0.05 0.02 0.045"/>
+      </geometry>
+      <origin xyz="0.072 0.428 0.040" rpy="0.0 0.0 0.0"/>
+    </collision>
+    <collision>
+      <geometry>
+        <box size="0.05 0.02 0.045"/>
+      </geometry>
+      <origin xyz="0.52 0.428 0.040" rpy="0.0 0.0 0.0"/>
     </collision>
   </link>

File: mppi_examples/mppi_manipulation/data/rd_raisim_cylinder.urdf (robot description, URDF)
Before this commit: robot panda, 35 links, 34 joints
Links:
- link base_link: geometry collision box size=1.5 0.75 0.65
- link panda_leftfinger: geometry collision cylinder length=0.07 radius=0.008; visual cylinder length=0.07 radius=0.008

Commit message: tuning of obj model and stuff for paper tests june 2nd and june 3rd

File: mppi_examples/mppi_manipulation/data/objects/zanussi/mobility.urdf.xacro (robot description, xacro)
@@ -84,5 +84,5 @@
     <child link="base"/>
     <!--<origin xyz="-1.156 1.46 1.01" rpy="0.0 0.0 1.57"/>-->
-    <origin xyz="-0.727 1.18 1.005" rpy="0.0 0.0 2.525"/>
+    <origin xyz="-0.015 -0.97 1.21" rpy="0.0 0.0 3.8"/>
     <axis xyz="1.0 0.0 0.0"/>
   </joint>
@@ -90,5 +90,8 @@
     <parent link="${prefix}link_3"/>
     <child link="${prefix}handle_link"/>
+    <!--open tasks-->
     <origin xyz="-0.594 -0.589 -0.015" rpy="0.0 0.0 0.0"/>
+    <!--close tasks-->
+    <!--<origin xyz="-0.594 -0.569 -0.035" rpy="0.0 0.0 0.0"/>-->
     <axis xyz="1.0 0.0 0.0"/>
     <limit effort="1000.0" velocity="1.0" lower="0.0" upper="1.5707963267948966"/>
